Commit message: sync https://www.lejuhub.com/highlydynamic/kuavo-ros-control/commit/0343b5884f373d04824aabc4896c068c4a212810

File: src/kuavo_assets/models/biped_s45/urdf/biped_s45_gazebo.urdf (robot description, URDF)
Before this commit: robot biped_s45, 47 links, 46 joints
Links:
- link zarm_l7_link: geometry collision mesh filename=package://kuavo_assets/models/biped_s45/meshes/l_hand_pitch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; visual mesh filename=package://kuavo_assets/models/biped_s45/meshes/l_hand_pitch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
- link zarm_r7_link: geometry collision mesh filename=package://kuavo_assets/models/biped_s45/meshes/r_hand_pitch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; visual mesh filename=package://kuavo_assets/models/biped_s45/meshes/r_hand_pitch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
Joints:
- joint l_foot_heel_joint: origin xyz=-0.073164 0.0 -0.0595 rpy=0 0 0 -> xyz=-0.0 0.04773 -0.0595 rpy=0 0 0
- joint l_foot_toe_joint: origin xyz=0.17084 0.0 -0.0595 rpy=0 0 0 -> xyz=0.0 -0.04773 -0.0595 rpy=0 0 0
- joint r_foot_heel_joint: origin xyz=-0.073164 0.0 -0.0595 rpy=0 0 0 -> xyz=-0.0 0.04773 -0.0595 rpy=0 0 0
- joint r_foot_toe_joint: origin xyz=0.17084 0.0 -0.0595 rpy=0 0 0 -> xyz=0.0 -0.04773 -0.0595 rpy=0 0 0
