Commit message: sync https://www.lejuhub.com/highlydynamic/kuavo-ros-control/commit/12ef80dede525adec576e5f6fb06f5e4c873c5dc

File: src/kuavo_assets/models/biped_s45/urdf/biped_s45.urdf (robot description, URDF)
Before this commit: robot biped_s45, 47 links, 46 joints
Links:
- added link l_hand_camera, mass 0.038145442577304; collision mesh filename=package://kuavo_assets/models/biped_s45/meshes/l_hand_camer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; visual mesh filename=package://kuavo_assets/models/biped_s45/meshes/l_hand_camer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
- added link l_hand_tripod, mass 0.0342669089979502; collision mesh filename=package://kuavo_assets/models/biped_s45/meshes/l_hand_tripo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; visual mesh filename=package://kuavo_assets/models/biped_s45/meshes/l_hand_tripo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
- added link r_hand_camera, mass 0.038145442577304; collision mesh filename=package://kuavo_assets/models/biped_s45/meshes/r_hand_camer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; visual mesh filename=package://kuavo_assets/models/biped_s45/meshes/r_hand_camer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
- added link r_hand_tripod, mass 0.034266881719861; collision mesh filename=package://kuavo_assets/models/biped_s45/meshes/r_hand_tripo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; visual mesh filename=package://kuavo_assets/models/biped_s45/meshes/r_hand_tripo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
- added link torso-camera, mass 0.1; collision mesh filename=package://kuavo_assets/models/biped_s45/meshes/torso-camera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; visual mesh filename=package://kuavo_assets/models/biped_s45/meshes/torso-camera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
- added link waist_camera, mass 0.237986769607677; collision mesh filename=package://kuavo_assets/models/biped_s45/meshes/waist_camera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; visual mesh filename=package://kuavo_assets/models/biped_s45/meshes/waist_camera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
- link base_link: mass 22.11293803 -> 21.63013803; geometry collision cylinder length=0.6 radius=0.15; visual mesh filename=package://kuavo_assets/models/biped_s45/meshes/torso.STL
- link zarm_l2_link: geometry collision cylinder length=0.3 radius=0.05; visual mesh filename=package://kuavo_assets/models/biped_s45/meshes/l_arm_roll.S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
- link zarm_l4_link: geometry collision cylinder length=0.26 radius=0.05; visual mesh filename=package://kuavo_assets/models/biped_s45/meshes/l_forearm.STL
- link zarm_l7_end_effector: geometry collision sphere radius=0.01
- link zarm_l7_link: geometry collision cylinder length=0.14 radius=0.04; visual mesh filename=package://kuavo_assets/models/biped_s45/meshes/l_hand_pitch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
- link zarm_r2_link: geometry collision cylinder length=0.3 radius=0.05; visual mesh filename=package://kuavo_assets/models/biped_s45/meshes/r_arm_roll.S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
- link zarm_r4_link: geometry collision cylinder length=0.26 radius=0.05; visual mesh filename=package://kuavo_assets/models/biped_s45/meshes/r_forearm.STL
- link zarm_r7_end_effector: geometry collision sphere radius=0.01
- link zarm_r7_link: geometry collision cylinder length=0.14 radius=0.04; visual mesh filename=package://kuavo_assets/models/biped_s45/meshes/r_hand_pitch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
- link zhead_1_link: geometry collision sphere radius=0.1; visual mesh filename=package://kuavo_assets/models/biped_s45/meshes/head_yaw.STL
Joints:
- removed joint dummy_to_base_link
- added joint base_link_to_dummy_link: type fixed, parent base_link, child dummy_link, origin xyz=0 0 0 rpy=0 0 0
- added joint l_hand_camera: type fixed, parent l_hand_tripod, child l_hand_camera, origin xyz=0.11540559159102 -0.0145586110669961 -0.110123491595499 rpy=-1.919862177193763 0.753528063917894 -2.897246568680842, axis 0 0 0
- added joint l_hand_tripod: type fixed, parent zarm_l7_link, child l_hand_tripod, origin xyz=0.0 0.0 0.0 rpy=0.0 0.0 0.0, axis 0 0 0
- added joint r_hand_camera: type fixed, parent r_hand_tripod, child r_hand_camera, origin xyz=0.115405591590931 0.0154312352120435 -0.107724128430896 rpy=1.208853693239594  0.751879414295006 2.888346587751982, axis 0 0 0
- added joint r_hand_tripod: type fixed, parent zarm_r7_link, child r_hand_tripod, origin xyz=0.0 0.0 0.0 rpy=0.0 0.0 0.0, axis 0 0 0
- added joint torso-camera: type fixed, parent base_link, child torso-camera, origin xyz=0.115535332475413 0.0175000000005085 0.2883441440894 rpy=0 0.732666 0, axis 0 0 0
- added joint waist_camera: type fixed, parent base_link, child waist_camera, origin xyz=0.168717483101422 0 0.01355599662743 rpy=0 0 0, axis 0 0 0

File: src/kuavo_assets/models/biped_s49/urdf/biped_s49.urdf (robot description, URDF)
Before this commit: robot biped_s49, 47 links, 46 joints
Links:
- added link l_hand_camera, mass 0.038145442577304; collision mesh filename=package://kuavo_assets/models/biped_s45/meshes/l_hand_camer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; visual mesh filename=package://kuavo_assets/models/biped_s45/meshes/l_hand_camer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
- added link l_hand_tripod, mass 0.0342669089979502; collision mesh filename=package://kuavo_assets/models/biped_s45/meshes/l_hand_tripo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; visual mesh filename=package://kuavo_assets/models/biped_s45/meshes/l_hand_tripo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
- added link r_hand_camera, mass 0.038145442577304; collision mesh filename=package://kuavo_assets/models/biped_s45/meshes/r_hand_camer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; visual mesh filename=package://kuavo_assets/models/biped_s45/meshes/r_hand_camer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
- added link r_hand_tripod, mass 0.034266881719861; collision mesh filename=package://kuavo_assets/models/biped_s45/meshes/r_hand_tripo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; visual mesh filename=package://kuavo_assets/models/biped_s45/meshes/r_hand_tripo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
- link base_link: geometry collision cylinder length=0.6 radius=0.15; visual mesh filename=package://kuavo_assets/models/biped_s49/meshes/torso.STL
- link zarm_l2_link: geometry collision cylinder length=0.3 radius=0.05; visual mesh filename=package://kuavo_assets/models/biped_s49/meshes/l_arm_roll.S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
- link zarm_l4_link: geometry collision cylinder length=0.26 radius=0.05; visual mesh filename=package://kuavo_assets/models/biped_s49/meshes/l_forearm.STL
- link zarm_l7_link: geometry collision cylinder length=0.14 radius=0.04; visual mesh filename=package://kuavo_assets/models/biped_s49/meshes/l_hand_pitch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
- link zarm_r2_link: geometry collision cylinder length=0.3 radius=0.05; visual mesh filename=package://kuavo_assets/models/biped_s49/meshes/r_arm_roll.S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
- link zarm_r4_link: geometry collision cylinder length=0.26 radius=0.05; visual mesh filename=package://kuavo_assets/models/biped_s49/meshes/r_forearm.STL
- link zarm_r7_link: geometry collision cylinder length=0.14 radius=0.04; visual mesh filename=package://kuavo_assets/models/biped_s49/meshes/r_hand_pitch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
- link zhead_1_link: geometry collision sphere radius=0.1; visual mesh filename=package://kuavo_assets/models/biped_s49/meshes/head_yaw.STL
Joints:
- removed joint dummy_to_base_link
- added joint base_link_to_dummy_link: type fixed, parent base_link, child dummy_link, origin xyz=0 0 0 rpy=0 0 0
- added joint l_hand_camera: type fixed, parent l_hand_tripod, child l_hand_camera, origin xyz=0.11540559159102 -0.0145586110669961 -0.110123491595499 rpy=-1.919862177193763 0.753528063917894 -2.897246568680842, axis 0 0 0
- added joint l_hand_tripod: type fixed, parent zarm_l7_link, child l_hand_tripod, origin xyz=0.0 0.0 0.0 rpy=0.0 0.0 0.0, axis 0 0 0
- added joint r_hand_camera: type fixed, parent r_hand_tripod, child r_hand_camera, origin xyz=0.115405591590931 0.0154312352120435 -0.107724128430896 rpy=1.208853693239594  0.751879414295006 2.888346587751982, axis 0 0 0
- added joint r_hand_tripod: type fixed, parent zarm_r7_link, child r_hand_tripod, origin xyz=0.0 0.0 0.0 rpy=0.0 0.0 0.0, axis 0 0 0

Commit message: sync https://www.lejuhub.com/highlydynamic/kuavo-ros-control/commit/b5f3928d4928bda2c6d9eaa3da7666e05882e12b

File: src/kuavo_assets/models/biped_s45/urdf/biped_s45.urdf (robot description, URDF)
Before this commit: robot biped_s45, 47 links, 46 joints
Links:
- added link l_hand_camera, mass 0.038145442577304; collision mesh filename=package://kuavo_assets/models/biped_s45/meshes/l_hand_camer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; visual mesh filename=package://kuavo_assets/models/biped_s45/meshes/l_hand_camer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
- added link l_hand_tripod, mass 0.0342669089979502; collision mesh filename=package://kuavo_assets/models/biped_s45/meshes/l_hand_tripo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; visual mesh filename=package://kuavo_assets/models/biped_s45/meshes/l_hand_tripo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
- added link r_hand_camera, mass 0.038145442577304; collision mesh filename=package://kuavo_assets/models/biped_s45/meshes/r_hand_camer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; visual mesh filename=package://kuavo_assets/models/biped_s45/meshes/r_hand_camer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
- added link r_hand_tripod, mass 0.034266881719861; collision mesh filename=package://kuavo_assets/models/biped_s45/meshes/r_hand_tripo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; visual mesh filename=package://kuavo_assets/models/biped_s45/meshes/r_hand_tripo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
- added link torso-camera, mass 0.1; collision mesh filename=package://kuavo_assets/models/biped_s45/meshes/torso-camera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; visual mesh filename=package://kuavo_assets/models/biped_s45/meshes/torso-camera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
- added link waist_camera, mass 0.237986769607677; collision mesh filename=package://kuavo_assets/models/biped_s45/meshes/waist_camera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; visual mesh filename=package://kuavo_assets/models/biped_s45/meshes/waist_camera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
- link base_link: mass 22.11293803 -> 27.41553803; geometry collision cylinder length=0.6 radius=0.15; visual mesh filename=package://kuavo_assets/models/biped_s45/meshes/torso.STL
- link zarm_l2_link: geometry collision cylinder length=0.3 radius=0.05; visual mesh filename=package://kuavo_assets/models/biped_s45/meshes/l_arm_roll.S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
- link zarm_l4_link: geometry collision cylinder length=0.26 radius=0.05; visual mesh filename=package://kuavo_assets/models/biped_s45/meshes/l_forearm.STL
- link zarm_l7_end_effector: geometry collision sphere radius=0.01
- link zarm_l7_link: geometry collision cylinder length=0.14 radius=0.04; visual mesh filename=package://kuavo_assets/models/biped_s45/meshes/l_hand_pitch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
- link zarm_r2_link: geometry collision cylinder length=0.3 radius=0.05; visual mesh filename=package://kuavo_assets/models/biped_s45/meshes/r_arm_roll.S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
- link zarm_r4_link: geometry collision cylinder length=0.26 radius=0.05; visual mesh filename=package://kuavo_assets/models/biped_s45/meshes/r_forearm.STL
- link zarm_r7_end_effector: geometry collision sphere radius=0.01
- link zarm_r7_link: geometry collision cylinder length=0.14 radius=0.04; visual mesh filename=package://kuavo_assets/models/biped_s45/meshes/r_hand_pitch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
- link zhead_1_link: geometry collision sphere radius=0.1; visual mesh filename=package://kuavo_assets/models/biped_s45/meshes/head_yaw.STL
Joints:
- removed joint dummy_to_base_link
- added joint base_link_to_dummy_link: type fixed, parent base_link, child dummy_link, origin xyz=0 0 0 rpy=0 0 0
- added joint l_hand_camera: type fixed, parent l_hand_tripod, child l_hand_camera, origin xyz=0.11540559159102 -0.0145586110669961 -0.110123491595499 rpy=1.919862177193763 0.753528063917894 -2.897246568680842, axis 0 0 0
- added joint l_hand_tripod: type fixed, parent zarm_l7_link, child l_hand_tripod, origin xyz=0.0 0.0 0.0 rpy=0.0 0.0 0.0, axis 0 0 0
- added joint r_hand_camera: type fixed, parent r_hand_tripod, child r_hand_camera, origin xyz=0.115405591590931 0.0154312352120435 -0.107724128430896 rpy=1.208853693239594  0.751879414295006 2.888346587751982, axis 0 0 0
- added joint r_hand_tripod: type fixed, parent zarm_r7_link, child r_hand_tripod, origin xyz=0.0 0.0 0.0 rpy=0.0 0.0 0.0, axis 0 0 0
- added joint torso-camera: type fixed, parent base_link, child torso-camera, origin xyz=0.115535332475413 0.0175000000005085 0.2883441440894 rpy=0 0.732666 0, axis 0 0 0
- added joint waist_camera: type fixed, parent base_link, child waist_camera, origin xyz=0.168717483101422 0 0.01355599662743 rpy=0 0 0, axis 0 0 0

File: src/kuavo_assets/models/biped_s48/urdf/biped_s48.urdf (robot description, URDF)
Before this commit: robot biped_s48, 69 links, 68 joints
Links:
- link base_link: geometry collision cylinder length=0.6 radius=0.15; visual mesh filename=package://kuavo_assets/models/biped_s48/meshes/torso.STL
- link zarm_l2_link: geometry collision cylinder length=0.3 radius=0.05; visual mesh filename=package://kuavo_assets/models/biped_s48/meshes/l_arm_roll.S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
- link zarm_l4_link: geometry collision cylinder length=0.26 radius=0.05; visual mesh filename=package://kuavo_assets/models/biped_s48/meshes/l_forearm.STL
- link zarm_l7_link: geometry collision cylinder length=0.14 radius=0.04; visual mesh filename=package://kuavo_assets/models/biped_s48/meshes/l_hand_pitch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
- link zarm_r2_link: geometry collision cylinder length=0.3 radius=0.05; visual mesh filename=package://kuavo_assets/models/biped_s48/meshes/r_arm_roll.S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
- link zarm_r4_link: geometry collision cylinder length=0.26 radius=0.05; visual mesh filename=package://kuavo_assets/models/biped_s48/meshes/r_forearm.STL
- link zarm_r7_link: geometry collision cylinder length=0.14 radius=0.04; visual mesh filename=package://kuavo_assets/models/biped_s48/meshes/r_hand_pitch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
- link zhead_2_link: geometry collision sphere radius=0.1; visual mesh filename=package://kuavo_assets/models/biped_s48/meshes/head_pitch.S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
Joints:
- removed joint dummy_to_base_link
- added joint base_link_to_dummy_link: type fixed, parent base_link, child dummy_link, origin xyz=0 0 0 rpy=0 0 0

File: src/kuavo_assets/models/biped_s49/urdf/biped_s49.urdf (robot description, URDF)
Before this commit: robot biped_s49, 47 links, 46 joints
Links:
- added link l_hand_camera, mass 0.038145442577304; collision mesh filename=package://kuavo_assets/models/biped_s45/meshes/l_hand_camer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; visual mesh filename=package://kuavo_assets/models/biped_s45/meshes/l_hand_camer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
- added link l_hand_tripod, mass 0.0342669089979502; collision mesh filename=package://kuavo_assets/models/biped_s45/meshes/l_hand_tripo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; visual mesh filename=package://kuavo_assets/models/biped_s45/meshes/l_hand_tripo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
- added link r_hand_camera, mass 0.038145442577304; collision mesh filename=package://kuavo_assets/models/biped_s45/meshes/r_hand_camer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; visual mesh filename=package://kuavo_assets/models/biped_s45/meshes/r_hand_camer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
- added link r_hand_tripod, mass 0.034266881719861; collision mesh filename=package://kuavo_assets/models/biped_s45/meshes/r_hand_tripo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; visual mesh filename=package://kuavo_assets/models/biped_s45/meshes/r_hand_tripo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
- link base_link: geometry collision cylinder length=0.6 radius=0.15; visual mesh filename=package://kuavo_assets/models/biped_s49/meshes/torso.STL
- link zarm_l2_link: geometry collision cylinder length=0.3 radius=0.05; visual mesh filename=package://kuavo_assets/models/biped_s49/meshes/l_arm_roll.S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
- link zarm_l4_link: geometry collision cylinder length=0.26 radius=0.05; visual mesh filename=package://kuavo_assets/models/biped_s49/meshes/l_forearm.STL
- link zarm_l7_link: geometry collision cylinder length=0.14 radius=0.04; visual mesh filename=package://kuavo_assets/models/biped_s49/meshes/l_hand_pitch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
- link zarm_r2_link: geometry collision cylinder length=0.3 radius=0.05; visual mesh filename=package://kuavo_assets/models/biped_s49/meshes/r_arm_roll.S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
- link zarm_r4_link: geometry collision cylinder length=0.26 radius=0.05; visual mesh filename=package://kuavo_assets/models/biped_s49/meshes/r_forearm.STL
- link zarm_r7_link: geometry collision cylinder length=0.14 radius=0.04; visual mesh filename=package://kuavo_assets/models/biped_s49/meshes/r_hand_pitch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
- link zhead_1_link: geometry collision sphere radius=0.1; visual mesh filename=package://kuavo_assets/models/biped_s49/meshes/head_yaw.STL
Joints:
- removed joint dummy_to_base_link
- added joint base_link_to_dummy_link: type fixed, parent base_link, child dummy_link, origin xyz=0 0 0 rpy=0 0 0
- added joint l_hand_camera: type fixed, parent l_hand_tripod, child l_hand_camera, origin xyz=0.11540559159102 -0.0145586110669961 -0.110123491595499 rpy=1.919862177193763 0.753528063917894 -2.897246568680842, axis 0 0 0
- added joint l_hand_tripod: type fixed, parent zarm_l7_link, child l_hand_tripod, origin xyz=0.0 0.0 0.0 rpy=0.0 0.0 0.0, axis 0 0 0
- added joint r_hand_camera: type fixed, parent r_hand_tripod, child r_hand_camera, origin xyz=0.115405591590931 0.0154312352120435 -0.107724128430896 rpy=1.208853693239594  0.751879414295006 2.888346587751982, axis 0 0 0
- added joint r_hand_tripod: type fixed, parent zarm_r7_link, child r_hand_tripod, origin xyz=0.0 0.0 0.0 rpy=0.0 0.0 0.0, axis 0 0 0

Commit message: sync https://www.lejuhub.com/highlydynamic/kuavo-ros-control/commit/fe4d17b4b012accb7a2349457309a505b3ce45d7

File: src/kuavo_assets/models/biped_s45/urdf/biped_s45.urdf (robot description, URDF)
Before this commit: robot biped_s45, 53 links, 52 joints
Joints:
- removed joint l_hand_camera
- removed joint l_hand_tripod
- removed joint r_hand_camera
- removed joint r_hand_tripod
- added joint l_hand_camera_joint: type fixed, parent l_hand_tripod, child l_hand_camera, origin xyz=0.11540559159102 -0.0145586110669961 -0.110123491595499 rpy=1.919862177193763 0.753528063917894 -2.897246568680842, axis 0 0 0
- added joint l_hand_tripod_joint: type fixed, parent zarm_l7_link, child l_hand_tripod, origin xyz=0.0 0.0 0.0 rpy=0.0 0.0 0.0, axis 0 0 0
- added joint r_hand_camera_joint: type fixed, parent r_hand_tripod, child r_hand_camera, origin xyz=0.115405591590931 0.0154312352120435 -0.107724128430896 rpy=1.208853693239594  0.751879414295006 2.888346587751982, axis 0 0 0
- added joint r_hand_tripod_joint: type fixed, parent zarm_r7_link, child r_hand_tripod, origin xyz=0.0 0.0 0.0 rpy=0.0 0.0 0.0, axis 0 0 0

File: src/kuavo_assets/models/biped_s49/urdf/biped_s49.urdf (robot description, URDF)
Before this commit: robot biped_s49, 51 links, 50 joints
Joints:
- removed joint l_hand_camera
- removed joint l_hand_tripod
- removed joint r_hand_camera
- removed joint r_hand_tripod
- added joint l_hand_camera_joint: type fixed, parent l_hand_tripod, child l_hand_camera, origin xyz=0.11540559159102 -0.0145586110669961 -0.110123491595499 rpy=1.919862177193763 0.753528063917894 -2.897246568680842, axis 0 0 0
- added joint l_hand_tripod_joint: type fixed, parent zarm_l7_link, child l_hand_tripod, origin xyz=0.0 0.0 0.0 rpy=0.0 0.0 0.0, axis 0 0 0
- added joint r_hand_camera_joint: type fixed, parent r_hand_tripod, child r_hand_camera, origin xyz=0.115405591590931 0.0154312352120435 -0.107724128430896 rpy=1.208853693239594  0.751879414295006 2.888346587751982, axis 0 0 0
- added joint r_hand_tripod_joint: type fixed, parent zarm_r7_link, child r_hand_tripod, origin xyz=0.0 0.0 0.0 rpy=0.0 0.0 0.0, axis 0 0 0

Commit message: sync https://www.lejuhub.com/highlydynamic/kuavo-ros-control/commit/7d3eb93aa09826fce18108d1a7cbc4da5f6d59a1

File: src/kuavo_assets/models/biped_s45/urdf/biped_s45.urdf (robot description, URDF)
Before this commit: robot biped_s45, 47 links, 46 joints
Links:
- added link l_hand_camera, mass 0.038145442577304; collision mesh filename=package://kuavo_assets/models/biped_s45/meshes/l_hand_camer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; visual mesh filename=package://kuavo_assets/models/biped_s45/meshes/l_hand_camer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
- added link l_hand_tripod, mass 0.0342669089979502; collision mesh filename=package://kuavo_assets/models/biped_s45/meshes/l_hand_tripo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; visual mesh filename=package://kuavo_assets/models/biped_s45/meshes/l_hand_tripo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
- added link r_hand_camera, mass 0.038145442577304; collision mesh filename=package://kuavo_assets/models/biped_s45/meshes/r_hand_camer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; visual mesh filename=package://kuavo_assets/models/biped_s45/meshes/r_hand_camer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
- added link r_hand_tripod, mass 0.034266881719861; collision mesh filename=package://kuavo_assets/models/biped_s45/meshes/r_hand_tripo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; visual mesh filename=package://kuavo_assets/models/biped_s45/meshes/r_hand_tripo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
- added link torso-camera, mass 0.1; collision mesh filename=package://kuavo_assets/models/biped_s45/meshes/torso-camera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; visual mesh filename=package://kuavo_assets/models/biped_s45/meshes/torso-camera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
- added link waist_camera, mass 0.237986769607677; collision mesh filename=package://kuavo_assets/models/biped_s45/meshes/waist_camera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; visual mesh filename=package://kuavo_assets/models/biped_s45/meshes/waist_camera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
- link base_link: mass 22.11293803 -> 21.63013803; geometry collision cylinder length=0.6 radius=0.15; visual mesh filename=package://kuavo_assets/models/biped_s45/meshes/torso.STL
- link zarm_l2_link: geometry collision cylinder length=0.3 radius=0.05; visual mesh filename=package://kuavo_assets/models/biped_s45/meshes/l_arm_roll.S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
- link zarm_l4_link: geometry collision cylinder length=0.26 radius=0.05; visual mesh filename=package://kuavo_assets/models/biped_s45/meshes/l_forearm.STL
- link zarm_l7_end_effector: geometry collision sphere radius=0.01
- link zarm_l7_link: geometry collision cylinder length=0.14 radius=0.04; visual mesh filename=package://kuavo_assets/models/biped_s45/meshes/l_hand_pitch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
- link zarm_r2_link: geometry collision cylinder length=0.3 radius=0.05; visual mesh filename=package://kuavo_assets/models/biped_s45/meshes/r_arm_roll.S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
- link zarm_r4_link: geometry collision cylinder length=0.26 radius=0.05; visual mesh filename=package://kuavo_assets/models/biped_s45/meshes/r_forearm.STL
- link zarm_r7_end_effector: geometry collision sphere radius=0.01
- link zarm_r7_link: geometry collision cylinder length=0.14 radius=0.04; visual mesh filename=package://kuavo_assets/models/biped_s45/meshes/r_hand_pitch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
- link zhead_1_link: geometry collision sphere radius=0.1; visual mesh filename=package://kuavo_assets/models/biped_s45/meshes/head_yaw.STL
Joints:
- removed joint dummy_to_base_link
- added joint base_link_to_dummy_link: type fixed, parent base_link, child dummy_link, origin xyz=0 0 0 rpy=0 0 0
- added joint l_hand_camera_joint: type fixed, parent l_hand_tripod, child l_hand_camera, origin xyz=0.11540559159102 -0.0145586110669961 -0.110123491595499 rpy=1.919862177193763 0.753528063917894 -2.897246568680842, axis 0 0 0
- added joint l_hand_tripod_joint: type fixed, parent zarm_l7_link, child l_hand_tripod, origin xyz=0.0 0.0 0.0 rpy=0.0 0.0 0.0, axis 0 0 0
- added joint r_hand_camera_joint: type fixed, parent r_hand_tripod, child r_hand_camera, origin xyz=0.115405591590931 0.0154312352120435 -0.107724128430896 rpy=1.208853693239594  0.751879414295006 2.888346587751982, axis 0 0 0
- added joint r_hand_tripod_joint: type fixed, parent zarm_r7_link, child r_hand_tripod, origin xyz=0.0 0.0 0.0 rpy=0.0 0.0 0.0, axis 0 0 0
- added joint torso-camera: type fixed, parent base_link, child torso-camera, origin xyz=0.115535332475413 0.0175000000005085 0.2883441440894 rpy=0 0.732666 0, axis 0 0 0
- added joint waist_camera: type fixed, parent base_link, child waist_camera, origin xyz=0.168717483101422 0 0.01355599662743 rpy=0 0 0, axis 0 0 0

Commit message: sync https://www.lejuhub.com/highlydynamic/kuavo-ros-control/commit/8b72d52095ccfee116500685ec09824b617d3814

File: src/kuavo_assets/models/biped_s45/urdf/biped_s45.urdf (robot description, URDF)
Before this commit: robot biped_s45, 53 links, 52 joints
Links:
- link base_link: mass 21.63013803 -> 27.41553803

File: src/kuavo_assets/models/biped_s45/urdf/biped_s45_gazebo.urdf (robot description, URDF)
Before this commit: robot biped_s45, 47 links, 46 joints
Links:
- link base_link: mass 22.11293803 -> 27.89833803
