Commit message: sync https://www.lejuhub.com/highlydynamic/kuavo-ros-control/commit/79757a37306faa535ba50c4952499f51b89ee460

File: src/kuavo_assets/models/biped_s14/urdf/biped_s14_gazebo.urdf (robot description, URDF)
Before this commit: robot biped_s14, 39 links, 38 joints
Joints:
- removed joint waist
- added joint waist_joint: type revolute, parent base_link, child waist, origin xyz=0 0 0 rpy=0 0 0, axis 0 0 1, limit lower=-2.0943951023932 upper=2.0943951023932 effort=36.0 velocity=23.0266666666667
- joint dummy_to_base_link: type floating -> fixed
