Commit message: sync https://www.lejuhub.com/highlydynamic/kuavo-ros-control/commit/58f1372b802e64e3bdcb57487377bea2b7efdd46

File: src/kuavo_assets/models/biped_s14/urdf/biped_s14.urdf (robot description, URDF)
Before this commit: robot biped_s14, 39 links, 38 joints
Links:
- link base_link: mass 8.017776 -> 8.620576

File: src/kuavo_assets/models/biped_s14/urdf/biped_s14_gazebo.urdf (robot description, URDF)
Before this commit: robot biped_s14, 39 links, 38 joints
Links:
- link base_link: mass 8.017776 -> 8.620576

File: src/kuavo_assets/models/biped_s14/urdf/drake/biped_v3.urdf (robot description, URDF)
Before this commit: robot biped_v3, 14 links, 13 joints
Links:
- link torso: mass 12.09718758 -> 12.69998758

File: src/kuavo_assets/models/biped_s14/urdf/drake/biped_v3_full.urdf (robot description, URDF)
Before this commit: robot biped_v3_full, 22 links, 21 joints
Links:
- link torso: mass 9.385076 -> 9.987876

Commit message: sync https://www.lejuhub.com/highlydynamic/kuavo-ros-control/commit/b3494837f6b8da48f79a0aa65cd6dfb5255f61b8

File: src/kuavo_assets/models/biped_s14/urdf/biped_s14.urdf (robot description, URDF)
Before this commit: robot biped_s14, 39 links, 38 joints
Links:
- added link camera, mass 0.011119; collision mesh filename=package://kuavo_assets/models/biped_s14/meshes/camera.STL; visual mesh filename=package://kuavo_assets/models/biped_s14/meshes/camera.STL
- added link camera_base, mass 3.927E-05; collision mesh filename=package://kuavo_assets/models/biped_s14/meshes/camera_base.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; visual mesh filename=package://kuavo_assets/models/biped_s14/meshes/camera_base.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
- link zhead_1_link: mass 1.03077542 -> 0.32829; geometry collision mesh filename=package://kuavo_assets/models/biped_s14/meshes/head_yaw.STL; visual mesh filename=package://kuavo_assets/models/biped_s14/meshes/head_yaw.STL
- link zhead_2_link: mass 0.33654975 -> 0.33162; geometry collision mesh filename=package://kuavo_assets/models/biped_s14/meshes/head_pitch.S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; visual mesh filename=package://kuavo_assets/models/biped_s14/meshes/head_pitch.S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
Joints:
- added joint camera_base_joint: type fixed, parent zhead_2_link, child camera_base, origin xyz=0.049912 0.0002 0.050414 rpy=0 0.27152 0, axis 0 0 0
- added joint camera_joint: type fixed, parent zhead_2_link, child camera, origin xyz=0.069468 0.0112 0.057945 rpy=-0.014569 0.27114 -0.054347, axis 0 0 0

File: src/kuavo_assets/models/biped_s14/urdf/biped_s14_gazebo.urdf (robot description, URDF)
Before this commit: robot biped_s14, 39 links, 38 joints
Links:
- added link camera, mass 0.011119; collision mesh filename=package://kuavo_assets/models/biped_s14/meshes/camera.STL; visual mesh filename=package://kuavo_assets/models/biped_s14/meshes/camera.STL
- added link camera_base, mass 3.927E-05; collision mesh filename=package://kuavo_assets/models/biped_s14/meshes/camera_base.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; visual mesh filename=package://kuavo_assets/models/biped_s14/meshes/camera_base.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
- link zhead_1_link: mass 1.03077542 -> 0.32829; geometry collision mesh filename=package://kuavo_assets/models/biped_s14/meshes/head_yaw.STL; visual mesh filename=package://kuavo_assets/models/biped_s14/meshes/head_yaw.STL
- link zhead_2_link: mass 0.33654975 -> 0.33162; geometry collision mesh filename=package://kuavo_assets/models/biped_s14/meshes/head_pitch.S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; visual mesh filename=package://kuavo_assets/models/biped_s14/meshes/head_pitch.S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
Joints:
- added joint camera_base_joint: type fixed, parent zhead_2_link, child camera_base, origin xyz=0.049912 0.0002 0.050414 rpy=0 0.27152 0
- added joint camera_joint: type fixed, parent zhead_2_link, child camera, origin xyz=0.069468 0.0112 0.057945 rpy=-0.014569 0.27114 -0.054347

File: src/kuavo_assets/models/biped_s14/urdf/biped_s14_gazebo.xacro (robot description, xacro)
@@ -6,5 +6,5 @@
   <xacro:include filename="$(find realsense_ros_gazebo)/xacro/depthcam.xacro"/>
   <!-- d435 声明 -->
-  <xacro:realsense_d435 sensor_name="camera" parent_link="camera_base" rate="30">
+  <xacro:realsense_d435 sensor_name="rs_camera" parent_link="camera_base" rate="30">
     <origin rpy="0 0 0 " xyz="0 0 0"/>
   </xacro:realsense_d435>

Commit message: sync https://www.lejuhub.com/highlydynamic/kuavo-ros-control/commit/5a76b533df55eaa21925730c6183a043de642185

File: src/kuavo_assets/models/biped_s14/urdf/biped_s14.urdf (robot description, URDF)
Before this commit: robot biped_s14, 39 links, 38 joints
Links:
- link base_link: mass 8.620576 -> 8.620776
- link leg_r1_link: mass 0.42877618 -> 0.42877473
- link leg_r2_link: mass 2.4999594 -> 2.50010758
- link leg_r3_link: mass 1.109669 -> 1.10966483
- link leg_r4_link: mass 1.55038362 -> 1.55001765
- link leg_r6_link: mass 0.34819511 -> 0.34819252
- link zarm_r1_link: mass 0.37301773 -> 0.3730157
- link zarm_r2_link: mass 0.15112665 -> 0.15112869
- link zarm_r4_link: mass 0.16269033 -> 0.16269441
Joints:
- joint leg_r4_joint: origin xyz=-0.0209999999999396 0 -0.182000000000001 rpy=0 0 0 -> xyz=-0.0209999999999696 0 -0.181999999999961 rpy=0 0 0
- joint leg_r5_joint: origin xyz=0.0209999999999936 0 -0.235 rpy=0 0 0 -> xyz=0.0209999999999503 0 -0.235000000000001 rpy=0 0 0
- joint ll_foot_toe_joint: origin xyz=0.121 0.04149834 -0.0435 rpy=0 0 0 -> xyz=0.121 0.03824834 -0.0435 rpy=0 0 0
- joint rl_foot_toe_joint: origin xyz=0.121 0.04149834 -0.0435 rpy=0 0 0 -> xyz=0.121 0.03824834 -0.0435 rpy=0 0 0
- joint zarm_r4_joint: origin xyz=0 0 -0.187999999999989 rpy=0 0 0 -> xyz=0 0 -0.187999999999999 rpy=0 0 0
- joint zhead_1_joint: origin xyz=0.00400001 2.92e-06 0.35618885 rpy=0 0 0 -> xyz=0 0 0.35618885 rpy=0 0 0

File: src/kuavo_assets/models/biped_s14/urdf/biped_s14_gazebo.urdf (robot description, URDF)
Before this commit: robot biped_s14, 39 links, 38 joints
Links:
- link base_link: mass 8.620576 -> 8.620776
- link leg_r1_link: mass 0.42877618 -> 0.42877473
- link leg_r2_link: mass 2.4999594 -> 2.50010758
- link leg_r3_link: mass 1.109669 -> 1.10966483
- link leg_r4_link: mass 1.55038362 -> 1.55001765
- link leg_r6_link: mass 0.34819511 -> 0.34819252
- link zarm_r1_link: mass 0.37301773 -> 0.3730157
- link zarm_r2_link: mass 0.15112665 -> 0.15112869
- link zarm_r4_link: mass 0.16269033 -> 0.16269441
Joints:
- joint leg_r4_joint: origin xyz=-0.0209999999999396 0 -0.182000000000001 rpy=0 0 0 -> xyz=-0.0209999999999696 0 -0.181999999999961 rpy=0 0 0
- joint leg_r5_joint: origin xyz=0.0209999999999936 0 -0.235 rpy=0 0 0 -> xyz=0.0209999999999503 0 -0.235000000000001 rpy=0 0 0
- joint ll_foot_toe_joint: origin xyz=0.121 0.04149834 -0.0435 rpy=0 0 0 -> xyz=0.121 0.03824834 -0.0435 rpy=0 0 0
- joint rl_foot_toe_joint: origin xyz=0.121 0.04149834 -0.0435 rpy=0 0 0 -> xyz=0.121 0.03824834 -0.0435 rpy=0 0 0
- joint zarm_r4_joint: origin xyz=0 0 -0.187999999999989 rpy=0 0 0 -> xyz=0 0 -0.187999999999999 rpy=0 0 0
- joint zhead_1_joint: origin xyz=0.00400001 2.92e-06 0.35618885 rpy=0 0 0 -> xyz=0 0 0.35618885 rpy=0 0 0

File: src/kuavo_assets/models/biped_s14/urdf/drake/biped_v3.urdf (robot description, URDF)
Before this commit: robot biped_v3, 14 links, 13 joints
Links:
- link leg_r1_link: mass 0.42877618 -> 0.42877473
- link leg_r2_link: mass 2.4999594 -> 2.50010758
- link leg_r3_link: mass 1.109669 -> 1.10966483
- link leg_r4_link: mass 1.55038362 -> 1.55001765
- link leg_r6_link: mass 0.34819511 -> 0.34819252
- link torso: mass 12.69998758 -> 12.700276
Joints:
- joint leg_r4_joint: origin xyz=-0.0209999999999396 0 -0.182000000000001 rpy=0 0 0 -> xyz=-0.0209999999999696 0 -0.181999999999961 rpy=0 0 0
- joint leg_r5_joint: origin xyz=0.0209999999999936 0 -0.235 rpy=0 0 0 -> xyz=0.0209999999999503 0 -0.235000000000001 rpy=0 0 0

Commit message: sync https://www.lejuhub.com/highlydynamic/kuavo-ros-control/commit/a974f9f4767e76a35a9b3bf09f5bcb4106ea93c5

File: src/kuavo_assets/models/biped_s14/urdf/biped_s14.urdf (robot description, URDF)
Before this commit: robot biped_s14, 41 links, 40 joints
Links:
- link camera_base: mass 3.927E-05 -> 0.001

File: src/kuavo_assets/models/biped_s52/urdf/drake/biped_v3_arm.urdf (robot description, URDF)
Before this commit: robot biped_s45, 17 links, 16 joints
Links:
- added link waist_yaw_link, mass 18.01415568; visual mesh filename=../../meshes/waist_yaw.STL
- link base_link: mass 22.11293803 -> 6.48663928
- link zarm_l1_link: mass 0.962 -> 0.91653322
- link zarm_l2_link: mass 0.57 -> 0.3876739
- link zarm_l3_link: mass 1.65 -> 1.77926875
- link zarm_l4_link: mass 0.429 -> 0.58507821
- link zarm_l5_link: mass 0.61 -> 0.68679955
- link zarm_l6_link: mass 0.331 -> 0.39387181
- link zarm_l7_link: mass 0.64 -> 0.61537779
- link zarm_r1_link: mass 0.962 -> 0.92062797
- link zarm_r2_link: mass 0.57 -> 0.38768053
- link zarm_r3_link: mass 1.65 -> 1.77969208
- link zarm_r4_link: mass 0.429 -> 0.58514611
- link zarm_r5_link: mass 0.61 -> 0.68473867
- link zarm_r6_link: mass 0.331 -> 0.39247462
- link zarm_r7_link: mass 0.64 -> 0.61562202
Joints:
- added joint waist_yaw_joint: type fixed, parent base_link, child waist_yaw_link, origin xyz=0 0 0.1114 rpy=0 0 0, axis 0 0 1, limit lower=-3.14159 upper=3.14159 effort=180.0 velocity=23.55
- joint zarm_l1_joint: origin xyz=-0.017499853 0.29269999999999996 0.4245 rpy=0 0 0 -> xyz=-0.003 0.1737 0.2831 rpy=0 0 0; parent base_link -> waist_yaw_link
- joint zarm_l2_joint: limit lower=-0.349065850398866 upper=2.0943951023932 effort=50.0 velocity=19.154 -> lower=-0.349065850398866 upper=2.0943951023932 effort=50.0 velocity=8.37333333333333; origin xyz=0 0 0 rpy=0 0 0 -> xyz=0 0.081 0 rpy=0 0 0
- joint zarm_l3_joint: limit lower=-1.5707963267949 upper=1.5707963267949 effort=39.0 velocity=18.84 -> lower=-1.5707963267949 upper=1.5707963267949 effort=36.0 velocity=9.94333333333333; origin xyz=0 0 0 rpy=0 0 0 -> xyz=0 0 -0.104 rpy=0 0 0
- joint zarm_l4_joint: limit lower=-2.61799387799149 upper=0.0 effort=50.0 velocity=18.84 -> lower=-2.61799387799149 upper=0.0 effort=50.0 velocity=8.37333333333333; origin xyz=0.0200000000000006 0 -0.283699999999996 rpy=0 0 0 -> xyz=0.02 0 -0.1797 rpy=0 0 0
- joint zarm_l5_joint: limit lower=-1.5707963267949 upper=1.5707963267949 effort=12.0 velocity=21.666 -> lower=-1.5707963267949 upper=1.5707963267949 effort=12.0 velocity=7.32666666666667; origin xyz=-0.0200000000000025 0 -0.127037274261591 rpy=0 0 0 -> xyz=-0.02 0 -0.1195 rpy=0 0 0
- joint zarm_l6_joint: limit lower=-1.30899693899575 upper=0.698131700797732 effort=12.0 velocity=21.666 -> lower=-1.30899693899575 upper=0.698131700797732 effort=12.0 velocity=7.32666666666667; origin xyz=0.000199999999999079 0 -0.106462725738415 rpy=0 0 0 -> xyz=0 0 -0.114 rpy=0 0 0
- joint zarm_l7_joint: limit lower=-0.698131700797732 upper=0.698131700797732 effort=12.0 velocity=21.666 -> lower=-0.698131700797732 upper=0.698131700797732 effort=12.0 velocity=7.32666666666667; origin xyz=0 0 -0.0210004653879916 rpy=0 0 0 -> xyz=-0.0002 0 -0.021 rpy=0 0 0
- joint zarm_r1_joint: origin xyz=-0.017499853 -0.29269999999999996 0.4245 rpy=0 0 0 -> xyz=-0.003 -0.1737 0.2831 rpy=0 0 0; parent base_link -> waist_yaw_link
- joint zarm_r2_joint: limit lower=-2.0943951023932 upper=0.349065850398866 effort=50.0 velocity=19.154 -> lower=-2.0943951023932 upper=0.349065850398866 effort=50.0 velocity=8.37333333333333; origin xyz=0 0 0 rpy=0 0 0 -> xyz=0 -0.081 0 rpy=0 0 0
- joint zarm_r3_joint: limit lower=-1.5707963267949 upper=1.5707963267949 effort=39.0 velocity=18.84 -> lower=-1.5707963267949 upper=1.5707963267949 effort=36.0 velocity=9.94333333333333; origin xyz=0 0 0 rpy=0 0 0 -> xyz=0 0 -0.104 rpy=0 0 0
- joint zarm_r4_joint: limit lower=-2.61799387799149 upper=0.0 effort=50.0 velocity=18.84 -> lower=-2.61799387799149 upper=0.0 effort=50.0 velocity=8.37333333333333; origin xyz=0.0200000000000024 0 -0.2837 rpy=0 0 0 -> xyz=0.02 0 -0.1797 rpy=0 0 0
- joint zarm_r5_joint: limit lower=-1.5707963267949 upper=1.5707963267949 effort=12.0 velocity=21.666 -> lower=-1.5707963267949 upper=1.5707963267949 effort=12.0 velocity=7.32666666666667; origin xyz=-0.0200000000000001 0 -0.127037274261587 rpy=0 0 0 -> xyz=-0.02 0 -0.1195 rpy=0 0 0
- joint zarm_r6_joint: limit lower=-0.698131700797732 upper=1.30899693899575 effort=12.0 velocity=21.666 -> lower=-0.698131700797732 upper=1.30899693899575 effort=12.0 velocity=7.32666666666667; origin xyz=0 0 -0.106462725738415 rpy=0 0 0 -> xyz=0 0 -0.114 rpy=0 0 0
- joint zarm_r7_joint: limit lower=-0.698131700797732 upper=0.698131700797732 effort=12.0 velocity=21.666 -> lower=-0.698131700797732 upper=0.698131700797732 effort=12.0 velocity=7.32666666666667; origin xyz=0 0 -0.0209999999999999 rpy=0 0 0 -> xyz=0 0 -0.022284 rpy=0 0 0

Commit message: sync https://www.lejuhub.com/highlydynamic/kuavo-ros-control/commit/cf9b9db4259f4b7882c028f149b66d0957840d73

File: src/kuavo_assets/models/biped_s14/urdf/biped_s14.urdf (robot description, URDF)
Before this commit: robot biped_s14, 41 links, 40 joints
Links:
- link base_link: mass 4.787076 -> 4.60775998
- link camera: mass 0.011119 -> 0.000011119
- link camera_base: mass 0.001 -> 0.00003927
- link leg_r1_link: mass 0.42877618 -> 0.42877473
- link leg_r2_link: mass 2.4999594 -> 2.50010758
- link leg_r3_link: mass 1.109669 -> 1.10966483
- link leg_r4_link: mass 1.55038362 -> 1.55001765
- link leg_r6_link: mass 0.34819511 -> 0.34819252
- link waist_yaw_link: mass 10.367276 -> 8.620776
- link zarm_r1_link: mass 0.37301773 -> 0.3730157
- link zarm_r2_link: mass 0.15112665 -> 0.15112869
- link zarm_r4_link: mass 0.16269033 -> 0.16269441
- link zhead_1_link: mass 0.32829 -> 1.03077542; geometry visual mesh filename=package://kuavo_assets/models/biped_s14/meshes/head_yaw.STL
- link zhead_2_link: mass 0.33162 -> 0.33654975; geometry visual mesh filename=package://kuavo_assets/models/biped_s14/meshes/head_pitch.S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
Joints:
- joint leg_r4_joint: origin xyz=-0.0209999999999396 0 -0.182000000000001 rpy=0 0 0 -> xyz=-0.0209999999999696 0 -0.181999999999961 rpy=0 0 0
- joint leg_r5_joint: origin xyz=0.0209999999999936 0 -0.235 rpy=0 0 0 -> xyz=0.0209999999999503 0 -0.235000000000001 rpy=0 0 0
- joint ll_foot_toe_joint: origin xyz=0.121 0.04149834 -0.0435 rpy=0 0 0 -> xyz=0.121 0.03824834 -0.0435 rpy=0 0 0
- joint rl_foot_toe_joint: origin xyz=0.121 0.04149834 -0.0435 rpy=0 0 0 -> xyz=0.121 0.03824834 -0.0435 rpy=0 0 0
- joint zarm_r4_joint: origin xyz=0 0 -0.187999999999989 rpy=0 0 0 -> xyz=0 0 -0.187999999999999 rpy=0 0 0
- joint zhead_1_joint: origin xyz=0.00400001 2.92e-06 0.35618885 rpy=0 0 0 -> xyz=0 0 0.35618885 rpy=0 0 0

File: src/kuavo_assets/models/biped_s14/urdf/biped_s14_gazebo.urdf (robot description, URDF)
Before this commit: robot biped_s14, 41 links, 40 joints
Links:
- link base_link: mass 6.620576 -> 4.60775998
- link camera: mass 0.011119 -> 0.000011119
- link camera_base: mass 3.927E-05 -> 0.00003927
- link leg_r1_link: mass 0.42877618 -> 0.42877473
- link leg_r2_link: mass 2.4999594 -> 2.50010758
- link leg_r3_link: mass 1.109669 -> 1.10966483
- link leg_r4_link: mass 1.55038362 -> 1.55001765
- link leg_r6_link: mass 0.34819511 -> 0.34819252
- link waist_yaw_link: mass 4.60775998 -> 8.620776
- link zarm_r1_link: mass 0.37301773 -> 0.3730157
- link zarm_r2_link: mass 0.15112665 -> 0.15112869
- link zarm_r4_link: mass 0.16269033 -> 0.16269441
- link zhead_1_link: mass 0.32829 -> 1.03077542; geometry visual mesh filename=package://kuavo_assets/models/biped_s14/meshes/head_yaw.STL
- link zhead_2_link: mass 0.33162 -> 0.33654975; geometry visual mesh filename=package://kuavo_assets/models/biped_s14/meshes/head_pitch.S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
Joints:
- joint l_foot_heel_joint: origin xyz=-0.084 0.0 -0.0435 rpy=0 0 0 -> xyz=-0.04 -0.03824834 -0.0435 rpy=0 0 0
- joint l_foot_toe_joint: origin xyz=0.121 0.0 -0.0435 rpy=0 0 0 -> xyz=-0.04 0.03824834 -0.0435 rpy=0 0 0
- joint leg_r4_joint: origin xyz=-0.0209999999999396 0 -0.182000000000001 rpy=0 0 0 -> xyz=-0.0209999999999696 0 -0.181999999999961 rpy=0 0 0
- joint leg_r5_joint: origin xyz=0.0209999999999936 0 -0.235 rpy=0 0 0 -> xyz=0.0209999999999503 0 -0.235000000000001 rpy=0 0 0
- joint ll_foot_toe_joint: origin xyz=0.121 0.04149834 -0.0435 rpy=0 0 0 -> xyz=0.121 0.03824834 -0.0435 rpy=0 0 0
- joint r_foot_heel_joint: origin xyz=-0.084 0.0 -0.0435 rpy=0 0 0 -> xyz=-0.04 -0.03824834 -0.0435 rpy=0 0 0
- joint r_foot_toe_joint: origin xyz=0.121 0.0 -0.0435 rpy=0 0 0 -> xyz=-0.04 0.03824834 -0.0435 rpy=0 0 0
- joint rl_foot_toe_joint: origin xyz=0.121 0.04149834 -0.0435 rpy=0 0 0 -> xyz=0.121 0.03824834 -0.0435 rpy=0 0 0
- joint zarm_r4_joint: origin xyz=0 0 -0.187999999999989 rpy=0 0 0 -> xyz=0 0 -0.187999999999999 rpy=0 0 0
- joint zhead_1_joint: origin xyz=0.00400001 2.92e-06 0.35618885 rpy=0 0 0 -> xyz=0 0 0.35618885 rpy=0 0 0

File: src/kuavo_assets/models/biped_s14/urdf/drake/biped_v3.urdf (robot description, URDF)
Before this commit: robot biped_v3, 14 links, 13 joints
Links:
- link leg_r1_link: mass 0.42877618 -> 0.42877473
- link leg_r2_link: mass 2.4999594 -> 2.50010758
- link leg_r3_link: mass 1.109669 -> 1.10966483
- link leg_r4_link: mass 1.55038362 -> 1.55001765
- link leg_r6_link: mass 0.34819511 -> 0.34819252
- link torso: mass 13.93068758 -> 12.700276
Joints:
- joint leg_r4_joint: origin xyz=-0.0209999999999396 0 -0.182000000000001 rpy=0 0 0 -> xyz=-0.0209999999999696 0 -0.181999999999961 rpy=0 0 0
- joint leg_r5_joint: origin xyz=0.0209999999999936 0 -0.235 rpy=0 0 0 -> xyz=0.0209999999999503 0 -0.235000000000001 rpy=0 0 0

File: src/kuavo_assets/models/biped_s14/urdf/drake/biped_v3_all_joint.urdf (robot description, URDF)
Before this commit: robot biped_v3_all_joint, 30 links, 25 joints
Links:
- link torso: mass 8.72811242 -> 7.49741242

File: src/kuavo_assets/models/biped_s14/urdf/drake/biped_v3_full.urdf (robot description, URDF)
Before this commit: robot biped_v3_full, 22 links, 21 joints
Links:
- link torso: mass 11.218576 -> 9.987876

Commit message: sync https://www.lejuhub.com/highlydynamic/kuavo-ros-control/commit/718500915a2698d8eefecab292ff79cb31b85ed3

File: src/kuavo_assets/models/biped_s14/urdf/biped_s14.urdf (robot description, URDF)
Before this commit: robot biped_s14, 41 links, 40 joints
Links:
- link zarm_l4_link: mass 0.16269441 -> 0.56269441
- link zarm_r4_link: mass 0.16269441 -> 0.56269441

File: src/kuavo_assets/models/biped_s14/urdf/biped_s14_gazebo.urdf (robot description, URDF)
Before this commit: robot biped_s14, 41 links, 40 joints
Links:
- link zarm_l4_link: mass 0.16269441 -> 0.56269441
- link zarm_r4_link: mass 0.16269441 -> 0.56269441
