Commit message: sync https://www.lejuhub.com/highlydynamic/kuavo-ros-control/commit/c82c88be048abfd2a3e150fcc05864eae1a36bba

File: src/kuavo_assets/models/biped_s14/urdf/biped_s14.urdf (robot description, URDF)
Before this commit: robot biped_s14, 41 links, 40 joints
Links:
- link base_link: mass 4.787076 -> 4.60775998
- link camera: mass 0.011119 -> 0.000011119
- link camera_base: mass 0.001 -> 0.00003927
- link leg_r1_link: mass 0.42877618 -> 0.42877473
- link leg_r2_link: mass 2.4999594 -> 2.50010758
- link leg_r3_link: mass 1.109669 -> 1.10966483
- link leg_r4_link: mass 1.55038362 -> 1.55001765
- link leg_r6_link: mass 0.34819511 -> 0.34819252
- link waist_yaw_link: mass 4.60775998 -> 8.620776
- link zarm_l4_link: mass 0.16269441 -> 0.56269441
- link zarm_r1_link: mass 0.37301773 -> 0.3730157
- link zarm_r2_link: mass 0.15112665 -> 0.15112869
- link zarm_r4_link: mass 0.16269033 -> 0.56269441
- link zhead_1_link: mass 0.32829 -> 1.03077542; geometry visual mesh filename=package://kuavo_assets/models/biped_s14/meshes/head_yaw.STL
- link zhead_2_link: mass 0.33162 -> 0.33654975; geometry visual mesh filename=package://kuavo_assets/models/biped_s14/meshes/head_pitch.S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
Joints:
- joint leg_r4_joint: origin xyz=-0.0209999999999396 0 -0.182000000000001 rpy=0 0 0 -> xyz=-0.0209999999999696 0 -0.181999999999961 rpy=0 0 0
- joint leg_r5_joint: origin xyz=0.0209999999999936 0 -0.235 rpy=0 0 0 -> xyz=0.0209999999999503 0 -0.235000000000001 rpy=0 0 0
- joint ll_foot_toe_joint: origin xyz=0.121 0.04149834 -0.0435 rpy=0 0 0 -> xyz=0.121 0.03824834 -0.0435 rpy=0 0 0
- joint rl_foot_toe_joint: origin xyz=0.121 0.04149834 -0.0435 rpy=0 0 0 -> xyz=0.121 0.03824834 -0.0435 rpy=0 0 0
- joint zarm_r4_joint: origin xyz=0 0 -0.187999999999989 rpy=0 0 0 -> xyz=0 0 -0.187999999999999 rpy=0 0 0
- joint zhead_1_joint: origin xyz=0.00400001 2.92e-06 0.35618885 rpy=0 0 0 -> xyz=0 0 0.35618885 rpy=0 0 0

File: src/kuavo_assets/models/biped_s14/urdf/biped_s14_gazebo.urdf (robot description, URDF)
Before this commit: robot biped_s14, 41 links, 40 joints
Links:
- link base_link: mass 4.787076 -> 4.60775998
- link camera: mass 0.011119 -> 0.000011119
- link camera_base: mass 3.927E-05 -> 0.00003927
- link leg_r1_link: mass 0.42877618 -> 0.42877473
- link leg_r2_link: mass 2.4999594 -> 2.50010758
- link leg_r3_link: mass 1.109669 -> 1.10966483
- link leg_r4_link: mass 1.55038362 -> 1.55001765
- link leg_r6_link: mass 0.34819511 -> 0.34819252
- link waist_yaw_link: mass 4.60775998 -> 8.620776
- link zarm_l4_link: mass 0.16269441 -> 0.56269441
- link zarm_r1_link: mass 0.37301773 -> 0.3730157
- link zarm_r2_link: mass 0.15112665 -> 0.15112869
- link zarm_r4_link: mass 0.16269033 -> 0.56269441
- link zhead_1_link: mass 0.32829 -> 1.03077542; geometry visual mesh filename=package://kuavo_assets/models/biped_s14/meshes/head_yaw.STL
- link zhead_2_link: mass 0.33162 -> 0.33654975; geometry visual mesh filename=package://kuavo_assets/models/biped_s14/meshes/head_pitch.S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
Joints:
- joint l_foot_heel_joint: origin xyz=-0.084 0.0 -0.0435 rpy=0 0 0 -> xyz=-0.04 -0.03824834 -0.0435 rpy=0 0 0
- joint l_foot_toe_joint: origin xyz=0.121 0.0 -0.0435 rpy=0 0 0 -> xyz=-0.04 0.03824834 -0.0435 rpy=0 0 0
- joint leg_r4_joint: origin xyz=-0.0209999999999396 0 -0.182000000000001 rpy=0 0 0 -> xyz=-0.0209999999999696 0 -0.181999999999961 rpy=0 0 0
- joint leg_r5_joint: origin xyz=0.0209999999999936 0 -0.235 rpy=0 0 0 -> xyz=0.0209999999999503 0 -0.235000000000001 rpy=0 0 0
- joint ll_foot_toe_joint: origin xyz=0.121 0.04149834 -0.0435 rpy=0 0 0 -> xyz=0.121 0.03824834 -0.0435 rpy=0 0 0
- joint r_foot_heel_joint: origin xyz=-0.084 0.0 -0.0435 rpy=0 0 0 -> xyz=-0.04 -0.03824834 -0.0435 rpy=0 0 0
- joint r_foot_toe_joint: origin xyz=0.121 0.0 -0.0435 rpy=0 0 0 -> xyz=-0.04 0.03824834 -0.0435 rpy=0 0 0
- joint rl_foot_toe_joint: origin xyz=0.121 0.04149834 -0.0435 rpy=0 0 0 -> xyz=0.121 0.03824834 -0.0435 rpy=0 0 0
- joint zarm_r4_joint: origin xyz=0 0 -0.187999999999989 rpy=0 0 0 -> xyz=0 0 -0.187999999999999 rpy=0 0 0
- joint zhead_1_joint: origin xyz=0.00400001 2.92e-06 0.35618885 rpy=0 0 0 -> xyz=0 0 0.35618885 rpy=0 0 0

File: src/kuavo_assets/models/biped_s14/urdf/drake/biped_v3.urdf (robot description, URDF)
Before this commit: robot biped_v3, 14 links, 13 joints
Links:
- link leg_r1_link: mass 0.42877618 -> 0.42877473
- link leg_r2_link: mass 2.4999594 -> 2.50010758
- link leg_r3_link: mass 1.109669 -> 1.10966483
- link leg_r4_link: mass 1.55038362 -> 1.55001765
- link leg_r6_link: mass 0.34819511 -> 0.34819252
- link torso: mass 12.09718758 -> 13.500276
Joints:
- joint leg_r4_joint: origin xyz=-0.0209999999999396 0 -0.182000000000001 rpy=0 0 0 -> xyz=-0.0209999999999696 0 -0.181999999999961 rpy=0 0 0
- joint leg_r5_joint: origin xyz=0.0209999999999936 0 -0.235 rpy=0 0 0 -> xyz=0.0209999999999503 0 -0.235000000000001 rpy=0 0 0
