Commit message: sync https://www.lejuhub.com/highlydynamic/kuavo-ros-control/commit/d6c2d163885a17925db87e64d0fcd454f5f1afd0

File: src/kuavo_assets/models/biped_s13/urdf/drake/biped_v3_all_joint.urdf (robot description, URDF)
Before this commit: robot biped_v3_all_joint, 30 links, 25 joints
Links:
- link torso: mass -.07761242 -> 0.07761242
