Commit message: sync https://www.lejuhub.com/highlydynamic/kuavo-ros-control/commit/885aa30a3f1bf7249755f8e9120c2c80b51279cf

File: src/kuavo_assets/models/biped_s49/urdf/biped_s49.urdf (robot description, URDF)
Before this commit: robot biped_s49, 73 links, 72 joints
Links:
- removed link l_Index_prox
- removed link l_hand_camera
- removed link l_hand_tripod
- removed link l_index_dist
- removed link l_little_dist
- removed link l_little_prox
- removed link l_middle_dist
- removed link l_middle_prox
- removed link l_palm
- removed link l_ring_dist
- removed link l_ring_prox
- removed link l_thumb_dist
- removed link l_thumb_prox
- removed link r_hand_camera
- removed link r_hand_tripod
- removed link r_index_dist
- removed link r_index_prox
- removed link r_little_dist
- removed link r_little_prox
- removed link r_middle_dist
- removed link r_middle_prox
- removed link r_palm
- removed link r_ring_dist
- removed link r_ring_prox
- removed link r_thumb_dist
- removed link r_thumb_prox
- added link l_b_bar-1, mass 0.045; visual mesh filename=package://kuavo_assets/models/biped_s49/meshes/l_b_bar-1.STL
- added link l_b_bar-2, mass 0.009; visual mesh filename=package://kuavo_assets/models/biped_s49/meshes/l_b_bar-2.STL
- added link l_b_bar-3, mass 0.013; visual mesh filename=package://kuavo_assets/models/biped_s49/meshes/l_b_bar-3.STL
- added link l_b_fingers, mass 0.014; visual mesh filename=package://kuavo_assets/models/biped_s49/meshes/l_b_fingers.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
- added link l_f_bar-1, mass 0.045; visual mesh filename=package://kuavo_assets/models/biped_s49/meshes/l_f_bar-1.STL
- added link l_f_bar-2, mass 0.009; visual mesh filename=package://kuavo_assets/models/biped_s49/meshes/l_f_bar-2.STL
- added link l_f_bar-3, mass 0.013; visual mesh filename=package://kuavo_assets/models/biped_s49/meshes/l_f_bar-3.STL
- added link l_f_fingers, mass 0.014; visual mesh filename=package://kuavo_assets/models/biped_s49/meshes/l_f_fingers.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
- added link r_b_bar-1, mass 0.045; visual mesh filename=package://kuavo_assets/models/biped_s49/meshes/r_b_bar-1.STL
- added link r_b_bar-2, mass 0.009; visual mesh filename=package://kuavo_assets/models/biped_s49/meshes/r_b_bar-2.STL
- added link r_b_bar-3, mass 0.013; visual mesh filename=package://kuavo_assets/models/biped_s49/meshes/r_b_bar-3.STL
- added link r_b_fingers, mass 0.014; visual mesh filename=package://kuavo_assets/models/biped_s49/meshes/r_b_fingers.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
- added link r_f_bar-1, mass 0.045; visual mesh filename=package://kuavo_assets/models/biped_s49/meshes/r_f_bar_1.STL
- added link r_f_bar-2, mass 0.009; visual mesh filename=package://kuavo_assets/models/biped_s49/meshes/r_f_bar-2.STL
- added link r_f_bar-3, mass 0.013; visual mesh filename=package://kuavo_assets/models/biped_s49/meshes/r_f_bar-3.STL
- added link r_f_fingers, mass 0.014; visual mesh filename=package://kuavo_assets/models/biped_s49/meshes/r_f_finger.S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
- link base_link: mass 27.41553803 -> 24.09723803; geometry visual mesh filename=package://kuavo_assets/models/biped_s49/meshes/torso.STL
- link camera_base: mass 0.0000392699081698732 -> 3.92699081698732E-05
- link zarm_l2_link: geometry visual mesh filename=package://kuavo_assets/models/biped_s49/meshes/l_arm_roll.S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
- link zarm_l4_link: geometry visual mesh filename=package://kuavo_assets/models/biped_s49/meshes/l_forearm.STL
- link zarm_l7_link: mass 0.0542110173081966 -> 0.64; geometry visual mesh filename=package://kuavo_assets/models/biped_s49/meshes/l_hand_pitch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
- link zarm_r2_link: geometry visual mesh filename=package://kuavo_assets/models/biped_s49/meshes/r_arm_roll.S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
- link zarm_r4_link: geometry visual mesh filename=package://kuavo_assets/models/biped_s49/meshes/r_forearm.STL
- link zarm_r7_link: mass 0.0542110173081966 -> 0.64; geometry visual mesh filename=package://kuavo_assets/models/biped_s49/meshes/r_hand_pitch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
- link zhead_1_link: geometry visual mesh filename=package://kuavo_assets/models/biped_s49/meshes/head_yaw.STL
Joints:
- removed joint base_link_to_dummy_link
- removed joint l_hand_camera_joint
- removed joint l_hand_tripod_joint
- removed joint l_indexMCP
- removed joint l_indexPIP
- removed joint l_littleMCP
- removed joint l_littlePIP
- removed joint l_middleMCP
- removed joint l_middlePIP
- removed joint l_palm_fixed_joint
- removed joint l_ringMCP
- removed joint l_ringPIP
- removed joint l_thumbCMC
- removed joint l_thumbMCP
- removed joint r_hand_camera_joint
- removed joint r_hand_tripod_joint
- removed joint r_indexMCP
- removed joint r_indexPIP
- removed joint r_littleMCP
- removed joint r_littlePIP
- removed joint r_middleMCP
- removed joint r_middlePIP
- removed joint r_palm_fixed_joint
- removed joint r_ringMCP
- removed joint r_ringPIP
- removed joint r_thumbCMC
- removed joint r_thumbMCP
- added joint dummy_to_base_link: type fixed, parent dummy_link, child base_link, origin xyz=0 0 0 rpy=0 0 0
- added joint l_b_bar-1: type revolute, parent zarm_l7_link, child l_b_bar-1, origin xyz=-0.0219999996097237 0 -0.1114 rpy=0 0 0, axis 0 1 0, limit lower=-0.698 upper=0.698 effort=5 velocity=5
- added joint l_b_bar-2: type fixed, parent l_b_bar-1, child l_b_bar-2, origin xyz=-0.0254380979411351 0 -0.0464962705293328 rpy=0 0 0, axis 0 1 0
- added joint l_b_bar-3: type revolute, parent zarm_l7_link, child l_b_bar-3, origin xyz=-0.0239578924930216 0 -0.135271672920607 rpy=0 0 0, axis 0 1 0, limit lower=-0.698 upper=0.698 effort=5 velocity=5
- added joint l_b_fingers: type fixed, parent l_b_bar-2, child l_b_fingers, origin xyz=0.0191548518271917 0 -0.0292932014550803 rpy=0 0 0, axis 0 1 0
- added joint l_f_bar-1_joint: type revolute, parent zarm_l7_link, child l_f_bar-1, origin xyz=0.0220000003906073 0 -0.111399999999999 rpy=0 0 0, axis 0 1 0, limit lower=-0.698 upper=0.698 effort=5 velocity=5
- added joint l_f_bar-2: type fixed, parent l_f_bar-1, child l_f_bar-2, origin xyz=0.025438097941138 0 -0.0464962705293307 rpy=0 0 0, axis 0 1 0
- added joint l_f_bar-3: type revolute, parent zarm_l7_link, child l_f_bar-3, origin xyz=0.0239578932739072 0 -0.135271672920607 rpy=0 0 0, axis 0 1 0, limit lower=-0.698 upper=0.698 effort=5 velocity=5
- added joint l_f_fingers: type fixed, parent l_f_bar-2, child l_f_fingers, origin xyz=-0.0191548518271909 0 -0.0292932014550821 rpy=0 0 0, axis 0 1 0
- added joint r_b_bar-1: type revolute, parent zarm_r7_link, child r_b_bar-1, origin xyz=-0.0219999996097237 0 -0.1114 rpy=0 0 0, axis 0 1 0, limit lower=-0.698 upper=0.698 effort=5 velocity=5
- added joint r_b_bar-2: type fixed, parent r_b_bar-1, child r_b_bar-2, origin xyz=-0.0254380979411353 0 -0.0464962705293326 rpy=0 0 0, axis 0 1 0
- added joint r_b_bar-3: type revolute, parent zarm_r7_link, child r_b_bar-3, origin xyz=-0.0239578932738948 0 -0.135271672920607 rpy=0 0 0, axis 0 1 0, limit lower=-0.698 upper=0.698 effort=5 velocity=5
- added joint r_b_fingers: type fixed, parent r_b_bar-2, child r_b_fingers, origin xyz=0.0191548518271923 0 -0.0292932014550809 rpy=0 0 0, axis 0 1 0
- added joint r_f_bar-1_joint: type revolute, parent zarm_r7_link, child r_f_bar-1, origin xyz=0.0220000003906073 0 -0.111399999999999 rpy=0 0 0, axis 0 1 0, limit lower=-0.698 upper=0.698 effort=5 velocity=5
- added joint r_f_bar-2: type fixed, parent r_f_bar-1, child r_f_bar-2, origin xyz=0.025438097941138 0 -0.0464962705293307 rpy=0 0 0, axis 0 1 0
- added joint r_f_bar-3: type revolute, parent zarm_r7_link, child r_f_bar-3, origin xyz=0.0239578932739072 0 -0.135271672920607 rpy=0 0 0, axis 0 1 0, limit lower=-0.698 upper=0.698 effort=5 velocity=5
- added joint r_f_fingers: type fixed, parent r_f_bar-2, child r_f_fingers, origin xyz=-0.0191548518271909 0 -0.0292932014550821 rpy=0 0 0, axis 0 1 0

Commit message: sync https://www.lejuhub.com/highlydynamic/kuavo-ros-control/commit/bbf749b54faba0b8fce634ed3222667027188a79

File: src/kuavo_assets/models/biped_s49/urdf/biped_s49.urdf (robot description, URDF)
Before this commit: robot biped_s49, 73 links, 72 joints
Links:
- link base_link: mass 27.41553803 -> 28.27893803
