Commit message: sync https://www.lejuhub.com/highlydynamic/kuavo-ros-control/commit/2d95e6e9b7659227cc9387dccb4a5949c482d226

File: src/kuavo_assets/models/biped_s47/urdf/biped_s47.urdf (robot description, URDF)
Before this commit: robot biped_s47, 62 links, 61 joints
Links:
- removed link l_b_claw_1
- removed link l_b_claw_2
- removed link l_b_claw_3
- removed link l_b_finger
- removed link l_f_claw_1
- removed link l_f_claw_2
- removed link l_f_claw_3
- removed link l_f_finger
- removed link r_b_claw_1
- removed link r_b_claw_2
- removed link r_b_claw_3
- removed link r_b_finger
- removed link r_f_claw_1
- removed link r_f_claw_2
- removed link r_f_claw_3
- removed link r_f_finger
- added link l_b_bar-1, mass 0.045; visual mesh filename=package://kuavo_assets/models/biped_s47/meshes/l_b_bar-1.STL
- added link l_b_bar-2, mass 0.009; visual mesh filename=package://kuavo_assets/models/biped_s47/meshes/l_b_bar-2.STL
- added link l_b_bar-3, mass 0.013; visual mesh filename=package://kuavo_assets/models/biped_s47/meshes/l_b_bar-3.STL
- added link l_b_fingers, mass 0.014; visual mesh filename=package://kuavo_assets/models/biped_s47/meshes/l_b_fingers.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
- added link l_f_bar-1, mass 0.045; visual mesh filename=package://kuavo_assets/models/biped_s47/meshes/l_f_bar-1.STL
- added link l_f_bar-2, mass 0.009; visual mesh filename=package://kuavo_assets/models/biped_s47/meshes/l_f_bar-2.STL
- added link l_f_bar-3, mass 0.013; visual mesh filename=package://kuavo_assets/models/biped_s47/meshes/l_f_bar-3.STL
- added link l_f_fingers, mass 0.014; visual mesh filename=package://kuavo_assets/models/biped_s47/meshes/l_f_fingers.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
- added link l_hand_camera, mass 0.038145442577304; collision mesh filename=package://kuavo_assets/models/biped_s47/meshes/l_hand_camer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; visual mesh filename=package://kuavo_assets/models/biped_s47/meshes/l_hand_camer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
- added link l_hand_tripod, mass 0.0342669089979502; collision mesh filename=package://kuavo_assets/models/biped_s47/meshes/l_hand_tripo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; visual mesh filename=package://kuavo_assets/models/biped_s47/meshes/l_hand_tripo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
- added link r_b_bar-1, mass 0.045; visual mesh filename=package://kuavo_assets/models/biped_s47/meshes/r_b_bar-1.STL
- added link r_b_bar-2, mass 0.009; visual mesh filename=package://kuavo_assets/models/biped_s47/meshes/r_b_bar-2.STL
- added link r_b_bar-3, mass 0.013; visual mesh filename=package://kuavo_assets/models/biped_s47/meshes/r_b_bar-3.STL
- added link r_b_fingers, mass 0.014; visual mesh filename=package://kuavo_assets/models/biped_s47/meshes/r_b_fingers.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
- added link r_f_bar-1, mass 0.045; visual mesh filename=package://kuavo_assets/models/biped_s47/meshes/r_f_bar_1.STL
- added link r_f_bar-2, mass 0.009; visual mesh filename=package://kuavo_assets/models/biped_s47/meshes/r_f_bar-2.STL
- added link r_f_bar-3, mass 0.013; visual mesh filename=package://kuavo_assets/models/biped_s47/meshes/r_f_bar-3.STL
- added link r_f_fingers, mass 0.014; visual mesh filename=package://kuavo_assets/models/biped_s47/meshes/r_f_finger.S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
- added link r_hand_camera, mass 0.038145442577304; collision mesh filename=package://kuavo_assets/models/biped_s47/meshes/r_hand_camer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; visual mesh filename=package://kuavo_assets/models/biped_s47/meshes/r_hand_camer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
- added link r_hand_tripod, mass 0.034266881719861; collision mesh filename=package://kuavo_assets/models/biped_s47/meshes/r_hand_tripo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; visual mesh filename=package://kuavo_assets/models/biped_s47/meshes/r_hand_tripo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
- link base_link: mass 27.65693803 -> 27.65133803
Joints:
- removed joint l_b_claw_1
- removed joint l_b_claw_2
- removed joint l_b_claw_3
- removed joint l_b_finger
- removed joint l_f_claw_1
- removed joint l_f_claw_2
- removed joint l_f_claw_3
- removed joint l_f_finger
- removed joint r_b_claw_1
- removed joint r_b_claw_2
- removed joint r_b_claw_3
- removed joint r_b_finger
- removed joint r_f_claw_1
- removed joint r_f_claw_2
- removed joint r_f_claw_3
- removed joint r_f_finger
- added joint l_b_bar-1: type revolute, parent zarm_l7_link, child l_b_bar-1, origin xyz=-0.0219999996097237 0 -0.1114 rpy=0 0 0, axis 0 1 0, limit lower=-0.698 upper=0.698 effort=5 velocity=5
- added joint l_b_bar-2: type fixed, parent l_b_bar-1, child l_b_bar-2, origin xyz=-0.0254380979411351 0 -0.0464962705293328 rpy=0 0 0, axis 0 1 0
- added joint l_b_bar-3: type revolute, parent zarm_l7_link, child l_b_bar-3, origin xyz=-0.0239578924930216 0 -0.135271672920607 rpy=0 0 0, axis 0 1 0, limit lower=-0.698 upper=0.698 effort=5 velocity=5
- added joint l_b_fingers: type fixed, parent l_b_bar-2, child l_b_fingers, origin xyz=0.0191548518271917 0 -0.0292932014550803 rpy=0 0 0, axis 0 1 0
- added joint l_f_bar-1_joint: type revolute, parent zarm_l7_link, child l_f_bar-1, origin xyz=0.0220000003906073 0 -0.111399999999999 rpy=0 0 0, axis 0 1 0, limit lower=-0.698 upper=0.698 effort=5 velocity=5
- added joint l_f_bar-2: type fixed, parent l_f_bar-1, child l_f_bar-2, origin xyz=0.025438097941138 0 -0.0464962705293307 rpy=0 0 0, axis 0 1 0
- added joint l_f_bar-3: type revolute, parent zarm_l7_link, child l_f_bar-3, origin xyz=0.0239578932739072 0 -0.135271672920607 rpy=0 0 0, axis 0 1 0, limit lower=-0.698 upper=0.698 effort=5 velocity=5
- added joint l_f_fingers: type fixed, parent l_f_bar-2, child l_f_fingers, origin xyz=-0.0191548518271909 0 -0.0292932014550821 rpy=0 0 0, axis 0 1 0
- added joint l_hand_camera_joint: type fixed, parent l_hand_tripod, child l_hand_camera, origin xyz=0.11540559159102 -0.0145586110669961 -0.110123491595499 rpy=1.919862177193763 0.753528063917894 -2.897246568680842, axis 0 0 0
- added joint l_hand_tripod_joint: type fixed, parent zarm_l7_link, child l_hand_tripod, origin xyz=0.0 0.0 0.0 rpy=0.0 0.0 0.0, axis 0 0 0
- added joint r_b_bar-1: type revolute, parent zarm_r7_link, child r_b_bar-1, origin xyz=-0.0219999996097237 0 -0.1114 rpy=0 0 0, axis 0 1 0, limit lower=-0.698 upper=0.698 effort=5 velocity=5
- added joint r_b_bar-2: type fixed, parent r_b_bar-1, child r_b_bar-2, origin xyz=-0.0254380979411353 0 -0.0464962705293326 rpy=0 0 0, axis 0 1 0
- added joint r_b_bar-3: type revolute, parent zarm_r7_link, child r_b_bar-3, origin xyz=-0.0239578932738948 0 -0.135271672920607 rpy=0 0 0, axis 0 1 0, limit lower=-0.698 upper=0.698 effort=5 velocity=5
- added joint r_b_fingers: type fixed, parent r_b_bar-2, child r_b_fingers, origin xyz=0.0191548518271923 0 -0.0292932014550809 rpy=0 0 0, axis 0 1 0
- added joint r_f_bar-1_joint: type revolute, parent zarm_r7_link, child r_f_bar-1, origin xyz=0.0220000003906073 0 -0.111399999999999 rpy=0 0 0, axis 0 1 0, limit lower=-0.698 upper=0.698 effort=5 velocity=5
- added joint r_f_bar-2: type fixed, parent r_f_bar-1, child r_f_bar-2, origin xyz=0.025438097941138 0 -0.0464962705293307 rpy=0 0 0, axis 0 1 0
- added joint r_f_bar-3: type revolute, parent zarm_r7_link, child r_f_bar-3, origin xyz=0.0239578932739072 0 -0.135271672920607 rpy=0 0 0, axis 0 1 0, limit lower=-0.698 upper=0.698 effort=5 velocity=5
- added joint r_f_fingers: type fixed, parent r_f_bar-2, child r_f_fingers, origin xyz=-0.0191548518271909 0 -0.0292932014550821 rpy=0 0 0, axis 0 1 0
- added joint r_hand_camera_joint: type fixed, parent r_hand_tripod, child r_hand_camera, origin xyz=0.115405591590931 0.0154312352120435 -0.107724128430896 rpy=1.208853693239594  0.751879414295006 2.888346587751982, axis 0 0 0
- added joint r_hand_tripod_joint: type fixed, parent zarm_r7_link, child r_hand_tripod, origin xyz=0.0 0.0 0.0 rpy=0.0 0.0 0.0, axis 0 0 0

File: src/kuavo_assets/models/biped_s49/urdf/biped_s49.urdf (robot description, URDF)
Before this commit: robot biped_s49, 63 links, 62 joints
Links:
- removed link l_b_bar-1
- removed link l_b_bar-2
- removed link l_b_bar-3
- removed link l_b_fingers
- removed link l_f_bar-1
- removed link l_f_bar-2
- removed link l_f_bar-3
- removed link l_f_fingers
- removed link r_b_bar-1
- removed link r_b_bar-2
- removed link r_b_bar-3
- removed link r_b_fingers
- removed link r_f_bar-1
- removed link r_f_bar-2
- removed link r_f_bar-3
- removed link r_f_fingers
- added link l_Index_prox, mass 0.008; collision mesh filename=package://kuavo_assets/models/biped_s49/meshes/l_Index_prox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; visual mesh filename=package://kuavo_assets/models/biped_s49/meshes/l_Index_prox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
- added link l_hand_camera, mass 0.038145442577304; collision mesh filename=package://kuavo_assets/models/biped_s49/meshes/l_hand_camer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; visual mesh filename=package://kuavo_assets/models/biped_s49/meshes/l_hand_camer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
- added link l_hand_tripod, mass 0.0342669089979502; collision mesh filename=package://kuavo_assets/models/biped_s49/meshes/l_hand_tripo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; visual mesh filename=package://kuavo_assets/models/biped_s49/meshes/l_hand_tripo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
- added link l_index_dist, mass 0.011; collision mesh filename=package://kuavo_assets/models/biped_s49/meshes/l_index_dist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; visual mesh filename=package://kuavo_assets/models/biped_s49/meshes/l_index_dist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
- added link l_little_dist, mass 0.008; collision mesh filename=package://kuavo_assets/models/biped_s49/meshes/l_little_dis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; visual mesh filename=package://kuavo_assets/models/biped_s49/meshes/l_little_dis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
- added link l_little_prox, mass 0.008; collision mesh filename=package://kuavo_assets/models/biped_s49/meshes/l_little_pro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; visual mesh filename=package://kuavo_assets/models/biped_s49/meshes/l_little_pro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
- added link l_middle_dist, mass 0.011; collision mesh filename=package://kuavo_assets/models/biped_s49/meshes/l_middle_dis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; visual mesh filename=package://kuavo_assets/models/biped_s49/meshes/l_middle_dis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
- added link l_middle_prox, mass 0.011; collision mesh filename=package://kuavo_assets/models/biped_s49/meshes/l_middle_pro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; visual mesh filename=package://kuavo_assets/models/biped_s49/meshes/l_middle_pro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
- added link l_palm, mass 0.427; collision mesh filename=package://kuavo_assets/models/biped_s49/meshes/l_palm.STL; visual mesh filename=package://kuavo_assets/models/biped_s49/meshes/l_palm.STL
- added link l_ring_dist, mass 0.008; collision mesh filename=package://kuavo_assets/models/biped_s49/meshes/l_ring_dist.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; visual mesh filename=package://kuavo_assets/models/biped_s49/meshes/l_ring_dist.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
- added link l_ring_prox, mass 0.011; collision mesh filename=package://kuavo_assets/models/biped_s49/meshes/l_ring_prox.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; visual mesh filename=package://kuavo_assets/models/biped_s49/meshes/l_ring_prox.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
- added link l_thumb_dist, mass 0.04; collision mesh filename=package://kuavo_assets/models/biped_s49/meshes/l_thumb_dist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; visual mesh filename=package://kuavo_assets/models/biped_s49/meshes/l_thumb_dist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
- added link l_thumb_prox, mass 0.005; collision mesh filename=package://kuavo_assets/models/biped_s49/meshes/l_thumb_prox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; visual mesh filename=package://kuavo_assets/models/biped_s49/meshes/l_thumb_prox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
- added link r_hand_camera, mass 0.038145442577304; collision mesh filename=package://kuavo_assets/models/biped_s49/meshes/r_hand_camer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; visual mesh filename=package://kuavo_assets/models/biped_s49/meshes/r_hand_camer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
- added link r_hand_tripod, mass 0.034266881719861; collision mesh filename=package://kuavo_assets/models/biped_s49/meshes/r_hand_tripo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; visual mesh filename=package://kuavo_assets/models/biped_s49/meshes/r_hand_tripo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
- added link r_index_dist, mass 0.011; collision mesh filename=package://kuavo_assets/models/biped_s49/meshes/r_index_dist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; visual mesh filename=package://kuavo_assets/models/biped_s49/meshes/r_index_dist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
- added link r_index_prox, mass 0.008; collision mesh filename=package://kuavo_assets/models/biped_s49/meshes/r_index_prox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; visual mesh filename=package://kuavo_assets/models/biped_s49/meshes/r_index_prox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
- added link r_little_dist, mass 0.008; collision mesh filename=package://kuavo_assets/models/biped_s49/meshes/r_little_dis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; visual mesh filename=package://kuavo_assets/models/biped_s49/meshes/r_little_dis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
- added link r_little_prox, mass 0.008; collision mesh filename=package://kuavo_assets/models/biped_s49/meshes/r_little_pro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; visual mesh filename=package://kuavo_assets/models/biped_s49/meshes/r_little_pro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
- added link r_middle_dist, mass 0.011; collision mesh filename=package://kuavo_assets/models/biped_s49/meshes/r_middle_dis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; visual mesh filename=package://kuavo_assets/models/biped_s49/meshes/r_middle_dis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
- added link r_middle_prox, mass 0.011; collision mesh filename=package://kuavo_assets/models/biped_s49/meshes/r_middle_pro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; visual mesh filename=package://kuavo_assets/models/biped_s49/meshes/r_middle_pro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
- added link r_palm, mass 0.427; collision mesh filename=package://kuavo_assets/models/biped_s49/meshes/r_palm.STL; visual mesh filename=package://kuavo_assets/models/biped_s49/meshes/r_palm.STL
- added link r_ring_dist, mass 0.008; collision mesh filename=package://kuavo_assets/models/biped_s49/meshes/r_ring_dist.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; visual mesh filename=package://kuavo_assets/models/biped_s49/meshes/r_ring_dist.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
- added link r_ring_prox, mass 0.011; collision mesh filename=package://kuavo_assets/models/biped_s49/meshes/r_ring_prox.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; visual mesh filename=package://kuavo_assets/models/biped_s49/meshes/r_ring_prox.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
- added link r_thumb_dist, mass 0.04; collision mesh filename=package://kuavo_assets/models/biped_s49/meshes/r_thumb_dist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; visual mesh filename=package://kuavo_assets/models/biped_s49/meshes/r_thumb_dist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
- added link r_thumb_prox, mass 0.005; collision mesh filename=package://kuavo_assets/models/biped_s49/meshes/r_thumb_prox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; visual mesh filename=package://kuavo_assets/models/biped_s49/meshes/r_thumb_prox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
- link base_link: mass 24.09723803 -> 28.27893803; geometry collision cylinder length=0.6 radius=0.15; visual mesh filename=package://kuavo_assets/models/biped_s49/meshes/torso.STL
- link camera_base: mass 3.92699081698732E-05 -> 0.0000392699081698732
- link zarm_l2_link: geometry collision cylinder length=0.3 radius=0.05; visual mesh filename=package://kuavo_assets/models/biped_s49/meshes/l_arm_roll.S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
- link zarm_l4_link: geometry collision cylinder length=0.26 radius=0.05; visual mesh filename=package://kuavo_assets/models/biped_s49/meshes/l_forearm.STL
- link zarm_l7_link: mass 0.64 -> 0.0542110173081966; geometry collision cylinder length=0.14 radius=0.04; visual mesh filename=package://kuavo_assets/models/biped_s49/meshes/l_hand_pitch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
- link zarm_r2_link: geometry collision cylinder length=0.3 radius=0.05; visual mesh filename=package://kuavo_assets/models/biped_s49/meshes/r_arm_roll.S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
- link zarm_r4_link: geometry collision cylinder length=0.26 radius=0.05; visual mesh filename=package://kuavo_assets/models/biped_s49/meshes/r_forearm.STL
- link zarm_r7_link: mass 0.64 -> 0.0542110173081966; geometry collision cylinder length=0.14 radius=0.04; visual mesh filename=package://kuavo_assets/models/biped_s49/meshes/r_hand_pitch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
- link zhead_1_link: geometry collision sphere radius=0.1; visual mesh filename=package://kuavo_assets/models/biped_s49/meshes/head_yaw.STL
Joints:
- removed joint dummy_to_base_link
- removed joint l_b_bar-1
- removed joint l_b_bar-2
- removed joint l_b_bar-3
- removed joint l_b_fingers
- removed joint l_f_bar-1_joint
- removed joint l_f_bar-2
- removed joint l_f_bar-3
- removed joint l_f_fingers
- removed joint r_b_bar-1
- removed joint r_b_bar-2
- removed joint r_b_bar-3
- removed joint r_b_fingers
- removed joint r_f_bar-1_joint
- removed joint r_f_bar-2
- removed joint r_f_bar-3
- removed joint r_f_fingers
- added joint base_link_to_dummy_link: type fixed, parent base_link, child dummy_link, origin xyz=0 0 0 rpy=0 0 0
- added joint l_hand_camera_joint: type fixed, parent l_hand_tripod, child l_hand_camera, origin xyz=0.11540559159102 -0.0145586110669961 -0.110123491595499 rpy=1.919862177193763 0.753528063917894 -2.897246568680842, axis 0 0 0
- added joint l_hand_tripod_joint: type fixed, parent zarm_l7_link, child l_hand_tripod, origin xyz=0.0 0.0 0.0 rpy=0.0 0.0 0.0, axis 0 0 0
- added joint l_indexMCP: type revolute, parent l_palm, child l_Index_prox, origin xyz=-0.029003 0.088291 0.0022155 rpy=-0.029415 0.05236 0.034907, axis 1 0 0, limit lower=0 upper=1.309 effort=0 velocity=0
- added joint l_indexPIP: type revolute, parent l_Index_prox, child l_index_dist, origin xyz=0 0.035 0 rpy=0.19353 0 0, axis 1 0 0, limit lower=0 upper=1.25 effort=0 velocity=0
- added joint l_littleMCP: type revolute, parent l_palm, child l_little_prox, origin xyz=0.033731 0.083777 0.0022155 rpy=-0.024909 -0.05236 -0.069813, axis 1 0 0, limit lower=0 upper=1.309 effort=0 velocity=0
- added joint l_littlePIP: type revolute, parent l_little_prox, child l_little_dist, origin xyz=0 0.035 0 rpy=0.20294 0 0, axis 1 0 0, limit lower=0 upper=1.25 effort=0 velocity=0
- added joint l_middleMCP: type revolute, parent l_palm, child l_middle_prox, origin xyz=-0.008 0.092284 -0.0017707 rpy=0 0 0, axis 1 0 0, limit lower=0 upper=1.309 effort=0 velocity=0
- added joint l_middlePIP: type revolute, parent l_middle_prox, child l_middle_dist, origin xyz=0 0.042 0 rpy=0.18357 0 0, axis 1 0 0, limit lower=0 upper=1.25 effort=0 velocity=0
- added joint l_palm_fixed_joint: type fixed, parent zarm_l7_link, child l_palm, origin xyz=0 0 -0.07 rpy=-1.57 0 -3.14
- added joint l_ringMCP: type revolute, parent l_palm, child l_ring_prox, origin xyz=0.013103 0.090291 -0.0017845 rpy=-0.0092374 -0.05236 -0.034907, axis 1 0 0, limit lower=0 upper=1.309 effort=0 velocity=0
- added joint l_ringPIP: type revolute, parent l_ring_prox, child l_ring_dist, origin xyz=0 0.042 0 rpy=0.16583 0 0, axis 1 0 0, limit lower=0 upper=1.25 effort=0 velocity=0
- added joint l_thumbCMC: type revolute, parent l_palm, child l_thumb_prox, origin xyz=-0.0245 0.022632 0.023263 rpy=0.14578 -1.0699 -0.12808, axis 0 1 0, limit lower=0 upper=1.5708 effort=0 velocity=0
- added joint l_thumbMCP: type revolute, parent l_thumb_prox, child l_thumb_dist, origin xyz=0 0 0.013647 rpy=0.87266 -0.49642 0, axis -1 0 0, limit lower=0 upper=0.8727 effort=0 velocity=0
- added joint r_hand_camera_joint: type fixed, parent r_hand_tripod, child r_hand_camera, origin xyz=0.115405591590931 0.0154312352120435 -0.107724128430896 rpy=1.208853693239594  0.751879414295006 2.888346587751982, axis 0 0 0
- added joint r_hand_tripod_joint: type fixed, parent zarm_r7_link, child r_hand_tripod, origin xyz=0.0 0.0 0.0 rpy=0.0 0.0 0.0, axis 0 0 0
- added joint r_indexMCP: type revolute, parent r_palm, child r_index_prox, origin xyz=0.029003 0.088231 -0.0039488 rpy=-0.09929 -0.054667 -0.031168, axis 1 0 0, limit lower=0 upper=1.309 effort=0 velocity=0
- added joint r_indexPIP: type revolute, parent r_index_prox, child r_index_dist, origin xyz=0 0.035 0 rpy=0.19353 0 0, axis 1 0 0, limit lower=0 upper=1.25 effort=0 velocity=0
- added joint r_littleMCP: type revolute, parent r_palm, child r_little_prox, origin xyz=-0.033731 0.083727 -0.0036339 rpy=-0.094666 0.057099 0.065996, axis 1 0 0, limit lower=0 upper=1.309 effort=0 velocity=0
- added joint r_littlePIP: type revolute, parent r_little_prox, child r_little_dist, origin xyz=0 0.035 0 rpy=0.20294 0 0, axis 1 0 0, limit lower=0 upper=1.25 effort=0 velocity=0
- added joint r_middleMCP: type revolute, parent r_palm, child r_middle_prox, origin xyz=0.008 0.091935 -0.0082038 rpy=-0.069813 0 0, axis 1 0 0, limit lower=0 upper=1.309 effort=0 velocity=0
- added joint r_middlePIP: type revolute, parent r_middle_prox, child r_middle_dist, origin xyz=0 0.042 0 rpy=0.18357 0 0, axis 1 0 0, limit lower=0 upper=1.25 effort=0 velocity=0
- added joint r_palm_fixed_joint: type fixed, parent zarm_r7_link, child r_palm, origin xyz=0 0 -0.07 rpy=-1.57 0 0
- added joint r_ringMCP: type revolute, parent r_palm, child r_ring_prox, origin xyz=-0.013103 0.089947 -0.0080786 rpy=-0.079113 0.054667 0.031168, axis 1 0 0, limit lower=0 upper=1.309 effort=0 velocity=0
- added joint r_ringPIP: type revolute, parent r_ring_prox, child r_ring_dist, origin xyz=0 0.042 0 rpy=0.16583 0 0, axis 1 0 0, limit lower=0 upper=1.25 effort=0 velocity=0
- added joint r_thumbCMC: type revolute, parent r_palm, child r_thumb_prox, origin xyz=0.0245 0.0242 0.021628 rpy=0 -0.49642 0, axis 0 -1 0, limit lower=0 upper=1.5708 effort=0 velocity=0
- added joint r_thumbMCP: type revolute, parent r_thumb_prox, child r_thumb_dist, origin xyz=0.013647 0 0 rpy=-0.39332 0.31115 -0.93514, axis 0 0 1, limit lower=0 upper=0.87266 effort=0 velocity=0

Commit message: sync https://www.lejuhub.com/highlydynamic/kuavo-ros-control/commit/e58a15283be3379c7e512221da8ed96b991c377d

File: src/kuavo_assets/models/biped_s47/urdf/biped_s47.urdf (robot description, URDF)
Before this commit: robot biped_s47, 66 links, 65 joints
Links:
- removed link l_hand_tripod
- removed link r_hand_tripod
- link l_hand_camera: mass 0.038145442577304 -> 3.8901417772519E-12
- link r_hand_camera: mass 0.038145442577304 -> 3.89014177725188E-12
Joints:
- removed joint l_hand_tripod_joint
- removed joint r_hand_tripod_joint
- joint l_hand_camera_joint: origin xyz=0.11540559159102 -0.0145586110669961 -0.110123491595499 rpy=1.919862177193763 0.753528063917894 -2.897246568680842 -> xyz=0 0.0334213029231864 -0.10658802837623 rpy=3.14159265358979 1.04719755119659 -1.57079632679489; parent l_hand_tripod -> zarm_l7_link
- joint r_hand_camera_joint: origin xyz=0.115405591590931 0.0154312352120435 -0.107724128430896 rpy=1.208853693239594  0.751879414295006 2.888346587751982 -> xyz=0 -0.0334213029231857 -0.10658802837623 rpy=3.14159265358976 1.04719755119665 1.57079632679484; parent r_hand_tripod -> zarm_r7_link
