Commit message: sync https://www.lejuhub.com/highlydynamic/kuavo-ros-control/commit/69817b9beccbf076e0bd51c3ae126df41a9e2097

File: src/kuavo_assets/models/biped_s45/urdf/drake/biped_v3_arm.urdf (robot description, URDF)
Before this commit: robot biped_s45, 17 links, 16 joints
Joints:
- joint zarm_l2_joint: limit lower=-0.349065850398866 upper=1.46 effort=50.0 velocity=19.154 -> lower=-0.349065850398866 upper=2.0943951023932 effort=50.0 velocity=19.154
- joint zarm_l3_joint: limit lower=-1.5707963267949 upper=0.46 effort=39.0 velocity=18.84 -> lower=-1.5707963267949 upper=1.5707963267949 effort=39.0 velocity=18.84
- joint zarm_r2_joint: limit lower=-1.46 upper=0.349065850398866 effort=50.0 velocity=19.154 -> lower=-2.0943951023932 upper=0.349065850398866 effort=50.0 velocity=19.154
- joint zarm_r3_joint: limit lower=-0.46 upper=1.5707963267949 effort=39.0 velocity=18.84 -> lower=-1.5707963267949 upper=1.5707963267949 effort=39.0 velocity=18.84

File: src/kuavo_assets/models/biped_s46/urdf/drake/biped_v3_arm.urdf (robot description, URDF)
Before this commit: robot biped_s46, 17 links, 16 joints
Joints:
- joint zarm_l2_joint: limit lower=-0.349065850398866 upper=1.46 effort=50.0 velocity=19.154 -> lower=-0.349065850398866 upper=2.0943951023932 effort=50.0 velocity=8.37333333333333
- joint zarm_l3_joint: limit lower=-1.5707963267949 upper=0.46 effort=39.0 velocity=18.84 -> lower=-1.5707963267949 upper=1.5707963267949 effort=39.0 velocity=19.3633333333333
- joint zarm_r2_joint: limit lower=-1.46 upper=0.349065850398866 effort=50.0 velocity=19.154 -> lower=-2.0943951023932 upper=0.349065850398866 effort=50.0 velocity=8.37333333333333
- joint zarm_r3_joint: limit lower=-0.46 upper=1.5707963267949 effort=39.0 velocity=18.84 -> lower=-1.5707963267949 upper=1.5707963267949 effort=39.0 velocity=18.84

File: src/kuavo_assets/models/biped_s47/urdf/biped_s47.urdf (robot description, URDF)
Before this commit: robot biped_s47, 64 links, 63 joints
Links:
- added link l_hand_tripod, mass 0.0342669089979502; collision mesh filename=package://kuavo_assets/models/biped_s47/meshes/l_hand_tripo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; visual mesh filename=package://kuavo_assets/models/biped_s47/meshes/l_hand_tripo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
- added link r_hand_tripod, mass 0.034266881719861; collision mesh filename=package://kuavo_assets/models/biped_s47/meshes/r_hand_tripo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; visual mesh filename=package://kuavo_assets/models/biped_s47/meshes/r_hand_tripo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
- link l_hand_camera: mass 3.8901417772519E-12 -> 0.038145442577304
- link r_hand_camera: mass 3.89014177725188E-12 -> 0.038145442577304
Joints:
- added joint l_hand_tripod_joint: type fixed, parent zarm_l7_link, child l_hand_tripod, origin xyz=0.0 0.0 0.0 rpy=0.0 0.0 0.0, axis 0 0 0
- added joint r_hand_tripod_joint: type fixed, parent zarm_r7_link, child r_hand_tripod, origin xyz=0.0 0.0 0.0 rpy=0.0 0.0 0.0, axis 0 0 0
- joint l_hand_camera_joint: origin xyz=0 0.0334213029231864 -0.10658802837623 rpy=3.14159265358979 1.04719755119659 -1.57079632679489 -> xyz=0.11540559159102 -0.0145586110669961 -0.110123491595499 rpy=1.919862177193763 0.753528063917894 -2.897246568680842; parent zarm_l7_link -> l_hand_tripod
- joint r_hand_camera_joint: origin xyz=0 -0.0334213029231857 -0.10658802837623 rpy=3.14159265358976 1.04719755119665 1.57079632679484 -> xyz=0.115405591590931 0.0154312352120435 -0.107724128430896 rpy=1.208853693239594  0.751879414295006 2.888346587751982; parent zarm_r7_link -> r_hand_tripod

File: src/kuavo_assets/models/biped_s47/urdf/drake/biped_v3_arm.urdf (robot description, URDF)
Before this commit: robot biped_s47, 17 links, 16 joints
Joints:
- joint zarm_l2_joint: limit lower=-0.349065850398866 upper=1.46 effort=50.0 velocity=19.154 -> lower=-0.349065850398866 upper=2.0943951023932 effort=50.0 velocity=8.37333333333333
- joint zarm_l3_joint: limit lower=-1.5707963267949 upper=0.46 effort=39.0 velocity=18.84 -> lower=-1.5707963267949 upper=1.5707963267949 effort=39.0 velocity=19.3633333333333
- joint zarm_r2_joint: limit lower=-1.46 upper=0.349065850398866 effort=50.0 velocity=19.154 -> lower=-2.0943951023932 upper=0.349065850398866 effort=50.0 velocity=8.37333333333333
- joint zarm_r3_joint: limit lower=-0.46 upper=1.5707963267949 effort=39.0 velocity=18.84 -> lower=-1.5707963267949 upper=1.5707963267949 effort=39.0 velocity=18.84

File: src/kuavo_assets/models/biped_s48/urdf/drake/biped_v3_arm.urdf (robot description, URDF)
Before this commit: robot biped_s48, 17 links, 16 joints
Joints:
- joint zarm_l2_joint: limit lower=-0.349065850398866 upper=1.46 effort=50.0 velocity=19.154 -> lower=-0.349065850398866 upper=2.0943951023932 effort=50.0 velocity=19.154
- joint zarm_l3_joint: limit lower=-1.5707963267949 upper=0.46 effort=39.0 velocity=18.84 -> lower=-1.5707963267949 upper=1.5707963267949 effort=39.0 velocity=18.84
- joint zarm_r2_joint: limit lower=-1.46 upper=0.349065850398866 effort=50.0 velocity=19.154 -> lower=-2.0943951023932 upper=0.349065850398866 effort=50.0 velocity=19.154
- joint zarm_r3_joint: limit lower=-0.46 upper=1.5707963267949 effort=39.0 velocity=18.84 -> lower=-1.5707963267949 upper=1.5707963267949 effort=39.0 velocity=18.84

File: src/kuavo_assets/models/biped_s49/urdf/drake/biped_v3_arm.urdf (robot description, URDF)
Before this commit: robot biped_s49, 17 links, 16 joints
Joints:
- joint zarm_l2_joint: limit lower=-0.349065850398866 upper=1.46 effort=50.0 velocity=19.154 -> lower=-0.349065850398866 upper=2.0943951023932 effort=50.0 velocity=19.154
- joint zarm_l3_joint: limit lower=-1.5707963267949 upper=0.46 effort=39.0 velocity=18.84 -> lower=-1.5707963267949 upper=1.5707963267949 effort=39.0 velocity=18.84
- joint zarm_r2_joint: limit lower=-1.46 upper=0.349065850398866 effort=50.0 velocity=19.154 -> lower=-2.0943951023932 upper=0.349065850398866 effort=50.0 velocity=19.154
- joint zarm_r3_joint: limit lower=-0.46 upper=1.5707963267949 effort=39.0 velocity=18.84 -> lower=-1.5707963267949 upper=1.5707963267949 effort=39.0 velocity=18.84
