Commit message: sync https://www.lejuhub.com/highlydynamic/kuavo-ros-control/commit/63733716f13fef1a6a9b2dac7658cb496648660f

File: src/kuavo_assets/models/apriltag/urdf/apriltag.xacro (robot description, xacro)
@@ -1,5 +1,5 @@
 <?xml version="1.0"?>
 <robot xmlns:xacro="http://ros.org/wiki/xacro" name="apriltag_marker">
-  <xacro:macro name="apriltag_marker" params="parent_link *origin id enable_collision:=true">
+  <xacro:macro name="apriltag_marker" params="parent_link *origin id enable_collision:=false">
     <!-- 定义二维码的Link -->
     <link name="apriltag_marker_${id}">

Commit message: sync https://www.lejuhub.com/highlydynamic/kuavo-ros-control/commit/e61f635b8aca76b76e47feeb3bbd11117c39dbe9

File: src/kuavo_assets/models/apriltag/urdf/apriltag.xacro (robot description, xacro)
@@ -1,5 +1,5 @@
 <?xml version="1.0"?>
 <robot xmlns:xacro="http://ros.org/wiki/xacro" name="apriltag_marker">
-  <xacro:macro name="apriltag_marker" params="parent_link *origin id">
+  <xacro:macro name="apriltag_marker" params="parent_link *origin id enable_collision:=false">
     <!-- 定义二维码的Link -->
     <link name="apriltag_marker_${id}">
@@ -10,9 +10,11 @@
         </geometry>
       </visual>
-      <collision>
-        <geometry>
-          <box size="0.11 0.11 0.001"/>
-        </geometry>
-      </collision>
+      <xacro:if value="${enable_collision}">
+        <collision>
+          <geometry>
+            <box size="0.11 0.11 0.001"/>
+          </geometry>
+        </collision>
+      </xacro:if>
     </link>
     <joint name="apriltag_joint_${id}" type="fixed">

File: src/kuavo_assets/models/biped_s13/urdf/biped_s13.urdf (robot description, URDF)
Before this commit: robot biped_s13, 39 links, 38 joints
Links:
- removed link waist
- added link waist_yaw_link, mass 4.09458758; visual mesh filename=package://kuavo_assets/models/biped_s13/meshes/torso.STL
- link base_link: mass 4.09458758 -> 5.17438719; geometry visual mesh filename=package://kuavo_assets/models/biped_s13/meshes/waist.STL
- link leg_l6_link: geometry collision box size=0.21 0.1 0.035; visual mesh filename=package://kuavo_assets/models/biped_s13/meshes/l_foot_roll_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
- link leg_r6_link: geometry collision box size=0.21 0.1 0.035; visual mesh filename=package://kuavo_assets/models/biped_s13/meshes/r_foot_roll_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
Joints:
- removed joint waist
- added joint waist_yaw_joint: type revolute, parent base_link, child waist_yaw_link, origin xyz=0 0 0 rpy=0 0 0, axis 0 0 1, limit lower=-2.0943951023932 upper=2.0943951023932 effort=50 velocity=8.37333333333333
- joint leg_l1_joint: parent waist -> base_link
- joint leg_r1_joint: parent waist -> base_link
- joint zarm_l1_joint: parent base_link -> waist_yaw_link
- joint zarm_r1_joint: parent base_link -> waist_yaw_link
- joint zhead_1_joint: parent base_link -> waist_yaw_link

File: src/kuavo_assets/models/biped_s13/urdf/biped_s13_gazebo.urdf (robot description, URDF)
Before this commit: robot biped_s13, 39 links, 38 joints
Links:
- removed link waist
- added link waist_yaw_link, mass 4.09458758; visual mesh filename=package://kuavo_assets/models/biped_s13/meshes/torso.STL
- link base_link: mass 4.60608758 -> 5.17438719; geometry visual mesh filename=package://kuavo_assets/models/biped_s13/meshes/waist.STL
- link zarm_l4_link: mass 0.2274965 -> 0.48320221; geometry visual mesh filename=package://kuavo_assets/models/biped_s13/meshes/l_forearm_ha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
- link zarm_r4_link: mass 0.22747514 -> 0.48320221; geometry visual mesh filename=package://kuavo_assets/models/biped_s13/meshes/r_forearm_ha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
Joints:
- removed joint waist_joint
- added joint waist_yaw_joint: type revolute, parent base_link, child waist_yaw_link, origin xyz=0 0 0 rpy=0 0 0, axis 0 0 1, limit lower=-2.0943951023932 upper=2.0943951023932 effort=50 velocity=8.37333333333333
- joint l_foot_heel_joint: origin xyz=-0.02 -0.05 -0.0435 rpy=0 0 0 -> xyz=-0.089 0.0 -0.0435 rpy=0 0 0
- joint l_foot_toe_joint: origin xyz=-0.02 0.05 -0.0435 rpy=0 0 0 -> xyz=0.126 0.0 -0.0435 rpy=0 0 0
- joint leg_l1_joint: parent waist -> base_link
- joint leg_r1_joint: parent waist -> base_link
- joint r_foot_heel_joint: origin xyz=-0.02 -0.05 -0.0435 rpy=0 0 0 -> xyz=-0.089 0.0 -0.0435 rpy=0 0 0
- joint r_foot_toe_joint: origin xyz=-0.02 0.05 -0.0435 rpy=0 0 0 -> xyz=0.126 0.0 -0.0435 rpy=0 0 0
- joint zarm_l1_joint: parent base_link -> waist_yaw_link
- joint zarm_r1_joint: parent base_link -> waist_yaw_link
- joint zhead_1_joint: parent base_link -> waist_yaw_link
- joint zhead_2_joint: limit lower=0.0 upper=0.523598775598299 effort=50 velocity=8.37333333333333 -> lower=-0.349065850398866 upper=0.523598775598299 effort=50 velocity=8.37333333333333

File: src/kuavo_assets/models/biped_s13/urdf/drake/biped_v3.urdf (robot description, URDF)
Before this commit: robot biped_v3, 14 links, 13 joints
Links:
- removed link waist
- added link waist_yaw_link, mass 11.23288758; visual mesh filename=../../meshes/torso.STL
- link torso: mass 11.23288758 -> 3.17438719; geometry visual mesh filename=../../meshes/waist.STL
Joints:
- removed joint waist
- added joint waist_yaw_joint: type fixed, parent torso, child waist_yaw_link, origin xyz=0 0 0 rpy=0 0 0, axis 0 0 1, limit lower=-2.0943951023932 upper=2.0943951023932 effort=50 velocity=8.37333333333333
- joint leg_l1_joint: parent waist -> torso
- joint leg_r1_joint: parent waist -> torso

File: src/kuavo_assets/models/biped_s13/urdf/drake/biped_v3_all_joint.urdf (robot description, URDF)
Before this commit: robot biped_v3_all_joint, 30 links, 25 joints
Links:
- link torso: mass -.07761242 -> 5.17741242

File: src/kuavo_assets/models/biped_s13/urdf/drake/biped_v3_arm.urdf (robot description, URDF)
Before this commit: robot biped_v3_arm, 10 links, 9 joints
Links:
- removed link waist
- added link waist_yaw_link, mass 7.34228758; visual mesh filename=../../meshes/torso.STL
- link torso: mass 7.34228758 -> 5.17438719; geometry visual mesh filename=../../meshes/waist.STL
Joints:
- removed joint waist
- added joint waist_yaw_joint: type fixed, parent torso, child waist_yaw_link, origin xyz=0 0 0 rpy=0 0 0, axis 0 0 1, limit lower=-2.0943951023932 upper=2.0943951023932 effort=50 velocity=8.37333333333333
- joint zarm_l1_joint: parent torso -> waist_yaw_link
- joint zarm_r1_joint: parent torso -> waist_yaw_link

File: src/kuavo_assets/models/biped_s45/urdf/biped_s45_gazebo.urdf (robot description, URDF)
Before this commit: robot biped_s45, 47 links, 46 joints
Links:
- link zarm_l7_link: geometry collision mesh filename=package://kuavo_assets/models/biped_s45/meshes/l_hand_pitch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; visual mesh filename=package://kuavo_assets/models/biped_s45/meshes/l_hand_pitch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
- link zarm_r7_link: geometry collision mesh filename=package://kuavo_assets/models/biped_s45/meshes/r_hand_pitch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; visual mesh filename=package://kuavo_assets/models/biped_s45/meshes/r_hand_pitch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

File: src/kuavo_assets/models/biped_s50/urdf/biped_s50.urdf (robot description, URDF)
Before this commit: robot biped_s50, 47 links, 46 joints
Links:
- removed link waist_yaw
- added link camera, mass 0.0497265773443356; visual mesh filename=package://kuavo_assets/models/biped_s49/meshes/camera.STL
- added link waist_camera, mass 0.237986769607677; collision mesh filename=package://kuavo_assets/models/biped_s45/meshes/waist_camera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; visual mesh filename=package://kuavo_assets/models/biped_s45/meshes/waist_camera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
- added link waist_yaw_link, mass 15.18745152; visual mesh filename=package://kuavo_assets/models/biped_s50/meshes/waist_yaw.STL
- link base_link: mass 6.7086837 -> 12.2561837
- link camera_base: mass 0.0482361371130408 -> 0.0000392699081698732; geometry collision mesh filename=package://kuavo_assets/models/biped_s49/meshes/camera_base.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; visual mesh filename=package://kuavo_assets/models/biped_s49/meshes/camera_base.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
- link leg_l6_link: geometry collision box size=0.25 0.1 0.04; visual mesh filename=package://kuavo_assets/models/biped_s50/meshes/l_foot_roll.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
- link leg_r6_link: geometry collision box size=0.25 0.1 0.04; visual mesh filename=package://kuavo_assets/models/biped_s50/meshes/r_foot_roll.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
- link radar: mass 0.137337293833749 -> 0.149896342265089; geometry visual mesh filename=package://kuavo_assets/models/biped_s49/meshes/radar.STL
- link zhead_1_link: mass 1.06289355 -> 0.35; geometry collision sphere radius=0.1; visual mesh filename=package://kuavo_assets/models/biped_s45/meshes/head_yaw.STL
- link zhead_2_link: mass 0.20029579 -> 0.5492; geometry visual mesh filename=package://kuavo_assets/models/biped_s45/meshes/head_pitch.S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
Joints:
- removed joint waist_yaw
- added joint camera: type fixed, parent zhead_2_link, child camera, origin xyz=0.102420738776518 -0.0475000000000003 0.126192926717169 rpy=3.14159265358979 0.383972435438723 0
- added joint waist_camera: type fixed, parent base_link, child waist_camera, origin xyz=0.168717483101422 0 0.01355599662743 rpy=0 0.8 0, axis 0 0 0
- added joint waist_yaw_joint: type revolute, parent base_link, child waist_yaw_link, origin xyz=0 0 0.107 rpy=0 0 0, axis 0 0 1, limit lower=-2.0943951023932 upper=2.0943951023932 effort=180.0 velocity=23.55
- joint camera_base: origin xyz=0.094395257832706 0 0.11395418930214 rpy=0 0.310766624316135 0 -> xyz=0.0932759773834307 0 0.145322661773667 rpy=3.14159265358979 0.383972435438723 0
- joint dummy_to_base_link: child base_link -> dummy_link; parent dummy_link -> base_link
- joint radar: origin xyz=0 0 -0.0264531741828733 rpy=0 0 0 -> xyz=0.0193616404443762 0 0.113041650167083 rpy=-3.14159265358784 0.242945586895529 0; parent zhead_1_link -> zhead_2_link
- joint zarm_l1_joint: parent waist_yaw -> waist_yaw_link
- joint zarm_r1_joint: parent waist_yaw -> waist_yaw_link
- joint zhead_1_joint: limit lower=-1.57 upper=1.57 effort=1.5 velocity=5.23 -> lower=-1.5707963267949 upper=1.5707963267949 effort=1.5 velocity=5.23333333333333; origin xyz=0.004 0.0 0.39985400000000004 rpy=0 0 0 -> xyz=-0.003 0.0 0.3804 rpy=0 0 0; parent waist_yaw -> waist_yaw_link
- joint zhead_2_joint: limit lower=-0.52 upper=0.52 effort=12.0 velocity=5.23 -> lower=-0.523598775598299 upper=0.523598775598299 effort=12.0 velocity=5.23333333333333

File: src/kuavo_assets/models/biped_s50/urdf/biped_s50_gazebo.urdf (robot description, URDF)
Before this commit: robot biped_s50, 47 links, 46 joints
Links:
- removed link waist_yaw
- added link camera, mass 0.0497265773443356; visual mesh filename=package://kuavo_assets/models/biped_s49/meshes/camera.STL
- added link waist_yaw_link, mass 15.18745152; visual mesh filename=package://kuavo_assets/models/biped_s50/meshes/waist_yaw.STL
- link base_link: mass 6.7086837 -> 12.8439837
- link camera_base: mass 0.0482361371130408 -> 0.0000392699081698732; geometry collision mesh filename=package://kuavo_assets/models/biped_s49/meshes/camera_base.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; visual mesh filename=package://kuavo_assets/models/biped_s49/meshes/camera_base.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
- link radar: mass 0.137337293833749 -> 0.149896342265089; geometry visual mesh filename=package://kuavo_assets/models/biped_s49/meshes/radar.STL
- link zarm_l7_link: geometry collision mesh filename=package://kuavo_assets/models/biped_s50/meshes/l_hand_pitch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; visual mesh filename=package://kuavo_assets/models/biped_s50/meshes/l_hand_pitch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
- link zarm_r7_link: geometry collision mesh filename=package://kuavo_assets/models/biped_s50/meshes/r_hand_pitch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; visual mesh filename=package://kuavo_assets/models/biped_s50/meshes/r_hand_pitch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
- link zhead_1_link: mass 1.06289355 -> 0.35; geometry visual mesh filename=package://kuavo_assets/models/biped_s45/meshes/head_yaw.STL
- link zhead_2_link: mass 0.20029579 -> 0.5492; geometry visual mesh filename=package://kuavo_assets/models/biped_s45/meshes/head_pitch.S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
Joints:
- removed joint waist_yaw
- added joint camera: type fixed, parent zhead_2_link, child camera, origin xyz=0.102420738776518 -0.0475000000000003 0.126192926717169 rpy=3.14159265358979 0.383972435438723 0
- added joint waist_yaw_joint: type revolute, parent base_link, child waist_yaw_link, origin xyz=0 0 0.107 rpy=0 0 0, axis 0 0 1, limit lower=-2.0943951023932 upper=2.0943951023932 effort=180.0 velocity=23.55
- joint camera_base: origin xyz=0.094395257832706 0 0.11395418930214 rpy=0 0.310766624316135 0 -> xyz=0.0932759773834307 0 0.145322661773667 rpy=3.14159265358979 0.383972435438723 0
- joint l_foot_heel_joint: origin xyz=-0.073164 0.0 -0.0595 rpy=0 0 0 -> xyz=-0.0 0.04773 -0.0595 rpy=0 0 0
- joint l_foot_toe_joint: origin xyz=0.17084 0.0 -0.0595 rpy=0 0 0 -> xyz=0.0 -0.04773 -0.0595 rpy=0 0 0
- joint r_foot_heel_joint: origin xyz=-0.073164 0.0 -0.0595 rpy=0 0 0 -> xyz=-0.0 0.04773 -0.0595 rpy=0 0 0
- joint r_foot_toe_joint: origin xyz=0.17084 0.0 -0.0595 rpy=0 0 0 -> xyz=0.0 -0.04773 -0.0595 rpy=0 0 0
- joint radar: origin xyz=0 0 -0.0264531741828733 rpy=0 0 0 -> xyz=0.0193616404443762 0 0.113041650167083 rpy=-3.14159265358784 0.242945586895529 0; parent zhead_1_link -> zhead_2_link
- joint zarm_l1_joint: parent waist_yaw -> waist_yaw_link
- joint zarm_r1_joint: parent waist_yaw -> waist_yaw_link
- joint zhead_1_joint: limit lower=-1.57 upper=1.57 effort=1.5 velocity=5.23 -> lower=-1.5707963267949 upper=1.5707963267949 effort=1.5 velocity=5.23333333333333; origin xyz=0.004 0.0 0.39985400000000004 rpy=0 0 0 -> xyz=-0.003 0.0 0.3804 rpy=0 0 0; parent waist_yaw -> waist_yaw_link
- joint zhead_2_joint: limit lower=-0.52 upper=0.52 effort=12.0 velocity=5.23 -> lower=-0.523598775598299 upper=0.523598775598299 effort=12.0 velocity=5.23333333333333

File: src/kuavo_assets/models/biped_s50/urdf/drake/biped_v3.urdf (robot description, URDF)
Before this commit: robot biped_v3, 14 links, 13 joints
Links:
- removed link waist_yaw
- added link waist_yaw_link, mass 15.18745152; visual mesh filename=../../meshes/waist_yaw.STL
- link torso: mass 18.5414837 -> 24.3268837
Joints:
- removed joint waist_yaw
- added joint waist_yaw_joint: type fixed, parent torso, child waist_yaw_link, origin xyz=0 0 0.107 rpy=0 0 0, axis 0 0 1, limit lower=-2.0943951023932 upper=2.0943951023932 effort=180.0 velocity=23.55

File: src/kuavo_assets/models/biped_s50/urdf/drake/biped_v3_arm.urdf (robot description, URDF)
Before this commit: robot biped_s45, 16 links, 15 joints
Links:
- removed link waist_yaw
- added link zarm_l7_end_effector; collision sphere radius=0.005
- added link zarm_r7_end_effector; collision sphere radius=0.005
- link base_link: mass 5.8663837 -> 22.11293803
Joints:
- removed joint waist_yaw
- added joint zarm_l7_end_effector_joint: type fixed, parent zarm_l7_link, child zarm_l7_end_effector, origin xyz=0 -0.03 -0.17 rpy=0 0 0
- added joint zarm_r7_end_effector_joint: type fixed, parent zarm_r7_link, child zarm_r7_end_effector, origin xyz=0 0.03 -0.17 rpy=0 0 0
- joint zarm_l1_joint: origin xyz=0.003 0.28569999999999995 0.2055 rpy=0 0 0 -> xyz=-0.017499853 0.29269999999999996 0.4245 rpy=0 0 0; parent waist_yaw -> base_link
- joint zarm_r1_joint: origin xyz=0.003 -0.28569999999999995 0.2055 rpy=0 0 0 -> xyz=-0.017499853 -0.29269999999999996 0.4245 rpy=0 0 0; parent waist_yaw -> base_link

File: src/kuavo_assets/models/biped_s50/urdf/drake/biped_v3_full.urdf (robot description, URDF)
Before this commit: robot biped_v3_full, 28 links, 27 joints
Links:
- removed link waist_yaw
- added link waist_yaw_link, mass 15.18745152; visual mesh filename=../../meshes/waist_yaw.STL
- link torso: mass 8.1574837 -> 13.9428837
Joints:
- removed joint waist_yaw
- added joint waist_yaw_joint: type fixed, parent biped_s50, child waist_yaw_link, origin xyz=0 0 0.107 rpy=0 0 0, axis 0 0 1, limit lower=-2.0943951023932 upper=2.0943951023932 effort=180.0 velocity=23.55
- joint zarm_l1_joint: parent waist_yaw -> waist_yaw_link
- joint zarm_r1_joint: parent waist_yaw -> waist_yaw_link
