Commit message: sync https://www.lejuhub.com/highlydynamic/kuavo-ros-control/commit/d54563a3c23cc8fe8e12f2b58551040e769adebc

File: src/kuavo_assets/models/apriltag/urdf/grab_box_table.xacro (robot description, xacro)
@@ -194,4 +194,42 @@
     </inertial>
   </link>
+  <link name="apriltag_box_tag2_base">
+    <visual>
+      <geometry>
+        <box size="0.1 0.1 0.1"/>
+      </geometry>
+      <material>
+        <color rgba="0.8 0.8 0.8 0.5"/>
+      </material>
+    </visual>
+    <collision>
+      <geometry>
+        <box size="0.1 0.1 0.1"/>
+      </geometry>
+    </collision>
+    <inertial>
+      <mass value="0.1"/>
+      <inertia ixx="0.0001" ixy="0" ixz="0" iyy="0.0001" iyz="0" izz="0.0001"/>
+    </inertial>
+  </link>
+  <link name="apriltag_box_tag3_base">
+    <visual>
+      <geometry>
+        <box size="0.1 0.1 0.1"/>
+      </geometry>
+      <material>
+        <color rgba="0.8 0.8 0.8 0.5"/>
+      </material>
+    </visual>
+    <collision>
+      <geometry>
+        <box size="0.1 0.1 0.1"/>
+      </geometry>
+    </collision>
+    <inertial>
+      <mass value="0.1"/>
+      <inertia ixx="0.0001" ixy="0" ixz="0" iyy="0.0001" iyz="0" izz="0.0001"/>
+    </inertial>
+  </link>
   <link name="apriltag_shelf_base">
     <visual>
@@ -219,4 +257,14 @@
     <origin xyz="0.0 -1.7 1.05" rpy="0 0 0"/>
   </joint>
+  <joint name="world_to_box_tag2_joint" type="fixed">
+    <parent link="world"/>
+    <child link="apriltag_box_tag2_base"/>
+    <origin xyz="0.5 -1.7 1.3" rpy="0 0 0"/>
+  </joint>
+  <joint name="world_to_box_tag3_joint" type="fixed">
+    <parent link="world"/>
+    <child link="apriltag_box_tag3_base"/>
+    <origin xyz="-0.5 -1.7 0.75" rpy="0 0 0"/>
+  </joint>
   <joint name="world_to_table_joint" type="fixed">
     <parent link="world"/>
@@ -227,4 +275,10 @@
     <origin xyz="0 -0.055 -0.165" rpy="1.5708 1.5708 0"/>
   </xacro:apriltag_marker>
+  <xacro:apriltag_marker parent_link="apriltag_box_tag2_base" id="2">
+    <origin xyz="0 -0.055 -0.165" rpy="1.5708 1.5708 0"/>
+  </xacro:apriltag_marker>
+  <xacro:apriltag_marker parent_link="apriltag_box_tag3_base" id="3">
+    <origin xyz="0 -0.055 -0.165" rpy="1.5708 1.5708 0"/>
+  </xacro:apriltag_marker>
   <xacro:apriltag_marker parent_link="apriltag_shelf_base" id="0">
     <origin xyz="0.055 0 -0.165" rpy="0 -1.5708 3.14159"/>

File: src/kuavo_assets/models/biped_s45/urdf/biped_s45.urdf (robot description, URDF)
Before this commit: robot biped_s45, 53 links, 52 joints
Links:
- link zarm_l1_link: mass 0.962 -> 0.95200000
- link zarm_l2_link: mass 0.57 -> 0.38500000
- link zarm_l3_link: mass 1.65 -> 1.75450000
- link zarm_l4_link: mass 0.429 -> 0.60780000
- link zarm_l5_link: mass 0.61 -> 0.63690000
- link zarm_l6_link: mass 0.331 -> 0.47390000
- link zarm_r1_link: mass 0.962 -> 0.95200000
- link zarm_r2_link: mass 0.57 -> 0.38500000
- link zarm_r3_link: mass 1.65 -> 1.75450000
- link zarm_r4_link: mass 0.429 -> 0.60780000
- link zarm_r5_link: mass 0.61 -> 0.63690000
- link zarm_r6_link: mass 0.331 -> 0.47390000

File: src/kuavo_assets/models/biped_s45/urdf/biped_s45_gazebo.urdf (robot description, URDF)
Before this commit: robot biped_s45, 47 links, 46 joints
Links:
- link zarm_l1_link: mass 0.962 -> 0.95200000
- link zarm_l2_link: mass 0.57 -> 0.38500000
- link zarm_l3_link: mass 1.65 -> 1.75450000
- link zarm_l4_link: mass 0.429 -> 0.60780000
- link zarm_l5_link: mass 0.61 -> 0.63690000
- link zarm_l6_link: mass 0.331 -> 0.47390000
- link zarm_r1_link: mass 0.962 -> 0.95200000
- link zarm_r2_link: mass 0.57 -> 0.38500000
- link zarm_r3_link: mass 1.65 -> 1.75450000
- link zarm_r4_link: mass 0.429 -> 0.60780000
- link zarm_r5_link: mass 0.61 -> 0.63690000
- link zarm_r6_link: mass 0.331 -> 0.47390000

File: src/kuavo_assets/models/biped_s45/urdf/drake/biped_v3_arm.urdf (robot description, URDF)
Before this commit: robot biped_s45, 19 links, 18 joints
Links:
- link zarm_l1_link: mass 0.962 -> 0.95200000
- link zarm_l2_link: mass 0.57 -> 0.38500000
- link zarm_l3_link: mass 1.65 -> 1.75450000
- link zarm_l4_link: mass 0.429 -> 0.60780000
- link zarm_l5_link: mass 0.61 -> 0.63690000
- link zarm_l6_link: mass 0.331 -> 0.47390000
- link zarm_r1_link: mass 0.962 -> 0.95200000
- link zarm_r2_link: mass 0.57 -> 0.38500000
- link zarm_r3_link: mass 1.65 -> 1.75450000
- link zarm_r4_link: mass 0.429 -> 0.60780000
- link zarm_r5_link: mass 0.61 -> 0.63690000
- link zarm_r6_link: mass 0.331 -> 0.47390000

File: src/kuavo_assets/models/biped_s46/urdf/biped_s46.urdf (robot description, URDF)
Before this commit: robot biped_s46, 46 links, 45 joints
Links:
- link zarm_l1_link: mass 0.962 -> 0.95200000
- link zarm_l2_link: mass 0.57 -> 0.38500000
- link zarm_l3_link: mass 1.65 -> 1.75450000
- link zarm_l4_link: mass 0.429 -> 0.60780000
- link zarm_l5_link: mass 0.61 -> 0.63690000
- link zarm_l6_link: mass 0.331 -> 0.47390000
- link zarm_r1_link: mass 0.962 -> 0.95200000
- link zarm_r2_link: mass 0.57 -> 0.38500000
- link zarm_r3_link: mass 1.65 -> 1.75450000
- link zarm_r4_link: mass 0.429 -> 0.60780000
- link zarm_r5_link: mass 0.61 -> 0.63690000
- link zarm_r6_link: mass 0.331 -> 0.47390000

File: src/kuavo_assets/models/biped_s46/urdf/biped_s46_gazebo.urdf (robot description, URDF)
Before this commit: robot biped_s46, 46 links, 45 joints
Links:
- link zarm_l1_link: mass 0.962 -> 0.95200000
- link zarm_l2_link: mass 0.57 -> 0.38500000
- link zarm_l3_link: mass 1.65 -> 1.75450000
- link zarm_l4_link: mass 0.429 -> 0.60780000
- link zarm_l5_link: mass 0.61 -> 0.63690000
- link zarm_l6_link: mass 0.331 -> 0.47390000
- link zarm_r1_link: mass 0.962 -> 0.95200000
- link zarm_r2_link: mass 0.57 -> 0.38500000
- link zarm_r3_link: mass 1.65 -> 1.75450000
- link zarm_r4_link: mass 0.429 -> 0.60780000
- link zarm_r5_link: mass 0.61 -> 0.63690000
- link zarm_r6_link: mass 0.331 -> 0.47390000

File: src/kuavo_assets/models/biped_s46/urdf/drake/biped_v3_arm.urdf (robot description, URDF)
Before this commit: robot biped_s46, 19 links, 18 joints
Links:
- link zarm_l1_link: mass 0.962 -> 0.95200000
- link zarm_l2_link: mass 0.57 -> 0.38500000
- link zarm_l3_link: mass 1.65 -> 1.75450000
- link zarm_l4_link: mass 0.429 -> 0.60780000
- link zarm_l5_link: mass 0.61 -> 0.63690000
- link zarm_l6_link: mass 0.331 -> 0.47390000
- link zarm_r1_link: mass 0.962 -> 0.95200000
- link zarm_r2_link: mass 0.57 -> 0.38500000
- link zarm_r3_link: mass 1.65 -> 1.75450000
- link zarm_r4_link: mass 0.429 -> 0.60780000
- link zarm_r5_link: mass 0.61 -> 0.63690000
- link zarm_r6_link: mass 0.331 -> 0.47390000

File: src/kuavo_assets/models/biped_s47/urdf/biped_s47.urdf (robot description, URDF)
Before this commit: robot biped_s47, 64 links, 63 joints
Links:
- link zarm_l1_link: mass 0.962 -> 0.95200000
- link zarm_l2_link: mass 0.57 -> 0.38500000
- link zarm_l3_link: mass 1.65 -> 1.75450000
- link zarm_l4_link: mass 0.429 -> 0.60780000
- link zarm_l5_link: mass 0.61 -> 0.63690000
- link zarm_l6_link: mass 0.331 -> 0.47390000
- link zarm_r1_link: mass 0.962 -> 0.95200000
- link zarm_r2_link: mass 0.57 -> 0.38500000
- link zarm_r3_link: mass 1.65 -> 1.75450000
- link zarm_r4_link: mass 0.429 -> 0.60780000
- link zarm_r5_link: mass 0.61 -> 0.63690000
- link zarm_r6_link: mass 0.331 -> 0.47390000

File: src/kuavo_assets/models/biped_s47/urdf/biped_s47_gazebo.urdf (robot description, URDF)
Before this commit: robot biped_s47, 63 links, 62 joints
Links:
- link zarm_l1_link: mass 0.962 -> 0.95200000
- link zarm_l2_link: mass 0.57 -> 0.38500000
- link zarm_l3_link: mass 1.65 -> 1.75450000
- link zarm_l4_link: mass 0.429 -> 0.60780000
- link zarm_l5_link: mass 0.61 -> 0.63690000
- link zarm_l6_link: mass 0.331 -> 0.47390000
- link zarm_r1_link: mass 0.962 -> 0.95200000
- link zarm_r2_link: mass 0.57 -> 0.38500000
- link zarm_r3_link: mass 1.65 -> 1.75450000
- link zarm_r4_link: mass 0.429 -> 0.60780000
- link zarm_r5_link: mass 0.61 -> 0.63690000
- link zarm_r6_link: mass 0.331 -> 0.47390000

File: src/kuavo_assets/models/biped_s47/urdf/drake/biped_v3_arm.urdf (robot description, URDF)
Before this commit: robot biped_s47, 19 links, 18 joints
Links:
- link zarm_l1_link: mass 0.962 -> 0.95200000
- link zarm_l2_link: mass 0.57 -> 0.38500000
- link zarm_l3_link: mass 1.65 -> 1.75450000
- link zarm_l4_link: mass 0.429 -> 0.60780000
- link zarm_l5_link: mass 0.61 -> 0.63690000
- link zarm_l6_link: mass 0.331 -> 0.47390000
- link zarm_r1_link: mass 0.962 -> 0.95200000
- link zarm_r2_link: mass 0.57 -> 0.38500000
- link zarm_r3_link: mass 1.65 -> 1.75450000
- link zarm_r4_link: mass 0.429 -> 0.60780000
- link zarm_r5_link: mass 0.61 -> 0.63690000
- link zarm_r6_link: mass 0.331 -> 0.47390000

File: src/kuavo_assets/models/biped_s48/urdf/biped_s48.urdf (robot description, URDF)
Before this commit: robot biped_s48, 69 links, 68 joints
Links:
- link zarm_l1_link: mass 0.962 -> 0.95200000
- link zarm_l2_link: mass 0.57 -> 0.38500000
- link zarm_l3_link: mass 1.65 -> 1.75450000
- link zarm_l4_link: mass 0.429 -> 0.60780000
- link zarm_l5_link: mass 0.61 -> 0.63690000
- link zarm_l6_link: mass 0.331 -> 0.47390000
- link zarm_r1_link: mass 0.962 -> 0.95200000
- link zarm_r2_link: mass 0.57 -> 0.38500000
- link zarm_r3_link: mass 1.65 -> 1.75450000
- link zarm_r4_link: mass 0.429 -> 0.60780000
- link zarm_r5_link: mass 0.61 -> 0.63690000
- link zarm_r6_link: mass 0.331 -> 0.47390000

File: src/kuavo_assets/models/biped_s48/urdf/biped_s48_gazebo.urdf (robot description, URDF)
Before this commit: robot biped_s48, 69 links, 68 joints
Links:
- link zarm_l1_link: mass 0.962 -> 0.95200000
- link zarm_l2_link: mass 0.57 -> 0.38500000
- link zarm_l3_link: mass 1.65 -> 1.75450000
- link zarm_l4_link: mass 0.429 -> 0.60780000
- link zarm_l5_link: mass 0.61 -> 0.63690000
- link zarm_l6_link: mass 0.331 -> 0.47390000
- link zarm_r1_link: mass 0.962 -> 0.95200000
- link zarm_r2_link: mass 0.57 -> 0.38500000
- link zarm_r3_link: mass 1.65 -> 1.75450000
- link zarm_r4_link: mass 0.429 -> 0.60780000
- link zarm_r5_link: mass 0.61 -> 0.63690000
- link zarm_r6_link: mass 0.331 -> 0.47390000

File: src/kuavo_assets/models/biped_s48/urdf/drake/biped_v3_arm.urdf (robot description, URDF)
Before this commit: robot biped_s48, 19 links, 18 joints
Links:
- link zarm_l1_link: mass 0.962 -> 0.95200000
- link zarm_l2_link: mass 0.57 -> 0.38500000
- link zarm_l3_link: mass 1.65 -> 1.75450000
- link zarm_l4_link: mass 0.429 -> 0.60780000
- link zarm_l5_link: mass 0.61 -> 0.63690000
- link zarm_l6_link: mass 0.331 -> 0.47390000
- link zarm_r1_link: mass 0.962 -> 0.95200000
- link zarm_r2_link: mass 0.57 -> 0.38500000
- link zarm_r3_link: mass 1.65 -> 1.75450000
- link zarm_r4_link: mass 0.429 -> 0.60780000
- link zarm_r5_link: mass 0.61 -> 0.63690000
- link zarm_r6_link: mass 0.331 -> 0.47390000

File: src/kuavo_assets/models/biped_s49/urdf/biped_s49.urdf (robot description, URDF)
Before this commit: robot biped_s49, 73 links, 72 joints
Links:
- link zarm_l1_link: mass 0.962 -> 0.95200000
- link zarm_l2_link: mass 0.57 -> 0.38500000
- link zarm_l3_link: mass 1.65 -> 1.75450000
- link zarm_l4_link: mass 0.429 -> 0.60780000
- link zarm_l5_link: mass 0.61 -> 0.63690000
- link zarm_l6_link: mass 0.331 -> 0.47390000
- link zarm_r1_link: mass 0.962 -> 0.95200000
- link zarm_r2_link: mass 0.57 -> 0.38500000
- link zarm_r3_link: mass 1.65 -> 1.75450000
- link zarm_r4_link: mass 0.429 -> 0.60780000
- link zarm_r5_link: mass 0.61 -> 0.63690000
- link zarm_r6_link: mass 0.331 -> 0.47390000
- link zarm_r7_link: mass 0.0542110173081966 -> 0.11660000

File: src/kuavo_assets/models/biped_s49/urdf/biped_s49_gazebo.urdf (robot description, URDF)
Before this commit: robot biped_s49, 69 links, 68 joints
Links:
- link zarm_l1_link: mass 0.962 -> 0.95200000
- link zarm_l2_link: mass 0.57 -> 0.38500000
- link zarm_l3_link: mass 1.65 -> 1.75450000
- link zarm_l4_link: mass 0.429 -> 0.60780000
- link zarm_l5_link: mass 0.61 -> 0.63690000
- link zarm_l6_link: mass 0.331 -> 0.47390000
- link zarm_r1_link: mass 0.962 -> 0.95200000
- link zarm_r2_link: mass 0.57 -> 0.38500000
- link zarm_r3_link: mass 1.65 -> 1.75450000
- link zarm_r4_link: mass 0.429 -> 0.60780000
- link zarm_r5_link: mass 0.61 -> 0.63690000
- link zarm_r6_link: mass 0.331 -> 0.47390000

File: src/kuavo_assets/models/biped_s49/urdf/drake/biped_v3_arm.urdf (robot description, URDF)
Before this commit: robot biped_s49, 19 links, 18 joints
Links:
- link zarm_l1_link: mass 0.962 -> 0.95200000
- link zarm_l2_link: mass 0.57 -> 0.38500000
- link zarm_l3_link: mass 1.65 -> 1.75450000
- link zarm_l4_link: mass 0.429 -> 0.60780000
- link zarm_l5_link: mass 0.61 -> 0.63690000
- link zarm_l6_link: mass 0.331 -> 0.47390000
- link zarm_r1_link: mass 0.962 -> 0.95200000
- link zarm_r2_link: mass 0.57 -> 0.38500000
- link zarm_r3_link: mass 1.65 -> 1.75450000
- link zarm_r4_link: mass 0.429 -> 0.60780000
- link zarm_r5_link: mass 0.61 -> 0.63690000
- link zarm_r6_link: mass 0.331 -> 0.47390000

File: src/kuavo_assets/models/biped_s52/urdf/biped_s52.urdf (robot description, URDF)
Before this commit: robot biped_s52, 47 links, 46 joints
Links:
- link base_link: mass 6.48663928 -> 9.69103928

File: src/kuavo_assets/models/biped_s52/urdf/biped_s52_gazebo.urdf (robot description, URDF)
Before this commit: robot biped_s52, 47 links, 46 joints
Links:
- link base_link: mass 6.29683928 -> 9.50123928

File: src/kuavo_assets/models/biped_s52/urdf/drake/biped_v3.urdf (robot description, URDF)
Before this commit: robot biped_v3, 14 links, 13 joints
Links:
- link torso: mass 18.99013928 -> 22.19453928

File: src/kuavo_assets/models/biped_s52/urdf/drake/biped_v3_all_joint.urdf (robot description, URDF)
Before this commit: robot biped_v3_all_joint, 35 links, 30 joints
Links:
- link torso: mass 33.93314316 -> 37.13754316
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