Commit message: sync https://www.lejuhub.com/highlydynamic/kuavo-ros-control/commit/1aaa743d73d0af61b21a004169238ed39b043eb8

File: src/kuavo_assets/models/apriltag/urdf/grab_box_table.xacro (robot description, xacro)
@@ -260,10 +260,10 @@
     <parent link="world"/>
     <child link="apriltag_box_tag2_base"/>
-    <origin xyz="0.5 -1.7 1.3" rpy="0 0 0"/>
+    <origin xyz="0.75 -1.7 1.3" rpy="0 0 0"/>
   </joint>
   <joint name="world_to_box_tag3_joint" type="fixed">
     <parent link="world"/>
     <child link="apriltag_box_tag3_base"/>
-    <origin xyz="-0.5 -1.7 0.75" rpy="0 0 0"/>
+    <origin xyz="-0.75 -1.7 0.75" rpy="0 0 0"/>
   </joint>
   <joint name="world_to_table_joint" type="fixed">

File: src/kuavo_assets/models/biped_s200062/urdf/biped_s200062.urdf (robot description, URDF)
Before this commit: robot biped_s200062, 64 links, 63 joints
Joints:
- removed joint l_f_bar_2
- removed joint r_f_bar_2
- added joint l_f_bar_2_joint: type revolute, parent l_f_bar_1, child l_f_bar_2, origin xyz=0.011329 0 0.0063767 rpy=0 0 0, axis 0 1 0, limit lower=-0.698 upper=0.698 effort=5 velocity=5
- added joint r_f_bar_2_joint: type revolute, parent r_f_bar_1, child r_f_bar_2, origin xyz=0.011329 0 0.0063767 rpy=0 0 0, axis 0 1 0, limit lower=-0.698 upper=0.698 effort=5 velocity=5
- joint camera: parent camera_base -> head_camera_base
- joint camera_base_joint: child camera_base -> head_camera_base
- joint l_b_bar_2_joint: axis (none) -> 0 1 0; limit (none) -> lower=-0.698 upper=0.698 effort=5 velocity=5; type fixed -> revolute
- joint l_b_bar_4_joint: axis (none) -> 0 1 0; limit (none) -> lower=-0.698 upper=0.698 effort=5 velocity=5; type fixed -> revolute
- joint l_b_finger_joint: axis (none) -> 0 1 0; limit (none) -> lower=-0.698 upper=0.698 effort=5 velocity=5; type fixed -> revolute
- joint l_f_bar_4_joint: axis (none) -> 0 1 0; limit (none) -> lower=-0.698 upper=0.698 effort=5 velocity=5; type fixed -> revolute
- joint l_f_finger_joint: axis (none) -> 0 1 0; limit (none) -> lower=-0.698 upper=0.698 effort=5 velocity=5; type fixed -> revolute
- joint r_b_bar_2_joint: axis (none) -> 0 1 0; limit (none) -> lower=-0.698 upper=0.698 effort=5 velocity=5; type fixed -> revolute
- joint r_b_bar_4_joint: axis (none) -> 0 1 0; limit (none) -> lower=-0.698 upper=0.698 effort=5 velocity=5; type fixed -> revolute
- joint r_b_finger_joint: axis (none) -> 0 1 0; limit (none) -> lower=-0.698 upper=0.698 effort=5 velocity=5; type fixed -> revolute
- joint r_f_bar_4_joint: axis (none) -> 0 1 0; limit (none) -> lower=-0.698 upper=0.698 effort=5 velocity=5; type fixed -> revolute
- joint r_f_finger_joint: axis (none) -> 0 1 0; limit (none) -> lower=-0.698 upper=0.698 effort=5 velocity=5; type fixed -> revolute
