Commit message: sync https://www.lejuhub.com/highlydynamic/kuavo-ros-control/commit/f53f0aca187bf01681cfffc0d36b3d60046a4884

File: src/kuavo_assets/models/apriltag/urdf/apriltag_cube.xacro (robot description, xacro)
@@ -8,40 +8,5 @@
       <origin xyz="0.055 0 -0.165" rpy="0 1.5708 0"/>
     </xacro:apriltag_marker>
-    <xacro:apriltag_marker parent_link="${parent_link}" id="1">
-      <origin xyz="-0.055 0 -0.165" rpy="0 1.5708 3.1415"/>
-    </xacro:apriltag_marker>
-    <xacro:apriltag_marker parent_link="${parent_link}" id="2">
-      <origin xyz="0 0.055 -0.165" rpy="0 1.5708 1.5708"/>
-    </xacro:apriltag_marker>
-    <xacro:apriltag_marker parent_link="${parent_link}" id="3">
-      <origin xyz="0 -0.055 -0.165" rpy="0 1.5708 -1.5708"/>
-    </xacro:apriltag_marker>
-    <xacro:apriltag_marker parent_link="${parent_link}" id="4">
-      <origin xyz="0 0 -0.22" rpy="0 3.1416 0"/>
-    </xacro:apriltag_marker>
-    <xacro:apriltag_marker parent_link="${parent_link}" id="111">
-      <origin xyz="0 0 -0.11" rpy="0 3.1416 0"/>
-    </xacro:apriltag_marker>
   </xacro:macro>
   <!-- 右臂AprilTag标记 -->
-  <xacro:macro name="right_arm_apriltags" params="parent_link">
-    <xacro:apriltag_marker parent_link="${parent_link}" id="5">
-      <origin xyz="0.055 0 -0.165" rpy="0 1.5708 0"/>
-    </xacro:apriltag_marker>
-    <xacro:apriltag_marker parent_link="${parent_link}" id="6">
-      <origin xyz="-0.055 0 -0.165" rpy="0 1.5708 3.1415"/>
-    </xacro:apriltag_marker>
-    <xacro:apriltag_marker parent_link="${parent_link}" id="7">
-      <origin xyz="0 0.055 -0.165" rpy="0 1.5708 1.5708"/>
-    </xacro:apriltag_marker>
-    <xacro:apriltag_marker parent_link="${parent_link}" id="8">
-      <origin xyz="0 -0.055 -0.165" rpy="0 1.5708 -1.5708"/>
-    </xacro:apriltag_marker>
-    <xacro:apriltag_marker parent_link="${parent_link}" id="9">
-      <origin xyz="0 0 -0.22" rpy="0 3.1416 0"/>
-    </xacro:apriltag_marker>
-    <xacro:apriltag_marker parent_link="${parent_link}" id="999">
-      <origin xyz="0 0 -0.11" rpy="0 3.1416 0"/>
-    </xacro:apriltag_marker>
-  </xacro:macro>
 </robot>

File: src/kuavo_assets/models/apriltag/urdf/grab_box_table.xacro (robot description, xacro)
@@ -194,5 +194,5 @@
     </inertial>
   </link>
-  <link name="apriltag_box_tag2_base">
+  <link name="apriltag_shelf_base">
     <visual>
       <geometry>
@@ -213,42 +213,4 @@
     </inertial>
   </link>
-  <link name="apriltag_box_tag3_base">
-    <visual>
-      <geometry>
-        <box size="0.1 0.1 0.1"/>
-      </geometry>
-      <material>
-        <color rgba="0.8 0.8 0.8 0.5"/>
-      </material>
-    </visual>
-    <collision>
-      <geometry>
-        <box size="0.1 0.1 0.1"/>
-      </geometry>
-    </collision>
-    <inertial>
-      <mass value="0.1"/>
-      <inertia ixx="0.0001" ixy="0" ixz="0" iyy="0.0001" iyz="0" izz="0.0001"/>
-    </inertial>
-  </link>
-  <link name="apriltag_shelf_base">
-    <visual>
-      <geometry>
-        <box size="0.1 0.1 0.1"/>
-      </geometry>
-      <material>
-        <color rgba="0.8 0.8 0.8 0.5"/>
-      </material>
-    </visual>
-    <collision>
-      <geometry>
-        <box size="0.1 0.1 0.1"/>
-      </geometry>
-    </collision>
-    <inertial>
-      <mass value="0.1"/>
-      <inertia ixx="0.0001" ixy="0" ixz="0" iyy="0.0001" iyz="0" izz="0.0001"/>
-    </inertial>
-  </link>
   <!-- 将立方体连接到世界坐标系 -->
   <joint name="world_to_box_tag_joint" type="fixed">
@@ -257,14 +219,4 @@
     <origin xyz="0.0 -1.7 1.05" rpy="0 0 0"/>
   </joint>
-  <joint name="world_to_box_tag2_joint" type="fixed">
-    <parent link="world"/>
-    <child link="apriltag_box_tag2_base"/>
-    <origin xyz="0.5 -1.7 1.3" rpy="0 0 0"/>
-  </joint>
-  <joint name="world_to_box_tag3_joint" type="fixed">
-    <parent link="world"/>
-    <child link="apriltag_box_tag3_base"/>
-    <origin xyz="-0.5 -1.7 0.75" rpy="0 0 0"/>
-  </joint>
   <joint name="world_to_table_joint" type="fixed">
     <parent link="world"/>
@@ -273,10 +225,4 @@
   </joint>
   <xacro:apriltag_marker parent_link="apriltag_box_base" id="1">
-    <origin xyz="0 -0.055 -0.165" rpy="1.5708 1.5708 0"/>
-  </xacro:apriltag_marker>
-  <xacro:apriltag_marker parent_link="apriltag_box_tag2_base" id="2">
-    <origin xyz="0 -0.055 -0.165" rpy="1.5708 1.5708 0"/>
-  </xacro:apriltag_marker>
-  <xacro:apriltag_marker parent_link="apriltag_box_tag3_base" id="3">
     <origin xyz="0 -0.055 -0.165" rpy="1.5708 1.5708 0"/>
   </xacro:apriltag_marker>

File: src/kuavo_assets/models/biped_s100045/urdf/drake/biped_v3_arm.urdf (robot description, URDF)
Before this commit: robot biped_s100045, 19 links, 18 joints
Links:
- removed link zarm_l7_virtual_thumb_link
- removed link zarm_r7_virtual_thumb_link
Joints:
- removed joint zarm_l7_virtual_thumb_joint_ee
- removed joint zarm_r7_virtual_thumb_joint_ee

File: src/kuavo_assets/models/biped_s100049/urdf/drake/biped_v3_arm.urdf (robot description, URDF)
Before this commit: robot biped_s100049, 19 links, 18 joints
Links:
- removed link zarm_l7_virtual_thumb_link
- removed link zarm_r7_virtual_thumb_link
Joints:
- removed joint zarm_l7_virtual_thumb_joint_ee
- removed joint zarm_r7_virtual_thumb_joint_ee

File: src/kuavo_assets/models/biped_s11/urdf/biped_s11.urdf (robot description, URDF)
Before this commit: robot biped_s11, 37 links, 36 joints
Joints:
- joint dummy_to_base_link: type fixed -> floating

File: src/kuavo_assets/models/biped_s13/urdf/biped_s13.urdf (robot description, URDF)
Before this commit: robot biped_s13, 39 links, 38 joints
Links:
- removed link waist_yaw_link
- added link waist_yaw, mass 4.09458758; visual mesh filename=package://kuavo_assets/models/biped_s13/meshes/torso.STL
Joints:
- joint base_link_to_dummy_link: type fixed -> floating
- joint waist_yaw_joint: child waist_yaw_link -> waist_yaw
- joint zarm_l1_joint: parent waist_yaw_link -> waist_yaw
- joint zarm_r1_joint: parent waist_yaw_link -> waist_yaw
- joint zhead_1_joint: parent waist_yaw_link -> waist_yaw

File: src/kuavo_assets/models/biped_s13/urdf/biped_s13_gazebo.urdf (robot description, URDF)
Before this commit: robot biped_s13, 39 links, 38 joints
Links:
- removed link waist_yaw_link
- added link waist_yaw, mass 4.09458758; visual mesh filename=package://kuavo_assets/models/biped_s13/meshes/torso.STL
Joints:
- joint waist_yaw_joint: child waist_yaw_link -> waist_yaw
- joint zarm_l1_joint: parent waist_yaw_link -> waist_yaw
- joint zarm_r1_joint: parent waist_yaw_link -> waist_yaw
- joint zhead_1_joint: parent waist_yaw_link -> waist_yaw

File: src/kuavo_assets/models/biped_s13/urdf/drake/biped_v3.urdf (robot description, URDF)
Before this commit: robot biped_v3, 14 links, 13 joints
Links:
- removed link waist_yaw_link
- added link waist_yaw, mass 11.23288758; visual mesh filename=../../meshes/torso.STL
Joints:
- joint waist_yaw_joint: child waist_yaw_link -> waist_yaw

File: src/kuavo_assets/models/biped_s13/urdf/drake/biped_v3_all_joint.urdf (robot description, URDF)
Before this commit: robot biped_v3_all_joint, 30 links, 25 joints
Links:
- link torso: mass 5.17741242 -> 0.07761242

File: src/kuavo_assets/models/biped_s13/urdf/drake/biped_v3_arm.urdf (robot description, URDF)
Before this commit: robot biped_v3_arm, 10 links, 9 joints
Links:
- removed link waist_yaw_link
- added link waist_yaw, mass 7.34228758; visual mesh filename=../../meshes/torso.STL
Joints:
- joint waist_yaw_joint: child waist_yaw_link -> waist_yaw
- joint zarm_l1_joint: parent waist_yaw_link -> waist_yaw
- joint zarm_r1_joint: parent waist_yaw_link -> waist_yaw

File: src/kuavo_assets/models/biped_s14/urdf/biped_s14.urdf (robot description, URDF)
Before this commit: robot biped_s14, 41 links, 40 joints
Links:
- link base_link: mass 4.60775998 -> 8.620576; geometry visual mesh filename=package://kuavo_assets/models/biped_s14/meshes/torso.STL
- link camera: mass 0.000011119 -> 0.011119
- link camera_base: mass 0.00003927 -> 3.927E-05
- link leg_r1_link: mass 0.42877473 -> 0.42877618
- link leg_r2_link: mass 2.50010758 -> 2.4999594
- link leg_r3_link: mass 1.10966483 -> 1.109669
- link leg_r4_link: mass 1.55001765 -> 1.55038362
- link leg_r6_link: mass 0.34819252 -> 0.34819511
- link waist_yaw_link: mass 8.620776 -> 4.60775998; geometry visual mesh filename=package://kuavo_assets/models/biped_s14/meshes/waist.STL
- link zarm_l4_link: mass 0.56269441 -> 0.16269441
- link zarm_r1_link: mass 0.3730157 -> 0.37301773
- link zarm_r2_link: mass 0.15112869 -> 0.15112665
- link zarm_r4_link: mass 0.56269441 -> 0.16269033
- link zhead_1_link: mass 1.03077542 -> 0.32829; geometry collision mesh filename=package://kuavo_assets/models/biped_s14/meshes/head_yaw.STL; visual mesh filename=package://kuavo_assets/models/biped_s14/meshes/head_yaw.STL
- link zhead_2_link: mass 0.33654975 -> 0.33162; geometry collision mesh filename=package://kuavo_assets/models/biped_s14/meshes/head_pitch.S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; visual mesh filename=package://kuavo_assets/models/biped_s14/meshes/head_pitch.S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
Joints:
- joint dummy_to_base_link: type fixed -> floating
- joint leg_r4_joint: origin xyz=-0.0209999999999696 0 -0.181999999999961 rpy=0 0 0 -> xyz=-0.0209999999999396 0 -0.182000000000001 rpy=0 0 0
- joint leg_r5_joint: origin xyz=0.0209999999999503 0 -0.235000000000001 rpy=0 0 0 -> xyz=0.0209999999999936 0 -0.235 rpy=0 0 0
- joint ll_foot_toe_joint: origin xyz=0.121 0.03824834 -0.0435 rpy=0 0 0 -> xyz=0.121 0.04149834 -0.0435 rpy=0 0 0
- joint rl_foot_toe_joint: origin xyz=0.121 0.03824834 -0.0435 rpy=0 0 0 -> xyz=0.121 0.04149834 -0.0435 rpy=0 0 0
- joint zarm_r4_joint: origin xyz=0 0 -0.187999999999999 rpy=0 0 0 -> xyz=0 0 -0.187999999999989 rpy=0 0 0
- joint zhead_1_joint: origin xyz=0 0 0.35618885 rpy=0 0 0 -> xyz=0.00400001 2.92e-06 0.35618885 rpy=0 0 0

File: src/kuavo_assets/models/biped_s14/urdf/biped_s14_gazebo.urdf (robot description, URDF)
Before this commit: robot biped_s14, 41 links, 40 joints
Links:
- link base_link: mass 4.60775998 -> 4.787076; geometry visual mesh filename=package://kuavo_assets/models/biped_s14/meshes/torso.STL
- link camera: mass 0.000011119 -> 0.011119
- link camera_base: mass 0.00003927 -> 3.927E-05
- link leg_r1_link: mass 0.42877473 -> 0.42877618
- link leg_r2_link: mass 2.50010758 -> 2.4999594
- link leg_r3_link: mass 1.10966483 -> 1.109669
- link leg_r4_link: mass 1.55001765 -> 1.55038362
- link leg_r6_link: mass 0.34819252 -> 0.34819511
- link waist_yaw_link: mass 8.620776 -> 4.60775998; geometry visual mesh filename=package://kuavo_assets/models/biped_s14/meshes/waist.STL
- link zarm_l4_link: mass 0.56269441 -> 0.16269441
- link zarm_r1_link: mass 0.3730157 -> 0.37301773
- link zarm_r2_link: mass 0.15112869 -> 0.15112665
- link zarm_r4_link: mass 0.56269441 -> 0.16269033
- link zhead_1_link: mass 1.03077542 -> 0.32829; geometry collision mesh filename=package://kuavo_assets/models/biped_s14/meshes/head_yaw.STL; visual mesh filename=package://kuavo_assets/models/biped_s14/meshes/head_yaw.STL
- link zhead_2_link: mass 0.33654975 -> 0.33162; geometry collision mesh filename=package://kuavo_assets/models/biped_s14/meshes/head_pitch.S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; visual mesh filename=package://kuavo_assets/models/biped_s14/meshes/head_pitch.S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
Joints:
- joint l_foot_heel_joint: origin xyz=-0.04 -0.03824834 -0.0435 rpy=0 0 0 -> xyz=-0.084 0.0 -0.0435 rpy=0 0 0
- joint l_foot_toe_joint: origin xyz=-0.04 0.03824834 -0.0435 rpy=0 0 0 -> xyz=0.121 0.0 -0.0435 rpy=0 0 0
- joint leg_r4_joint: origin xyz=-0.0209999999999696 0 -0.181999999999961 rpy=0 0 0 -> xyz=-0.0209999999999396 0 -0.182000000000001 rpy=0 0 0
- joint leg_r5_joint: origin xyz=0.0209999999999503 0 -0.235000000000001 rpy=0 0 0 -> xyz=0.0209999999999936 0 -0.235 rpy=0 0 0
- joint ll_foot_toe_joint: origin xyz=0.121 0.03824834 -0.0435 rpy=0 0 0 -> xyz=0.121 0.04149834 -0.0435 rpy=0 0 0
- joint r_foot_heel_joint: origin xyz=-0.04 -0.03824834 -0.0435 rpy=0 0 0 -> xyz=-0.084 0.0 -0.0435 rpy=0 0 0
- joint r_foot_toe_joint: origin xyz=-0.04 0.03824834 -0.0435 rpy=0 0 0 -> xyz=0.121 0.0 -0.0435 rpy=0 0 0
- joint rl_foot_toe_joint: origin xyz=0.121 0.03824834 -0.0435 rpy=0 0 0 -> xyz=0.121 0.04149834 -0.0435 rpy=0 0 0
- joint zarm_r4_joint: origin xyz=0 0 -0.187999999999999 rpy=0 0 0 -> xyz=0 0 -0.187999999999989 rpy=0 0 0
- joint zhead_1_joint: origin xyz=0 0 0.35618885 rpy=0 0 0 -> xyz=0.00400001 2.92e-06 0.35618885 rpy=0 0 0

File: src/kuavo_assets/models/biped_s14/urdf/drake/biped_v3.urdf (robot description, URDF)
Before this commit: robot biped_v3, 14 links, 13 joints
Links:
- link leg_r1_link: mass 0.42877473 -> 0.42877618
- link leg_r2_link: mass 2.50010758 -> 2.4999594
- link leg_r3_link: mass 1.10966483 -> 1.109669
- link leg_r4_link: mass 1.55001765 -> 1.55038362
- link leg_r6_link: mass 0.34819252 -> 0.34819511
- link torso: mass 13.500276 -> 12.69998758
Joints:
- joint leg_r4_joint: origin xyz=-0.0209999999999696 0 -0.181999999999961 rpy=0 0 0 -> xyz=-0.0209999999999396 0 -0.182000000000001 rpy=0 0 0
- joint leg_r5_joint: origin xyz=0.0209999999999503 0 -0.235000000000001 rpy=0 0 0 -> xyz=0.0209999999999936 0 -0.235 rpy=0 0 0

File: src/kuavo_assets/models/biped_s14/urdf/drake/biped_v3_all_joint.urdf (robot description, URDF)
Before this commit: robot biped_v3_all_joint, 30 links, 25 joints
Links:
- link torso: mass 8.29741242 -> 0.07761242

File: src/kuavo_assets/models/biped_s14/urdf/drake/biped_v3_full.urdf (robot description, URDF)
Before this commit: robot biped_v3_full, 22 links, 21 joints
Links:
- link torso: mass 10.787876 -> 9.987876

File: src/kuavo_assets/models/biped_s45/urdf/biped_s45.urdf (robot description, URDF)
Before this commit: robot biped_s45, 53 links, 52 joints
Links:
- link base_link: mass 27.41553803 -> 21.63013803

File: src/kuavo_assets/models/biped_s45/urdf/biped_s45_gazebo.urdf (robot description, URDF)
Before this commit: robot biped_s45, 47 links, 46 joints
Links:
- link base_link: mass 27.89833803 -> 22.11293803

File: src/kuavo_assets/models/biped_s45/urdf/drake/biped_v3.urdf (robot description, URDF)
Before this commit: robot biped_v3, 13 links, 12 joints
Links:
- link torso: mass 39.51433803 -> 33.72893803

File: src/kuavo_assets/models/biped_s45/urdf/drake/biped_v3_all_joint.urdf (robot description, URDF)
Before this commit: robot biped_v3_all_joint, 35 links, 30 joints
Links:
- link torso: mass 28.48754316 -> 22.70214316

File: src/kuavo_assets/models/biped_s45/urdf/drake/biped_v3_arm.urdf (robot description, URDF)
Before this commit: robot biped_s45, 19 links, 18 joints
Links:
- removed link zarm_l7_virtual_thumb_link
- removed link zarm_r7_virtual_thumb_link
Joints:
- removed joint zarm_l7_virtual_thumb_joint_ee
- removed joint zarm_r7_virtual_thumb_joint_ee
- joint zarm_l2_joint: limit lower=-0.349065850398866 upper=1.46 effort=50.0 velocity=19.154 -> lower=-0.349065850398866 upper=2.0943951023932 effort=50.0 velocity=19.154
- joint zarm_l3_joint: limit lower=-1.5707963267949 upper=0.46 effort=39.0 velocity=18.84 -> lower=-1.5707963267949 upper=1.5707963267949 effort=39.0 velocity=18.84
- joint zarm_r2_joint: limit lower=-1.46 upper=0.349065850398866 effort=50.0 velocity=19.154 -> lower=-2.0943951023932 upper=0.349065850398866 effort=50.0 velocity=19.154
- joint zarm_r3_joint: limit lower=-0.46 upper=1.5707963267949 effort=39.0 velocity=18.84 -> lower=-1.5707963267949 upper=1.5707963267949 effort=39.0 velocity=18.84
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