Commit message: sync https://www.lejuhub.com/highlydynamic/kuavo-ros-control/commit/3aef0862d6b6fe1a91b6fd0f5977d42a207e0bc0

File: src/kuavo_assets/models/biped_s43/urdf/biped_s43.urdf (robot description, URDF)
Before this commit: robot biped_s43, 46 links, 45 joints
Links:
- link base_link: geometry visual mesh filename=package://kuavo_assets/models/biped_s43/meshes/base_link.STL
- link zarm_l2_link: geometry visual mesh filename=package://kuavo_assets/models/biped_s43/meshes/l_arm_roll.S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
- link zarm_l4_link: geometry visual mesh filename=package://kuavo_assets/models/biped_s43/meshes/l_forearm.STL
- link zarm_l7_link: geometry visual mesh filename=package://kuavo_assets/models/biped_s43/meshes/l_hand_pitch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
- link zarm_r2_link: geometry visual mesh filename=package://kuavo_assets/models/biped_s43/meshes/r_arm_roll.S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
- link zarm_r4_link: geometry visual mesh filename=package://kuavo_assets/models/biped_s43/meshes/r_forearm.STL
- link zarm_r7_link: geometry visual mesh filename=package://kuavo_assets/models/biped_s43/meshes/r_hand_pitch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
- link zhead_1_link: geometry visual mesh filename=package://kuavo_assets/models/biped_s43/meshes/head_yaw.STL

File: src/kuavo_assets/models/biped_s45/urdf/biped_s45.urdf (robot description, URDF)
Before this commit: robot biped_s45, 53 links, 52 joints
Links:
- removed link l_hand_camera
- removed link l_hand_tripod
- removed link r_hand_camera
- removed link r_hand_tripod
- link base_link: mass 27.41553803 -> 21.77493803; geometry visual mesh filename=package://kuavo_assets/models/biped_s45/meshes/torso.STL
- link zarm_l2_link: geometry visual mesh filename=package://kuavo_assets/models/biped_s45/meshes/l_arm_roll.S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
- link zarm_l4_link: geometry visual mesh filename=package://kuavo_assets/models/biped_s45/meshes/l_forearm.STL
- link zarm_l7_end_effector: geometry collision sphere radius=0.005
- link zarm_l7_link: geometry visual mesh filename=package://kuavo_assets/models/biped_s45/meshes/l_hand_pitch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
- link zarm_r2_link: geometry visual mesh filename=package://kuavo_assets/models/biped_s45/meshes/r_arm_roll.S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
- link zarm_r4_link: geometry visual mesh filename=package://kuavo_assets/models/biped_s45/meshes/r_forearm.STL
- link zarm_r7_end_effector: geometry collision sphere radius=0.005
- link zarm_r7_link: geometry visual mesh filename=package://kuavo_assets/models/biped_s45/meshes/r_hand_pitch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
- link zhead_1_link: geometry visual mesh filename=package://kuavo_assets/models/biped_s45/meshes/head_yaw.STL
Joints:
- removed joint l_hand_camera_joint
- removed joint l_hand_tripod_joint
- removed joint r_hand_camera_joint
- removed joint r_hand_tripod_joint

File: src/kuavo_assets/models/biped_s45/urdf/drake/biped_v3_arm.urdf (robot description, URDF)
Before this commit: robot biped_s45, 17 links, 16 joints
Joints:
- joint zarm_l1_joint: limit lower=-2.4 upper=0.6 effort=100.0 velocity=41.3433333333333 -> lower=-3.14159265358979 upper=1.5707963267949 effort=100.0 velocity=41.3433333333333
- joint zarm_l2_joint: limit lower=-0.349065850398866 upper=1.46 effort=50.0 velocity=19.154 -> lower=-0.349065850398866 upper=2.0943951023932 effort=50.0 velocity=19.154
- joint zarm_l3_joint: limit lower=-1.5707963267949 upper=0.46 effort=39.0 velocity=18.84 -> lower=-1.5707963267949 upper=1.5707963267949 effort=39.0 velocity=18.84
- joint zarm_r1_joint: limit lower=-2.4 upper=0.6 effort=100.0 velocity=41.3433333333333 -> lower=-3.14159265358979 upper=1.5707963267949 effort=100.0 velocity=41.3433333333333
- joint zarm_r2_joint: limit lower=-1.46 upper=0.349065850398866 effort=50.0 velocity=19.154 -> lower=-2.0943951023932 upper=0.349065850398866 effort=50.0 velocity=19.154
- joint zarm_r3_joint: limit lower=-0.46 upper=1.5707963267949 effort=39.0 velocity=18.84 -> lower=-1.5707963267949 upper=1.5707963267949 effort=39.0 velocity=18.84

File: src/kuavo_assets/models/biped_s46/urdf/biped_s46.urdf (robot description, URDF)
Before this commit: robot biped_s46, 46 links, 45 joints
Links:
- link base_link: geometry visual mesh filename=package://kuavo_assets/models/biped_s46/meshes/torso.STL
- link zarm_l2_link: geometry visual mesh filename=package://kuavo_assets/models/biped_s46/meshes/l_arm_roll.S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
- link zarm_l4_link: geometry visual mesh filename=package://kuavo_assets/models/biped_s46/meshes/l_forearm.STL
- link zarm_l7_link: geometry visual mesh filename=package://kuavo_assets/models/biped_s46/meshes/l_hand_pitch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
- link zarm_r2_link: geometry visual mesh filename=package://kuavo_assets/models/biped_s46/meshes/r_arm_roll.S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
- link zarm_r4_link: geometry visual mesh filename=package://kuavo_assets/models/biped_s46/meshes/r_forearm.STL
- link zarm_r7_link: geometry visual mesh filename=package://kuavo_assets/models/biped_s46/meshes/r_hand_pitch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
- link zhead_1_link: geometry visual mesh filename=package://kuavo_assets/models/biped_s46/meshes/head_yaw.STL

File: src/kuavo_assets/models/biped_s46/urdf/drake/biped_v3_arm.urdf (robot description, URDF)
Before this commit: robot biped_s46, 17 links, 16 joints
Joints:
- joint zarm_l1_joint: limit lower=-2.4 upper=0.6 effort=100.0 velocity=41.3433333333333 -> lower=-3.14159265358979 upper=1.5707963267949 effort=100.0 velocity=41.3433333333333
- joint zarm_l2_joint: limit lower=-0.349065850398866 upper=1.46 effort=50.0 velocity=19.154 -> lower=-0.349065850398866 upper=2.0943951023932 effort=50.0 velocity=8.37333333333333
- joint zarm_l3_joint: limit lower=-1.5707963267949 upper=0.46 effort=39.0 velocity=18.84 -> lower=-1.5707963267949 upper=1.5707963267949 effort=39.0 velocity=19.3633333333333
- joint zarm_r1_joint: limit lower=-2.4 upper=0.6 effort=100.0 velocity=41.3433333333333 -> lower=-3.14159265358979 upper=1.5707963267949 effort=100.0 velocity=41.3433333333333
- joint zarm_r2_joint: limit lower=-1.46 upper=0.349065850398866 effort=50.0 velocity=19.154 -> lower=-2.0943951023932 upper=0.349065850398866 effort=50.0 velocity=8.37333333333333
- joint zarm_r3_joint: limit lower=-0.46 upper=1.5707963267949 effort=39.0 velocity=18.84 -> lower=-1.5707963267949 upper=1.5707963267949 effort=39.0 velocity=18.84

File: src/kuavo_assets/models/biped_s47/urdf/biped_s47.urdf (robot description, URDF)
Before this commit: robot biped_s47, 64 links, 63 joints
Links:
- removed link l_b_bar-1
- removed link l_b_bar-2
- removed link l_b_bar-3
- removed link l_b_fingers
- removed link l_f_bar-1
- removed link l_f_bar-2
- removed link l_f_bar-3
- removed link l_f_fingers
- removed link l_hand_camera
- removed link r_b_bar-1
- removed link r_b_bar-2
- removed link r_b_bar-3
- removed link r_b_fingers
- removed link r_f_bar-1
- removed link r_f_bar-2
- removed link r_f_bar-3
- removed link r_f_fingers
- removed link r_hand_camera
- added link l_b_claw_1, mass 0.045; visual mesh filename=package://kuavo_assets/models/biped_s47/meshes/l_b_claw_1.S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
- added link l_b_claw_2, mass 0.009; visual mesh filename=package://kuavo_assets/models/biped_s47/meshes/l_b_claw_2.S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
- added link l_b_claw_3, mass 0.013; visual mesh filename=package://kuavo_assets/models/biped_s47/meshes/l_b_claw_3.S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
- added link l_b_finger, mass 0.014; visual mesh filename=package://kuavo_assets/models/biped_s47/meshes/l_b_finger.S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
- added link l_f_claw_1, mass 0.045; visual mesh filename=package://kuavo_assets/models/biped_s47/meshes/l_f_claw_1.S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
- added link l_f_claw_2, mass 0.009; visual mesh filename=package://kuavo_assets/models/biped_s47/meshes/l_f_claw_2.S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
- added link l_f_claw_3, mass 0.013; visual mesh filename=package://kuavo_assets/models/biped_s47/meshes/l_f_claw_3.S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
- added link l_f_finger, mass 0.014; visual mesh filename=package://kuavo_assets/models/biped_s47/meshes/l_f_finger.S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
- added link r_b_claw_1, mass 0.045; visual mesh filename=package://kuavo_assets/models/biped_s47/meshes/r_b_claw_1.S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
- added link r_b_claw_2, mass 0.009; visual mesh filename=package://kuavo_assets/models/biped_s47/meshes/r_b_claw_2.S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
- added link r_b_claw_3, mass 0.013; visual mesh filename=package://kuavo_assets/models/biped_s47/meshes/r_b_claw_3.S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
- added link r_b_finger, mass 0.014; visual mesh filename=package://kuavo_assets/models/biped_s47/meshes/r_b_finger.S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
- added link r_f_claw_1, mass 0.045; visual mesh filename=package://kuavo_assets/models/biped_s47/meshes/r_f_claw_1.S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
- added link r_f_claw_2, mass 0.0034; visual mesh filename=package://kuavo_assets/models/biped_s47/meshes/r_f_claw_2.S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
- added link r_f_claw_3, mass 0.013; visual mesh filename=package://kuavo_assets/models/biped_s47/meshes/r_f_claw_3.S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
- added link r_f_finger, mass 0.014; visual mesh filename=package://kuavo_assets/models/biped_s47/meshes/r_f_finger.S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
- link base_link: mass 27.65133803 -> 27.65693803; geometry visual mesh filename=package://kuavo_assets/models/biped_s47/meshes/torso.STL
- link zarm_l2_link: geometry visual mesh filename=package://kuavo_assets/models/biped_s47/meshes/l_arm_roll.S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
- link zarm_l4_link: geometry visual mesh filename=package://kuavo_assets/models/biped_s47/meshes/l_forearm.STL
- link zarm_l7_link: geometry visual mesh filename=package://kuavo_assets/models/biped_s47/meshes/l_hand_pitch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
- link zarm_r2_link: geometry visual mesh filename=package://kuavo_assets/models/biped_s47/meshes/r_arm_roll.S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
- link zarm_r4_link: geometry visual mesh filename=package://kuavo_assets/models/biped_s47/meshes/r_forearm.STL
- link zarm_r7_link: geometry visual mesh filename=package://kuavo_assets/models/biped_s47/meshes/r_hand_pitch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
- link zhead_1_link: geometry visual mesh filename=package://kuavo_assets/models/biped_s47/meshes/head_yaw.STL
Joints:
- removed joint l_b_bar-1
- removed joint l_b_bar-2
- removed joint l_b_bar-3
- removed joint l_b_fingers
- removed joint l_f_bar-1_joint
- removed joint l_f_bar-2
- removed joint l_f_bar-3
- removed joint l_f_fingers
- removed joint l_hand_camera_joint
- removed joint r_b_bar-1
- removed joint r_b_bar-2
- removed joint r_b_bar-3
- removed joint r_b_fingers
- removed joint r_f_bar-1_joint
- removed joint r_f_bar-2
- removed joint r_f_bar-3
- removed joint r_f_fingers
- removed joint r_hand_camera_joint
- added joint l_b_claw_1: type fixed, parent zarm_l7_link, child l_b_claw_1, origin xyz=-0.0219999996097237 0 -0.1114 rpy=0 0 0, axis 0 1 0
- added joint l_b_claw_2: type fixed, parent l_b_claw_1, child l_b_claw_2, origin xyz=-0.0254380979411351 0 -0.0464962705293328 rpy=0 0 0, axis 0 1 0
- added joint l_b_claw_3: type fixed, parent zarm_l7_link, child l_b_claw_3, origin xyz=-0.0239578924930216 0 -0.135271672920607 rpy=0 0 0, axis 0 1 0
- added joint l_b_finger: type fixed, parent l_b_claw_2, child l_b_finger, origin xyz=0.0191548518271917 0 -0.0292932014550803 rpy=0 0 0, axis 0 1 0
- added joint l_f_claw_1: type fixed, parent zarm_l7_link, child l_f_claw_1, origin xyz=0.0220000003906073 0 -0.111399999999999 rpy=0 0 0, axis 0 1 0, limit lower=-0.698 upper=0.698 effort=0 velocity=0
- added joint l_f_claw_2: type fixed, parent l_f_claw_1, child l_f_claw_2, origin xyz=0.025438097941138 0 -0.0464962705293307 rpy=0 0 0, axis 0 1 0
- added joint l_f_claw_3: type fixed, parent zarm_l7_link, child l_f_claw_3, origin xyz=0.0239578932739072 0 -0.135271672920607 rpy=0 0 0, axis 0 1 0
- added joint l_f_finger: type fixed, parent l_f_claw_2, child l_f_finger, origin xyz=-0.0191548518271909 0 -0.0292932014550821 rpy=0 0 0, axis 0 1 0
- added joint r_b_claw_1: type fixed, parent zarm_r7_link, child r_b_claw_1, origin xyz=-0.022000000390599 -0.000500000000001402 -0.111399999999999 rpy=0 0 0, axis 0 1 0
- added joint r_b_claw_2: type fixed, parent r_b_claw_1, child r_b_claw_2, origin xyz=-0.0254380979411353 0 -0.0464962705293326 rpy=0 0 0, axis 0 1 0
- added joint r_b_claw_3: type fixed, parent zarm_r7_link, child r_b_claw_3, origin xyz=-0.0239578932738948 -0.000500000000001666 -0.135271672920607 rpy=0 0 0
- added joint r_b_finger: type fixed, parent r_b_claw_2, child r_b_finger, origin xyz=0.0191548518271923 0 -0.0292932014550809 rpy=0 0 0, axis 0 1 0
- added joint r_f_claw_1: type fixed, parent zarm_r7_link, child r_f_claw_1, origin xyz=0.0219999996097342 -0.000500000000000958 -0.1114 rpy=0 0 0, axis 0 1 0, limit lower=-0.698 upper=0.698 effort=0 velocity=0
- added joint r_f_claw_2: type fixed, parent r_f_claw_1, child r_f_claw_2, origin xyz=0.0254380979411394 0 -0.0464962705293306 rpy=0 0 0, axis 0 1 0
- added joint r_f_claw_3: type fixed, parent zarm_r7_link, child r_f_claw_3, origin xyz=0.023957892493034 -0.000500000000001166 -0.135271672920607 rpy=0 0 0, axis 0 1 0
- added joint r_f_finger: type fixed, parent r_f_claw_2, child r_f_finger, origin xyz=-0.0191548518271941 0 -0.0292932014550819 rpy=0 0 0, axis 0 1 0

File: src/kuavo_assets/models/biped_s47/urdf/drake/biped_v3_arm.urdf (robot description, URDF)
Before this commit: robot biped_s47, 17 links, 16 joints
Joints:
- joint zarm_l1_joint: limit lower=-2.4 upper=0.6 effort=100.0 velocity=41.3433333333333 -> lower=-3.14159265358979 upper=1.5707963267949 effort=100.0 velocity=41.3433333333333
- joint zarm_l2_joint: limit lower=-0.349065850398866 upper=1.46 effort=50.0 velocity=19.154 -> lower=-0.349065850398866 upper=2.0943951023932 effort=50.0 velocity=8.37333333333333
- joint zarm_l3_joint: limit lower=-1.5707963267949 upper=0.46 effort=39.0 velocity=18.84 -> lower=-1.5707963267949 upper=1.5707963267949 effort=39.0 velocity=19.3633333333333
- joint zarm_r1_joint: limit lower=-2.4 upper=0.6 effort=100.0 velocity=41.3433333333333 -> lower=-3.14159265358979 upper=1.5707963267949 effort=100.0 velocity=41.3433333333333
- joint zarm_r2_joint: limit lower=-1.46 upper=0.349065850398866 effort=50.0 velocity=19.154 -> lower=-2.0943951023932 upper=0.349065850398866 effort=50.0 velocity=8.37333333333333
- joint zarm_r3_joint: limit lower=-0.46 upper=1.5707963267949 effort=39.0 velocity=18.84 -> lower=-1.5707963267949 upper=1.5707963267949 effort=39.0 velocity=18.84

File: src/kuavo_assets/models/biped_s48/urdf/biped_s48.urdf (robot description, URDF)
Before this commit: robot biped_s48, 69 links, 68 joints
Links:
- link base_link: mass 27.41553803 -> 22.11293803; geometry visual mesh filename=package://kuavo_assets/models/biped_s48/meshes/torso.STL
- link zarm_l2_link: geometry visual mesh filename=package://kuavo_assets/models/biped_s48/meshes/l_arm_roll.S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
- link zarm_l4_link: geometry visual mesh filename=package://kuavo_assets/models/biped_s48/meshes/l_forearm.STL
- link zarm_l7_link: geometry visual mesh filename=package://kuavo_assets/models/biped_s48/meshes/l_hand_pitch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
- link zarm_r2_link: geometry visual mesh filename=package://kuavo_assets/models/biped_s48/meshes/r_arm_roll.S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
- link zarm_r4_link: geometry visual mesh filename=package://kuavo_assets/models/biped_s48/meshes/r_forearm.STL
- link zarm_r7_link: geometry visual mesh filename=package://kuavo_assets/models/biped_s48/meshes/r_hand_pitch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
- link zhead_2_link: geometry visual mesh filename=package://kuavo_assets/models/biped_s48/meshes/head_pitch.S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

File: src/kuavo_assets/models/biped_s48/urdf/drake/biped_v3_arm.urdf (robot description, URDF)
Before this commit: robot biped_s48, 17 links, 16 joints
Joints:
- joint zarm_l1_joint: limit lower=-2.4 upper=0.6 effort=100.0 velocity=41.3433333333333 -> lower=-3.14159265358979 upper=1.5707963267949 effort=100.0 velocity=41.3433333333333
- joint zarm_l2_joint: limit lower=-0.349065850398866 upper=1.46 effort=50.0 velocity=19.154 -> lower=-0.349065850398866 upper=2.0943951023932 effort=50.0 velocity=19.154
- joint zarm_l3_joint: limit lower=-1.5707963267949 upper=0.46 effort=39.0 velocity=18.84 -> lower=-1.5707963267949 upper=1.5707963267949 effort=39.0 velocity=18.84
- joint zarm_r1_joint: limit lower=-2.4 upper=0.6 effort=100.0 velocity=41.3433333333333 -> lower=-3.14159265358979 upper=1.5707963267949 effort=100.0 velocity=41.3433333333333
- joint zarm_r2_joint: limit lower=-1.46 upper=0.349065850398866 effort=50.0 velocity=19.154 -> lower=-2.0943951023932 upper=0.349065850398866 effort=50.0 velocity=19.154
- joint zarm_r3_joint: limit lower=-0.46 upper=1.5707963267949 effort=39.0 velocity=18.84 -> lower=-1.5707963267949 upper=1.5707963267949 effort=39.0 velocity=18.84

File: src/kuavo_assets/models/biped_s49/urdf/biped_s49.urdf (robot description, URDF)
Before this commit: robot biped_s49, 73 links, 72 joints
Links:
- removed link l_Index_prox
- removed link l_hand_camera
- removed link l_hand_tripod
- removed link l_index_dist
- removed link l_little_dist
- removed link l_little_prox
- removed link l_middle_dist
- removed link l_middle_prox
- removed link l_palm
- removed link l_ring_dist
- removed link l_ring_prox
- removed link l_thumb_dist
- removed link l_thumb_prox
- removed link r_hand_camera
- removed link r_hand_tripod
- removed link r_index_dist
- removed link r_index_prox
- removed link r_little_dist
- removed link r_little_prox
- removed link r_middle_dist
- removed link r_middle_prox
- removed link r_palm
- removed link r_ring_dist
- removed link r_ring_prox
- removed link r_thumb_dist
- removed link r_thumb_prox
- link base_link: mass 28.27893803 -> 28.34823803; geometry visual mesh filename=package://kuavo_assets/models/biped_s49/meshes/torso.STL
- link zarm_l2_link: geometry visual mesh filename=package://kuavo_assets/models/biped_s49/meshes/l_arm_roll.S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
- link zarm_l4_link: geometry visual mesh filename=package://kuavo_assets/models/biped_s49/meshes/l_forearm.STL
- link zarm_l7_link: mass 0.0542110173081966 -> 0.64; geometry visual mesh filename=package://kuavo_assets/models/biped_s49/meshes/l_hand_pitch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
- link zarm_r2_link: geometry visual mesh filename=package://kuavo_assets/models/biped_s49/meshes/r_arm_roll.S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
- link zarm_r4_link: geometry visual mesh filename=package://kuavo_assets/models/biped_s49/meshes/r_forearm.STL
- link zarm_r7_link: mass 0.0542110173081966 -> 0.64; geometry visual mesh filename=package://kuavo_assets/models/biped_s49/meshes/r_hand_pitch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
- link zhead_1_link: geometry visual mesh filename=package://kuavo_assets/models/biped_s49/meshes/head_yaw.STL
Joints:
- removed joint l_hand_camera_joint
- removed joint l_hand_tripod_joint
- removed joint l_indexMCP
- removed joint l_indexPIP
- removed joint l_littleMCP
- removed joint l_littlePIP
- removed joint l_middleMCP
- removed joint l_middlePIP
- removed joint l_palm_fixed_joint
- removed joint l_ringMCP
- removed joint l_ringPIP
- removed joint l_thumbCMC
- removed joint l_thumbMCP
- removed joint r_hand_camera_joint
- removed joint r_hand_tripod_joint
- removed joint r_indexMCP
- removed joint r_indexPIP
- removed joint r_littleMCP
- removed joint r_littlePIP
- removed joint r_middleMCP
- removed joint r_middlePIP
- removed joint r_palm_fixed_joint
- removed joint r_ringMCP
- removed joint r_ringPIP
- removed joint r_thumbCMC
- removed joint r_thumbMCP

File: src/kuavo_assets/models/biped_s49/urdf/drake/biped_v3_arm.urdf (robot description, URDF)
Before this commit: robot biped_s49, 17 links, 16 joints
Joints:
- joint zarm_l1_joint: limit lower=-2.4 upper=0.6 effort=100.0 velocity=41.3433333333333 -> lower=-3.14159265358979 upper=1.5707963267949 effort=100.0 velocity=41.3433333333333
- joint zarm_l2_joint: limit lower=-0.349065850398866 upper=1.46 effort=50.0 velocity=19.154 -> lower=-0.349065850398866 upper=2.0943951023932 effort=50.0 velocity=19.154
- joint zarm_l3_joint: limit lower=-1.5707963267949 upper=0.46 effort=39.0 velocity=18.84 -> lower=-1.5707963267949 upper=1.5707963267949 effort=39.0 velocity=18.84
- joint zarm_r1_joint: limit lower=-2.4 upper=0.6 effort=100.0 velocity=41.3433333333333 -> lower=-3.14159265358979 upper=1.5707963267949 effort=100.0 velocity=41.3433333333333
- joint zarm_r2_joint: limit lower=-1.46 upper=0.349065850398866 effort=50.0 velocity=19.154 -> lower=-2.0943951023932 upper=0.349065850398866 effort=50.0 velocity=19.154
- joint zarm_r3_joint: limit lower=-0.46 upper=1.5707963267949 effort=39.0 velocity=18.84 -> lower=-1.5707963267949 upper=1.5707963267949 effort=39.0 velocity=18.84
