Commit message: sync https://www.lejuhub.com/highlydynamic/kuavo-ros-control/commit/f9e3145c5cf180d7dfa9c408153e3d4951e30a8f

File: src/kuavo_assets/models/biped_s11/urdf/biped_s11.urdf (robot description, URDF)
Before this commit: robot biped_s11, 37 links, 36 joints
Joints:
- joint dummy_to_base_link: type floating -> fixed

File: src/kuavo_assets/models/biped_s13/urdf/biped_s13.urdf (robot description, URDF)
Before this commit: robot biped_s13, 39 links, 38 joints
Joints:
- joint base_link_to_dummy_link: type floating -> fixed

File: src/kuavo_assets/models/biped_s14/urdf/biped_s14.urdf (robot description, URDF)
Before this commit: robot biped_s14, 41 links, 40 joints
Joints:
- joint dummy_to_base_link: type floating -> fixed

File: src/kuavo_assets/models/biped_s200049/urdf/biped_s200049.urdf (robot description, URDF)
Before this commit: robot biped_s200049, 65 links, 64 joints
Joints:
- joint dummy_to_base_link: type floating -> fixed

File: src/kuavo_assets/models/biped_s46/urdf/biped_s46.urdf (robot description, URDF)
Before this commit: robot biped_s46, 46 links, 45 joints
Joints:
- joint dummy_to_base_link: type floating -> fixed

File: src/kuavo_assets/models/biped_s46/urdf/biped_s46_gazebo.urdf (robot description, URDF)
Before this commit: robot biped_s46, 46 links, 45 joints
Joints:
- joint dummy_to_base_link: type floating -> fixed

File: src/kuavo_assets/models/biped_s47/urdf/biped_s47.urdf (robot description, URDF)
Before this commit: robot biped_s47, 64 links, 63 joints
Joints:
- joint dummy_to_base_link: type floating -> fixed

File: src/kuavo_assets/models/biped_s50/urdf/biped_s50.urdf (robot description, URDF)
Before this commit: robot biped_s50, 49 links, 48 joints
Joints:
- joint dummy_to_base_link: type floating -> fixed

File: src/kuavo_assets/models/biped_s51/urdf/biped_s51.urdf (robot description, URDF)
Before this commit: robot biped_s51, 47 links, 46 joints
Joints:
- joint dummy_to_base_link: type floating -> fixed

File: src/kuavo_assets/models/biped_s52/urdf/biped_s52.urdf (robot description, URDF)
Before this commit: robot biped_s52, 47 links, 46 joints
Joints:
- joint dummy_to_base_link: type floating -> fixed
