Commit message: sync https://www.lejuhub.com/highlydynamic/kuavo-ros-control/commit/54c86d0b06c5471aa393407d048285bdb94db5dd

File: src/kuavo_assets/models/biped_s13/urdf/biped_s13_gazebo.urdf (robot description, URDF)
Before this commit: robot biped_s13, 39 links, 38 joints
Joints:
- removed joint dummy_to_base_link
- added joint base_link_to_dummy_link: type fixed, parent base_link, child dummy_link, origin xyz=0 0 0 rpy=0 0 0

File: src/kuavo_assets/models/biped_s14/urdf/biped_s14_gazebo.urdf (robot description, URDF)
Before this commit: robot biped_s14, 41 links, 40 joints
Joints:
- removed joint dummy_to_base_link
- added joint base_link_to_dummy_link: type fixed, parent base_link, child dummy_link, origin xyz=0 0 0 rpy=0 0 0

File: src/kuavo_assets/models/biped_s16/urdf/biped_s16_gazebo.urdf (robot description, URDF)
Before this commit: robot biped_s16, 41 links, 40 joints
Joints:
- removed joint dummy_to_base_link
- added joint base_link_to_dummy_link: type fixed, parent base_link, child dummy_link, origin xyz=0 0 0 rpy=0 0 0

File: src/kuavo_assets/models/biped_s17/urdf/biped_s17.urdf (robot description, URDF)
Before this commit: robot biped_s17, 43 links, 42 joints
Joints:
- removed joint dummy_to_base_link
- added joint base_link_to_dummy_link: type fixed, parent base_link, child dummy_link, origin xyz=0 0 0 rpy=0 0 0
- joint zhead_1_joint: origin xyz=0.0042 0 0.35369 rpy=0 0 0 -> xyz=0.0042 0 0.35469 rpy=0 0 0

File: src/kuavo_assets/models/biped_s17/urdf/biped_s17_gazebo.urdf (robot description, URDF)
Before this commit: robot biped_s17, 43 links, 42 joints
Joints:
- removed joint dummy_to_base_link
- added joint base_link_to_dummy_link: type fixed, parent base_link, child dummy_link, origin xyz=0 0 0 rpy=0 0 0
- joint zhead_1_joint: origin xyz=0.0042 0 0.35369 rpy=0 0 0 -> xyz=0.0042 0 0.35469 rpy=0 0 0

File: src/kuavo_assets/models/biped_s40/urdf/biped_s40_gazebo.urdf (robot description, URDF)
Before this commit: robot biped_s40, 46 links, 45 joints
Links:
- link base_link: mass 22.6889 -> 22.6719
Joints:
- removed joint dummy_to_base_link
- added joint base_link_to_dummy_link: type fixed, parent base_link, child dummy_link, origin xyz=0 0 0 rpy=0 0 0
