Commit message: sync https://www.lejuhub.com/highlydynamic/kuavo-ros-control/commit/d849ca18f85e3b9de947c9a2558a2f34144f0cd2

File: src/kuavo_assets/models/biped_s100045/urdf/drake/biped_v3_arm.urdf (robot description, URDF)
Before this commit: robot biped_s100045, 17 links, 16 joints
Links:
- added link zarm_l7_virtual_thumb_link; collision sphere radius=0.005
- added link zarm_r7_virtual_thumb_link; collision sphere radius=0.005
Joints:
- added joint zarm_l7_virtual_thumb_joint_ee: type fixed, parent zarm_l7_end_effector, child zarm_l7_virtual_thumb_link, origin xyz=0.15 0 0 rpy=0 0 0
- added joint zarm_r7_virtual_thumb_joint_ee: type fixed, parent zarm_r7_end_effector, child zarm_r7_virtual_thumb_link, origin xyz=0.15 0 0 rpy=0 0 0

File: src/kuavo_assets/models/biped_s100049/urdf/drake/biped_v3_arm.urdf (robot description, URDF)
Before this commit: robot biped_s100049, 17 links, 16 joints
Links:
- added link zarm_l7_virtual_thumb_link; collision sphere radius=0.005
- added link zarm_r7_virtual_thumb_link; collision sphere radius=0.005
Joints:
- added joint zarm_l7_virtual_thumb_joint_ee: type fixed, parent zarm_l7_end_effector, child zarm_l7_virtual_thumb_link, origin xyz=0.15 0 0 rpy=0 0 0
- added joint zarm_r7_virtual_thumb_joint_ee: type fixed, parent zarm_r7_end_effector, child zarm_r7_virtual_thumb_link, origin xyz=0.15 0 0 rpy=0 0 0

File: src/kuavo_assets/models/biped_s200049/urdf/drake/biped_v3_arm.urdf (robot description, URDF)
Before this commit: robot biped_s200049, 17 links, 16 joints
Links:
- added link zarm_l7_virtual_thumb_link; collision sphere radius=0.005
- added link zarm_r7_virtual_thumb_link; collision sphere radius=0.005
Joints:
- added joint zarm_l7_virtual_thumb_joint_ee: type fixed, parent zarm_l7_end_effector, child zarm_l7_virtual_thumb_link, origin xyz=0.15 0 0 rpy=0 0 0
- added joint zarm_r7_virtual_thumb_joint_ee: type fixed, parent zarm_r7_end_effector, child zarm_r7_virtual_thumb_link, origin xyz=0.15 0 0 rpy=0 0 0
