Commit message: sync https://www.lejuhub.com/highlydynamic/kuavo-ros-control/commit/0814304cd0ff346c69c2893130130d50b7bd6b1f

File: src/kuavo_assets/models/biped_s52/urdf/drake/biped_v3_arm.urdf (robot description, URDF)
Before this commit: robot biped_s52, 18 links, 17 joints
Joints:
- joint zarm_l1_joint: limit lower=-3.14159265358979 upper=1.5707963267949 effort=100.0 velocity=41.3433333333333 -> lower=-2.4 upper=0.6 effort=100.0 velocity=41.3433333333333; origin xyz=-0.003 0.1737 0.2831 rpy=0 0 0 -> xyz=-0.003 0.2547 0.2831 rpy=0 0 0
- joint zarm_l2_joint: limit lower=-0.349065850398866 upper=2.0943951023932 effort=50.0 velocity=8.37333333333333 -> lower=-0.349065850398866 upper=1.46 effort=50.0 velocity=19.154; origin xyz=0 0.081 0 rpy=0 0 0 -> xyz=0 0 0 rpy=0 0 0
- joint zarm_l3_joint: limit lower=-1.5707963267949 upper=1.5707963267949 effort=36.0 velocity=9.94333333333333 -> lower=-1.5707963267949 upper=0.46 effort=39.0 velocity=18.84
- joint zarm_l4_joint: limit lower=-2.61799387799149 upper=0.0 effort=50.0 velocity=8.37333333333333 -> lower=-2.61799387799149 upper=0.0 effort=50.0 velocity=18.84
- joint zarm_l5_joint: limit lower=-1.5707963267949 upper=1.5707963267949 effort=12.0 velocity=7.32666666666667 -> lower=-1.5707963267949 upper=1.5707963267949 effort=12.0 velocity=21.666
- joint zarm_l6_joint: limit lower=-1.30899693899575 upper=0.698131700797732 effort=12.0 velocity=7.32666666666667 -> lower=-1.30899693899575 upper=0.698131700797732 effort=12.0 velocity=21.666
- joint zarm_l7_joint: limit lower=-0.698131700797732 upper=0.698131700797732 effort=12.0 velocity=7.32666666666667 -> lower=-0.698131700797732 upper=0.698131700797732 effort=12.0 velocity=21.666
- joint zarm_r1_joint: limit lower=-3.14159265358979 upper=1.5707963267949 effort=100.0 velocity=41.3433333333333 -> lower=-2.4 upper=0.6 effort=100.0 velocity=41.3433333333333; origin xyz=-0.003 -0.1737 0.2831 rpy=0 0 0 -> xyz=-0.003 -0.2547 0.2831 rpy=0 0 0
- joint zarm_r2_joint: limit lower=-2.0943951023932 upper=0.349065850398866 effort=50.0 velocity=8.37333333333333 -> lower=-1.46 upper=0.349065850398866 effort=50.0 velocity=19.154; origin xyz=0 -0.081 0 rpy=0 0 0 -> xyz=0 0 0 rpy=0 0 0
- joint zarm_r3_joint: limit lower=-1.5707963267949 upper=1.5707963267949 effort=36.0 velocity=9.94333333333333 -> lower=-0.46 upper=1.5707963267949 effort=39.0 velocity=18.84
- joint zarm_r4_joint: limit lower=-2.61799387799149 upper=0.0 effort=50.0 velocity=8.37333333333333 -> lower=-2.61799387799149 upper=0.0 effort=50.0 velocity=18.84
- joint zarm_r5_joint: limit lower=-1.5707963267949 upper=1.5707963267949 effort=12.0 velocity=7.32666666666667 -> lower=-1.5707963267949 upper=1.5707963267949 effort=12.0 velocity=21.666
- joint zarm_r6_joint: limit lower=-0.698131700797732 upper=1.30899693899575 effort=12.0 velocity=7.32666666666667 -> lower=-0.698131700797732 upper=1.30899693899575 effort=12.0 velocity=21.666
- joint zarm_r7_joint: limit lower=-0.698131700797732 upper=0.698131700797732 effort=12.0 velocity=7.32666666666667 -> lower=-0.698131700797732 upper=0.698131700797732 effort=12.0 velocity=21.666

Commit message: sync https://www.lejuhub.com/highlydynamic/kuavo-ros-control/commit/94a6cbcd6b420f3c4529b6ab37c0e815bb9e4f0e

File: src/kuavo_assets/models/biped_s52/urdf/drake/biped_v3_arm.urdf (robot description, URDF)
Before this commit: robot biped_s45, 17 links, 16 joints
Links:
- added link waist_yaw_link, mass 18.01415568; visual mesh filename=../../meshes/waist_yaw.STL
- link base_link: mass 22.11293803 -> 6.48663928
- link zarm_l1_link: mass 0.962 -> 0.91653322
- link zarm_l2_link: mass 0.57 -> 0.3876739
- link zarm_l3_link: mass 1.65 -> 1.77926875
- link zarm_l4_link: mass 0.429 -> 0.58507821
- link zarm_l5_link: mass 0.61 -> 0.68679955
- link zarm_l6_link: mass 0.331 -> 0.39387181
- link zarm_l7_link: mass 0.64 -> 0.61537779
- link zarm_r1_link: mass 0.962 -> 0.92062797
- link zarm_r2_link: mass 0.57 -> 0.38768053
- link zarm_r3_link: mass 1.65 -> 1.77969208
- link zarm_r4_link: mass 0.429 -> 0.58514611
- link zarm_r5_link: mass 0.61 -> 0.68473867
- link zarm_r6_link: mass 0.331 -> 0.39247462
- link zarm_r7_link: mass 0.64 -> 0.61562202
Joints:
- added joint waist_yaw_joint: type fixed, parent base_link, child waist_yaw_link, origin xyz=0 0 0.1114 rpy=0 0 0, axis 0 0 1, limit lower=-3.14159 upper=3.14159 effort=180.0 velocity=23.55
- joint zarm_l1_joint: limit lower=-3.14159265358979 upper=1.5707963267949 effort=100.0 velocity=41.3433333333333 -> lower=-2.4 upper=0.6 effort=100.0 velocity=41.3433333333333; origin xyz=-0.017499853 0.29269999999999996 0.4245 rpy=0 0 0 -> xyz=-0.003 0.2547 0.2831 rpy=0 0 0; parent base_link -> waist_yaw_link
- joint zarm_l2_joint: limit lower=-0.349065850398866 upper=2.0943951023932 effort=50.0 velocity=19.154 -> lower=-0.349065850398866 upper=1.46 effort=50.0 velocity=19.154
- joint zarm_l3_joint: limit lower=-1.5707963267949 upper=1.5707963267949 effort=39.0 velocity=18.84 -> lower=-1.5707963267949 upper=0.46 effort=39.0 velocity=18.84; origin xyz=0 0 0 rpy=0 0 0 -> xyz=0 0 -0.104 rpy=0 0 0
- joint zarm_l4_joint: origin xyz=0.0200000000000006 0 -0.283699999999996 rpy=0 0 0 -> xyz=0.02 0 -0.1797 rpy=0 0 0
- joint zarm_l5_joint: origin xyz=-0.0200000000000025 0 -0.127037274261591 rpy=0 0 0 -> xyz=-0.02 0 -0.1195 rpy=0 0 0
- joint zarm_l6_joint: origin xyz=0.000199999999999079 0 -0.106462725738415 rpy=0 0 0 -> xyz=0 0 -0.114 rpy=0 0 0
- joint zarm_l7_joint: origin xyz=0 0 -0.0210004653879916 rpy=0 0 0 -> xyz=-0.0002 0 -0.021 rpy=0 0 0
- joint zarm_r1_joint: limit lower=-3.14159265358979 upper=1.5707963267949 effort=100.0 velocity=41.3433333333333 -> lower=-2.4 upper=0.6 effort=100.0 velocity=41.3433333333333; origin xyz=-0.017499853 -0.29269999999999996 0.4245 rpy=0 0 0 -> xyz=-0.003 -0.2547 0.2831 rpy=0 0 0; parent base_link -> waist_yaw_link
- joint zarm_r2_joint: limit lower=-2.0943951023932 upper=0.349065850398866 effort=50.0 velocity=19.154 -> lower=-1.46 upper=0.349065850398866 effort=50.0 velocity=19.154
- joint zarm_r3_joint: limit lower=-1.5707963267949 upper=1.5707963267949 effort=39.0 velocity=18.84 -> lower=-0.46 upper=1.5707963267949 effort=39.0 velocity=18.84; origin xyz=0 0 0 rpy=0 0 0 -> xyz=0 0 -0.104 rpy=0 0 0
- joint zarm_r4_joint: origin xyz=0.0200000000000024 0 -0.2837 rpy=0 0 0 -> xyz=0.02 0 -0.1797 rpy=0 0 0
- joint zarm_r5_joint: origin xyz=-0.0200000000000001 0 -0.127037274261587 rpy=0 0 0 -> xyz=-0.02 0 -0.1195 rpy=0 0 0
- joint zarm_r6_joint: origin xyz=0 0 -0.106462725738415 rpy=0 0 0 -> xyz=0 0 -0.114 rpy=0 0 0
- joint zarm_r7_joint: origin xyz=0 0 -0.0209999999999999 rpy=0 0 0 -> xyz=0 0 -0.022284 rpy=0 0 0

Commit message: sync https://www.lejuhub.com/highlydynamic/kuavo-ros-control/commit/6167e30c8938f6f0287ae14819da6bcd53681b7d

File: src/kuavo_assets/models/biped_s52/urdf/drake/biped_v3_arm.urdf (robot description, URDF)
Before this commit: robot biped_s52, 18 links, 17 joints
Joints:
- joint zarm_l1_joint: limit lower=-2.4 upper=0.6 effort=100.0 velocity=41.3433333333333 -> lower=-3.14159265358979 upper=1.5707963267949 effort=100.0 velocity=41.3433333333333; origin xyz=-0.003 0.2547 0.2831 rpy=0 0 0 -> xyz=-0.003 0.1737 0.2831 rpy=0 0 0
- joint zarm_l2_joint: limit lower=-0.349065850398866 upper=1.46 effort=50.0 velocity=19.154 -> lower=-0.349065850398866 upper=2.0943951023932 effort=50.0 velocity=8.37333333333333; origin xyz=0 0 0 rpy=0 0 0 -> xyz=0 0.081 0 rpy=0 0 0
- joint zarm_l3_joint: limit lower=-1.5707963267949 upper=0.46 effort=39.0 velocity=18.84 -> lower=-1.5707963267949 upper=1.5707963267949 effort=36.0 velocity=9.94333333333333
- joint zarm_l4_joint: limit lower=-2.61799387799149 upper=0.0 effort=50.0 velocity=18.84 -> lower=-2.61799387799149 upper=0.0 effort=50.0 velocity=8.37333333333333
- joint zarm_l5_joint: limit lower=-1.5707963267949 upper=1.5707963267949 effort=12.0 velocity=21.666 -> lower=-1.5707963267949 upper=1.5707963267949 effort=12.0 velocity=7.32666666666667
- joint zarm_l6_joint: limit lower=-1.30899693899575 upper=0.698131700797732 effort=12.0 velocity=21.666 -> lower=-1.30899693899575 upper=0.698131700797732 effort=12.0 velocity=7.32666666666667
- joint zarm_l7_joint: limit lower=-0.698131700797732 upper=0.698131700797732 effort=12.0 velocity=21.666 -> lower=-0.698131700797732 upper=0.698131700797732 effort=12.0 velocity=7.32666666666667
- joint zarm_r1_joint: limit lower=-2.4 upper=0.6 effort=100.0 velocity=41.3433333333333 -> lower=-3.14159265358979 upper=1.5707963267949 effort=100.0 velocity=41.3433333333333; origin xyz=-0.003 -0.2547 0.2831 rpy=0 0 0 -> xyz=-0.003 -0.1737 0.2831 rpy=0 0 0
- joint zarm_r2_joint: limit lower=-1.46 upper=0.349065850398866 effort=50.0 velocity=19.154 -> lower=-2.0943951023932 upper=0.349065850398866 effort=50.0 velocity=8.37333333333333; origin xyz=0 0 0 rpy=0 0 0 -> xyz=0 -0.081 0 rpy=0 0 0
- joint zarm_r3_joint: limit lower=-0.46 upper=1.5707963267949 effort=39.0 velocity=18.84 -> lower=-1.5707963267949 upper=1.5707963267949 effort=36.0 velocity=9.94333333333333
- joint zarm_r4_joint: limit lower=-2.61799387799149 upper=0.0 effort=50.0 velocity=18.84 -> lower=-2.61799387799149 upper=0.0 effort=50.0 velocity=8.37333333333333
- joint zarm_r5_joint: limit lower=-1.5707963267949 upper=1.5707963267949 effort=12.0 velocity=21.666 -> lower=-1.5707963267949 upper=1.5707963267949 effort=12.0 velocity=7.32666666666667
- joint zarm_r6_joint: limit lower=-0.698131700797732 upper=1.30899693899575 effort=12.0 velocity=21.666 -> lower=-0.698131700797732 upper=1.30899693899575 effort=12.0 velocity=7.32666666666667
- joint zarm_r7_joint: limit lower=-0.698131700797732 upper=0.698131700797732 effort=12.0 velocity=21.666 -> lower=-0.698131700797732 upper=0.698131700797732 effort=12.0 velocity=7.32666666666667
