Commit message: sync https://www.lejuhub.com/highlydynamic/kuavo-ros-control/commit/cb2c4a41fb965bdb2379ccd1a0d34a307da00ee8

File: src/kuavo_assets/models/biped_s52/urdf/drake/biped_v3_arm.urdf (robot description, URDF)
Before this commit: robot biped_s52, 20 links, 19 joints
Links:
- added link zarm_r7_virtual_thumb_link; collision sphere radius=0.005
Joints:
- added joint zarm_r7_virtual_thumb_joint_ee: type fixed, parent zarm_r7_end_effector, child zarm_r7_virtual_thumb_link, origin xyz=0.15 0 0 rpy=0 0 0
