Commit message: sync https://www.lejuhub.com/highlydynamic/kuavo-ros-control/commit/ac970558bd7270ea5cd45652e86b41193692604a

File: src/kuavo_assets/models/biped_s14/urdf/drake/biped_v3_arm.urdf (robot description, URDF)
Before this commit: robot biped_v3_arm, 10 links, 9 joints
Links:
- added link zarm_l7_end_effector; collision sphere radius=0.005
- added link zarm_r7_end_effector; collision sphere radius=0.005
Joints:
- added joint zarm_l7_end_effector_joint: type fixed, parent zarm_l4_link, child zarm_l7_end_effector, origin xyz=0 -0.03 -0.17 rpy=0 0 0
- added joint zarm_r7_end_effector_joint: type fixed, parent zarm_r4_link, child zarm_r7_end_effector, origin xyz=0 0.03 -0.17 rpy=0 0 0
