Commit message: sync https://www.lejuhub.com/highlydynamic/kuavo-ros-control/commit/221df4f296ba380ccfca1b788ea5a4b9019aecfe

File: src/kuavo_assets/models/biped_s14/urdf/drake/biped_v3.urdf (robot description, URDF)
Before this commit: robot biped_v3, 14 links, 13 joints
Links:
- link torso: mass 13.500276 -> 12.097476

File: src/kuavo_assets/models/biped_s14/urdf/drake/biped_v3_all_joint.urdf (robot description, URDF)
Before this commit: robot biped_v3_all_joint, 30 links, 25 joints
Links:
- link torso: mass 8.29741242 -> 6.89461242

File: src/kuavo_assets/models/biped_s14/urdf/drake/biped_v3_full.urdf (robot description, URDF)
Before this commit: robot biped_v3_full, 22 links, 21 joints
Links:
- link torso: mass 10.787876 -> 9.385076

File: src/kuavo_assets/models/biped_s52/urdf/biped_s52.urdf (robot description, URDF)
Before this commit: robot biped_s52, 48 links, 47 joints
Joints:
- joint leg_l6_joint: limit lower=-0.261799387799149 upper=0.261799387799149 effort=30.0 velocity=17.8 -> lower=-0.261799387799149 upper=0.261799387799149 effort=68.4 velocity=17.8
- joint leg_r6_joint: limit lower=-0.261799387799149 upper=0.261799387799149 effort=30.0 velocity=17.8 -> lower=-0.261799387799149 upper=0.261799387799149 effort=68.4 velocity=17.8

File: src/kuavo_assets/models/biped_s52/urdf/biped_s52_gazebo.urdf (robot description, URDF)
Before this commit: robot biped_s52, 48 links, 47 joints
Joints:
- joint leg_l6_joint: limit lower=-0.261799387799149 upper=0.261799387799149 effort=30.0 velocity=17.8 -> lower=-0.261799387799149 upper=0.261799387799149 effort=68.4 velocity=17.8
- joint leg_r6_joint: limit lower=-0.261799387799149 upper=0.261799387799149 effort=30.0 velocity=17.8 -> lower=-0.261799387799149 upper=0.261799387799149 effort=68.4 velocity=17.8

File: src/kuavo_assets/models/biped_s53/urdf/biped_s53.urdf (robot description, URDF)
Before this commit: robot biped_s53, 48 links, 47 joints
Joints:
- joint leg_l6_joint: limit lower=-0.261799387799149 upper=0.261799387799149 effort=30.0 velocity=17.8 -> lower=-0.261799387799149 upper=0.261799387799149 effort=68.4 velocity=17.8
- joint leg_r6_joint: limit lower=-0.261799387799149 upper=0.261799387799149 effort=30.0 velocity=17.8 -> lower=-0.261799387799149 upper=0.261799387799149 effort=68.4 velocity=17.8

File: src/kuavo_assets/models/biped_s53/urdf/biped_s53_gazebo.urdf (robot description, URDF)
Before this commit: robot biped_s53, 48 links, 47 joints
Joints:
- joint leg_l6_joint: limit lower=-0.261799387799149 upper=0.261799387799149 effort=30.0 velocity=17.8 -> lower=-0.261799387799149 upper=0.261799387799149 effort=68.4 velocity=17.8
- joint leg_r6_joint: limit lower=-0.261799387799149 upper=0.261799387799149 effort=30.0 velocity=17.8 -> lower=-0.261799387799149 upper=0.261799387799149 effort=68.4 velocity=17.8

File: src/kuavo_assets/models/biped_s54/urdf/biped_s54.urdf (robot description, URDF)
Before this commit: robot biped_s54, 48 links, 47 joints
Joints:
- joint leg_l6_joint: limit lower=-0.261799387799149 upper=0.261799387799149 effort=30.0 velocity=17.8 -> lower=-0.261799387799149 upper=0.261799387799149 effort=68.4 velocity=17.8
- joint leg_r6_joint: limit lower=-0.261799387799149 upper=0.261799387799149 effort=30.0 velocity=17.8 -> lower=-0.261799387799149 upper=0.261799387799149 effort=68.4 velocity=17.8

File: src/kuavo_assets/models/biped_s54/urdf/biped_s54_gazebo.urdf (robot description, URDF)
Before this commit: robot biped_s54, 48 links, 47 joints
Joints:
- joint leg_l6_joint: limit lower=-0.261799387799149 upper=0.261799387799149 effort=30.0 velocity=17.8 -> lower=-0.261799387799149 upper=0.261799387799149 effort=68.4 velocity=17.8
- joint leg_r6_joint: limit lower=-0.261799387799149 upper=0.261799387799149 effort=30.0 velocity=17.8 -> lower=-0.261799387799149 upper=0.261799387799149 effort=68.4 velocity=17.8
