Commit message: sync https://www.lejuhub.com/highlydynamic/kuavo-ros-control/commit/257f037af1d14992c8da04362176e6d05ea47d04

File: src/kuavo_assets/models/biped_s16/urdf/biped_s16.urdf (robot description, URDF)
Before this commit: robot biped_s16, 41 links, 40 joints
Links:
- link camera: mass 0.151390657704653 -> 0.000011119
- link camera_base: mass 3.92699081698722E-05 -> 0.00003927
- link zarm_l4_link: mass 0.16269441 -> 0.56269441
- link zarm_r4_link: mass 0.16269441 -> 0.56269441
- link zhead_1_link: mass 0.328285020254512 -> 1.03077542
- link zhead_2_link: mass 0.330948706392445 -> 0.33654975
Joints:
- joint dummy_to_base_link: type floating -> fixed

File: src/kuavo_assets/models/biped_s16/urdf/biped_s16_gazebo.urdf (robot description, URDF)
Before this commit: robot biped_s16, 41 links, 40 joints
Links:
- link zarm_l4_link: mass 0.16269441 -> 0.56269441
- link zarm_r4_link: mass 0.16269441 -> 0.56269441

File: src/kuavo_assets/models/biped_s16/urdf/drake/biped_v3.urdf (robot description, URDF)
Before this commit: robot biped_v3, 14 links, 13 joints
Links:
- link torso: mass 12.700276 -> 13.500276

File: src/kuavo_assets/models/biped_s16/urdf/drake/biped_v3_all_joint.urdf (robot description, URDF)
Before this commit: robot biped_v3_all_joint, 30 links, 25 joints
Links:
- link torso: mass 7.49741242 -> 8.29741242

File: src/kuavo_assets/models/biped_s16/urdf/drake/biped_v3_full.urdf (robot description, URDF)
Before this commit: robot biped_v3_full, 22 links, 21 joints
Links:
- link torso: mass 9.987876 -> 10.787876

File: src/kuavo_assets/models/biped_s52/urdf/drake/biped_v3_arm.urdf (robot description, URDF)
Before this commit: robot biped_s52, 18 links, 17 joints
Links:
- added link zarm_l7_virtual_thumb_link; collision sphere radius=0.005
- added link zarm_r7_virtual_thumb_link; collision sphere radius=0.005
Joints:
- added joint zarm_l7_virtual_thumb_joint_ee: type fixed, parent zarm_l7_end_effector, child zarm_l7_virtual_thumb_link, origin xyz=0.15 0 0 rpy=0 0 0
- added joint zarm_r7_virtual_thumb_joint_ee: type fixed, parent zarm_r7_end_effector, child zarm_r7_virtual_thumb_link, origin xyz=0.15 0 0 rpy=0 0 0
