Commit message: sync https://www.lejuhub.com/highlydynamic/kuavo-ros-control/commit/7488a27a16517dc3bd23901d85c4fc8988546303

File: src/kuavo_assets/models/biped_s53/urdf/biped_s53_gazebo.urdf (robot description, URDF)
Before this commit: robot biped_s53, 48 links, 47 joints
Links:
- link waist_yaw_link: mass 20.63616 -> 21.63516

File: src/kuavo_assets/models/biped_s53/urdf/drake/biped_v3.urdf (robot description, URDF)
Before this commit: robot biped_v3, 14 links, 13 joints
Links:
- link waist_yaw_link: mass 33.54346 -> 34.54246

File: src/kuavo_assets/models/biped_s53/urdf/drake/biped_v3_all_joint.urdf (robot description, URDF)
Before this commit: robot biped_v3_all_joint, 35 links, 30 joints
Links:
- link torso: mass 38.42194316 -> 39.42094316

File: src/kuavo_assets/models/biped_s53/urdf/drake/biped_v3_full.urdf (robot description, URDF)
Before this commit: robot biped_s53, 32 links, 31 joints
Links:
- link waist_yaw_link: mass 22.55935568 -> 23.55835568
