Commit message: sync https://www.lejuhub.com/highlydynamic/kuavo-ros-control/commit/6cbf3cecbab821ddfb6e6c2b68b835e3f7d079f8

File: src/kuavo_assets/models/biped_s53/urdf/drake/biped_v3.urdf (robot description, URDF)
Before this commit: robot biped_v3, 14 links, 13 joints
Links:
- link leg_l1_link: mass 1.63858534 -> 1.55641
- link leg_l2_link: mass 0.70575545 -> 0.75873
- link leg_l3_link: mass 5.93791258 -> 6.68074
- link leg_l4_link: mass 4.02498548 -> 3.64666
- link leg_l5_link: mass 0.07848005 -> 0.07848
- link leg_l6_link: mass 0.58491513 -> 0.69242
- link leg_r1_link: mass 1.63861324 -> 1.55641
- link leg_r2_link: mass 0.70575545 -> 0.75873
- link leg_r3_link: mass 5.93791831 -> 6.68074
- link leg_r4_link: mass 4.02498548 -> 3.64666
- link leg_r5_link: mass 0.07848005 -> 0.07848
- link leg_r6_link: mass 0.58491513 -> 0.69242
- link torso: mass 18.99013928 -> 7.06405; geometry visual mesh filename=../../meshes/torso.STL
- link waist_yaw_link: mass 18.01415568 -> 34.54246
Joints:
- joint leg_l1_joint: limit lower=-0.314159265358979 upper=0.663225115757845 effort=180.0 velocity=23.55 -> lower=-0.314159265358979 upper=0.663225115757845 effort=127.0 velocity=10.4
- joint leg_l2_joint: limit lower=-1.91986217719376 upper=0.785398163397448 effort=100.0 velocity=41.3433333333333 -> lower=-0.785398163397448 upper=1.91986217719376 effort=71.0 velocity=8.7
- joint leg_l3_joint: limit lower=-1.91986217719376 upper=1.5707963267949 effort=100.0 velocity=41.3433333333333 -> lower=-1.91986217719376 upper=1.5707963267949 effort=132 velocity=12.7
- joint leg_l4_joint: limit lower=0.0 upper=2.53072741539178 effort=180.0 velocity=23.55 -> lower=0.0 upper=2.53072741539178 effort=280.0 velocity=10.4; origin xyz=0 0 -0.284 rpy=0 0 0 -> xyz=-0.0011639 0 -0.284 rpy=0 0 0
- joint leg_l5_joint: limit lower=-0.872664625997165 upper=0.349065850398866 effort=36.0 velocity=23.0266666666667 -> lower=-0.872664625997165 upper=0.349065850398866 effort=91.6 velocity=17.8; origin xyz=0.002 0.0003 -0.416 rpy=0 0 0 -> xyz=0.002 0 -0.416 rpy=0 0 0
- joint leg_l6_joint: limit lower=-0.261799387799149 upper=0.261799387799149 effort=36.0 velocity=23.0266666666667 -> lower=-0.261799387799149 upper=0.261799387799149 effort=30.0 velocity=17.8
- joint leg_r1_joint: limit lower=-0.663225115757845 upper=0.314159265358979 effort=180.0 velocity=23.55 -> lower=-0.663225115757845 upper=0.314159265358979 effort=127.0 velocity=10.4
- joint leg_r2_joint: limit lower=-0.785398163397448 upper=1.91986217719376 effort=100.0 velocity=41.3433333333333 -> lower=-1.91986217719376 upper=0.785398163397448 effort=71.0 velocity=8.7
- joint leg_r3_joint: limit lower=-1.91986217719376 upper=1.5707963267949 effort=100.0 velocity=41.3433333333333 -> lower=-1.91986217719376 upper=1.5707963267949 effort=132.0 velocity=12.7
- joint leg_r4_joint: limit lower=0.0 upper=2.53072741539178 effort=180.0 velocity=23.55 -> lower=0.0 upper=2.53072741539178 effort=280.0 velocity=10.4; origin xyz=0 0 -0.284 rpy=0 0 0 -> xyz=-0.0011639 0 -0.284 rpy=0 0 0
- joint leg_r5_joint: limit lower=-0.872664625997165 upper=0.349065850398866 effort=36.0 velocity=23.0266666666667 -> lower=-0.872664625997165 upper=0.349065850398866 effort=91.6 velocity=17.8; origin xyz=0.00199999999983541 -0.000300000028212572 -0.415999999987417 rpy=0 0 0 -> xyz=0.002 0 -0.416 rpy=0 0 0
- joint leg_r6_joint: limit lower=-0.261799387799149 upper=0.261799387799149 effort=36.0 velocity=23.0266666666667 -> lower=-0.261799387799149 upper=0.261799387799149 effort=30.0 velocity=17.8
- joint waist_yaw_joint: limit lower=-2.0943951023932 upper=2.0943951023932 effort=180.0 velocity=23.55 -> lower=-3.14159 upper=3.14159 effort=102.0 velocity=8.7

File: src/kuavo_assets/models/biped_s53/urdf/drake/biped_v3_all_joint.urdf (robot description, URDF)
Before this commit: robot biped_v3_all_joint, 35 links, 30 joints
Links:
- link torso: mass 33.93314316 -> 39.42094316

File: src/kuavo_assets/models/biped_s53/urdf/drake/biped_v3_arm.urdf (robot description, URDF)
Before this commit: robot biped_s53, 18 links, 17 joints
Links:
- added link zarm_l7_virtual_thumb_link; collision sphere radius=0.005
- added link zarm_r7_virtual_thumb_link; collision sphere radius=0.005
- link base_link: mass 6.48663928 -> 7.06405; geometry visual mesh filename=../../meshes/torso.STL
- link waist_yaw_link: mass 18.01415568 -> 20.63616
- link zarm_l1_link: mass 0.91653322 -> 0.94521
- link zarm_l2_link: mass 0.3876739 -> 0.41921
- link zarm_l3_link: mass 1.77926875 -> 1.78857
- link zarm_l4_link: mass 0.58507821 -> 0.63149
- link zarm_l5_link: mass 0.68679955 -> 0.60828
- link zarm_l6_link: mass 0.39387181 -> 0.50616
- link zarm_l7_end_effector: geometry 
- link zarm_l7_link: mass 0.61537779 -> 0.7374; geometry visual mesh filename=../../meshes/l_hand_pitch_nohand.STL
- link zarm_r1_link: mass 0.92062797 -> 0.92947
- link zarm_r2_link: mass 0.38768053 -> 0.41523
- link zarm_r3_link: mass 1.77969208 -> 1.78473
- link zarm_r4_link: mass 0.58514611 -> 0.63548
- link zarm_r5_link: mass 0.68473867 -> 0.61021
- link zarm_r6_link: mass 0.39247462 -> 0.53821
- link zarm_r7_end_effector: geometry 
- link zarm_r7_link: mass 0.61562202 -> 0.7374; geometry visual mesh filename=../../meshes/r_hand_pitch_nohand.STL
Joints:
- added joint zarm_l7_virtual_thumb_joint_ee: type fixed, parent zarm_l7_end_effector, child zarm_l7_virtual_thumb_link, origin xyz=0.15 0 0 rpy=0 0 0
- added joint zarm_r7_virtual_thumb_joint_ee: type fixed, parent zarm_r7_end_effector, child zarm_r7_virtual_thumb_link, origin xyz=0.15 0 0 rpy=0 0 0
- joint waist_yaw_joint: limit lower=-3.14159 upper=3.14159 effort=180.0 velocity=23.55 -> lower=-3.14159 upper=3.14159 effort=102.0 velocity=8.7
- joint zarm_l1_joint: limit lower=-2.4 upper=0.6 effort=100.0 velocity=41.3433333333333 -> lower=-3.14159265358979 upper=1.5707963267949 effort=66.0 velocity=18.8; origin xyz=-0.003 0.2547 0.2831 rpy=0 0 0 -> xyz=-0.003 0.2527 0.283 rpy=0 0 0
- joint zarm_l2_joint: limit lower=-0.349065850398866 upper=1.46 effort=50.0 velocity=19.154 -> lower=-0.349065850398866 upper=3.49065850398866 effort=75.0 velocity=8.0
- joint zarm_l3_joint: limit lower=-1.5707963267949 upper=0.46 effort=39.0 velocity=18.84 -> lower=-1.48352986419518 upper=1.48352986419518 effort=57.0 velocity=7.5; origin xyz=0 0 -0.104 rpy=0 0 0 -> xyz=0 0 0 rpy=0 0 0
- joint zarm_l4_joint: limit lower=-2.61799387799149 upper=0.0 effort=50.0 velocity=18.84 -> lower=-2.61799387799149 upper=0.0 effort=75.0 velocity=8.0; origin xyz=0.02 0 -0.1797 rpy=0 0 0 -> xyz=0.02 0 -0.2837 rpy=0 0 0
- joint zarm_l5_joint: limit lower=-1.5707963267949 upper=1.5707963267949 effort=12.0 velocity=21.666 -> lower=-1.5707963267949 upper=1.5707963267949 effort=14.1 velocity=17.5; origin xyz=-0.02 0 -0.1195 rpy=0 0 0 -> xyz=-0.02 0 -0.1201 rpy=0 0 0
- joint zarm_l6_joint: limit lower=-1.30899693899575 upper=0.698131700797732 effort=12.0 velocity=21.666 -> lower=-1.30899693899575 upper=0.698131700797732 effort=14.1 velocity=17.5; origin xyz=0 0 -0.114 rpy=0 0 0 -> xyz=0.0 0 -0.114 rpy=0 0 0
- joint zarm_l7_end_effector_joint: origin xyz=0 -0.03 -0.17 rpy=0 0 0 -> xyz=0 0.0 -0.17 rpy=0 0 0
- joint zarm_l7_joint: limit lower=-0.698131700797732 upper=0.698131700797732 effort=12.0 velocity=21.666 -> lower=-0.698131700797732 upper=0.698131700797732 effort=14.1 velocity=17.5; origin xyz=-0.0002 0 -0.021 rpy=0 0 0 -> xyz=0 0 -0.021 rpy=0 0 0
- joint zarm_r1_joint: limit lower=-2.4 upper=0.6 effort=100.0 velocity=41.3433333333333 -> lower=-3.14159265358979 upper=1.5707963267949 effort=66.0 velocity=18.8; origin xyz=-0.003 -0.2547 0.2831 rpy=0 0 0 -> xyz=-0.003 -0.2527 0.283 rpy=0 0 0
- joint zarm_r2_joint: limit lower=-1.46 upper=0.349065850398866 effort=50.0 velocity=19.154 -> lower=-3.49065850398866 upper=0.349065850398866 effort=75.0 velocity=8.0
- joint zarm_r3_joint: limit lower=-0.46 upper=1.5707963267949 effort=39.0 velocity=18.84 -> lower=-1.48352986419518 upper=1.48352986419518 effort=57.0 velocity=7.5; origin xyz=0 0 -0.104 rpy=0 0 0 -> xyz=0 0 0 rpy=0 0 0
- joint zarm_r4_joint: limit lower=-2.61799387799149 upper=0.0 effort=50.0 velocity=18.84 -> lower=-2.61799387799149 upper=0.0 effort=75.0 velocity=8.0; origin xyz=0.02 0 -0.1797 rpy=0 0 0 -> xyz=0.02 0 -0.2837 rpy=0 0 0
- joint zarm_r5_joint: limit lower=-1.5707963267949 upper=1.5707963267949 effort=12.0 velocity=21.666 -> lower=-1.5707963267949 upper=1.5707963267949 effort=14.1 velocity=17.5; origin xyz=-0.02 0 -0.1195 rpy=0 0 0 -> xyz=-0.02 0 -0.1201 rpy=0 0 0
- joint zarm_r6_joint: limit lower=-0.698131700797732 upper=1.30899693899575 effort=12.0 velocity=21.666 -> lower=-0.698131700797732 upper=1.30899693899575 effort=14.1 velocity=17.5; origin xyz=0 0 -0.114 rpy=0 0 0 -> xyz=0.0 0 -0.114 rpy=0 0 0
- joint zarm_r7_end_effector_joint: origin xyz=0 0.03 -0.17 rpy=0 0 0 -> xyz=0 0.0 -0.17 rpy=0 0 0
- joint zarm_r7_joint: limit lower=-0.698131700797732 upper=0.698131700797732 effort=12.0 velocity=21.666 -> lower=-0.698131700797732 upper=0.698131700797732 effort=14.1 velocity=17.5; origin xyz=0 0 -0.022284 rpy=0 0 0 -> xyz=0.0 0 -0.021 rpy=0 0 0

File: src/kuavo_assets/models/biped_s53/urdf/drake/biped_v3_full.urdf (robot description, URDF)
Before this commit: robot biped_v3_full, 28 links, 27 joints
Links:
- removed link torso
- added link base_link, mass 6.48663928; visual mesh filename=../../meshes/base_link.STL
- added link dummy_link
- added link head_camera, mass 0.0400617267216207; visual mesh filename=../../meshes/head_camera.STL
- added link zhead_1_link, mass 0.87117795; visual mesh filename=../../meshes/head_yaw.STL
- added link zhead_2_link, mass 0.80529305; visual mesh filename=../../meshes/head_pitch.STL
- link leg_l1_link: mass 1.71093115 -> 1.63858534
- link leg_l2_link: mass 0.58029165 -> 0.70575545
- link leg_l3_link: mass 4.50393141 -> 5.93791258
- link leg_l4_link: mass 1.62776815 -> 4.02498548
- link leg_l5_link: mass 0.07193524 -> 0.07848005
- link leg_l6_link: mass 0.49861272 -> 0.58491513
- link leg_r1_link: mass 1.71093008 -> 1.63861324
- link leg_r2_link: mass 0.58029165 -> 0.70575545
- link leg_r3_link: mass 4.50385993 -> 5.93791831
- link leg_r4_link: mass 1.62655699 -> 4.02498548
- link leg_r5_link: mass 0.07193524 -> 0.07848005
- link leg_r6_link: mass 0.49861272 -> 0.58491513
- link waist_yaw_link: mass 15.18745152 -> 23.55835568
- link zarm_l1_link: mass 0.962 -> 0.91653322
- link zarm_l2_link: mass 0.57 -> 0.3876739
- link zarm_l3_link: mass 1.65 -> 1.77926875
- link zarm_l4_link: mass 0.429 -> 0.58507821
- link zarm_l5_link: mass 0.61 -> 0.68679955
- link zarm_l6_link: mass 0.331 -> 0.39387181
- link zarm_l7_link: mass 0.64 -> 0.61537779
- link zarm_r1_link: mass 0.962 -> 0.92062797
- link zarm_r2_link: mass 0.57 -> 0.38768053
- link zarm_r3_link: mass 1.65 -> 1.77969208
- link zarm_r4_link: mass 0.429 -> 0.58514611
- link zarm_r5_link: mass 0.61 -> 0.68473867
- link zarm_r6_link: mass 0.331 -> 0.39247462
- link zarm_r7_link: mass 0.64 -> 0.61562202
Joints:
- added joint dummy_to_base_link: type fixed, parent dummy_link, child base_link, origin xyz=0 0 0 rpy=0 0 0
- added joint head_camera: type fixed, parent zhead_2_link, child head_camera, origin xyz=0.119717018973535 0.0237514612535074 0.0262044145991832 rpy=0 0.480224871300295 0
- added joint zhead_1_joint: type revolute, parent waist_yaw_link, child zhead_1_link, origin xyz=-0.003 0.0 0.3715 rpy=0 0 0, axis 0 0 1, limit lower=-1.5707963267949 upper=1.5707963267949 effort=1.5 velocity=5.23
- added joint zhead_2_joint: type revolute, parent zhead_1_link, child zhead_2_link, origin xyz=0 0 0.137954074182872 rpy=0 0 0, axis 0 1 0, limit lower=-0.349065850398866 upper=0.785398163397448 effort=12.0 velocity=5.23
- joint leg_l1_joint: origin xyz=-0.0024999 0.087 -0.066 rpy=0 0 0 -> xyz=0.0 0.095075 -0.066 rpy=0 0 0; parent torso -> base_link
- joint leg_l3_joint: origin xyz=0.000500354536093913 -0.00100000000000011 -0.1287 rpy=0 0 0 -> xyz=0 0 -0.1437 rpy=0 0 0
- joint leg_l4_joint: origin xyz=-6.87185435835039E-05 0 -0.284 rpy=0 0 0 -> xyz=0 0 -0.284 rpy=0 0 0
- joint leg_l5_joint: origin xyz=-0.000431635992531742 0 -0.346000000000001 rpy=0 0 0 -> xyz=0.002 0.0003 -0.416 rpy=0 0 0
- joint leg_r1_joint: origin xyz=-0.0024999 -0.087 -0.066 rpy=0 0 0 -> xyz=0.0 -0.095075 -0.066 rpy=0 0 0; parent torso -> base_link
- joint leg_r3_joint: origin xyz=-4.88006581312577E-05 0 -0.1287 rpy=0 0 0 -> xyz=0 0 -0.1437 rpy=0 0 0
- joint leg_r4_joint: origin xyz=0.000147138572785148 0 -0.283999982974744 rpy=0 0 0 -> xyz=0 0 -0.284 rpy=0 0 0
- joint leg_r5_joint: origin xyz=0.000119806050928577 0 -0.345999979257963 rpy=0 0 0 -> xyz=0.00199999999983541 -0.000300000028212572 -0.415999999987417 rpy=0 0 0
- joint waist_yaw_joint: limit lower=-0.314159265358979 upper=0.663225115757845 effort=180.0 velocity=23.55 -> lower=-3.14159 upper=3.14159 effort=180.0 velocity=23.55; origin xyz=0 0 0.107 rpy=0 0 0 -> xyz=0 0 0.1114 rpy=0 0 0; parent biped_s50 -> base_link; type fixed -> revolute
- joint zarm_l1_joint: origin xyz=0.003 0.28569999999999995 0.2055 rpy=0 0 0 -> xyz=-0.003 0.1737 0.2831 rpy=0 0 0
- joint zarm_l2_joint: limit lower=-0.349065850398866 upper=2.0943951023932 effort=50.0 velocity=19.154 -> lower=-0.349065850398866 upper=2.0943951023932 effort=50.0 velocity=8.37333333333333; origin xyz=0 0 0 rpy=0 0 0 -> xyz=0 0.081 0 rpy=0 0 0
- joint zarm_l3_joint: limit lower=-1.5707963267949 upper=1.5707963267949 effort=39.0 velocity=18.84 -> lower=-1.5707963267949 upper=1.5707963267949 effort=36.0 velocity=9.94333333333333; origin xyz=0 0 0 rpy=0 0 0 -> xyz=0 0 -0.104 rpy=0 0 0
- joint zarm_l4_joint: limit lower=-2.61799387799149 upper=0.0 effort=50.0 velocity=18.84 -> lower=-2.61799387799149 upper=0.0 effort=50.0 velocity=8.37333333333333; origin xyz=0.0200000000000006 0 -0.283699999999996 rpy=0 0 0 -> xyz=0.02 0 -0.1797 rpy=0 0 0
- joint zarm_l5_joint: limit lower=-1.5707963267949 upper=1.5707963267949 effort=12.0 velocity=21.666 -> lower=-1.5707963267949 upper=1.5707963267949 effort=12.0 velocity=7.32666666666667; origin xyz=-0.0200000000000025 0 -0.127037274261591 rpy=0 0 0 -> xyz=-0.02 0 -0.1195 rpy=0 0 0
- joint zarm_l6_joint: limit lower=-1.30899693899575 upper=0.698131700797732 effort=12.0 velocity=21.666 -> lower=-1.30899693899575 upper=0.698131700797732 effort=12.0 velocity=7.32666666666667; origin xyz=0.000199999999999079 0 -0.106462725738415 rpy=0 0 0 -> xyz=0 0 -0.114 rpy=0 0 0
- joint zarm_l7_joint: limit lower=-0.698131700797732 upper=0.698131700797732 effort=12.0 velocity=21.666 -> lower=-0.698131700797732 upper=0.698131700797732 effort=12.0 velocity=7.32666666666667; origin xyz=0 0 -0.0210004653879916 rpy=0 0 0 -> xyz=-0.0002 0 -0.021 rpy=0 0 0
- joint zarm_r1_joint: origin xyz=0.003 -0.28569999999999995 0.2055 rpy=0 0 0 -> xyz=-0.003 -0.1737 0.2831 rpy=0 0 0
- joint zarm_r2_joint: limit lower=-2.0943951023932 upper=0.349065850398866 effort=50.0 velocity=19.154 -> lower=-2.0943951023932 upper=0.349065850398866 effort=50.0 velocity=8.37333333333333; origin xyz=0 0 0 rpy=0 0 0 -> xyz=0 -0.081 0 rpy=0 0 0
- joint zarm_r3_joint: limit lower=-1.5707963267949 upper=1.5707963267949 effort=39.0 velocity=18.84 -> lower=-1.5707963267949 upper=1.5707963267949 effort=36.0 velocity=9.94333333333333; origin xyz=0 0 0 rpy=0 0 0 -> xyz=0 0 -0.104 rpy=0 0 0
- joint zarm_r4_joint: limit lower=-2.61799387799149 upper=0.0 effort=50.0 velocity=18.84 -> lower=-2.61799387799149 upper=0.0 effort=50.0 velocity=8.37333333333333; origin xyz=0.0200000000000024 0 -0.2837 rpy=0 0 0 -> xyz=0.02 0 -0.1797 rpy=0 0 0
- joint zarm_r5_joint: limit lower=-1.5707963267949 upper=1.5707963267949 effort=12.0 velocity=21.666 -> lower=-1.5707963267949 upper=1.5707963267949 effort=12.0 velocity=7.32666666666667; origin xyz=-0.0200000000000001 0 -0.127037274261587 rpy=0 0 0 -> xyz=-0.02 0 -0.1195 rpy=0 0 0
- joint zarm_r6_joint: limit lower=-0.698131700797732 upper=1.30899693899575 effort=12.0 velocity=21.666 -> lower=-0.698131700797732 upper=1.30899693899575 effort=12.0 velocity=7.32666666666667; origin xyz=0 0 -0.106462725738415 rpy=0 0 0 -> xyz=0 0 -0.114 rpy=0 0 0
- joint zarm_r7_joint: limit lower=-0.698131700797732 upper=0.698131700797732 effort=12.0 velocity=21.666 -> lower=-0.698131700797732 upper=0.698131700797732 effort=12.0 velocity=7.32666666666667; origin xyz=0 0 -0.0209999999999999 rpy=0 0 0 -> xyz=0 0 -0.022284 rpy=0 0 0

File: src/kuavo_assets/models/biped_s54/urdf/drake/biped_v3.urdf (robot description, URDF)
Before this commit: robot biped_v3, 14 links, 13 joints
Links:
- link waist_yaw_link: mass 33.70038 -> 33.70028

Commit message: sync https://www.lejuhub.com/highlydynamic/kuavo-ros-control/commit/861af0abeafd1c22183ad570be314f8fd6e3dffa

File: src/kuavo_assets/models/biped_s53/urdf/biped_s53.urdf (robot description, URDF)
Before this commit: robot biped_s53, 51 links, 50 joints
Links:
- link waist_yaw_link: mass 19.98201 -> 19.98191
Joints:
- joint dummy_to_base_link: type floating -> fixed

File: src/kuavo_assets/models/biped_s53/urdf/biped_s53_gazebo.urdf (robot description, URDF)
Before this commit: robot biped_s53, 51 links, 50 joints
Links:
- link waist_yaw_link: mass 21.90016 -> 21.81526

File: src/kuavo_assets/models/biped_s55/urdf/biped_s55.urdf (robot description, URDF)
Before this commit: robot biped_s55, 51 links, 50 joints
Joints:
- joint dummy_to_base_link: type floating -> fixed
