Commit message: sync https://www.lejuhub.com/highlydynamic/kuavo-ros-control/commit/a6332d61858921d58efcf6b158754dbab501a6e9

File: src/kuavo_assets/models/biped_s62/urdf/biped_s62_gazebo.urdf (robot description, URDF)
Before this commit: robot biped_s62, 39 links, 38 joints
Links:
- link waist_yaw_link: mass 120.2954 -> 11.56094002
