Commit message: sync https://www.lejuhub.com/highlydynamic/kuavo-ros-control/commit/73ea64e140a88fd76ef00b13fd9dd51bac8702df

File: src/kuavo_assets/models/biped_s62/urdf/biped_s62.urdf (robot description, URDF)
Before this commit: robot biped_s62, 36 links, 35 joints
Joints:
- joint base_to_joint: origin xyz=0.098 0 0.27064321 rpy=0 0 0 -> xyz=0.098 0 0.31 rpy=0 0 0

Commit message: sync https://www.lejuhub.com/highlydynamic/kuavo-ros-control/commit/dc11f7dbee2100ac6c16123316b322ad7cb0e598

File: src/kuavo_assets/models/biped_s62/urdf/biped_s62.urdf (robot description, URDF)
Before this commit: robot biped_s62, 36 links, 35 joints
Joints:
- removed joint floating_base
- added joint base_link_to_dummy_link: type fixed, parent base_link, child dummy_link, origin xyz=0 0 0 rpy=0 0 0
- joint base_to_joint: origin xyz=0.098 0 0.27064321 rpy=0 0 0 -> xyz=0.098 0 0.31 rpy=0 0 0

File: src/kuavo_assets/models/biped_s63/urdf/biped_s63.urdf (robot description, URDF)
Before this commit: robot biped_s63, 36 links, 35 joints
Joints:
- removed joint floating_base
- added joint base_link_to_dummy_link: type fixed, parent base_link, child dummy_link, origin xyz=0 0 0 rpy=0 0 0
- joint zhead_1_joint: origin xyz=0 0 0.43485 rpy=0 0 0 -> xyz=0 0 0.43935 rpy=0 0 0

File: src/kuavo_assets/models/biped_s63/urdf/biped_s63_gazebo.urdf (robot description, URDF)
Before this commit: robot biped_s63, 40 links, 39 joints
Joints:
- removed joint floating_base
- added joint base_link_to_dummy_link: type fixed, parent base_link, child dummy_link, origin xyz=0 0 0 rpy=0 0 0
- joint zhead_1_joint: origin xyz=0 0 0.43485 rpy=0 0 0 -> xyz=0 0 0.43935 rpy=0 0 0
