Commit message: sync https://www.lejuhub.com/highlydynamic/kuavo-ros-control/commit/26df00cc169f5f8104c28eed44b3dc14037d417c

File: src/kuavo_assets/models/biped_s17/urdf/drake/biped_v3_full.urdf (robot description, URDF)
Before this commit: robot biped_v3_full, 22 links, 21 joints
Links:
- link leg_r1_link: mass 0.42877618 -> 0.62568928
- link leg_r2_link: mass 2.4999594 -> 2.03159924
