Commit message: sync https://www.lejuhub.com/highlydynamic/kuavo-ros-control/commit/b576acf114137607e0cc4e26130252421c337b5a

File: src/kuavo_assets/models/biped_s400049/urdf/biped_s400049.urdf (robot description, URDF)
Before this commit: robot biped_s400049, 73 links, 72 joints
Links:
- removed link l_Index_prox
- removed link l_index_dist
- removed link l_little_dist
- removed link l_little_prox
- removed link l_middle_dist
- removed link l_middle_prox
- removed link l_palm
- removed link l_ring_dist
- removed link l_ring_prox
- removed link l_thumb_dist
- removed link l_thumb_prox
- removed link r_index_dist
- removed link r_index_prox
- removed link r_little_dist
- removed link r_little_prox
- removed link r_middle_dist
- removed link r_middle_prox
- removed link r_palm
- removed link r_ring_dist
- removed link r_ring_prox
- removed link r_thumb_dist
- removed link r_thumb_prox
- added link l_hand_base_link, mass 0.0672935238166485; collision mesh filename=package://kuavo_assets/models/biped_s400049/o6/left/meshes/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; visual mesh filename=package://kuavo_assets/models/biped_s400049/o6/left/meshes/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
- added link l_index_distal, mass 0.00376951085886838; collision mesh filename=package://kuavo_assets/models/biped_s400049/o6/left/meshes/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; visual mesh filename=package://kuavo_assets/models/biped_s400049/o6/left/meshes/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
- added link l_index_proximal, mass 0.00253174651934627; collision mesh filename=package://kuavo_assets/models/biped_s400049/o6/left/meshes/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; visual mesh filename=package://kuavo_assets/models/biped_s400049/o6/left/meshes/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
- added link l_middle_distal, mass 0.00376952789210256; collision mesh filename=package://kuavo_assets/models/biped_s400049/o6/left/meshes/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; visual mesh filename=package://kuavo_assets/models/biped_s400049/o6/left/meshes/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
- added link l_middle_proximal, mass 0.00253177375206983; collision mesh filename=package://kuavo_assets/models/biped_s400049/o6/left/meshes/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; visual mesh filename=package://kuavo_assets/models/biped_s400049/o6/left/meshes/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
- added link l_pinky_distal, mass 0.00376948071276134; collision mesh filename=package://kuavo_assets/models/biped_s400049/o6/left/meshes/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; visual mesh filename=package://kuavo_assets/models/biped_s400049/o6/left/meshes/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
- added link l_pinky_proximal, mass 0.00253185993162408; collision mesh filename=package://kuavo_assets/models/biped_s400049/o6/left/meshes/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; visual mesh filename=package://kuavo_assets/models/biped_s400049/o6/left/meshes/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
- added link l_ring_distal, mass 0.00376949588316609; collision mesh filename=package://kuavo_assets/models/biped_s400049/o6/left/meshes/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; visual mesh filename=package://kuavo_assets/models/biped_s400049/o6/left/meshes/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
- added link l_ring_proximal, mass 0.00253182223645066; collision mesh filename=package://kuavo_assets/models/biped_s400049/o6/left/meshes/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; visual mesh filename=package://kuavo_assets/models/biped_s400049/o6/left/meshes/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
- added link l_thumb_distal, mass 0.00763332957284057; collision mesh filename=package://kuavo_assets/models/biped_s400049/o6/left/meshes/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; visual mesh filename=package://kuavo_assets/models/biped_s400049/o6/left/meshes/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
- added link l_thumb_metacarpals, mass 0.0123381586619931; collision mesh filename=package://kuavo_assets/models/biped_s400049/o6/left/meshes/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; visual mesh filename=package://kuavo_assets/models/biped_s400049/o6/left/meshes/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
- added link l_thumb_metacarpals_base2, mass 0.00138588296544333; collision mesh filename=package://kuavo_assets/models/biped_s400049/o6/left/meshes/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; visual mesh filename=package://kuavo_assets/models/biped_s400049/o6/left/meshes/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
- added link r_hand_base_link, mass 0.06740077960995; collision mesh filename=package://kuavo_assets/models/biped_s400049/o6/right/meshes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; visual mesh filename=package://kuavo_assets/models/biped_s400049/o6/right/meshes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
- added link r_index_distal, mass 0.00376787129082313; collision mesh filename=package://kuavo_assets/models/biped_s400049/o6/right/meshes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; visual mesh filename=package://kuavo_assets/models/biped_s400049/o6/right/meshes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
- added link r_index_proximal, mass 0.00253178529301663; collision mesh filename=package://kuavo_assets/models/biped_s400049/o6/right/meshes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; visual mesh filename=package://kuavo_assets/models/biped_s400049/o6/right/meshes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
- added link r_middle_distal, mass 0.00376786259758948; collision mesh filename=package://kuavo_assets/models/biped_s400049/o6/right/meshes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; visual mesh filename=package://kuavo_assets/models/biped_s400049/o6/right/meshes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
- added link r_middle_proximal, mass 0.00253175497594429; collision mesh filename=package://kuavo_assets/models/biped_s400049/o6/right/meshes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; visual mesh filename=package://kuavo_assets/models/biped_s400049/o6/right/meshes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
- added link r_pinky_distal, mass 0.00376782669873412; collision mesh filename=package://kuavo_assets/models/biped_s400049/o6/right/meshes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; visual mesh filename=package://kuavo_assets/models/biped_s400049/o6/right/meshes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
- added link r_pinky_proximal, mass 0.00253167400540778; collision mesh filename=package://kuavo_assets/models/biped_s400049/o6/right/meshes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; visual mesh filename=package://kuavo_assets/models/biped_s400049/o6/right/meshes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
- added link r_ring_distal, mass 0.0037678395356105; collision mesh filename=package://kuavo_assets/models/biped_s400049/o6/right/meshes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; visual mesh filename=package://kuavo_assets/models/biped_s400049/o6/right/meshes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
- added link r_ring_proximal, mass 0.00253170963529411; collision mesh filename=package://kuavo_assets/models/biped_s400049/o6/right/meshes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; visual mesh filename=package://kuavo_assets/models/biped_s400049/o6/right/meshes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
- added link r_thumb_distal, mass 0.00763302603723749; collision mesh filename=package://kuavo_assets/models/biped_s400049/o6/right/meshes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; visual mesh filename=package://kuavo_assets/models/biped_s400049/o6/right/meshes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
- added link r_thumb_metacarpals, mass 0.0123381607727595; collision mesh filename=package://kuavo_assets/models/biped_s400049/o6/right/meshes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; visual mesh filename=package://kuavo_assets/models/biped_s400049/o6/right/meshes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
- added link r_thumb_metacarpals_base2, mass 0.00138591070212997; collision mesh filename=package://kuavo_assets/models/biped_s400049/o6/right/meshes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; visual mesh filename=package://kuavo_assets/models/biped_s400049/o6/right/meshes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
Joints:
- removed joint l_indexMCP
- removed joint l_indexPIP
- removed joint l_littleMCP
- removed joint l_littlePIP
- removed joint l_middleMCP
- removed joint l_middlePIP
- removed joint l_palm_fixed_joint
- removed joint l_ringMCP
- removed joint l_ringPIP
- removed joint l_thumbCMC
- removed joint l_thumbMCP
- removed joint r_indexMCP
- removed joint r_indexPIP
- removed joint r_littleMCP
- removed joint r_littlePIP
- removed joint r_middleMCP
- removed joint r_middlePIP
- removed joint r_palm_fixed_joint
- removed joint r_ringMCP
- removed joint r_ringPIP
- removed joint r_thumbCMC
- removed joint r_thumbMCP
- added joint l_index_dip: type revolute, parent l_index_proximal, child l_index_distal, origin xyz=-0.0052516 0 0.036625 rpy=0 0 0, axis 0 1 0, limit lower=0 upper=1.43 effort=100 velocity=1, mimic joint=l_index_mcp_pitch multiplier=0.89 offset=0
- added joint l_index_mcp_pitch: type revolute, parent l_hand_base_link, child l_index_proximal, origin xyz=0.0024758 -0.02419 0.103779 rpy=0.05236 0 0, axis 0 1 0, limit lower=0 upper=1.60 effort=100 velocity=1
- added joint l_middle_dip: type revolute, parent l_middle_proximal, child l_middle_distal, origin xyz=-0.0052516 0 0.036625 rpy=0 0 0, axis 0 1 0, limit lower=0 upper=1.43 effort=100 velocity=1, mimic joint=l_middle_mcp_pitch multiplier=0.89 offset=0
- added joint l_middle_mcp_pitch: type revolute, parent l_hand_base_link, child l_middle_proximal, origin xyz=0.00052576 -0.00634 0.1077 rpy=0 0 0, axis 0 1 0, limit lower=0 upper=1.60 effort=100 velocity=1
- added joint l_pinky_dip: type revolute, parent l_pinky_proximal, child l_pinky_distal, origin xyz=-0.0052516 0 0.036625 rpy=0 0 0, axis 0 1 0, limit lower=0 upper=1.43 effort=100 velocity=1, mimic joint=l_pinky_mcp_pitch multiplier=0.89 offset=0
- added joint l_pinky_mcp_pitch: type revolute, parent l_hand_base_link, child l_pinky_proximal, origin xyz=0.0024758 0.028372 0.097741 rpy=-0.087266 0 0, axis 0 1 0, limit lower=0 upper=1.60 effort=100 velocity=1
- added joint l_ring_dip: type revolute, parent l_ring_proximal, child l_ring_distal, origin xyz=-0.0052516 0 0.036625 rpy=0 0 0, axis 0 1 0, limit lower=0 upper=1.43 effort=100 velocity=1, mimic joint=l_ring_mcp_pitch multiplier=0.89 offset=0
- added joint l_ring_mcp_pitch: type revolute, parent l_hand_base_link, child l_ring_proximal, origin xyz=0.0010258 0.011135 0.103767 rpy=-0.05236 0 0, axis 0 1 0, limit lower=0 upper=1.60 effort=100 velocity=1
- added joint l_thumb_cmc_pitch: type revolute, parent l_thumb_metacarpals_base2, child l_thumb_metacarpals, origin xyz=0.0061649 -0.010678 -0.004891 rpy=0 -1.1529 2.0944, axis 0 1 0, limit lower=0 upper=0.58 effort=100 velocity=1
- added joint l_thumb_cmc_yaw: type revolute, parent l_hand_base_link, child l_thumb_metacarpals_base2, origin xyz=0.011508 -0.022975 0.037794 rpy=0 0 0, axis 0 0 1, limit lower=0 upper=1.3 effort=100 velocity=1
- added joint l_thumb_ip: type revolute, parent l_thumb_metacarpals, child l_thumb_distal, origin xyz=0.0037776 0 0.045368 rpy=0 0 0, axis 0 1 0, limit lower=0 upper=1.08 effort=100 velocity=1, mimic joint=l_thumb_cmc_pitch multiplier=2.29 offset=0
- added joint r_index_dip: type revolute, parent r_index_proximal, child r_index_distal, origin xyz=-0.0052516 0 0.036625 rpy=0 0 0, axis 0 1 0, limit lower=0 upper=1.43 effort=100 velocity=1, mimic joint=r_index_mcp_pitch multiplier=0.89 offset=0
- added joint r_index_mcp_pitch: type revolute, parent r_hand_base_link, child r_index_proximal, origin xyz=0.0024758 0.02419 0.103779 rpy=-0.05236 0 0, axis 0 1 0, limit lower=0 upper=1.60 effort=100 velocity=1
- added joint r_middle_dip: type revolute, parent r_middle_proximal, child r_middle_distal, origin xyz=-0.0052516 0 0.036625 rpy=0 0 0, axis 0 1 0, limit lower=0 upper=1.43 effort=100 velocity=1, mimic joint=r_middle_mcp_pitch multiplier=0.89 offset=0
- added joint r_middle_mcp_pitch: type revolute, parent r_hand_base_link, child r_middle_proximal, origin xyz=0.00052576 0.00634 0.1077 rpy=0 0 0, axis 0 1 0, limit lower=0 upper=1.60 effort=100 velocity=1
- added joint r_pinky_dip: type revolute, parent r_pinky_proximal, child r_pinky_distal, origin xyz=-0.0052516 0 0.036625 rpy=0 0 0, axis 0 1 0, limit lower=0 upper=1.43 effort=100 velocity=1, mimic joint=r_pinky_mcp_pitch multiplier=0.89 offset=0
- added joint r_pinky_mcp_pitch: type revolute, parent r_hand_base_link, child r_pinky_proximal, origin xyz=0.0024758 -0.028372 0.097741 rpy=0.087266 0 0, axis 0 1 0, limit lower=0 upper=1.60 effort=100 velocity=1
- added joint r_ring_dip: type revolute, parent r_ring_proximal, child r_ring_distal, origin xyz=-0.0052516 0 0.036625 rpy=0 0 0, axis 0 1 0, limit lower=0 upper=1.43 effort=100 velocity=1, mimic joint=r_ring_mcp_pitch multiplier=0.89 offset=0
- added joint r_ring_mcp_pitch: type revolute, parent r_hand_base_link, child r_ring_proximal, origin xyz=0.0010258 -0.011135 0.103767 rpy=0.05236 0 0, axis 0 1 0, limit lower=0 upper=1.60 effort=100 velocity=1
- added joint r_thumb_cmc_pitch: type revolute, parent r_thumb_metacarpals_base2, child r_thumb_metacarpals, origin xyz=0.0061649 0.010678 -0.004891 rpy=0 -1.1529 -2.0944, axis 0 1 0, limit lower=0 upper=0.58 effort=100 velocity=1
- added joint r_thumb_cmc_yaw: type revolute, parent r_hand_base_link, child r_thumb_metacarpals_base2, origin xyz=0.011508 0.022975 0.037794 rpy=0 0 0, axis 0 0 -1, limit lower=0 upper=1.36 effort=100 velocity=1
- added joint r_thumb_ip: type revolute, parent r_thumb_metacarpals, child r_thumb_distal, origin xyz=0.0037776 0 0.045368 rpy=0 0 0, axis 0 1 0, limit lower=0 upper=1.08 effort=100 velocity=1, mimic joint=r_thumb_cmc_pitch multiplier=1.86 offset=0
- added joint zarm_l7_to_l_hand_base_link: type fixed, parent zarm_l7_link, child l_hand_base_link, origin xyz=0 0 -0.05 rpy=3.14159265 0 -1.57079633
- added joint zarm_r7_to_r_hand_base_link: type fixed, parent zarm_r7_link, child r_hand_base_link, origin xyz=0 0 -0.05 rpy=3.14159265 0 1.57079633
