Commit message: sync https://www.lejuhub.com/highlydynamic/kuavo-ros-control/commit/cd4a9605096e84a3058116a70025b4b628d4ab99

File: src/kuavo_assets/models/biped_s61/urdf/biped_s61.urdf (robot description, URDF)
Before this commit: robot biped_s61, 36 links, 35 joints
Joints:
- joint floating_base: child base_link -> dummy_link; parent dummy_link -> base_link

File: src/kuavo_assets/models/biped_s61/urdf/biped_s61_gazebo.urdf (robot description, URDF)
Before this commit: robot biped_s61, 39 links, 38 joints
Joints:
- joint floating_base: child base_link -> dummy_link; parent dummy_link -> base_link

File: src/kuavo_assets/models/biped_s62/urdf/biped_s62.urdf (robot description, URDF)
Before this commit: robot biped_s62, 36 links, 35 joints
Joints:
- joint floating_base: child base_link -> dummy_link; parent dummy_link -> base_link

File: src/kuavo_assets/models/biped_s62/urdf/biped_s62_gazebo.urdf (robot description, URDF)
Before this commit: robot biped_s62, 39 links, 38 joints
Joints:
- joint floating_base: child base_link -> dummy_link; parent dummy_link -> base_link
