Commit message: sync https://www.lejuhub.com/highlydynamic/kuavo-ros-control/commit/6d2dcd681ab52f340f9e43293e9701f2ca2b1ab4

File: src/kuavo_assets/models/biped_s60/urdf/drake/biped_v3_arm.urdf (robot description, URDF)
Before this commit: robot biped_s60, 23 links, 22 joints
Joints:
- joint zarm_l4_joint: limit lower=-2.61799387799149 upper=-0.2 effort=75.0 velocity=8.0 -> lower=-2.61799387799149 upper=0.0 effort=75.0 velocity=8.0
- joint zarm_r4_joint: limit lower=-2.61799387799149 upper=-0.2 effort=75.0 velocity=8.0 -> lower=-2.61799387799149 upper=0.0 effort=75.0 velocity=8.0

File: src/kuavo_assets/models/biped_s62/urdf/drake/biped_v3_arm.urdf (robot description, URDF)
Before this commit: robot biped_s45, 17 links, 16 joints
Links:
- added link base_to_joint, mass 7.27493629; visual mesh filename=../../meshes/knee_link.STL
- added link knee_link, mass 13.41361777; visual mesh filename=../../meshes/leg_Link.STL
- added link leg_link, mass 9.78118294; visual mesh filename=../../meshes/waist_pitch_Link.STL
- added link waist_link, mass 4.65997944; visual mesh filename=../../meshes/waist_yaw_Link.STL
- added link waist_yaw_link, mass 11.56094002; collision cylinder length=0.6 radius=0.15; visual mesh filename=../../meshes/torso.STL
- added link zarm_l7_end_effector_1
- added link zarm_l7_end_effector_2
- added link zarm_l7_virtual_thumb_link; collision sphere radius=0.005
- added link zarm_r7_end_effector_1
- added link zarm_r7_end_effector_2
- added link zarm_r7_virtual_thumb_link; collision sphere radius=0.005
- link base_link: mass 11.56094002 -> 121.0; geometry collision cylinder length=0.32 radius=0.37; visual mesh filename=../../meshes/base_link.STL
Joints:
- added joint base_to_joint: type fixed, parent base_link, child base_to_joint, origin xyz=0.098 0 0.27064321 rpy=0 0 0
- added joint knee_joint: type revolute, parent base_to_joint, child knee_link, origin xyz=0 0 0.1055 rpy=0 0 0, axis 0 1 0, limit lower=0 upper=1.448 effort=668.53 velocity=25.33
- added joint leg_joint: type revolute, parent knee_link, child leg_link, origin xyz=-0.46521 0 0.18325 rpy=0 0 0, axis 0 1 0, limit lower=-2.81 upper=0.0 effort=668.53 velocity=25.33
- added joint waist_pitch_joint: type revolute, parent leg_link, child waist_link, origin xyz=0.48296 0 0.12941 rpy=0 0 0, axis 0 1 0, limit lower=0.0 upper=0.9 effort=618.48 velocity=25.33
- added joint waist_yaw_joint: type revolute, parent waist_link, child waist_yaw_link, origin xyz=0 0 0.235 rpy=0 0 0, axis 0 0 1, limit lower=-3.14159265358979 upper=3.14159265358979 effort=618.48 velocity=25.33
- added joint zarm_l7_end_effector_1_joint: type fixed, parent zarm_l7_link, child zarm_l7_end_effector_1, origin xyz=0 0.0 -0.08 rpy=0 0 0
- added joint zarm_l7_end_effector_2_joint: type fixed, parent zarm_l7_link, child zarm_l7_end_effector_2, origin xyz=0.03 0.0 -0.17 rpy=0 0 0
- added joint zarm_l7_virtual_thumb_joint_ee: type fixed, parent zarm_l7_end_effector, child zarm_l7_virtual_thumb_link, origin xyz=0.15 0 0 rpy=0 0 0
- added joint zarm_r7_end_effector_1_joint: type fixed, parent zarm_r7_link, child zarm_r7_end_effector_1, origin xyz=0 0.0 -0.08 rpy=0 0 0
- added joint zarm_r7_end_effector_2_joint: type fixed, parent zarm_r7_link, child zarm_r7_end_effector_2, origin xyz=0.03 0.0 -0.17 rpy=0 0 0
- added joint zarm_r7_virtual_thumb_joint_ee: type fixed, parent zarm_r7_end_effector, child zarm_r7_virtual_thumb_link, origin xyz=0.15 0 0 rpy=0 0 0
- joint zarm_l1_joint: parent base_link -> waist_yaw_link
- joint zarm_r1_joint: parent base_link -> waist_yaw_link
