Commit message: sync https://www.lejuhub.com/highlydynamic/kuavo-ros-control/commit/b782eca73b9baa1f5670f521f25fafa4d4d75ddc

File: src/kuavo_assets/models/biped_s62/urdf/drake/biped_v3_arm.urdf (robot description, URDF)
Before this commit: robot biped_s62, 28 links, 27 joints
Joints:
- joint waist_pitch_joint: limit lower=0.0 upper=0.9 effort=618.48 velocity=25.33 -> lower=-0.15707963267949 upper=2.9845130209103 effort=618.48 velocity=25.33
- joint zarm_l1_joint: limit lower=-3.14159265358979 upper=1.5707963267949 effort=66.0 velocity=18.8 -> lower=-2.4 upper=0.6 effort=66.0 velocity=18.8
- joint zarm_l2_joint: limit lower=-0.349065850398866 upper=3.49065850398866 effort=75.0 velocity=8.0 -> lower=-0.349065850398866 upper=1.46 effort=75.0 velocity=8.0
- joint zarm_l3_joint: limit lower=-1.48352986419518 upper=1.48352986419518 effort=57.0 velocity=7.5 -> lower=-1.5707963267949 upper=0.46 effort=57.0 velocity=7.5
- joint zarm_r1_joint: limit lower=-3.14159265358979 upper=1.5707963267949 effort=66.0 velocity=18.8 -> lower=-2.4 upper=0.6 effort=66.0 velocity=18.8
- joint zarm_r2_joint: limit lower=-3.49065850398866 upper=0.349065850398866 effort=75.0 velocity=8.0 -> lower=-1.46 upper=0.349065850398866 effort=75.0 velocity=8.0
- joint zarm_r3_joint: limit lower=-1.48352986419518 upper=1.48352986419518 effort=57.0 velocity=7.5 -> lower=-0.46 upper=1.5707963267949 effort=57.0 velocity=7.5
