Commit message: sync https://www.lejuhub.com/highlydynamic/kuavo-ros-control/commit/b8ffa8b480dc22aa818fa32bad5dea70898e3f93

File: src/kuavo_assets/models/biped_s63/urdf/biped_s63.urdf (robot description, URDF)
Before this commit: robot biped_s63, 36 links, 35 joints
Links:
- link base_link: mass 121.0 -> 114.0
- link wheel_left_behind: mass 6.0 -> 3.85
- link wheel_left_front: mass 6.0 -> 3.85
- link wheel_right_behind: mass 6.0 -> 3.85
- link wheel_right_front: mass 6.0 -> 3.85
Joints:
- joint base_to_joint: origin xyz=0.098 0 0.27064321 rpy=0 0 0 -> xyz=0.093 -0.0165 0.40635 rpy=0 0 0
- joint wheel_left_behind_joint: origin xyz=-0.23248871 0.23248871 0.13035 rpy=0 0 2.356194372 -> xyz=-0.23865 0.23865 0.13035 rpy=0 0 2.3562
- joint wheel_left_front_joint: origin xyz=0.23248871 0.23248871 0.13035 rpy=0 0 0.785398163 -> xyz=0.23865 0.23865 0.13035 rpy=0 0 0.7854
- joint wheel_right_behind_joint: origin xyz=-0.23248871 -0.23248871 0.13035 rpy=0 0 -2.356194372 -> xyz=-0.23865 -0.23865 0.13035 rpy=0 0 -2.3562
- joint wheel_right_front_joint: origin xyz=0.23248871 -0.23248871 0.13035 rpy=0 0 -0.785398163 -> xyz=0.23865 -0.23865 0.13035 rpy=0 0 -0.7854

File: src/kuavo_assets/models/biped_s63/urdf/biped_s63_gazebo.urdf (robot description, URDF)
Before this commit: robot biped_s63, 39 links, 38 joints
Links:
- link base_link: mass 121.0 -> 114.0
Joints:
- joint LB_wheel_yaw_joint: origin xyz=-0.23248871 0.23248871 0.13035 rpy=0 0 0 -> xyz=-0.23865 0.23865 0.13035 rpy=0 0 0
- joint LF_wheel_yaw_joint: origin xyz=0.23248871 0.23248871 0.13035 rpy=0 0 0 -> xyz=0.23865 0.23865 0.13035 rpy=0 0 0
- joint RB_wheel_yaw_joint: origin xyz=-0.23248871 -0.23248871 0.13035 rpy=0 0 0 -> xyz=-0.23865 -0.23865 0.13035 rpy=0 0 0
- joint RF_wheel_yaw_joint: origin xyz=0.23248871 -0.23248871 0.13035 rpy=0 0 0 -> xyz=0.23865 -0.23865 0.13035 rpy=0 0 0
- joint base_to_joint: origin xyz=0.098 0 0.27064321 rpy=0 0 0 -> xyz=0.093 -0.0165 0.40635 rpy=0 0 0
- joint wheel_left_behind_joint: origin xyz=-0.23248871 0.23248871 0.13035 rpy=0 0 2.356194372 -> xyz=-0.23865 0.23865 0.13035 rpy=0 0 2.3562
- joint wheel_left_front_joint: origin xyz=0.23248871 0.23248871 0.13035 rpy=0 0 0.785398163 -> xyz=0.23865 0.23865 0.13035 rpy=0 0 0.7854
- joint wheel_right_behind_joint: origin xyz=-0.23248871 -0.23248871 0.13035 rpy=0 0 -2.356194372 -> xyz=-0.23865 -0.23865 0.13035 rpy=0 0 -2.3562
- joint wheel_right_front_joint: origin xyz=0.23248871 -0.23248871 0.13035 rpy=0 0 -0.785398163 -> xyz=0.23865 -0.23865 0.13035 rpy=0 0 -0.7854

Commit message: sync https://www.lejuhub.com/highlydynamic/kuavo-ros-control/commit/c4f410eae794fa46eeb32472e1a96cd75fac56f0

File: src/kuavo_assets/models/biped_s63/urdf/biped_s63.urdf (robot description, URDF)
Before this commit: robot biped_s63, 36 links, 35 joints
Joints:
- joint zarm_l1_joint: limit lower=-3.14159265358979 upper=1.5707963267949 effort=66.0 velocity=18.8 -> lower=-3.14159265358979 upper=1.5707963267949 effort=85.0 velocity=13.0
- joint zarm_r1_joint: limit lower=-3.14159265358979 upper=1.5707963267949 effort=66.0 velocity=18.8 -> lower=-3.14159265358979 upper=1.5707963267949 effort=85.0 velocity=13.0

File: src/kuavo_assets/models/biped_s63/urdf/biped_s63_gazebo.urdf (robot description, URDF)
Before this commit: robot biped_s63, 39 links, 38 joints
Joints:
- joint zarm_l1_joint: limit lower=-3.14159265358979 upper=1.5707963267949 effort=66.0 velocity=18.8 -> lower=-3.14159265358979 upper=1.5707963267949 effort=85.0 velocity=13.0
- joint zarm_r1_joint: limit lower=-3.14159265358979 upper=1.5707963267949 effort=66.0 velocity=18.8 -> lower=-3.14159265358979 upper=1.5707963267949 effort=85.0 velocity=13.0

Commit message: sync https://www.lejuhub.com/highlydynamic/kuavo-ros-control/commit/718ca73a74a5b9e97b376c146936596f6d29860e

File: src/kuavo_assets/models/biped_s63/urdf/biped_s63.urdf (robot description, URDF)
Before this commit: robot biped_s63, 36 links, 35 joints
Links:
- link base_link: mass 114.0 -> 129.40001; geometry collision cylinder length=0.32 radius=0.37; visual mesh filename=package://kuavo_assets/models/biped_s63/meshes/chassis.STL
- link base_to_joint: mass 7.27493629 -> 7.34488200
- link camera: mass 0.0482361371130408 -> 0.0; geometry visual mesh filename=package://kuavo_assets/models/biped_s63/meshes/head_camera_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
- link camera_base: mass 0.0482361371130408 -> 0.0; geometry visual mesh filename=package://kuavo_assets/models/biped_s63/meshes/head_camera_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
- link knee_link: mass 13.41361777 -> 13.60706531; geometry visual mesh filename=package://kuavo_assets/models/biped_s63/meshes/knee_pitch.S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
- link leg_link: mass 9.78118294 -> 9.43091394; geometry visual mesh filename=package://kuavo_assets/models/biped_s63/meshes/leg_pitch.STL
- link radar: mass 0.001 -> 0.0
- link waist_link: mass 4.65997944 -> 8.15311772; geometry visual mesh filename=package://kuavo_assets/models/biped_s63/meshes/waist_pitch.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
- link waist_yaw_link: mass 11.56094002 -> 12.64200813
- link zarm_l1_link: mass 0.91653322 -> 1.01295970
- link zarm_l2_link: mass 0.38767390 -> 0.43788857
- link zarm_l3_link: mass 1.77926875 -> 1.83544700
- link zarm_l4_link: mass 0.58507821 -> 0.65770374
- link zarm_l5_link: mass 0.68679955 -> 0.67878399
- link zarm_l6_link: mass 0.39387181 -> 0.51230538
- link zarm_l7_link: mass 0.71537800 -> 0.7374
- link zarm_r1_link: mass 0.91653322 -> 1.01295970
- link zarm_r2_link: mass 0.38767390 -> 0.43788857
- link zarm_r3_link: mass 1.77926875 -> 1.83544700
- link zarm_r4_link: mass 0.58507821 -> 0.65770374
- link zarm_r5_link: mass 0.68679955 -> 0.67878399
- link zarm_r6_link: mass 0.39387181 -> 0.51230538
- link zarm_r7_link: mass 0.71537800 -> 0.7374
- link zhead_1_link: mass 0.83597358 -> 0.81695367
- link zhead_2_link: mass 0.75473516 -> 0.82379681
Joints:
- joint base_to_joint: origin xyz=0.093 -0.0165 0.40635 rpy=0 0 0 -> xyz=0.093 0 0.30085 rpy=0 0 0
- joint camera_base_joint: origin xyz=0.099478 0 0.032897 rpy=0 0.35805 0 -> xyz=0.099619 0 0.032844 rpy=0 0.3406 0
- joint radar: origin xyz=0 0 0.059701 rpy=0 0 0 -> xyz=0 0 -0.078453 rpy=0 0 0
- joint waist_yaw_joint: origin xyz=0 0 0.235 rpy=0 0 0 -> xyz=0 0 0.25 rpy=0 0 0
- joint zarm_l1_joint: origin xyz=0 0.2527 0.242 rpy=0 0 0 -> xyz=0 0.253 0.227 rpy=0 0 0
- joint zarm_r1_joint: origin xyz=0 -0.2527 0.242 rpy=0 0 0 -> xyz=0 -0.253 0.227 rpy=0 0 0
- joint zhead_1_joint: origin xyz=0 0 0.3164 rpy=0 0 0 -> xyz=0 0 0.43485 rpy=0 0 0
- joint zhead_2_joint: origin xyz=0 0 0.13795 rpy=0 0 0 -> xyz=0 0 0 rpy=0 0 0

File: src/kuavo_assets/models/biped_s63/urdf/biped_s63_gazebo.urdf (robot description, URDF)
Before this commit: robot biped_s63, 39 links, 38 joints
Links:
- removed link waist_pitch_link
- added link waist_link, mass 8.15311772; visual mesh filename=package://kuavo_assets/models/biped_s63/meshes/waist_pitch.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
- link base_link: mass 114.0 -> 129.40001; geometry visual mesh filename=package://kuavo_assets/models/biped_s63/meshes/chassis.STL
- link base_to_joint: mass 7.27493629 -> 7.34488200
- link camera: mass 0.001 -> 0.0; geometry visual mesh filename=package://kuavo_assets/models/biped_s63/meshes/head_camera_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
- link knee_link: mass 13.41361777 -> 13.60706531; geometry visual mesh filename=package://kuavo_assets/models/biped_s63/meshes/knee_pitch.S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
- link leg_link: mass 9.78118294 -> 9.43091394; geometry visual mesh filename=package://kuavo_assets/models/biped_s63/meshes/leg_pitch.STL
- link radar: mass 0.001 -> 0.0
- link waist_yaw_link: mass 11.56094002 -> 12.64200813; geometry visual mesh filename=package://kuavo_assets/models/biped_s63/meshes/waist_yaw.STL
- link wheel_left_behind: mass 0.1 -> 3.85
- link wheel_right_behind: mass 0.1 -> 3.85
- link wheel_right_front: mass 0.1 -> 3.85
- link zarm_l1_link: mass 0.91653322 -> 1.01295970
- link zarm_l2_link: mass 0.38767390 -> 0.43788857
- link zarm_l3_link: mass 1.77926875 -> 1.83544700
- link zarm_l4_link: mass 0.58507821 -> 0.65770374
- link zarm_l5_link: mass 0.68679955 -> 0.67878399
- link zarm_l6_link: mass 0.39387181 -> 0.51230538
- link zarm_l7_link: mass 0.71537800 -> 0.7374
- link zarm_r1_link: mass 0.91653322 -> 1.01295970
- link zarm_r2_link: mass 0.38767390 -> 0.43788857
- link zarm_r3_link: mass 1.77926875 -> 1.83544700
- link zarm_r4_link: mass 0.58507821 -> 0.65770374
- link zarm_r5_link: mass 0.68679955 -> 0.67878399
- link zarm_r6_link: mass 0.39387181 -> 0.51230538
- link zarm_r7_link: mass 0.71537800 -> 0.7374
- link zhead_1_link: mass 0.83597358 -> 0.81695367
- link zhead_2_link: mass 0.75473516 -> 0.82379681
Joints:
- joint base_to_joint: origin xyz=0.093 -0.0165 0.40635 rpy=0 0 0 -> xyz=0.093 0 0.30085 rpy=0 0 0
- joint camera: origin xyz=0.099478 0 0.032897 rpy=0 0.35805 0 -> xyz=0.011715 0.0475 0.014311 rpy=0 0 0; parent zhead_2_link -> camera_base
- joint radar: origin xyz=0 0 0.059701 rpy=0 0 0 -> xyz=0 0 -0.078453 rpy=0 0 0
- joint waist_pitch_joint: child waist_pitch_link -> waist_link
- joint waist_yaw_joint: origin xyz=0 0 0.235 rpy=0 0 0 -> xyz=0 0 0.25 rpy=0 0 0; parent waist_pitch_link -> waist_link
- joint zarm_l1_joint: origin xyz=0 0.2527 0.242 rpy=0 0 0 -> xyz=0 0.253 0.227 rpy=0 0 0
- joint zarm_r1_joint: origin xyz=0 -0.2527 0.242 rpy=0 0 0 -> xyz=0 -0.253 0.227 rpy=0 0 0
- joint zhead_1_joint: origin xyz=0 0 0.3164 rpy=0 0 0 -> xyz=0 0 0.43485 rpy=0 0 0
- joint zhead_2_joint: origin xyz=0 0 0.13795 rpy=0 0 0 -> xyz=0 0 0 rpy=0 0 0
