Commit message: sync https://www.lejuhub.com/highlydynamic/kuavo-ros-control/commit/981334288c83172b992b48f384bd6a17eb1dd070

File: src/Camera_Calibration/biped_v3_arm.urdf (robot description, URDF)
Before this commit: robot biped_s52, 30 links, 29 joints
Links:
- added link head_camera_color_optical_frame_0; visual sphere radius=0.001
Joints:
- added joint head_camera_color_optical_frame_joint_0: type fixed, parent camera_base, child head_camera_color_optical_frame_0, origin xyz=0 0 0 rpy=-1.57079632679 0 -1.57079632679
- joint head_camera_color_optical_frame_joint: origin xyz=0 0 0 rpy=-1.57079632679 0 -1.57079632679 -> xyz=0.02375 0 0 rpy=0 0 0; parent camera_base -> head_camera_color_optical_frame_0
