Commit message: sync https://www.lejuhub.com/highlydynamic/kuavo-ros-control/commit/728295f27882a6c6541176c1f8de088274419044

File: src/Camera_Calibration/biped_v3_arm_s56.urdf (robot description, URDF)
Before this commit: robot biped_s56, 31 links, 30 joints
Links:
- removed link head_camera_color_optical_frame_0
- link camera_base: geometry visual mesh filename=package://kuavo_assets/models/biped_s56/meshes/head_camera_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
- link zhead_1_link: geometry collision sphere radius=0.1; visual mesh filename=package://kuavo_assets/models/biped_s56/meshes/head_yaw.STL
- link zhead_2_link: geometry visual mesh filename=package://kuavo_assets/models/biped_s56/meshes/head_pitch.S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
Joints:
- removed joint head_camera_color_optical_frame_joint_0
- joint camera_base: origin xyz=0.129717018973535 0.0237514612535074 0.0262044145991832 rpy=0 0.480224871300295 0 -> xyz=0.099619 0 0.032844 rpy=0 0.340224871300295 0
- joint checkerboard_joint: origin xyz=1.01327467669963 -0.176934723317098 -0.17142623754583 rpy=-2.1510713166199 -0.0125236852930088 -1.57002984265249 -> xyz=1.1885083 -0.26639257 -0.23387741 rpy=-2.0934448 0.025182935 -1.5475454
- joint head_camera_color_optical_frame_joint: origin xyz=0.02375 0 0 rpy=0 0 0 -> xyz=0.011715 0.02375 0.014312 rpy=-1.57079632679 0 -1.57079632679; parent head_camera_color_optical_frame_0 -> camera_base
- joint zhead_1_joint: origin xyz=-0.003 0.0 0.3715 rpy=0 0 0 -> xyz=-0.003 0.0 0.49535 rpy=0 0 0
- joint zhead_2_joint: origin xyz=0 0 0.137954074182872 rpy=0 0 0 -> xyz=0 0 0 rpy=0 0 0

File: src/Camera_Calibration/biped_v3_arm_s62.urdf (robot description, URDF)
Before this commit: robot biped_s62, 31 links, 30 joints
Links:
- removed link head_camera_color_optical_frame_0
Joints:
- removed joint head_camera_color_optical_frame_joint_0
- joint camera_base: origin xyz=0.119717018973535 0.0237514612535074 0.0262044145991832 rpy=0 0.480224871300295 0 -> xyz=0.099619 0 0.032844 rpy=0 0.3406 0
- joint head_camera_color_optical_frame_joint: origin xyz=0.02375 0 0 rpy=0 0 0 -> xyz=0.01172 0.02375 0.01431 rpy=-1.57079632679 0 -1.57079632679; parent head_camera_color_optical_frame_0 -> camera_base

Commit message: sync https://www.lejuhub.com/highlydynamic/kuavo-ros-control/commit/034fc9dce5bb0c41cbf1a93da115bb7a0a515321

File: src/Camera_Calibration/biped_v3_arm_s56.urdf (robot description, URDF)
Before this commit: robot biped_s56, 30 links, 29 joints
Joints:
- joint zarm_l1_ref_joint: origin xyz=-0.003 0.1737 0.2831 rpy=0 0 0 -> xyz=-0.003 0.2527 0.2831 rpy=0 0 0
- joint zarm_l2_joint: origin xyz=0 0.081 0 rpy=0 0 0 -> xyz=0 0 0 rpy=0 0 0
- joint zarm_l7_end_effector_joint: origin xyz=0 -0.03 -0.17 rpy=0 0 0 -> xyz=0 0 -0.17 rpy=0 0 0
- joint zarm_r1_joint: origin xyz=-0.003 -0.1737 0.2831 rpy=0 0 0 -> xyz=-0.003 -0.2527 0.2831 rpy=0 0 0
- joint zarm_r2_joint: origin xyz=0 -0.081 0 rpy=0 0 0 -> xyz=0 0 0 rpy=0 0 0
- joint zarm_r7_end_effector_joint: origin xyz=0 0.03 -0.17 rpy=0 0 0 -> xyz=0 0 -0.17 rpy=0 0 0
- joint zarm_r7_joint: origin xyz=0 0 -0.022284 rpy=0 0 0 -> xyz=0 0 -0.021 rpy=0 0 0
