Commit message: sync https://www.lejuhub.com/highlydynamic/kuavo-ros-control/commit/6c0f7ec1efdb0732dab68b9b48e0c57907ced8f3

File: src/Camera_Calibration/biped_v3_arm_calibrated.urdf (robot description, URDF)
Before this commit: robot biped_s52, 30 links, 29 joints
Links:
- added link head_camera_color_optical_frame_0; visual sphere radius=0.001
Joints:
- added joint head_camera_color_optical_frame_joint_0: type fixed, parent camera_base, child head_camera_color_optical_frame_0, origin xyz=0 0 0 rpy=-1.57079632679 0 -1.57079632679
- joint camera_base: origin xyz=0.119717018973535 0.0237514612535074 0.0262044145991832 rpy=0 0.480224871300295 0 -> xyz=0.115442 0.047500 0.042420 rpy=0 0.3406 0
- joint checkerboard_joint: origin xyz=1.00327467669963 -0.176934723317098 -0.17142623754583 rpy=-2.15010713166199 -0.0125236852930088 -1.57002984265249 -> xyz=0.97327467669963 -0.175934723317098 -0.17142623754583 rpy=-2.08010713166199 -0.0125236852930088 -1.50002984265249
- joint head_camera_color_optical_frame_joint: origin xyz=0 0 0 rpy=-1.57079632679 0 -1.57079632679 -> xyz=0.02375 0 0 rpy=0 0 0; parent camera_base -> head_camera_color_optical_frame_0
- joint r_hand_tripod_joint: origin xyz=0.0 0.0 0.0 rpy=0.0 0.0 0.0 -> xyz=0.00881126 -0.00953293 -0.00286888 rpy=0.05840253 -0.00094767 0.03244089
- joint zarm_l1_ref_joint: origin xyz=-0.003 0.1737 0.2831 rpy=0 0 0 -> xyz=-0.003 0.2527 0.283 rpy=0 0 0
- joint zarm_l2_joint: origin xyz=0 0.081 0 rpy=0 0 0 -> xyz=0 0 0 rpy=0 0 0
- joint zarm_l3_joint: origin xyz=0 0 -0.104 rpy=0 0 0 -> xyz=0 0 0 rpy=0 0 0
- joint zarm_l4_joint: origin xyz=0.02 0 -0.1797 rpy=0 0 0 -> xyz=0.02 0 -0.2837 rpy=0 0 0
- joint zarm_l5_joint: origin xyz=-0.02 0 -0.1195 rpy=0 0 0 -> xyz=-0.02 0 -0.1201 rpy=0 0 0
- joint zarm_r1_joint: origin xyz=-0.003 -0.1737 0.2831 rpy=0 0 0 -> xyz=-0.003 -0.2527 0.283 rpy=0 0 0
- joint zarm_r2_joint: origin xyz=0 -0.081 0 rpy=0 0 0 -> xyz=0 0 0 rpy=0 0 0
- joint zarm_r3_joint: origin xyz=0 0 -0.104 rpy=0 0 0 -> xyz=0 0 0 rpy=0 0 0
- joint zarm_r4_joint: origin xyz=0.02 0 -0.1797 rpy=0 0 0 -> xyz=0.02 0 -0.2837 rpy=0 0 0
- joint zarm_r5_joint: origin xyz=-0.02 0 -0.1195 rpy=0 0 0 -> xyz=-0.02 0 -0.1201 rpy=0 0 0
- joint zarm_r7_joint: origin xyz=0 0 -0.022284 rpy=0 0 0 -> xyz=0 0 -0.021 rpy=0 0 0
- joint zhead_1_joint: origin xyz=-0.003 0.0 0.3715 rpy=0 0 0 -> xyz=-0.003 0.0 0.49535 rpy=0 0 0
- joint zhead_2_joint: axis 0 -1 0 -> 0 1 0; origin xyz=0 0 0.137954074182872 rpy=0 0 0 -> xyz=0 0 0 rpy=0 0 0

Commit message: sync https://www.lejuhub.com/highlydynamic/kuavo-ros-control/commit/93e48cf6399cacf801d9649ce5d84ac3e8678a80

File: src/Camera_Calibration/biped_v3_arm_calibrated.urdf (robot description, URDF)
Before this commit: robot biped_s56, 31 links, 30 joints
Links:
- removed link head_camera_color_optical_frame_0
Joints:
- removed joint head_camera_color_optical_frame_joint_0
- joint camera_base: origin xyz=0.115442 0.047500 0.042420 rpy=0 0.3406 0 -> xyz=0.119717018973535 0.0237514612535074 0.0262044145991832 rpy=0 0.480224871300295 0
- joint checkerboard_joint: origin xyz=0.97327467669963 -0.175934723317098 -0.17142623754583 rpy=-2.08010713166199 -0.0125236852930088 -1.50002984265249 -> xyz=1.00327467669963 -0.176934723317098 -0.17142623754583 rpy=-2.15010713166199 -0.0125236852930088 -1.57002984265249
- joint head_camera_color_optical_frame_joint: origin xyz=0.02375 0 0 rpy=0 0 0 -> xyz=0 0 0 rpy=-1.57079632679 0 -1.57079632679; parent head_camera_color_optical_frame_0 -> camera_base
- joint r_hand_tripod_joint: origin xyz=0.00881126 -0.00953293 -0.00286888 rpy=0.05840253 -0.00094767 0.03244089 -> xyz=0.0 0.0 0.0 rpy=0.0 0.0 0.0
- joint zarm_l1_ref_joint: origin xyz=-0.003 0.2527 0.283 rpy=0 0 0 -> xyz=-0.003 0.1737 0.2831 rpy=0 0 0
- joint zarm_l2_joint: origin xyz=0 0 0 rpy=0 0 0 -> xyz=0 0.081 0 rpy=0 0 0
- joint zarm_l3_joint: origin xyz=0 0 0 rpy=0 0 0 -> xyz=0 0 -0.104 rpy=0 0 0
- joint zarm_l4_joint: origin xyz=0.02 0 -0.2837 rpy=0 0 0 -> xyz=0.02 0 -0.1797 rpy=0 0 0
- joint zarm_l5_joint: origin xyz=-0.02 0 -0.1201 rpy=0 0 0 -> xyz=-0.02 0 -0.1195 rpy=0 0 0
- joint zarm_r1_joint: origin xyz=-0.003 -0.2527 0.283 rpy=0 0 0 -> xyz=-0.003 -0.1737 0.2831 rpy=0 0 0
- joint zarm_r2_joint: origin xyz=0 0 0 rpy=0 0 0 -> xyz=0 -0.081 0 rpy=0 0 0
- joint zarm_r3_joint: origin xyz=0 0 0 rpy=0 0 0 -> xyz=0 0 -0.104 rpy=0 0 0
- joint zarm_r4_joint: origin xyz=0.02 0 -0.2837 rpy=0 0 0 -> xyz=0.02 0 -0.1797 rpy=0 0 0
- joint zarm_r5_joint: origin xyz=-0.02 0 -0.1201 rpy=0 0 0 -> xyz=-0.02 0 -0.1195 rpy=0 0 0
- joint zarm_r7_joint: origin xyz=0 0 -0.021 rpy=0 0 0 -> xyz=0 0 -0.022284 rpy=0 0 0
- joint zhead_1_joint: origin xyz=-0.003 0.0 0.49535 rpy=0 0 0 -> xyz=-0.003 0.0 0.3715 rpy=0 0 0
- joint zhead_2_joint: axis 0 1 0 -> 0 -1 0; origin xyz=0 0 0 rpy=0 0 0 -> xyz=0 0 0.137954074182872 rpy=0 0 0

File: src/kuavo_assets/models/apriltag/urdf/grab_box_table.xacro (robot description, xacro)
@@ -260,10 +260,10 @@
     <parent link="world"/>
     <child link="apriltag_box_tag2_base"/>
-    <origin xyz="0.75 -1.7 1.3" rpy="0 0 0"/>
+    <origin xyz="0.5 -1.7 1.3" rpy="0 0 0"/>
   </joint>
   <joint name="world_to_box_tag3_joint" type="fixed">
     <parent link="world"/>
     <child link="apriltag_box_tag3_base"/>
-    <origin xyz="-0.75 -1.7 0.75" rpy="0 0 0"/>
+    <origin xyz="-0.5 -1.7 0.75" rpy="0 0 0"/>
   </joint>
   <joint name="world_to_table_joint" type="fixed">

File: src/kuavo_assets/models/biped_s200062/urdf/biped_s200062.urdf (robot description, URDF)
Before this commit: robot biped_s200062, 64 links, 63 joints
Joints:
- removed joint l_f_bar_2_joint
- removed joint r_f_bar_2_joint
- added joint l_f_bar_2: type fixed, parent l_f_bar_1, child l_f_bar_2, origin xyz=0.011329 0 0.0063767 rpy=0 0 0
- added joint r_f_bar_2: type fixed, parent r_f_bar_1, child r_f_bar_2, origin xyz=0.011329 0 0.0063767 rpy=0 0 0
- joint camera: parent head_camera_base -> camera_base
- joint camera_base_joint: child head_camera_base -> camera_base
- joint l_b_bar_2_joint: axis 0 1 0 -> (none); limit lower=-0.698 upper=0.698 effort=5 velocity=5 -> (none); type revolute -> fixed
- joint l_b_bar_4_joint: axis 0 1 0 -> (none); limit lower=-0.698 upper=0.698 effort=5 velocity=5 -> (none); type revolute -> fixed
- joint l_b_finger_joint: axis 0 1 0 -> (none); limit lower=-0.698 upper=0.698 effort=5 velocity=5 -> (none); type revolute -> fixed
- joint l_f_bar_4_joint: axis 0 1 0 -> (none); limit lower=-0.698 upper=0.698 effort=5 velocity=5 -> (none); type revolute -> fixed
- joint l_f_finger_joint: axis 0 1 0 -> (none); limit lower=-0.698 upper=0.698 effort=5 velocity=5 -> (none); type revolute -> fixed
- joint r_b_bar_2_joint: axis 0 1 0 -> (none); limit lower=-0.698 upper=0.698 effort=5 velocity=5 -> (none); type revolute -> fixed
- joint r_b_bar_4_joint: axis 0 1 0 -> (none); limit lower=-0.698 upper=0.698 effort=5 velocity=5 -> (none); type revolute -> fixed
- joint r_b_finger_joint: axis 0 1 0 -> (none); limit lower=-0.698 upper=0.698 effort=5 velocity=5 -> (none); type revolute -> fixed
- joint r_f_bar_4_joint: axis 0 1 0 -> (none); limit lower=-0.698 upper=0.698 effort=5 velocity=5 -> (none); type revolute -> fixed
- joint r_f_finger_joint: axis 0 1 0 -> (none); limit lower=-0.698 upper=0.698 effort=5 velocity=5 -> (none); type revolute -> fixed
