Commit message: sync https://www.lejuhub.com/highlydynamic/kuavo-ros-control/commit/00f0d403472bc55ef767134ad88a662a416ffada

File: src/Camera_Calibration/biped_v3_arm_s62.urdf (robot description, URDF)
Before this commit: robot biped_s62, 30 links, 29 joints
Joints:
- joint zarm_l1_ref_joint: origin xyz=0.0 0.2527 0.242 rpy=0 0 0 -> xyz=0.0 0.2527 0.227 rpy=0 0 0
- joint zarm_r1_joint: origin xyz=0.0 -0.2527 0.242 rpy=0 0 0 -> xyz=0.0 -0.2527 0.227 rpy=0 0 0
- joint zhead_1_joint: origin xyz=0 0 0.45435 rpy=0 0 0 -> xyz=0 0 0.43935 rpy=0 0 0

File: src/kuavo_assets/models/biped_s62/urdf/biped_s62.urdf (robot description, URDF)
Before this commit: robot biped_s62, 36 links, 35 joints
Joints:
- joint zarm_l1_joint: origin xyz=0 0.2527 0.242 rpy=0 0 0 -> xyz=0 0.2527 0.227 rpy=0 0 0
- joint zarm_r1_joint: origin xyz=0 -0.2527 0.242 rpy=0 0 0 -> xyz=0 -0.2527 0.227 rpy=0 0 0
- joint zhead_1_joint: origin xyz=0 0 0.3164 rpy=0 0 0 -> xyz=0 0 0.43935 rpy=0 0 0
- joint zhead_2_joint: origin xyz=0 0 0.13795 rpy=0 0 0 -> xyz=0 0 0 rpy=0 0 0

File: src/kuavo_assets/models/biped_s62/urdf/biped_s62_gazebo.urdf (robot description, URDF)
Before this commit: robot biped_s62, 40 links, 39 joints
Joints:
- joint zarm_l1_joint: origin xyz=0 0.2527 0.242 rpy=0 0 0 -> xyz=0 0.2527 0.227 rpy=0 0 0
- joint zarm_r1_joint: origin xyz=0 -0.2527 0.242 rpy=0 0 0 -> xyz=0 -0.2527 0.227 rpy=0 0 0
- joint zhead_1_joint: origin xyz=0 0 0.3164 rpy=0 0 0 -> xyz=0 0 0.43935 rpy=0 0 0
- joint zhead_2_joint: origin xyz=0 0 0.13795 rpy=0 0 0 -> xyz=0 0 0 rpy=0 0 0

File: src/kuavo_assets/models/biped_s62/urdf/drake/biped_v3_arm.urdf (robot description, URDF)
Before this commit: robot biped_s62, 28 links, 27 joints
Joints:
- joint zarm_l1_joint: origin xyz=0 0.2527 0.242 rpy=0 0 0 -> xyz=0 0.2527 0.227 rpy=0 0 0
- joint zarm_r1_joint: origin xyz=0 -0.2527 0.242 rpy=0 0 0 -> xyz=0 -0.2527 0.227 rpy=0 0 0

File: src/kuavo_assets/models/biped_s62/urdf/drake/biped_v3_arm_only.urdf (robot description, URDF)
Before this commit: robot biped_s62, 28 links, 27 joints
Joints:
- joint zarm_l1_joint: origin xyz=0 0.2527 0.242 rpy=0 0 0 -> xyz=0 0.2527 0.227 rpy=0 0 0
- joint zarm_r1_joint: origin xyz=0 -0.2527 0.242 rpy=0 0 0 -> xyz=0 -0.2527 0.227 rpy=0 0 0
