Commit message: sync https://www.lejuhub.com/highlydynamic/kuavo-ros-control/commit/ec83b4b7359f074a15db47d2e9f41cc40c866f0b

File: src/kuavo_assets/models/biped_s200062/urdf/biped_s200062.urdf (robot description, URDF)
Before this commit: robot biped_s200062, 64 links, 63 joints
Links:
- removed link camera_base
- added link head_camera_base, mass 0.0482361371130408; visual mesh filename=package://kuavo_assets/models/biped_s200062/meshes/head_cam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
Joints:
- joint zarm_l1_joint: limit lower=-3.14159265358979 upper=1.5707963267949 effort=66.0 velocity=18.8 -> lower=-3.14159265358979 upper=1.5707963267949 effort=85.0 velocity=13.0
- joint zarm_r1_joint: limit lower=-3.14159265358979 upper=1.5707963267949 effort=66.0 velocity=18.8 -> lower=-3.14159265358979 upper=1.5707963267949 effort=85.0 velocity=13.0

File: src/kuavo_assets/models/biped_s300062/urdf/biped_s300062.urdf (robot description, URDF)
Before this commit: robot biped_s300062, 64 links, 63 joints
Joints:
- joint zarm_l1_joint: limit lower=-3.14159265358979 upper=1.5707963267949 effort=66.0 velocity=18.8 -> lower=-3.14159265358979 upper=1.5707963267949 effort=85.0 velocity=13.0
- joint zarm_r1_joint: limit lower=-3.14159265358979 upper=1.5707963267949 effort=66.0 velocity=18.8 -> lower=-3.14159265358979 upper=1.5707963267949 effort=85.0 velocity=13.0
