Commit message: sync https://www.lejuhub.com/highlydynamic/kuavo-ros-control/commit/23d19c80cb86d690701a107f743550492fbab8c0

File: src/kuavo_assets/models/biped_s200062/urdf/biped_s200062.urdf (robot description, URDF)
Before this commit: robot biped_s200062, 64 links, 63 joints
Links:
- removed link l_d405_camera_base
- removed link r_d405_camera_base
- added link cam_h_link
- added link cam_l_link
- added link cam_r_link
- added link camera_l_base; visual mesh filename=package://kuavo_assets/models/biped_s200062/meshes/l_d405_c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
- added link camera_l_color_link
- added link camera_l_depth_link
- added link camera_r_base; visual mesh filename=package://kuavo_assets/models/biped_s200062/meshes/r_d405_c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
- added link camera_r_color_link
- added link camera_r_depth_link
Joints:
- removed joint l_d405_camera_base_joint
- removed joint r_d405_camera_base_joint
- added joint camera_l_color_frame: type fixed, parent camera_l_base, child camera_l_color_link, origin xyz=0.0109 0.009 0.021 rpy=0 0 0
- added joint camera_l_depth_frame: type fixed, parent camera_l_base, child camera_l_depth_link, origin xyz=0.0109 -0.009 0.021 rpy=0 0 0
- added joint camera_r_color_frame: type fixed, parent camera_r_base, child camera_r_color_link, origin xyz=0.0109 0.009 0.021 rpy=0 0 0
- added joint camera_r_depth_frame: type fixed, parent camera_r_base, child camera_r_depth_link, origin xyz=0.0109 -0.009 0.021 rpy=0 0 0
- added joint camera_to_realcam_h_frame: type fixed, parent camera, child cam_h_link, origin xyz=0 0 0 rpy=0 0 0
- added joint camera_to_realcam_l_frame: type fixed, parent camera_l_base, child cam_l_link, origin xyz=0.0146 0.00 0.021 rpy=0 0 0
- added joint camera_to_realcam_r_frame: type fixed, parent camera_r_base, child cam_r_link, origin xyz=0.0146 0.00 0.021 rpy=0 0 0
- added joint l_hand_camera_joint: type fixed, parent l_d405_camera_connect, child camera_l_base, origin xyz=0.00835 0 -0.021 rpy=0 0 0
- added joint r_hand_camera_joint: type fixed, parent r_d405_camera_connect, child camera_r_base, origin xyz=0.00835 0 -0.021 rpy=0 0 0
- joint base_to_joint: origin xyz=0.098 0 0.27064321 rpy=0 0 0 -> xyz=0.098 0 0.31064321 rpy=0 0 0
- joint camera_base_joint: origin xyz=0.099478 0 0.032897 rpy=0 0.35805 0 -> xyz=0.099478 0 0.032897 rpy=0 0.3406 0
- joint l_camera_joint: parent l_d405_camera_base -> camera_l_base
- joint r_camera_joint: parent r_d405_camera_base -> camera_r_base
- joint zarm_l1_joint: origin xyz=0 0.2527 0.242 rpy=0 0 0 -> xyz=0 0.2527 0.227 rpy=0 0 0
- joint zarm_r1_joint: origin xyz=0 -0.2527 0.242 rpy=0 0 0 -> xyz=0 -0.2527 0.227 rpy=0 0 0
- joint zhead_1_joint: origin xyz=0 0 0.3164 rpy=0 0 0 -> xyz=0 0 0.43935 rpy=0 0 0
- joint zhead_2_joint: origin xyz=0 0 0.13795 rpy=0 0 0 -> xyz=0 0 0 rpy=0 0 0

File: src/kuavo_assets/models/biped_s200062/urdf/biped_s200062_gazebo.urdf (robot description, URDF)
Before this commit: robot biped_s200062, 39 links, 38 joints
Links:
- added link cam_h_link
- added link cam_l_link
- added link cam_r_link
- added link camera_l_base
- added link camera_l_color_link
- added link camera_l_depth_link
- added link camera_r_base
- added link camera_r_color_link
- added link camera_r_depth_link
Joints:
- added joint camera_l_color_frame: type fixed, parent camera_l_base, child camera_l_color_link, origin xyz=0.0109 0.009 0.021 rpy=0 0 0
- added joint camera_l_depth_frame: type fixed, parent camera_l_base, child camera_l_depth_link, origin xyz=0.0109 -0.009 0.021 rpy=0 0 0
- added joint camera_r_color_frame: type fixed, parent camera_r_base, child camera_r_color_link, origin xyz=0.0109 0.009 0.021 rpy=0 0 0
- added joint camera_r_depth_frame: type fixed, parent camera_r_base, child camera_r_depth_link, origin xyz=0.0109 -0.009 0.021 rpy=0 0 0
- added joint camera_to_realcam_h_frame: type fixed, parent camera, child cam_h_link, origin xyz=0 0 0 rpy=0 0 0
- added joint camera_to_realcam_l_frame: type fixed, parent camera_l_base, child cam_l_link, origin xyz=0.0146 0.00 0.021 rpy=0 0 0
- added joint camera_to_realcam_r_frame: type fixed, parent camera_r_base, child cam_r_link, origin xyz=0.0146 0.00 0.021 rpy=0 0 0
- added joint l_hand_camera_joint: type fixed, parent zarm_l7_link, child camera_l_base, origin xyz=7.21360860434e-08 0.0334214585163 -0.106588366881 rpy=-3.1416 1.0472 -1.5708
- added joint r_hand_camera_joint: type fixed, parent zarm_r7_link, child camera_r_base, origin xyz=-2.36413142634e-07 -0.0334214585174 -0.106588366881 rpy=-3.1416 1.0472 1.5708
- joint camera: origin xyz=0.099478 0 0.032897 rpy=0 0.35805 0 -> xyz=0.099478 0 0.032897 rpy=0 0.3406 0
- joint zarm_l1_joint: origin xyz=0 0.2527 0.242 rpy=0 0 0 -> xyz=0 0.2527 0.227 rpy=0 0 0
- joint zarm_r1_joint: origin xyz=0 -0.2527 0.242 rpy=0 0 0 -> xyz=0 -0.2527 0.227 rpy=0 0 0
- joint zhead_1_joint: origin xyz=0 0 0.3164 rpy=0 0 0 -> xyz=0 0 0.43935 rpy=0 0 0
- joint zhead_2_joint: origin xyz=0 0 0.13795 rpy=0 0 0 -> xyz=0 0 0 rpy=0 0 0

File: src/kuavo_assets/models/biped_s200062/urdf/drake/biped_v3_arm.urdf (robot description, URDF)
Before this commit: robot biped_s200062, 28 links, 27 joints
Joints:
- joint base_to_joint: origin xyz=0.098 0 0.27064321 rpy=0 0 0 -> xyz=0.098 0 0.31064321 rpy=0 0 0
- joint zarm_l1_joint: origin xyz=0 0.2527 0.242 rpy=0 0 0 -> xyz=0 0.2527 0.227 rpy=0 0 0
- joint zarm_r1_joint: origin xyz=0 -0.2527 0.242 rpy=0 0 0 -> xyz=0 -0.2527 0.227 rpy=0 0 0

File: src/kuavo_assets/models/biped_s200062/urdf/drake/biped_v3_upper_body.urdf (robot description, URDF)
Before this commit: robot biped_s200062, 28 links, 27 joints
Joints:
- joint zarm_l1_joint: origin xyz=0 0.2527 0.242 rpy=0 0 0 -> xyz=0 0.2527 0.227 rpy=0 0 0
- joint zarm_r1_joint: origin xyz=0 -0.2527 0.242 rpy=0 0 0 -> xyz=0 -0.2527 0.227 rpy=0 0 0

File: src/kuavo_assets/models/biped_s300062/urdf/biped_s300062.urdf (robot description, URDF)
Before this commit: robot biped_s300062, 64 links, 63 joints
Links:
- removed link l_d405_camera_base
- removed link r_d405_camera_base
- added link cam_h_link
- added link cam_l_link
- added link cam_r_link
- added link camera_l_base, mass 0.0001; collision box size=0.03 0.09 0.025; visual mesh filename=package://kuavo_assets/models/biped_s300062/meshes/l_d405_c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
- added link camera_l_color_link
- added link camera_l_depth_link
- added link camera_r_base, mass 0.0001; collision box size=0.03 0.09 0.025; visual mesh filename=package://kuavo_assets/models/biped_s300062/meshes/r_d405_c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
- added link camera_r_color_link
- added link camera_r_depth_link
Joints:
- removed joint l_d405_camera_base_joint
- removed joint r_d405_camera_base_joint
- added joint camera_l_color_frame: type fixed, parent camera_l_base, child camera_l_color_link, origin xyz=0.0109 0.009 0.021 rpy=0 0 0
- added joint camera_l_depth_frame: type fixed, parent camera_l_base, child camera_l_depth_link, origin xyz=0.0109 -0.009 0.021 rpy=0 0 0
- added joint camera_r_color_frame: type fixed, parent camera_r_base, child camera_r_color_link, origin xyz=0.0109 0.009 0.021 rpy=0 0 0
- added joint camera_r_depth_frame: type fixed, parent camera_r_base, child camera_r_depth_link, origin xyz=0.0109 -0.009 0.021 rpy=0 0 0
- added joint camera_to_realcam_h_frame: type fixed, parent camera, child cam_h_link, origin xyz=0 0 0 rpy=0 0 0
- added joint camera_to_realcam_l_frame: type fixed, parent camera_l_base, child cam_l_link, origin xyz=0.0146 0.00 0.021 rpy=0 0 0
- added joint camera_to_realcam_r_frame: type fixed, parent camera_r_base, child cam_r_link, origin xyz=0.0146 0.00 0.021 rpy=0 0 0
- added joint l_hand_camera_joint: type fixed, parent zarm_l7_link, child camera_l_base, origin xyz=0.12576 -0.033035 -0.092883 rpy=1.933 0.75188 -2.8883
- added joint r_hand_camera_joint: type fixed, parent zarm_r7_link, child camera_r_base, origin xyz=0.12576 0.033035 -0.092883 rpy=-1.933 0.75188 2.8883
- joint base_to_joint: origin xyz=0.098 0 0.27064321 rpy=0 0 0 -> xyz=0.098 0 0.31 rpy=0 0 0
- joint camera: origin xyz=0.011715 0.0475 0.014311 rpy=0 0 0 -> xyz=0.115300652811 0.0475 0.042472468866 rpy=0 0.3406 0; parent camera_base -> zhead_2_link
- joint camera_base_joint: origin xyz=0.099478 0 0.032897 rpy=0 0.35805 0 -> xyz=0.099478 0 0.032897 rpy=0 0.3406 0
- joint l_d405_camera_joint: parent l_d405_camera_base -> camera_l_base
- joint r_d405_camera_joint: parent r_d405_camera_base -> camera_r_base
- joint zarm_l1_joint: origin xyz=0 0.2527 0.242 rpy=0 0 0 -> xyz=0 0.2527 0.227 rpy=0 0 0
- joint zarm_r1_joint: origin xyz=0 -0.2527 0.242 rpy=0 0 0 -> xyz=0 -0.2527 0.227 rpy=0 0 0
- joint zhead_1_joint: origin xyz=0 0 0.3164 rpy=0 0 0 -> xyz=0 0 0.43935 rpy=0 0 0
- joint zhead_2_joint: origin xyz=0 0 0.13795 rpy=0 0 0 -> xyz=0 0 0 rpy=0 0 0

File: src/kuavo_assets/models/biped_s300062/urdf/biped_s300062_gazebo.urdf (robot description, URDF)
Before this commit: robot biped_s300062, 39 links, 38 joints
Links:
- added link cam_h_link
- added link cam_l_link
- added link cam_r_link
- added link camera_l_base
- added link camera_l_color_link
- added link camera_l_depth_link
- added link camera_r_base
- added link camera_r_color_link
- added link camera_r_depth_link
Joints:
- added joint camera_l_color_frame: type fixed, parent camera_l_base, child camera_l_color_link, origin xyz=0.0109 0.009 0.021 rpy=0 0 0
- added joint camera_l_depth_frame: type fixed, parent camera_l_base, child camera_l_depth_link, origin xyz=0.0109 -0.009 0.021 rpy=0 0 0
- added joint camera_r_color_frame: type fixed, parent camera_r_base, child camera_r_color_link, origin xyz=0.0109 0.009 0.021 rpy=0 0 0
- added joint camera_r_depth_frame: type fixed, parent camera_r_base, child camera_r_depth_link, origin xyz=0.0109 -0.009 0.021 rpy=0 0 0
- added joint camera_to_realcam_h_frame: type fixed, parent camera, child cam_h_link, origin xyz=0 0 0 rpy=0 0 0
- added joint camera_to_realcam_l_frame: type fixed, parent camera_l_base, child cam_l_link, origin xyz=0.0146 0.00 0.021 rpy=0 0 0
- added joint camera_to_realcam_r_frame: type fixed, parent camera_r_base, child cam_r_link, origin xyz=0.0146 0.00 0.021 rpy=0 0 0
- added joint l_hand_camera_joint: type fixed, parent zarm_l7_link, child camera_l_base, origin xyz=0.12576 -0.033035 -0.092883 rpy=1.933 0.75188 -2.8883
- added joint r_hand_camera_joint: type fixed, parent zarm_r7_link, child camera_r_base, origin xyz=0.12576 0.033035 -0.092883 rpy=-1.933 0.75188 2.8883
- joint camera: origin xyz=0.099478 0 0.032897 rpy=0 0.35805 0 -> xyz=0.099478 0 0.032897 rpy=0 0.3406 0
- joint zarm_l1_joint: origin xyz=0 0.2527 0.242 rpy=0 0 0 -> xyz=0 0.2527 0.227 rpy=0 0 0
- joint zarm_r1_joint: origin xyz=0 -0.2527 0.242 rpy=0 0 0 -> xyz=0 -0.2527 0.227 rpy=0 0 0
- joint zhead_1_joint: origin xyz=0 0 0.3164 rpy=0 0 0 -> xyz=0 0 0.43935 rpy=0 0 0
- joint zhead_2_joint: origin xyz=0 0 0.13795 rpy=0 0 0 -> xyz=0 0 0 rpy=0 0 0

File: src/kuavo_assets/models/biped_s300062/urdf/drake/biped_v3_arm.urdf (robot description, URDF)
Before this commit: robot biped_s300062, 28 links, 27 joints
Joints:
- joint base_to_joint: origin xyz=0.098 0 0.27064321 rpy=0 0 0 -> xyz=0.098 0 0.31 rpy=0 0 0
- joint zarm_l1_joint: origin xyz=0 0.2527 0.242 rpy=0 0 0 -> xyz=0 0.2527 0.227 rpy=0 0 0
- joint zarm_r1_joint: origin xyz=0 -0.2527 0.242 rpy=0 0 0 -> xyz=0 -0.2527 0.227 rpy=0 0 0

File: src/kuavo_assets/models/biped_s400062/urdf/biped_s400062.urdf (robot description, URDF)
Before this commit: robot biped_s400062, 68 links, 67 joints
Links:
- removed link head_camera_base
- added link camera, mass 0.0482361371130408
- added link camera_base, mass 0.0482361371130408; visual mesh filename=package://kuavo_assets/models/biped_s400062/meshes/head_cam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
- link cam_h_link: mass 0.0482361371130408 -> None
Joints:
- removed joint cam_h_link_joint
- removed joint camera_l_base_joint
- removed joint camera_r_base_joint
- removed joint head_camera_base_joint
- added joint camera: type fixed, parent zhead_2_link, child camera, origin xyz=0.115300652811 0.0475 0.042472468866 rpy=0 0.3406 0
- added joint camera_base_joint: type fixed, parent zhead_2_link, child camera_base, origin xyz=0.099478 0 0.032897 rpy=0 0.3406 0
- added joint camera_to_realcam_h_frame: type fixed, parent camera, child cam_h_link, origin xyz=0 0 0 rpy=0 0 0
- added joint l_hand_camera_joint: type fixed, parent zarm_l7_link, child camera_l_base, origin xyz=0.093563 -0.015735 0.021967 rpy=-2.2353 1.1377 -2.1889, axis 0 0 0
- added joint r_hand_camera_joint: type fixed, parent zarm_r7_link, child camera_r_base, origin xyz=0.134 0.015735 0.0111 rpy=2.2353 1.1377 2.1889, axis 0 0 0
- joint camera_r_color_frame: origin xyz=0.0109 0.009 -0.021 rpy=3.14159265358979 0 0 -> xyz=0.0109 -0.009 -0.021 rpy=3.14159265358979 0 0
- joint camera_r_depth_frame: origin xyz=0.0109 -0.009 -0.021 rpy=3.14159265358979 0 0 -> xyz=0.0109 0.009 -0.021 rpy=3.14159265358979 0 0
- joint zarm_l1_joint: origin xyz=0 0.2527 0.242 rpy=0 0 0 -> xyz=0 0.2527 0.227 rpy=0 0 0
- joint zarm_r1_joint: origin xyz=0 -0.2527 0.242 rpy=0 0 0 -> xyz=0 -0.2527 0.227 rpy=0 0 0
- joint zhead_1_joint: origin xyz=0 0 0.3164 rpy=0 0 0 -> xyz=0 0 0.43935 rpy=0 0 0
- joint zhead_2_joint: origin xyz=0 0 0.13795 rpy=0 0 0 -> xyz=0 0 0 rpy=0 0 0

File: src/kuavo_assets/models/biped_s400062/urdf/biped_s400062_gazebo.urdf (robot description, URDF)
Before this commit: robot biped_s400062, 64 links, 63 joints
Links:
- removed link head_camera_base
- added link cam_l_link
- added link cam_r_link
- added link camera, mass 0.001; visual mesh filename=package://kuavo_assets/models/biped_s400062/meshes/head_cam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
- added link camera_l_base
- added link camera_l_color_link
- added link camera_l_depth_link
- added link camera_r_base
- added link camera_r_color_link
- added link camera_r_depth_link
- link cam_h_link: mass 0.001 -> None
Joints:
- removed joint cam_h_link_joint
- removed joint head_camera_base_joint
- added joint camera: type fixed, parent zhead_2_link, child camera, origin xyz=0.099478 0 0.032897 rpy=0 0.3406 0
- added joint camera_l_color_frame: type fixed, parent camera_l_base, child camera_l_color_link, origin xyz=0.0109 0.009 0.021 rpy=0 0 0
- added joint camera_l_depth_frame: type fixed, parent camera_l_base, child camera_l_depth_link, origin xyz=0.0109 -0.009 0.021 rpy=0 0 0
- added joint camera_r_color_frame: type fixed, parent camera_r_base, child camera_r_color_link, origin xyz=0.0109 -0.009 -0.021 rpy=3.14159265358979 0 0
- added joint camera_r_depth_frame: type fixed, parent camera_r_base, child camera_r_depth_link, origin xyz=0.0109 0.009 -0.021 rpy=3.14159265358979 0 0
- added joint camera_to_realcam_h_frame: type fixed, parent camera, child cam_h_link, origin xyz=0 0 0 rpy=0 0 0
- added joint camera_to_realcam_l_frame: type fixed, parent camera_l_base, child cam_l_link, origin xyz=0.0146 0.00 0.021 rpy=0 0 0
- added joint camera_to_realcam_r_frame: type fixed, parent camera_r_base, child cam_r_link, origin xyz=0.0146 0.00 -0.021 rpy=3.14159265358979 0 0
- added joint l_hand_camera_joint: type fixed, parent zarm_l7_link, child camera_l_base, origin xyz=0.093563 -0.015735 0.021967 rpy=-2.2353 1.1377 -2.1889
- added joint r_hand_camera_joint: type fixed, parent zarm_r7_link, child camera_r_base, origin xyz=0.134 0.015735 0.0111 rpy=2.2353 1.1377 2.1889
- joint zarm_l1_joint: origin xyz=0 0.2527 0.242 rpy=0 0 0 -> xyz=0 0.2527 0.227 rpy=0 0 0
- joint zarm_r1_joint: origin xyz=0 -0.2527 0.242 rpy=0 0 0 -> xyz=0 -0.2527 0.227 rpy=0 0 0
- joint zhead_1_joint: origin xyz=0 0 0.3164 rpy=0 0 0 -> xyz=0 0 0.43935 rpy=0 0 0
- joint zhead_2_joint: origin xyz=0 0 0.13795 rpy=0 0 0 -> xyz=0 0 0 rpy=0 0 0

File: src/kuavo_assets/models/biped_s400062/urdf/drake/biped_v3_arm.urdf (robot description, URDF)
Before this commit: robot biped_s400062, 52 links, 51 joints
Joints:
- joint base_to_joint: origin xyz=0.098 0 0.27064321 rpy=0 0 0 -> xyz=0.098 0 0.31 rpy=0 0 0
- joint zarm_l1_joint: origin xyz=0 0.2527 0.242 rpy=0 0 0 -> xyz=0 0.2527 0.227 rpy=0 0 0
- joint zarm_r1_joint: origin xyz=0 -0.2527 0.242 rpy=0 0 0 -> xyz=0 -0.2527 0.227 rpy=0 0 0

File: src/kuavo_assets/models/biped_s400062/urdf/drake/biped_v3_arm_only.urdf (robot description, URDF)
Before this commit: robot biped_s400062, 52 links, 51 joints
Joints:
- joint zarm_l1_joint: origin xyz=0 0.2527 0.242 rpy=0 0 0 -> xyz=0 0.2527 0.227 rpy=0 0 0
- joint zarm_r1_joint: origin xyz=0 -0.2527 0.242 rpy=0 0 0 -> xyz=0 -0.2527 0.227 rpy=0 0 0

File: src/kuavo_assets/models/biped_s400062/urdf/drake/biped_v3_upper_body.urdf (robot description, URDF)
Before this commit: robot biped_s400062, 47 links, 46 joints
Joints:
- joint zarm_l1_joint: origin xyz=0 0.2527 0.242 rpy=0 0 0 -> xyz=0 0.2527 0.227 rpy=0 0 0
- joint zarm_r1_joint: origin xyz=0 -0.2527 0.242 rpy=0 0 0 -> xyz=0 -0.2527 0.227 rpy=0 0 0

File: src/kuavo_assets/models/biped_s400063/urdf/biped_s400063.urdf (robot description, URDF)
Before this commit: robot biped_s400063, 68 links, 67 joints
Links:
- removed link head_camera_base
- added link camera, mass 0.0482361371130408
- added link camera_base, mass 0.0482361371130408; visual mesh filename=package://kuavo_assets/models/biped_s400063/meshes/head_cam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
- link cam_h_link: mass 0.0 -> None; geometry 
Joints:
- removed joint cam_h_link_joint
- removed joint camera_l_base_joint
- removed joint camera_r_base_joint
- removed joint head_camera_base_joint
- added joint camera: type fixed, parent zhead_2_link, child camera, origin xyz=0.115300652811 0.0475 0.042472468866 rpy=0 0.3406 0
- added joint camera_base_joint: type fixed, parent zhead_2_link, child camera_base, origin xyz=0.099478 0 0.032897 rpy=0 0.3406 0
- added joint camera_to_realcam_h_frame: type fixed, parent camera, child cam_h_link, origin xyz=0 0 0 rpy=0 0 0
- added joint l_hand_camera_joint: type fixed, parent zarm_l7_link, child camera_l_base, origin xyz=0.093563 -0.015735 0.021967 rpy=-2.2353 1.1377 -2.1889, axis 0 0 0
- added joint r_hand_camera_joint: type fixed, parent zarm_r7_link, child camera_r_base, origin xyz=0.134 0.015735 0.0111 rpy=2.2353 1.1377 2.1889, axis 0 0 0
- joint camera_r_color_frame: origin xyz=0.0109 0.009 -0.021 rpy=3.14159265358979 0 0 -> xyz=0.0109 -0.009 -0.021 rpy=3.14159265358979 0 0
- joint camera_r_depth_frame: origin xyz=0.0109 -0.009 -0.021 rpy=3.14159265358979 0 0 -> xyz=0.0109 0.009 -0.021 rpy=3.14159265358979 0 0

File: src/kuavo_assets/models/biped_s400063/urdf/biped_s400063_gazebo.urdf (robot description, URDF)
Before this commit: robot biped_s400063, 64 links, 63 joints
Links:
- removed link head_camera_base
- added link cam_l_link
- added link cam_r_link
- added link camera, mass 0.0; visual mesh filename=package://kuavo_assets/models/biped_s400063/meshes/head_cam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
- added link camera_l_base
- added link camera_l_color_link
- added link camera_l_depth_link
- added link camera_r_base
- added link camera_r_color_link
- added link camera_r_depth_link
- link cam_h_link: mass 0.0 -> None; geometry 
Joints:
- removed joint cam_h_link_joint
- removed joint head_camera_base_joint
- added joint camera: type fixed, parent zhead_2_link, child camera, origin xyz=0.099478 0 0.032897 rpy=0 0.3406 0
- added joint camera_l_color_frame: type fixed, parent camera_l_base, child camera_l_color_link, origin xyz=0.0109 0.009 0.021 rpy=0 0 0
- added joint camera_l_depth_frame: type fixed, parent camera_l_base, child camera_l_depth_link, origin xyz=0.0109 -0.009 0.021 rpy=0 0 0
- added joint camera_r_color_frame: type fixed, parent camera_r_base, child camera_r_color_link, origin xyz=0.0109 -0.009 -0.021 rpy=3.14159265358979 0 0
- added joint camera_r_depth_frame: type fixed, parent camera_r_base, child camera_r_depth_link, origin xyz=0.0109 0.009 -0.021 rpy=3.14159265358979 0 0
- added joint camera_to_realcam_h_frame: type fixed, parent camera, child cam_h_link, origin xyz=0 0 0 rpy=0 0 0
- added joint camera_to_realcam_l_frame: type fixed, parent camera_l_base, child cam_l_link, origin xyz=0.0146 0.00 0.021 rpy=0 0 0
- added joint camera_to_realcam_r_frame: type fixed, parent camera_r_base, child cam_r_link, origin xyz=0.0146 0.00 -0.021 rpy=3.14159265358979 0 0
- added joint l_hand_camera_joint: type fixed, parent zarm_l7_link, child camera_l_base, origin xyz=0.093563 -0.015735 0.021967 rpy=-2.2353 1.1377 -2.1889
- added joint r_hand_camera_joint: type fixed, parent zarm_r7_link, child camera_r_base, origin xyz=0.134 0.015735 0.0111 rpy=2.2353 1.1377 2.1889

File: src/kuavo_assets/models/biped_s62/urdf/biped_s62_gazebo.urdf (robot description, URDF)
Before this commit: robot biped_s62, 40 links, 39 joints
Joints:
- joint base_to_joint: origin xyz=0.098 0 0.27064321 rpy=0 0 0 -> xyz=0.098 0 0.31 rpy=0 0 0

File: src/kuavo_assets/models/biped_s62/urdf/drake/biped_v3_arm.urdf (robot description, URDF)
Before this commit: robot biped_s62, 28 links, 27 joints
Joints:
- joint base_to_joint: origin xyz=0.098 0 0.27064321 rpy=0 0 0 -> xyz=0.098 0 0.31 rpy=0 0 0

File: src/kuavo_assets/models/biped_s62/urdf/drake/biped_v3_arm_only.urdf (robot description, URDF)
Before this commit: robot biped_s62, 28 links, 27 joints
Joints:
- joint base_to_joint: origin xyz=0.098 0 0.27064321 rpy=0 0 0 -> xyz=0.098 0 0.31 rpy=0 0 0
