Commit message: sync https://www.lejuhub.com/highlydynamic/kuavo-ros-control/commit/02aba90958101c97808f24d6d370e8f0fc8d096a

File: src/kuavo_assets/models/biped_s200062/urdf/biped_s200062.urdf (robot description, URDF)
Before this commit: robot biped_s200062, 71 links, 70 joints
Joints:
- joint waist_yaw_joint: origin xyz=0 0 0.235 rpy=0 0 0 -> xyz=0 0 0.250 rpy=0 0 0

File: src/kuavo_assets/models/biped_s200062/urdf/biped_s200062_gazebo.urdf (robot description, URDF)
Before this commit: robot biped_s200062, 48 links, 47 joints
Joints:
- joint waist_yaw_joint: origin xyz=0 0 0.235 rpy=0 0 0 -> xyz=0 0 0.250 rpy=0 0 0

File: src/kuavo_assets/models/biped_s200062/urdf/drake/biped_v3_arm.urdf (robot description, URDF)
Before this commit: robot biped_s200062, 28 links, 27 joints
Joints:
- joint waist_yaw_joint: origin xyz=0 0 0.235 rpy=0 0 0 -> xyz=0 0 0.250 rpy=0 0 0

File: src/kuavo_assets/models/biped_s200062/urdf/drake/biped_v3_upper_body.urdf (robot description, URDF)
Before this commit: robot biped_s200062, 28 links, 27 joints
Joints:
- joint waist_yaw_joint: origin xyz=0 0 0.235 rpy=0 0 0 -> xyz=0 0 0.250 rpy=0 0 0

File: src/kuavo_assets/models/biped_s300062/urdf/biped_s300062.urdf (robot description, URDF)
Before this commit: robot biped_s300062, 71 links, 70 joints
Joints:
- joint waist_yaw_joint: origin xyz=0 0 0.235 rpy=0 0 0 -> xyz=0 0 0.250 rpy=0 0 0

File: src/kuavo_assets/models/biped_s300062/urdf/biped_s300062_gazebo.urdf (robot description, URDF)
Before this commit: robot biped_s300062, 48 links, 47 joints
Joints:
- joint waist_yaw_joint: origin xyz=0 0 0.235 rpy=0 0 0 -> xyz=0 0 0.250 rpy=0 0 0

File: src/kuavo_assets/models/biped_s300062/urdf/drake/biped_v3_arm.urdf (robot description, URDF)
Before this commit: robot biped_s300062, 28 links, 27 joints
Joints:
- joint waist_yaw_joint: origin xyz=0 0 0.235 rpy=0 0 0 -> xyz=0 0 0.250 rpy=0 0 0

File: src/kuavo_assets/models/biped_s400055/urdf/biped_s400055.urdf (robot description, URDF)
Before this commit: robot biped_s400055, 74 links, 73 joints
Links:
- added link cam_h_link
- added link cam_l_link
- added link cam_r_link
- added link camera
- added link camera_base, mass 0.00000000; visual mesh filename=package://kuavo_assets/models/biped_s400055/meshes/head_cam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
- added link camera_l_base, mass 0.00010000; collision mesh filename=package://kuavo_assets/models/biped_s400055/meshes/l_d405_c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; visual mesh filename=package://kuavo_assets/models/biped_s400055/meshes/l_d405_c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
- added link camera_l_color_link
- added link camera_l_depth_link
- added link camera_r_base, mass 0.00010000; collision mesh filename=package://kuavo_assets/models/biped_s400055/meshes/r_d405_c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; visual mesh filename=package://kuavo_assets/models/biped_s400055/meshes/r_d405_c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
- added link camera_r_color_link
- added link camera_r_depth_link
- added link l_d405_camera, mass 0.00006545; collision mesh filename=package://kuavo_assets/models/biped_s400055/meshes/l_d405_c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; visual mesh filename=package://kuavo_assets/models/biped_s400055/meshes/l_d405_c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
- added link r_d405_camera, mass 0.00006545; collision mesh filename=package://kuavo_assets/models/biped_s400055/meshes/r_d405_c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; visual mesh filename=package://kuavo_assets/models/biped_s400055/meshes/r_d405_c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
- added link radar, mass 0.00000; visual mesh filename=package://kuavo_assets/models/biped_s400055/meshes/head_rad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
- added link zarm_l7_end_effector_1
- added link zarm_l7_end_effector_2
- added link zarm_r7_end_effector_1
- added link zarm_r7_end_effector_2
Joints:
- added joint camera: type fixed, parent zhead_2_link, child camera, origin xyz=0.099619 0 0.032844 rpy=0 0.3406 0
- added joint camera_base_joint: type fixed, parent zhead_2_link, child camera_base, origin xyz=0.099619 0 0.032844 rpy=0 0.3406 0
- added joint camera_l_color_frame: type fixed, parent camera_l_base, child camera_l_color_link, origin xyz=0.0109 0.009 0.021 rpy=0 0 0
- added joint camera_l_depth_frame: type fixed, parent camera_l_base, child camera_l_depth_link, origin xyz=0.0109 -0.009 0.021 rpy=0 0 0
- added joint camera_r_color_frame: type fixed, parent camera_r_base, child camera_r_color_link, origin xyz=0.0109 0.009 0.021 rpy=0 0 0
- added joint camera_r_depth_frame: type fixed, parent camera_r_base, child camera_r_depth_link, origin xyz=0.0109 -0.009 0.021 rpy=0 0 0
- added joint camera_to_realcam_h_frame: type fixed, parent camera, child cam_h_link, origin xyz=0 0 0 rpy=0 0 0
- added joint camera_to_realcam_l_frame: type fixed, parent camera_l_base, child cam_l_link, origin xyz=0.0146 0.00 0.021 rpy=0 0 0
- added joint camera_to_realcam_r_frame: type fixed, parent camera_r_base, child cam_r_link, origin xyz=0.0146 0.00 0.021 rpy=0 0 0
- added joint l_camera_joint: type fixed, parent camera_l_base, child l_d405_camera, origin xyz=0.01085 0.009 0.021 rpy=0 0 0
- added joint l_hand_camera_joint: type fixed, parent zarm_l7_link, child camera_l_base, origin xyz=7.21360860434e-08 0.0334214585163 -0.106588366881 rpy=-3.1416 1.0472 -1.5708
- added joint r_camera_joint: type fixed, parent camera_r_base, child r_d405_camera, origin xyz=0.01085 -0.009 0.021 rpy=0 0 0
- added joint r_hand_camera_joint: type fixed, parent zarm_r7_link, child camera_r_base, origin xyz=-2.36413142634e-07 -0.0334214585174 -0.106588366881 rpy=-3.1416 1.0472 1.5708
- added joint radar: type fixed, parent zhead_1_link, child radar, origin xyz=0 0 -0.078253 rpy=0 0 0, axis 0 0 0
- added joint zarm_l7_end_effector_1_joint: type fixed, parent zarm_l7_link, child zarm_l7_end_effector_1, origin xyz=0 0.0 -0.08 rpy=0 0 0
- added joint zarm_l7_end_effector_2_joint: type fixed, parent zarm_l7_link, child zarm_l7_end_effector_2, origin xyz=0.03 0.0 -0.17 rpy=0 0 0
- added joint zarm_r7_end_effector_1_joint: type fixed, parent zarm_r7_link, child zarm_r7_end_effector_1, origin xyz=0 0.0 -0.08 rpy=0 0 0
- added joint zarm_r7_end_effector_2_joint: type fixed, parent zarm_r7_link, child zarm_r7_end_effector_2, origin xyz=0.03 0.0 -0.17 rpy=0 0 0

File: src/kuavo_assets/models/biped_s400055/urdf/biped_s400055_gazebo.urdf (robot description, URDF)
Before this commit: robot biped_s400055, 74 links, 73 joints
Links:
- added link cam_h_link
- added link cam_l_link
- added link cam_r_link
- added link camera
- added link camera_base, mass 0.00000000; visual mesh filename=package://kuavo_assets/models/biped_s400055/meshes/head_cam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
- added link camera_l_base
- added link camera_l_color_link
- added link camera_l_depth_link
- added link camera_r_base
- added link camera_r_color_link
- added link camera_r_depth_link
- added link radar, mass 0.26500; visual mesh filename=package://kuavo_assets/models/biped_s53/meshes/head_rader.S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
- added link zarm_l7_end_effector_1
- added link zarm_l7_end_effector_2
- added link zarm_r7_end_effector_1
- added link zarm_r7_end_effector_2
Joints:
- added joint camera: type fixed, parent zhead_2_link, child camera, origin xyz=0.099619 0 0.032844 rpy=0 0.3406 0
- added joint camera_base_joint: type fixed, parent zhead_2_link, child camera_base, origin xyz=0.099619 0 0.032844 rpy=0 0.3406 0
- added joint camera_l_color_frame: type fixed, parent camera_l_base, child camera_l_color_link, origin xyz=0.0109 0.009 0.021 rpy=0 0 0
- added joint camera_l_depth_frame: type fixed, parent camera_l_base, child camera_l_depth_link, origin xyz=0.0109 -0.009 0.021 rpy=0 0 0
- added joint camera_r_color_frame: type fixed, parent camera_r_base, child camera_r_color_link, origin xyz=0.0109 0.009 0.021 rpy=0 0 0
- added joint camera_r_depth_frame: type fixed, parent camera_r_base, child camera_r_depth_link, origin xyz=0.0109 -0.009 0.021 rpy=0 0 0
- added joint camera_to_realcam_h_frame: type fixed, parent camera, child cam_h_link, origin xyz=0 0 0 rpy=0 0 0
- added joint camera_to_realcam_l_frame: type fixed, parent camera_l_base, child cam_l_link, origin xyz=0.0146 0.00 0.021 rpy=0 0 0
- added joint camera_to_realcam_r_frame: type fixed, parent camera_r_base, child cam_r_link, origin xyz=0.0146 0.00 0.021 rpy=0 0 0
- added joint l_hand_camera_joint: type fixed, parent zarm_l7_link, child camera_l_base, origin xyz=7.21360860434e-08 0.0334214585163 -0.106588366881 rpy=-3.1416 1.0472 -1.5708
- added joint r_hand_camera_joint: type fixed, parent zarm_r7_link, child camera_r_base, origin xyz=-2.36413142634e-07 -0.0334214585174 -0.106588366881 rpy=-3.1416 1.0472 1.5708
- added joint radar: type fixed, parent zhead_1_link, child radar, origin xyz=0 0 -0.078253 rpy=0 0 0, axis 0 0 0
- added joint zarm_l7_end_effector_1_joint: type fixed, parent zarm_l7_link, child zarm_l7_end_effector_1, origin xyz=0 0.0 -0.08 rpy=0 0 0
- added joint zarm_l7_end_effector_2_joint: type fixed, parent zarm_l7_link, child zarm_l7_end_effector_2, origin xyz=0.03 0.0 -0.17 rpy=0 0 0
- added joint zarm_r7_end_effector_1_joint: type fixed, parent zarm_r7_link, child zarm_r7_end_effector_1, origin xyz=0 0.0 -0.08 rpy=0 0 0
- added joint zarm_r7_end_effector_2_joint: type fixed, parent zarm_r7_link, child zarm_r7_end_effector_2, origin xyz=0.03 0.0 -0.17 rpy=0 0 0

File: src/kuavo_assets/models/biped_s400055/urdf/drake/biped_v3_all_joint.urdf (robot description, URDF)
Before this commit: robot biped_v3_all_joint, 59 links, 54 joints
Links:
- added link cam_l_link
- added link cam_r_link
- added link camera_l_base, mass 0.00010000; visual mesh filename=../../meshes/l_d405_camera_base.STL
- added link camera_l_color_link
- added link camera_l_depth_link
- added link camera_r_base, mass 0.00010000; visual mesh filename=../../meshes/r_d405_camera_base.STL
- added link camera_r_color_link
- added link camera_r_depth_link
- added link l_d405_camera, mass 0.00006545; visual mesh filename=../../meshes/l_d405_camera.STL
- added link r_d405_camera, mass 0.00006545; visual mesh filename=../../meshes/r_d405_camera.STL
- added link zarm_l7_end_effector
- added link zarm_l7_end_effector_1
- added link zarm_l7_end_effector_2
- added link zarm_r7_end_effector
- added link zarm_r7_end_effector_1
- added link zarm_r7_end_effector_2
Joints:
- added joint camera_l_color_frame: type fixed, parent camera_l_base, child camera_l_color_link, origin xyz=0.0109 0.009 0.021 rpy=0 0 0
- added joint camera_l_depth_frame: type fixed, parent camera_l_base, child camera_l_depth_link, origin xyz=0.0109 -0.009 0.021 rpy=0 0 0
- added joint camera_r_color_frame: type fixed, parent camera_r_base, child camera_r_color_link, origin xyz=0.0109 0.009 0.021 rpy=0 0 0
- added joint camera_r_depth_frame: type fixed, parent camera_r_base, child camera_r_depth_link, origin xyz=0.0109 -0.009 0.021 rpy=0 0 0
- added joint camera_to_realcam_l_frame: type fixed, parent camera_l_base, child cam_l_link, origin xyz=0.0146 0.00 0.021 rpy=0 0 0
- added joint camera_to_realcam_r_frame: type fixed, parent camera_r_base, child cam_r_link, origin xyz=0.0146 0.00 0.021 rpy=0 0 0
- added joint l_camera_joint: type fixed, parent camera_l_base, child l_d405_camera, origin xyz=0.01085 0.009 0.021 rpy=0 0 0
- added joint l_hand_camera_joint: type fixed, parent zarm_l7_link, child camera_l_base, origin xyz=7.21360860434e-08 0.0334214585163 -0.106588366881 rpy=-3.1416 1.0472 -1.5708
- added joint r_camera_joint: type fixed, parent camera_r_base, child r_d405_camera, origin xyz=0.01085 -0.009 0.021 rpy=0 0 0
- added joint r_hand_camera_joint: type fixed, parent zarm_r7_link, child camera_r_base, origin xyz=-2.36413142634e-07 -0.0334214585174 -0.106588366881 rpy=-3.1416 1.0472 1.5708
- added joint zarm_l7_end_effector_1_joint: type fixed, parent zarm_l7_link, child zarm_l7_end_effector_1, origin xyz=0 0.0 -0.08 rpy=0 0 0
- added joint zarm_l7_end_effector_2_joint: type fixed, parent zarm_l7_link, child zarm_l7_end_effector_2, origin xyz=0.03 0.0 -0.17 rpy=0 0 0
- added joint zarm_l7_end_effector_joint: type fixed, parent zarm_l7_link, child zarm_l7_end_effector, origin xyz=0 0.0 -0.17 rpy=0 0 0
- added joint zarm_r7_end_effector_1_joint: type fixed, parent zarm_r7_link, child zarm_r7_end_effector_1, origin xyz=0 0.0 -0.08 rpy=0 0 0
- added joint zarm_r7_end_effector_2_joint: type fixed, parent zarm_r7_link, child zarm_r7_end_effector_2, origin xyz=0.03 0.0 -0.17 rpy=0 0 0
- added joint zarm_r7_end_effector_joint: type fixed, parent zarm_r7_link, child zarm_r7_end_effector, origin xyz=0 0.0 -0.17 rpy=0 0 0

File: src/kuavo_assets/models/biped_s400055/urdf/drake/biped_v3_arm.urdf (robot description, URDF)
Before this commit: robot biped_s400055, 44 links, 43 joints
Links:
- added link cam_l_link
- added link cam_r_link
- added link camera_l_base, mass 0.00010000; visual mesh filename=../../meshes/l_d405_camera_base.STL
- added link camera_l_color_link
- added link camera_l_depth_link
- added link camera_r_base, mass 0.00010000; visual mesh filename=../../meshes/r_d405_camera_base.STL
- added link camera_r_color_link
- added link camera_r_depth_link
- added link l_d405_camera, mass 0.00006545; visual mesh filename=../../meshes/l_d405_camera.STL
- added link r_d405_camera, mass 0.00006545; visual mesh filename=../../meshes/r_d405_camera.STL
- added link zarm_l7_end_effector_1
- added link zarm_l7_end_effector_2
- added link zarm_r7_end_effector_1
- added link zarm_r7_end_effector_2
Joints:
- added joint camera_l_color_frame: type fixed, parent camera_l_base, child camera_l_color_link, origin xyz=0.0109 0.009 0.021 rpy=0 0 0
- added joint camera_l_depth_frame: type fixed, parent camera_l_base, child camera_l_depth_link, origin xyz=0.0109 -0.009 0.021 rpy=0 0 0
- added joint camera_r_color_frame: type fixed, parent camera_r_base, child camera_r_color_link, origin xyz=0.0109 0.009 0.021 rpy=0 0 0
- added joint camera_r_depth_frame: type fixed, parent camera_r_base, child camera_r_depth_link, origin xyz=0.0109 -0.009 0.021 rpy=0 0 0
- added joint camera_to_realcam_l_frame: type fixed, parent camera_l_base, child cam_l_link, origin xyz=0.0146 0.00 0.021 rpy=0 0 0
- added joint camera_to_realcam_r_frame: type fixed, parent camera_r_base, child cam_r_link, origin xyz=0.0146 0.00 0.021 rpy=0 0 0
- added joint l_camera_joint: type fixed, parent camera_l_base, child l_d405_camera, origin xyz=0.01085 0.009 0.021 rpy=0 0 0
- added joint l_hand_camera_joint: type fixed, parent zarm_l7_link, child camera_l_base, origin xyz=7.21360860434e-08 0.0334214585163 -0.106588366881 rpy=-3.1416 1.0472 -1.5708
- added joint r_camera_joint: type fixed, parent camera_r_base, child r_d405_camera, origin xyz=0.01085 -0.009 0.021 rpy=0 0 0
- added joint r_hand_camera_joint: type fixed, parent zarm_r7_link, child camera_r_base, origin xyz=-2.36413142634e-07 -0.0334214585174 -0.106588366881 rpy=-3.1416 1.0472 1.5708
- added joint zarm_l7_end_effector_1_joint: type fixed, parent zarm_l7_link, child zarm_l7_end_effector_1, origin xyz=0 0.0 -0.08 rpy=0 0 0
- added joint zarm_l7_end_effector_2_joint: type fixed, parent zarm_l7_link, child zarm_l7_end_effector_2, origin xyz=0.03 0.0 -0.17 rpy=0 0 0
- added joint zarm_r7_end_effector_1_joint: type fixed, parent zarm_r7_link, child zarm_r7_end_effector_1, origin xyz=0 0.0 -0.08 rpy=0 0 0
- added joint zarm_r7_end_effector_2_joint: type fixed, parent zarm_r7_link, child zarm_r7_end_effector_2, origin xyz=0.03 0.0 -0.17 rpy=0 0 0

File: src/kuavo_assets/models/biped_s400055/urdf/drake/biped_v3_full.urdf (robot description, URDF)
Before this commit: robot biped_s400055, 56 links, 55 joints
Links:
- added link cam_h_link
- added link cam_l_link
- added link cam_r_link
- added link camera, mass 0.0400617267216207; visual mesh filename=../../meshes/head_camera.STL
- added link camera_base, mass 0.00000000; visual mesh filename=../../meshes/head_camera_base.STL
- added link camera_l_base, mass 0.00010000; visual mesh filename=../../meshes/l_d405_camera_base.STL
- added link camera_l_color_link
- added link camera_l_depth_link
- added link camera_r_base, mass 0.00010000; visual mesh filename=../../meshes/r_d405_camera_base.STL
- added link camera_r_color_link
- added link camera_r_depth_link
- added link head_camera_depth, mass 0.0000785398163397463; visual mesh filename=../../meshes/head_camera_depth.STL
- added link l_d405_camera, mass 0.00006545; visual mesh filename=../../meshes/l_d405_camera.STL
- added link r_d405_camera, mass 0.00006545; visual mesh filename=../../meshes/r_d405_camera.STL
- added link radar, mass 0.00000; visual mesh filename=../../meshes/head_rader.STL
- added link zarm_l7_end_effector
- added link zarm_l7_end_effector_1
- added link zarm_l7_end_effector_2
- added link zarm_r7_end_effector
- added link zarm_r7_end_effector_1
- added link zarm_r7_end_effector_2
Joints:
- added joint camera: type fixed, parent zhead_2_link, child camera, origin xyz=0.099619 0 0.032844 rpy=0 0.3406 0
- added joint camera_base_joint: type fixed, parent zhead_2_link, child camera_base, origin xyz=0.099619 0 0.032844 rpy=0 0.3406 0
- added joint camera_l_color_frame: type fixed, parent camera_l_base, child camera_l_color_link, origin xyz=0.0109 0.009 0.021 rpy=0 0 0
- added joint camera_l_depth_frame: type fixed, parent camera_l_base, child camera_l_depth_link, origin xyz=0.0109 -0.009 0.021 rpy=0 0 0
- added joint camera_r_color_frame: type fixed, parent camera_r_base, child camera_r_color_link, origin xyz=0.0109 0.009 0.021 rpy=0 0 0
- added joint camera_r_depth_frame: type fixed, parent camera_r_base, child camera_r_depth_link, origin xyz=0.0109 -0.009 0.021 rpy=0 0 0
- added joint camera_to_realcam_h_frame: type fixed, parent camera, child cam_h_link, origin xyz=0 0 0 rpy=0 0 0
- added joint camera_to_realcam_l_frame: type fixed, parent camera_l_base, child cam_l_link, origin xyz=0.0146 0.00 0.021 rpy=0 0 0
- added joint camera_to_realcam_r_frame: type fixed, parent camera_r_base, child cam_r_link, origin xyz=0.0146 0.00 0.021 rpy=0 0 0
- added joint head_camera_depth_joint: type fixed, parent camera, child head_camera_depth, origin xyz=0.011715 0.0475 0.014312 rpy=0 0 0
- added joint l_camera_joint: type fixed, parent camera_l_base, child l_d405_camera, origin xyz=0.01085 0.009 0.021 rpy=0 0 0
- added joint l_hand_camera_joint: type fixed, parent zarm_l7_link, child camera_l_base, origin xyz=7.21360860434e-08 0.0334214585163 -0.106588366881 rpy=-3.1416 1.0472 -1.5708
- added joint r_camera_joint: type fixed, parent camera_r_base, child r_d405_camera, origin xyz=0.01085 -0.009 0.021 rpy=0 0 0
- added joint r_hand_camera_joint: type fixed, parent zarm_r7_link, child camera_r_base, origin xyz=-2.36413142634e-07 -0.0334214585174 -0.106588366881 rpy=-3.1416 1.0472 1.5708
- added joint radar: type fixed, parent zhead_1_link, child radar, origin xyz=0 0 -0.078253 rpy=0 0 0
- added joint zarm_l7_end_effector_1_joint: type fixed, parent zarm_l7_link, child zarm_l7_end_effector_1, origin xyz=0 0.0 -0.08 rpy=0 0 0
- added joint zarm_l7_end_effector_2_joint: type fixed, parent zarm_l7_link, child zarm_l7_end_effector_2, origin xyz=0.03 0.0 -0.17 rpy=0 0 0
- added joint zarm_l7_end_effector_joint: type fixed, parent zarm_l7_link, child zarm_l7_end_effector, origin xyz=0 0.0 -0.17 rpy=0 0 0
- added joint zarm_r7_end_effector_1_joint: type fixed, parent zarm_r7_link, child zarm_r7_end_effector_1, origin xyz=0 0.0 -0.08 rpy=0 0 0
- added joint zarm_r7_end_effector_2_joint: type fixed, parent zarm_r7_link, child zarm_r7_end_effector_2, origin xyz=0.03 0.0 -0.17 rpy=0 0 0
- added joint zarm_r7_end_effector_joint: type fixed, parent zarm_r7_link, child zarm_r7_end_effector, origin xyz=0 0.0 -0.17 rpy=0 0 0

File: src/kuavo_assets/models/biped_s400062/urdf/biped_s400062.urdf (robot description, URDF)
Before this commit: robot biped_s400062, 69 links, 68 joints
Joints:
- joint waist_yaw_joint: origin xyz=0 0 0.235 rpy=0 0 0 -> xyz=0 0 0.250 rpy=0 0 0

File: src/kuavo_assets/models/biped_s400062/urdf/biped_s400062_gazebo.urdf (robot description, URDF)
Before this commit: robot biped_s400062, 72 links, 71 joints
Joints:
- joint waist_yaw_joint: origin xyz=0 0 0.235 rpy=0 0 0 -> xyz=0 0 0.250 rpy=0 0 0

File: src/kuavo_assets/models/biped_s400062/urdf/drake/biped_v3_arm.urdf (robot description, URDF)
Before this commit: robot biped_s400062, 52 links, 51 joints
Joints:
- joint waist_yaw_joint: origin xyz=0 0 0.235 rpy=0 0 0 -> xyz=0 0 0.250 rpy=0 0 0

File: src/kuavo_assets/models/biped_s400062/urdf/drake/biped_v3_arm_only.urdf (robot description, URDF)
Before this commit: robot biped_s400062, 52 links, 51 joints
Joints:
- joint waist_yaw_joint: origin xyz=0 0 0.235 rpy=0 0 0 -> xyz=0 0 0.250 rpy=0 0 0

File: src/kuavo_assets/models/biped_s500062/urdf/biped_s500062.urdf (robot description, URDF)
Before this commit: robot biped_s500062, 73 links, 72 joints
Joints:
- joint waist_yaw_joint: origin xyz=0 0 0.235 rpy=0 0 0 -> xyz=0 0 0.250 rpy=0 0 0

File: src/kuavo_assets/models/biped_s500062/urdf/biped_s500062_gazebo.urdf (robot description, URDF)
Before this commit: robot biped_s500062, 76 links, 75 joints
Joints:
- joint waist_yaw_joint: origin xyz=0 0 0.235 rpy=0 0 0 -> xyz=0 0 0.250 rpy=0 0 0

File: src/kuavo_assets/models/biped_s500062/urdf/drake/biped_v3_arm.urdf (robot description, URDF)
Before this commit: robot biped_s500062, 52 links, 51 joints
Joints:
- joint waist_yaw_joint: origin xyz=0 0 0.235 rpy=0 0 0 -> xyz=0 0 0.250 rpy=0 0 0

File: src/kuavo_assets/models/biped_s500062/urdf/drake/biped_v3_arm_only.urdf (robot description, URDF)
Before this commit: robot biped_s500062, 52 links, 51 joints
Joints:
- joint waist_yaw_joint: origin xyz=0 0 0.235 rpy=0 0 0 -> xyz=0 0 0.250 rpy=0 0 0
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