Commit message: sync https://www.lejuhub.com/highlydynamic/kuavo-ros-control/commit/f643e5d04c0f1a23596abbacea3be65c2b99ead0

File: src/kuavo_assets/models/biped_s52/urdf/biped_s52.urdf (robot description, URDF)
Before this commit: robot biped_s52, 47 links, 46 joints
Links:
- link waist_yaw_link: mass 18.01415568 -> 22.01415568

File: src/kuavo_assets/models/biped_s52/urdf/biped_s52_gazebo.urdf (robot description, URDF)
Before this commit: robot biped_s52, 47 links, 46 joints
Links:
- link waist_yaw_link: mass 18.01415568 -> 22.01415568

File: src/kuavo_assets/models/biped_s52/urdf/drake/biped_v3.urdf (robot description, URDF)
Before this commit: robot biped_v3, 14 links, 13 joints
Links:
- link torso: mass 18.99013928 -> 6.99013928
- link waist_yaw_link: mass 18.01415568 -> 34.01415568

File: src/kuavo_assets/models/biped_s52/urdf/drake/biped_v3_all_joint.urdf (robot description, URDF)
Before this commit: robot biped_v3_all_joint, 35 links, 30 joints
Links:
- link torso: mass 33.93314316 -> 37.93314316

File: src/kuavo_assets/models/biped_s52/urdf/drake/biped_v3_full.urdf (robot description, URDF)
Before this commit: robot biped_s52, 32 links, 31 joints
Links:
- link waist_yaw_link: mass 18.01415568 -> 22.07055568

Commit message: sync https://www.lejuhub.com/highlydynamic/kuavo-ros-control/commit/087367adf6670419e4651555bb34fec8ce958ffd

File: src/kuavo_assets/models/biped_s52/urdf/biped_s52.urdf (robot description, URDF)
Before this commit: robot biped_s52, 47 links, 46 joints
Links:
- link base_link: mass 9.69103928 -> 6.69103928
- link waist_yaw_link: mass 18.01415568 -> 21.61115568

File: src/kuavo_assets/models/biped_s52/urdf/biped_s52_gazebo.urdf (robot description, URDF)
Before this commit: robot biped_s52, 47 links, 46 joints
Links:
- link base_link: mass 9.50123928 -> 6.50123928
- link waist_yaw_link: mass 18.01415568 -> 21.61115568

File: src/kuavo_assets/models/biped_s52/urdf/drake/biped_v3.urdf (robot description, URDF)
Before this commit: robot biped_v3, 14 links, 13 joints
Links:
- link torso: mass 22.39313928 -> 6.99013928
- link waist_yaw_link: mass 18.01415568 -> 34.01415568

File: src/kuavo_assets/models/biped_s52/urdf/drake/biped_v3_all_joint.urdf (robot description, URDF)
Before this commit: robot biped_v3_all_joint, 35 links, 30 joints
Links:
- link torso: mass 37.33614316 -> 37.93314316

Commit message: sync https://www.lejuhub.com/highlydynamic/kuavo-ros-control/commit/54a0b4a65756afa80f4b8838e8d538d4186c01f4

File: src/kuavo_assets/models/biped_s52/urdf/biped_s52.urdf (robot description, URDF)
Before this commit: robot biped_s52, 47 links, 46 joints
Links:
- added link head_rader, mass 0.26500; visual mesh filename=package://kuavo_assets/models/biped_s52/meshes/head_rader.S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
- link base_link: mass 6.69103928 -> 7.06405; geometry collision cylinder length=0.24 radius=0.06; collision cylinder length=0.24 radius=0.06
- link camera_base: mass 0.0482361371130408 -> 0.00000000
- link leg_l1_link: mass 1.63858534 -> 1.55641
- link leg_l2_link: mass 0.70575545 -> 0.75873
- link leg_l3_link: mass 5.93791258 -> 6.68074
- link leg_l4_link: mass 4.02498548 -> 3.64666
- link leg_l5_link: mass 0.07848005 -> 0.07848
- link leg_l6_link: mass 0.58491513 -> 0.69242
- link leg_r1_link: mass 1.63861324 -> 1.55641
- link leg_r2_link: mass 0.70575545 -> 0.75873
- link leg_r3_link: mass 5.93791831 -> 6.68074
- link leg_r4_link: mass 4.02498548 -> 3.64666
- link leg_r5_link: mass 0.07848005 -> 0.07848
- link leg_r6_link: mass 0.58491513 -> 0.69242
- link waist_yaw_link: mass 21.61115568 -> 20.63616
- link zarm_l1_link: mass 0.91653322 -> 0.94521
- link zarm_l2_link: mass 0.38767390 -> 0.41921
- link zarm_l3_link: mass 1.77926875 -> 1.78857
- link zarm_l4_link: mass 0.58507821 -> 0.63149
- link zarm_l5_link: mass 0.68679955 -> 0.60828
- link zarm_l6_link: mass 0.39387181 -> 0.50616
- link zarm_l7_link: mass 0.71537800 -> 0.18940
- link zarm_r1_link: mass 0.91653322 -> 0.92947
- link zarm_r2_link: mass 0.38767390 -> 0.41523
- link zarm_r3_link: mass 1.77926875 -> 1.78473
- link zarm_r4_link: mass 0.58507821 -> 0.63548
- link zarm_r5_link: mass 0.68679955 -> 0.61021
- link zarm_r6_link: mass 0.39387181 -> 0.53821
- link zarm_r7_link: mass 0.71537800 -> 0.19960
- link zhead_1_link: mass 0.87117795 -> 0.57250
- link zhead_2_link: mass 0.80529305 -> 0.73448
Joints:
- added joint head_rader_joint: type fixed, parent zhead_1_link, child head_rader, origin xyz=0 0 -0.078253 rpy=0 0 0, axis 0 0 0
- joint camera_base: origin xyz=0.119717018973535 0.0237514612535074 0.0262044145991832 rpy=0 0.480224871300295 0 -> xyz=0.093839 0.0475 0.050077 rpy=0 0.3406 0
- joint leg_l4_joint: origin xyz=0 0 -0.284 rpy=0 0 0 -> xyz=-0.0011639 0 -0.284 rpy=0 0 0
- joint leg_l5_joint: origin xyz=0.002 0.0003 -0.416 rpy=0 0 0 -> xyz=0.002 0 -0.416 rpy=0 0 0
- joint leg_r4_joint: origin xyz=0 0 -0.284 rpy=0 0 0 -> xyz=-0.0011639 0 -0.284 rpy=0 0 0
- joint leg_r5_joint: origin xyz=0.00199999999983541 -0.000300000028212572 -0.415999999987417 rpy=0 0 0 -> xyz=0.002 0 -0.416 rpy=0 0 0
- joint waist_yaw_joint: origin xyz=0 0 0.1114 rpy=0 0 0 -> xyz=0 0 0.1115 rpy=0 0 0
- joint zarm_l1_joint: origin xyz=0 0.2527 0.2831 rpy=0 0 0 -> xyz=-0.003 0.2527 0.283 rpy=0 0 0
- joint zarm_l5_joint: origin xyz=-0.02 0 -0.1195 rpy=0 0 0 -> xyz=-0.02 0 -0.1201 rpy=0 0 0
- joint zarm_r1_joint: origin xyz=0 -0.2527 0.2831 rpy=0 0 0 -> xyz=-0.003 -0.2527 0.283 rpy=0 0 0
- joint zarm_r5_joint: origin xyz=-0.02 0 -0.1195 rpy=0 0 0 -> xyz=-0.02 0 -0.1201 rpy=0 0 0
- joint zhead_1_joint: origin xyz=-0.003 0.0 0.3715 rpy=0 0 0 -> xyz=-0.003 0.0 0.49535 rpy=0 0 0
- joint zhead_2_joint: origin xyz=0 0 0.137954074182872 rpy=0 0 0 -> xyz=0 0 0 rpy=0 0 0

File: src/kuavo_assets/models/biped_s52/urdf/biped_s52_gazebo.urdf (robot description, URDF)
Before this commit: robot biped_s52, 47 links, 46 joints
Links:
- link waist_yaw_link: mass 21.61115568 -> 21.01415568

File: src/kuavo_assets/models/biped_s52/urdf/drake/biped_v3.urdf (robot description, URDF)
Before this commit: robot biped_v3, 14 links, 13 joints
Links:
- link waist_yaw_link: mass 34.01415568 -> 33.41715568

File: src/kuavo_assets/models/biped_s52/urdf/drake/biped_v3_all_joint.urdf (robot description, URDF)
Before this commit: robot biped_v3_all_joint, 35 links, 30 joints
Links:
- link torso: mass 37.93314316 -> 37.33614316

File: src/kuavo_assets/models/biped_s52/urdf/drake/biped_v3_full.urdf (robot description, URDF)
Before this commit: robot biped_s52, 32 links, 31 joints
Links:
- link waist_yaw_link: mass 22.07055568 -> 21.47355568
