Commit message: sync https://www.lejuhub.com/highlydynamic/kuavo-ros-control/commit/9d19635bafeabe2c52050378b3e6927c0fa8ace9

File: src/kuavo_assets/models/biped_s52/urdf/biped_s52.urdf (robot description, URDF)
Before this commit: robot biped_s52, 48 links, 47 joints
Joints:
- joint leg_l5_joint: limit lower=-0.872664625997165 upper=0.349065850398866 effort=57.0 velocity=17.8 -> lower=-0.872664625997165 upper=0.349065850398866 effort=102.6 velocity=17.8
- joint leg_l6_joint: limit lower=-0.261799387799149 upper=0.261799387799149 effort=57.0 velocity=17.8 -> lower=-0.261799387799149 upper=0.261799387799149 effort=102.6 velocity=17.8
- joint leg_r5_joint: limit lower=-0.872664625997165 upper=0.349065850398866 effort=57.0 velocity=17.8 -> lower=-0.872664625997165 upper=0.349065850398866 effort=102.6 velocity=17.8
- joint leg_r6_joint: limit lower=-0.261799387799149 upper=0.261799387799149 effort=57.0 velocity=17.8 -> lower=-0.261799387799149 upper=0.261799387799149 effort=102.6 velocity=17.8
- joint waist_yaw_joint: origin xyz=0 0 0.1115 rpy=0 0 0 -> xyz=0 0 0.1114 rpy=0 0 0

File: src/kuavo_assets/models/biped_s52/urdf/biped_s52_gazebo.urdf (robot description, URDF)
Before this commit: robot biped_s52, 47 links, 46 joints
Links:
- added link head_rader, mass 0.26500; visual mesh filename=package://kuavo_assets/models/biped_s52/meshes/head_rader.S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
- link base_link: mass 6.50123928 -> 7.06405; geometry visual mesh filename=package://kuavo_assets/models/biped_s52/meshes/torso.STL
- link camera_base: mass 0.0482361371130408 -> 0.00000000
- link leg_l1_link: mass 1.63858534 -> 1.55641
- link leg_l2_link: mass 0.70575545 -> 0.75873
- link leg_l3_link: mass 5.93791258 -> 6.68074
- link leg_l4_link: mass 4.02498548 -> 3.64666
- link leg_l5_link: mass 0.07848005 -> 0.07848
- link leg_l6_link: mass 0.58491513 -> 0.69242
- link leg_r1_link: mass 1.63861324 -> 1.55641
- link leg_r2_link: mass 0.70575545 -> 0.75873
- link leg_r3_link: mass 5.93791831 -> 6.68074
- link leg_r4_link: mass 4.02498548 -> 3.64666
- link leg_r5_link: mass 0.07848005 -> 0.07848
- link leg_r6_link: mass 0.58491513 -> 0.69242
- link waist_camera: mass 0.237986769607677 -> 0.048238; geometry visual mesh filename=package://kuavo_assets/models/biped_s52/meshes/waist_camera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
- link waist_yaw_link: mass 21.01415568 -> 20.63616
- link zarm_l1_link: mass 0.91653322 -> 0.94521
- link zarm_l2_link: mass 0.38767390 -> 0.41921
- link zarm_l3_link: mass 1.77926875 -> 1.78857
- link zarm_l4_link: mass 0.58507821 -> 0.63149
- link zarm_l5_link: mass 0.68679955 -> 0.60828
- link zarm_l6_link: mass 0.39387181 -> 0.50616
- link zarm_l7_link: mass 0.71537800 -> 0.18940
- link zarm_r1_link: mass 0.91653322 -> 0.92947
- link zarm_r2_link: mass 0.38767390 -> 0.41523
- link zarm_r3_link: mass 1.77926875 -> 1.78473
- link zarm_r4_link: mass 0.58507821 -> 0.63548
- link zarm_r5_link: mass 0.68679955 -> 0.61021
- link zarm_r6_link: mass 0.39387181 -> 0.53821
- link zarm_r7_end_effector: geometry 
- link zarm_r7_link: mass 0.71537800 -> 0.19960
- link zhead_1_link: mass 0.87117795 -> 0.57250
- link zhead_2_link: mass 0.80529305 -> 0.73448
Joints:
- added joint head_rader_joint: type fixed, parent zhead_1_link, child head_rader, origin xyz=0 0 -0.078253 rpy=0 0 0, axis 0 0 0
- joint camera_base: origin xyz=0.119717018973535 0.0237514612535074 0.0262044145991832 rpy=0 0.480224871300295 0 -> xyz=0.093839 0.0475 0.050077 rpy=0 0.3406 0
- joint leg_l4_joint: origin xyz=0 0 -0.284 rpy=0 0 0 -> xyz=-0.0011639 0 -0.284 rpy=0 0 0
- joint leg_l5_joint: limit lower=-0.872664625997165 upper=0.349065850398866 effort=57.0 velocity=17.8 -> lower=-0.872664625997165 upper=0.349065850398866 effort=102.6 velocity=17.8; origin xyz=0.002 0.0003 -0.416 rpy=0 0 0 -> xyz=0.002 0 -0.416 rpy=0 0 0
- joint leg_l6_joint: limit lower=-0.261799387799149 upper=0.261799387799149 effort=57.0 velocity=17.8 -> lower=-0.261799387799149 upper=0.261799387799149 effort=102.6 velocity=17.8
- joint leg_r4_joint: origin xyz=0 0 -0.284 rpy=0 0 0 -> xyz=-0.0011639 0 -0.284 rpy=0 0 0
- joint leg_r5_joint: limit lower=-0.872664625997165 upper=0.349065850398866 effort=57.0 velocity=17.8 -> lower=-0.872664625997165 upper=0.349065850398866 effort=102.6 velocity=17.8; origin xyz=0.00199999999983541 -0.000300000028212572 -0.415999999987417 rpy=0 0 0 -> xyz=0.002 0 -0.416 rpy=0 0 0
- joint leg_r6_joint: limit lower=-0.261799387799149 upper=0.261799387799149 effort=57.0 velocity=17.8 -> lower=-0.261799387799149 upper=0.261799387799149 effort=102.6 velocity=17.8
- joint waist_camera: origin xyz=0 0 0 rpy=0 0 0 -> xyz=0.0787 0 -0.028449 rpy=0 0.59341 0; parent base_link -> waist_yaw_link
- joint zarm_l1_joint: origin xyz=0 0.2527 0.2831 rpy=0 0 0 -> xyz=-0.003 0.2527 0.283 rpy=0 0 0
- joint zarm_l5_joint: origin xyz=-0.02 0 -0.1195 rpy=0 0 0 -> xyz=-0.02 0 -0.1201 rpy=0 0 0
- joint zarm_r1_joint: origin xyz=0 -0.2527 0.2831 rpy=0 0 0 -> xyz=-0.003 -0.2527 0.283 rpy=0 0 0
- joint zarm_r5_joint: origin xyz=-0.02 0 -0.1195 rpy=0 0 0 -> xyz=-0.02 0 -0.1201 rpy=0 0 0
- joint zhead_1_joint: origin xyz=-0.003 0.0 0.3715 rpy=0 0 0 -> xyz=-0.003 0.0 0.49535 rpy=0 0 0
- joint zhead_2_joint: limit lower=-0.349065850398866 upper=0.785398163397448 effort=12.0 velocity=5.23 -> lower=-0.523598775598299 upper=0.523598775598299 effort=12.0 velocity=5.23; origin xyz=0 0 0.137954074182872 rpy=0 0 0 -> xyz=0 0 0 rpy=0 0 0

File: src/kuavo_assets/models/biped_s52/urdf/drake/biped_v3.urdf (robot description, URDF)
Before this commit: robot biped_v3, 14 links, 13 joints
Links:
- link leg_l1_link: mass 1.63858534 -> 1.55641
- link leg_l2_link: mass 0.70575545 -> 0.75873
- link leg_l3_link: mass 5.93791258 -> 6.68074
- link leg_l4_link: mass 4.02498548 -> 3.64666
- link leg_l5_link: mass 0.07848005 -> 0.07848
- link leg_l6_link: mass 0.58491513 -> 0.69242
- link leg_r1_link: mass 1.63861324 -> 1.55641
- link leg_r2_link: mass 0.70575545 -> 0.75873
- link leg_r3_link: mass 5.93791831 -> 6.68074; geometry visual mesh filename=package://kuavo_assets/models/biped_s52/meshes/r_leg_pitch.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
- link leg_r4_link: mass 4.02498548 -> 3.64666
- link leg_r5_link: mass 0.07848005 -> 0.07848
- link leg_r6_link: mass 0.58491513 -> 0.69242
- link torso: mass 6.99013928 -> 7.06405; geometry visual mesh filename=../../meshes/torso.STL
- link waist_yaw_link: mass 33.41715568 -> 32.45766
Joints:
- joint leg_l1_joint: limit lower=-0.314159265358979 upper=0.663225115757845 effort=180.0 velocity=23.55 -> lower=-0.314159265358979 upper=0.663225115757845 effort=127.0 velocity=10.4
- joint leg_l2_joint: limit lower=-1.91986217719376 upper=0.785398163397448 effort=100.0 velocity=41.3433333333333 -> lower=-0.785398163397448 upper=1.91986217719376 effort=71.0 velocity=8.7
- joint leg_l3_joint: limit lower=-1.91986217719376 upper=1.5707963267949 effort=100.0 velocity=41.3433333333333 -> lower=-1.91986217719376 upper=1.5707963267949 effort=132 velocity=12.7
- joint leg_l4_joint: limit lower=0.0 upper=2.53072741539178 effort=180.0 velocity=23.55 -> lower=0.0 upper=2.53072741539178 effort=280.0 velocity=10.4; origin xyz=0 0 -0.284 rpy=0 0 0 -> xyz=-0.0011639 0 -0.284 rpy=0 0 0
- joint leg_l5_joint: limit lower=-0.872664625997165 upper=0.349065850398866 effort=36.0 velocity=23.0266666666667 -> lower=-0.872664625997165 upper=0.349065850398866 effort=102.6 velocity=17.8; origin xyz=0.002 0.0003 -0.416 rpy=0 0 0 -> xyz=0.002 0 -0.416 rpy=0 0 0
- joint leg_l6_joint: limit lower=-0.261799387799149 upper=0.261799387799149 effort=36.0 velocity=23.0266666666667 -> lower=-0.261799387799149 upper=0.261799387799149 effort=102.6 velocity=17.8
- joint leg_r1_joint: limit lower=-0.663225115757845 upper=0.314159265358979 effort=180.0 velocity=23.55 -> lower=-0.663225115757845 upper=0.314159265358979 effort=127.0 velocity=10.4
- joint leg_r2_joint: limit lower=-0.785398163397448 upper=1.91986217719376 effort=100.0 velocity=41.3433333333333 -> lower=-1.91986217719376 upper=0.785398163397448 effort=71.0 velocity=8.7
- joint leg_r3_joint: limit lower=-1.91986217719376 upper=1.5707963267949 effort=100.0 velocity=41.3433333333333 -> lower=-1.91986217719376 upper=1.5707963267949 effort=132.0 velocity=12.7
- joint leg_r4_joint: limit lower=0.0 upper=2.53072741539178 effort=180.0 velocity=23.55 -> lower=0.0 upper=2.53072741539178 effort=280.0 velocity=10.4; origin xyz=0 0 -0.284 rpy=0 0 0 -> xyz=-0.0011639 0 -0.284 rpy=0 0 0
- joint leg_r5_joint: limit lower=-0.872664625997165 upper=0.349065850398866 effort=36.0 velocity=23.0266666666667 -> lower=-0.872664625997165 upper=0.349065850398866 effort=102.6 velocity=17.8; origin xyz=0.00199999999983541 -0.000300000028212572 -0.415999999987417 rpy=0 0 0 -> xyz=0.002 0 -0.416 rpy=0 0 0
- joint leg_r6_joint: limit lower=-0.261799387799149 upper=0.261799387799149 effort=36.0 velocity=23.0266666666667 -> lower=-0.261799387799149 upper=0.261799387799149 effort=102.6 velocity=17.8
- joint waist_yaw_joint: limit lower=-2.0943951023932 upper=2.0943951023932 effort=180.0 velocity=23.55 -> lower=-3.14159 upper=3.14159 effort=102.0 velocity=8.7

File: src/kuavo_assets/models/biped_s52/urdf/drake/biped_v3_arm.urdf (robot description, URDF)
Before this commit: robot biped_s52, 20 links, 19 joints
Links:
- link base_link: mass 6.48663928 -> 7.06405; geometry visual mesh filename=../../meshes/torso.STL
- link waist_yaw_link: mass 18.01415568 -> 20.63616
- link zarm_l1_link: mass 0.91653322 -> 0.94521
- link zarm_l2_link: mass 0.3876739 -> 0.41921
- link zarm_l3_link: mass 1.77926875 -> 1.78857
- link zarm_l4_link: mass 0.58507821 -> 0.63149
- link zarm_l5_link: mass 0.68679955 -> 0.60828
- link zarm_l6_link: mass 0.39387181 -> 0.50616
- link zarm_l7_end_effector: geometry 
- link zarm_l7_link: mass 0.61537779 -> 0.18940
- link zarm_r1_link: mass 0.92062797 -> 0.92947
- link zarm_r2_link: mass 0.38768053 -> 0.41523
- link zarm_r3_link: mass 1.77969208 -> 1.78473
- link zarm_r4_link: mass 0.58514611 -> 0.63548
- link zarm_r5_link: mass 0.68473867 -> 0.61021
- link zarm_r6_link: mass 0.39247462 -> 0.53821
- link zarm_r7_end_effector: geometry 
- link zarm_r7_link: mass 0.61562202 -> 0.19960
Joints:
- joint waist_yaw_joint: limit lower=-3.14159 upper=3.14159 effort=180.0 velocity=23.55 -> lower=-3.14159 upper=3.14159 effort=102.0 velocity=8.7
- joint zarm_l1_joint: limit lower=-3.14159265358979 upper=1.5707963267949 effort=100.0 velocity=41.3433333333333 -> lower=-3.14159265358979 upper=1.5707963267949 effort=66.0 velocity=18.8; origin xyz=-0.003 0.1737 0.2831 rpy=0 0 0 -> xyz=-0.003 0.2527 0.283 rpy=0 0 0
- joint zarm_l2_joint: limit lower=-0.349065850398866 upper=2.0943951023932 effort=50.0 velocity=8.37333333333333 -> lower=-0.349065850398866 upper=3.49065850398866 effort=75.0 velocity=8.0; origin xyz=0 0.081 0 rpy=0 0 0 -> xyz=0 0 0 rpy=0 0 0
- joint zarm_l3_joint: limit lower=-1.5707963267949 upper=1.5707963267949 effort=36.0 velocity=9.94333333333333 -> lower=-1.48352986419518 upper=1.48352986419518 effort=57.0 velocity=7.5; origin xyz=0 0 -0.104 rpy=0 0 0 -> xyz=0 0 0 rpy=0 0 0
- joint zarm_l4_joint: limit lower=-2.61799387799149 upper=0.0 effort=50.0 velocity=8.37333333333333 -> lower=-2.61799387799149 upper=0.0 effort=75.0 velocity=8.0; origin xyz=0.02 0 -0.1797 rpy=0 0 0 -> xyz=0.02 0 -0.2837 rpy=0 0 0
- joint zarm_l5_joint: limit lower=-1.5707963267949 upper=1.5707963267949 effort=12.0 velocity=7.32666666666667 -> lower=-1.5707963267949 upper=1.5707963267949 effort=14.1 velocity=17.5; origin xyz=-0.02 0 -0.1195 rpy=0 0 0 -> xyz=-0.02 0 -0.1201 rpy=0 0 0
- joint zarm_l6_joint: limit lower=-1.30899693899575 upper=0.698131700797732 effort=12.0 velocity=7.32666666666667 -> lower=-1.30899693899575 upper=0.698131700797732 effort=14.1 velocity=17.5; origin xyz=0 0 -0.114 rpy=0 0 0 -> xyz=0.0 0 -0.114 rpy=0 0 0
- joint zarm_l7_end_effector_joint: origin xyz=0 -0.03 -0.17 rpy=0 0 0 -> xyz=0 0.0 -0.17 rpy=0 0 0
- joint zarm_l7_joint: limit lower=-0.698131700797732 upper=0.698131700797732 effort=12.0 velocity=7.32666666666667 -> lower=-0.698131700797732 upper=0.698131700797732 effort=14.1 velocity=17.5; origin xyz=-0.0002 0 -0.021 rpy=0 0 0 -> xyz=0 0 -0.021 rpy=0 0 0
- joint zarm_r1_joint: limit lower=-3.14159265358979 upper=1.5707963267949 effort=100.0 velocity=41.3433333333333 -> lower=-3.14159265358979 upper=1.5707963267949 effort=66.0 velocity=18.8; origin xyz=-0.003 -0.1737 0.2831 rpy=0 0 0 -> xyz=-0.003 -0.2527 0.283 rpy=0 0 0
- joint zarm_r2_joint: limit lower=-2.0943951023932 upper=0.349065850398866 effort=50.0 velocity=8.37333333333333 -> lower=-3.49065850398866 upper=0.349065850398866 effort=75.0 velocity=8.0; origin xyz=0 -0.081 0 rpy=0 0 0 -> xyz=0 0 0 rpy=0 0 0
- joint zarm_r3_joint: limit lower=-1.5707963267949 upper=1.5707963267949 effort=36.0 velocity=9.94333333333333 -> lower=-1.48352986419518 upper=1.48352986419518 effort=57.0 velocity=7.5; origin xyz=0 0 -0.104 rpy=0 0 0 -> xyz=0 0 0 rpy=0 0 0
- joint zarm_r4_joint: limit lower=-2.61799387799149 upper=0.0 effort=50.0 velocity=8.37333333333333 -> lower=-2.61799387799149 upper=0.0 effort=75.0 velocity=8.0; origin xyz=0.02 0 -0.1797 rpy=0 0 0 -> xyz=0.02 0 -0.2837 rpy=0 0 0
- joint zarm_r5_joint: limit lower=-1.5707963267949 upper=1.5707963267949 effort=12.0 velocity=7.32666666666667 -> lower=-1.5707963267949 upper=1.5707963267949 effort=14.1 velocity=17.5; origin xyz=-0.02 0 -0.1195 rpy=0 0 0 -> xyz=-0.02 0 -0.1201 rpy=0 0 0
- joint zarm_r6_joint: limit lower=-0.698131700797732 upper=1.30899693899575 effort=12.0 velocity=7.32666666666667 -> lower=-0.698131700797732 upper=1.30899693899575 effort=14.1 velocity=17.5; origin xyz=0 0 -0.114 rpy=0 0 0 -> xyz=0.0 0 -0.114 rpy=0 0 0
- joint zarm_r7_end_effector_joint: origin xyz=0 0.03 -0.17 rpy=0 0 0 -> xyz=0 0.0 -0.17 rpy=0 0 0
- joint zarm_r7_joint: limit lower=-0.698131700797732 upper=0.698131700797732 effort=12.0 velocity=7.32666666666667 -> lower=-0.698131700797732 upper=0.698131700797732 effort=14.1 velocity=17.5; origin xyz=0 0 -0.022284 rpy=0 0 0 -> xyz=0.0 0 -0.021 rpy=0 0 0

Commit message: sync https://www.lejuhub.com/highlydynamic/kuavo-ros-control/commit/bb30d59265697824406293a211519c9c33ec93da

File: src/kuavo_assets/models/biped_s52/urdf/biped_s52.urdf (robot description, URDF)
Before this commit: robot biped_s52, 48 links, 47 joints
Links:
- link waist_yaw_link: mass 20.63616 -> 19.54016
- link zarm_l7_link: mass 0.18940 -> 0.7374
- link zarm_r7_link: mass 0.19960 -> 0.7374

File: src/kuavo_assets/models/biped_s52/urdf/biped_s52_gazebo.urdf (robot description, URDF)
Before this commit: robot biped_s52, 48 links, 47 joints
Links:
- link waist_yaw_link: mass 20.63616 -> 19.54016
- link zarm_l7_link: mass 0.18940 -> 0.7374
- link zarm_r7_link: mass 0.19960 -> 0.7374; geometry collision box size=0.08 0.05 0.16; collision cylinder length=0.08 radius=0.01

File: src/kuavo_assets/models/biped_s52/urdf/drake/biped_v3.urdf (robot description, URDF)
Before this commit: robot biped_v3, 14 links, 13 joints
Links:
- link leg_r3_link: geometry visual mesh filename=../../meshes/r_leg_pitch.STL
- link waist_yaw_link: mass 32.45766 -> 33.54346

File: src/kuavo_assets/models/biped_s52/urdf/drake/biped_v3_arm.urdf (robot description, URDF)
Before this commit: robot biped_s52, 20 links, 19 joints
Links:
- link zarm_l7_link: mass 0.18940 -> 0.7374; geometry visual mesh filename=../../meshes/l_hand_pitch_nohand.STL
- link zarm_r7_link: mass 0.19960 -> 0.7374; geometry visual mesh filename=../../meshes/r_hand_pitch_nohand.STL

File: src/kuavo_assets/models/biped_s52/urdf/drake/biped_v3_full.urdf (robot description, URDF)
Before this commit: robot biped_s52, 32 links, 31 joints
Links:
- link waist_yaw_link: mass 21.47355568 -> 22.55935568
