Commit message: sync https://www.lejuhub.com/highlydynamic/kuavo-ros-control/commit/508a907f99f7a5ae59bb918141667d4ed1ef8e22

File: src/kuavo_assets/models/biped_s52/urdf/drake/biped_v3.urdf (robot description, URDF)
Before this commit: robot biped_v3, 14 links, 13 joints
Links:
- link leg_l1_link: mass 1.63858534 -> 1.55641
- link leg_l2_link: mass 0.70575545 -> 0.75873
- link leg_l3_link: mass 5.93791258 -> 6.68074
- link leg_l4_link: mass 4.02498548 -> 3.64666
- link leg_l5_link: mass 0.07848005 -> 0.07848
- link leg_l6_link: mass 0.58491513 -> 0.69242
- link leg_r1_link: mass 1.63861324 -> 1.55641
- link leg_r2_link: mass 0.70575545 -> 0.75873
- link leg_r3_link: mass 5.93791831 -> 6.68074
- link leg_r4_link: mass 4.02498548 -> 3.64666
- link leg_r5_link: mass 0.07848005 -> 0.07848
- link leg_r6_link: mass 0.58491513 -> 0.69242
- link torso: mass 18.99013928 -> 7.06405; geometry visual mesh filename=../../meshes/torso.STL
- link waist_yaw_link: mass 18.01415568 -> 33.54346
Joints:
- joint leg_l1_joint: limit lower=-0.314159265358979 upper=0.663225115757845 effort=180.0 velocity=23.55 -> lower=-0.314159265358979 upper=0.663225115757845 effort=127.0 velocity=10.4
- joint leg_l2_joint: limit lower=-1.91986217719376 upper=0.785398163397448 effort=100.0 velocity=41.3433333333333 -> lower=-0.785398163397448 upper=1.91986217719376 effort=71.0 velocity=8.7
- joint leg_l3_joint: limit lower=-1.91986217719376 upper=1.5707963267949 effort=100.0 velocity=41.3433333333333 -> lower=-1.91986217719376 upper=1.5707963267949 effort=132 velocity=12.7
- joint leg_l4_joint: limit lower=0.0 upper=2.53072741539178 effort=180.0 velocity=23.55 -> lower=0.0 upper=2.53072741539178 effort=280.0 velocity=10.4; origin xyz=0 0 -0.284 rpy=0 0 0 -> xyz=-0.0011639 0 -0.284 rpy=0 0 0
- joint leg_l5_joint: limit lower=-0.872664625997165 upper=0.349065850398866 effort=36.0 velocity=23.0266666666667 -> lower=-0.872664625997165 upper=0.349065850398866 effort=91.6 velocity=17.8; origin xyz=0.002 0.0003 -0.416 rpy=0 0 0 -> xyz=0.002 0 -0.416 rpy=0 0 0
- joint leg_l6_joint: limit lower=-0.261799387799149 upper=0.261799387799149 effort=36.0 velocity=23.0266666666667 -> lower=-0.261799387799149 upper=0.261799387799149 effort=30.0 velocity=17.8
- joint leg_r1_joint: limit lower=-0.663225115757845 upper=0.314159265358979 effort=180.0 velocity=23.55 -> lower=-0.663225115757845 upper=0.314159265358979 effort=127.0 velocity=10.4
- joint leg_r2_joint: limit lower=-0.785398163397448 upper=1.91986217719376 effort=100.0 velocity=41.3433333333333 -> lower=-1.91986217719376 upper=0.785398163397448 effort=71.0 velocity=8.7
- joint leg_r3_joint: limit lower=-1.91986217719376 upper=1.5707963267949 effort=100.0 velocity=41.3433333333333 -> lower=-1.91986217719376 upper=1.5707963267949 effort=132.0 velocity=12.7
- joint leg_r4_joint: limit lower=0.0 upper=2.53072741539178 effort=180.0 velocity=23.55 -> lower=0.0 upper=2.53072741539178 effort=280.0 velocity=10.4; origin xyz=0 0 -0.284 rpy=0 0 0 -> xyz=-0.0011639 0 -0.284 rpy=0 0 0
- joint leg_r5_joint: limit lower=-0.872664625997165 upper=0.349065850398866 effort=36.0 velocity=23.0266666666667 -> lower=-0.872664625997165 upper=0.349065850398866 effort=91.6 velocity=17.8; origin xyz=0.00199999999983541 -0.000300000028212572 -0.415999999987417 rpy=0 0 0 -> xyz=0.002 0 -0.416 rpy=0 0 0
- joint leg_r6_joint: limit lower=-0.261799387799149 upper=0.261799387799149 effort=36.0 velocity=23.0266666666667 -> lower=-0.261799387799149 upper=0.261799387799149 effort=30.0 velocity=17.8
- joint waist_yaw_joint: limit lower=-2.0943951023932 upper=2.0943951023932 effort=180.0 velocity=23.55 -> lower=-3.14159 upper=3.14159 effort=102.0 velocity=8.7

File: src/kuavo_assets/models/biped_s52/urdf/drake/biped_v3_arm.urdf (robot description, URDF)
Before this commit: robot biped_s52, 20 links, 19 joints
Links:
- link base_link: mass 6.48663928 -> 7.06405; geometry visual mesh filename=../../meshes/torso.STL
- link waist_yaw_link: mass 18.01415568 -> 20.63616
- link zarm_l1_link: mass 0.91653322 -> 0.94521
- link zarm_l2_link: mass 0.3876739 -> 0.41921
- link zarm_l3_link: mass 1.77926875 -> 1.78857
- link zarm_l4_link: mass 0.58507821 -> 0.63149
- link zarm_l5_link: mass 0.68679955 -> 0.60828
- link zarm_l6_link: mass 0.39387181 -> 0.50616
- link zarm_l7_end_effector: geometry 
- link zarm_l7_link: mass 0.61537779 -> 0.7374; geometry visual mesh filename=../../meshes/l_hand_pitch_nohand.STL
- link zarm_r1_link: mass 0.92062797 -> 0.92947
- link zarm_r2_link: mass 0.38768053 -> 0.41523
- link zarm_r3_link: mass 1.77969208 -> 1.78473
- link zarm_r4_link: mass 0.58514611 -> 0.63548
- link zarm_r5_link: mass 0.68473867 -> 0.61021
- link zarm_r6_link: mass 0.39247462 -> 0.53821
- link zarm_r7_end_effector: geometry 
- link zarm_r7_link: mass 0.61562202 -> 0.7374; geometry visual mesh filename=../../meshes/r_hand_pitch_nohand.STL
Joints:
- joint waist_yaw_joint: limit lower=-3.14159 upper=3.14159 effort=180.0 velocity=23.55 -> lower=-3.14159 upper=3.14159 effort=102.0 velocity=8.7
- joint zarm_l1_joint: limit lower=-3.14159265358979 upper=1.5707963267949 effort=100.0 velocity=41.3433333333333 -> lower=-3.14159265358979 upper=1.5707963267949 effort=66.0 velocity=18.8; origin xyz=-0.003 0.1737 0.2831 rpy=0 0 0 -> xyz=-0.003 0.2527 0.283 rpy=0 0 0
- joint zarm_l2_joint: limit lower=-0.349065850398866 upper=2.0943951023932 effort=50.0 velocity=8.37333333333333 -> lower=-0.349065850398866 upper=3.49065850398866 effort=75.0 velocity=8.0; origin xyz=0 0.081 0 rpy=0 0 0 -> xyz=0 0 0 rpy=0 0 0
- joint zarm_l3_joint: limit lower=-1.5707963267949 upper=1.5707963267949 effort=36.0 velocity=9.94333333333333 -> lower=-1.48352986419518 upper=1.48352986419518 effort=57.0 velocity=7.5; origin xyz=0 0 -0.104 rpy=0 0 0 -> xyz=0 0 0 rpy=0 0 0
- joint zarm_l4_joint: limit lower=-2.61799387799149 upper=0.0 effort=50.0 velocity=8.37333333333333 -> lower=-2.61799387799149 upper=0.0 effort=75.0 velocity=8.0; origin xyz=0.02 0 -0.1797 rpy=0 0 0 -> xyz=0.02 0 -0.2837 rpy=0 0 0
- joint zarm_l5_joint: limit lower=-1.5707963267949 upper=1.5707963267949 effort=12.0 velocity=7.32666666666667 -> lower=-1.5707963267949 upper=1.5707963267949 effort=14.1 velocity=17.5; origin xyz=-0.02 0 -0.1195 rpy=0 0 0 -> xyz=-0.02 0 -0.1201 rpy=0 0 0
- joint zarm_l6_joint: limit lower=-1.30899693899575 upper=0.698131700797732 effort=12.0 velocity=7.32666666666667 -> lower=-1.30899693899575 upper=0.698131700797732 effort=14.1 velocity=17.5; origin xyz=0 0 -0.114 rpy=0 0 0 -> xyz=0.0 0 -0.114 rpy=0 0 0
- joint zarm_l7_end_effector_joint: origin xyz=0 -0.03 -0.17 rpy=0 0 0 -> xyz=0 0.0 -0.17 rpy=0 0 0
- joint zarm_l7_joint: limit lower=-0.698131700797732 upper=0.698131700797732 effort=12.0 velocity=7.32666666666667 -> lower=-0.698131700797732 upper=0.698131700797732 effort=14.1 velocity=17.5; origin xyz=-0.0002 0 -0.021 rpy=0 0 0 -> xyz=0 0 -0.021 rpy=0 0 0
- joint zarm_r1_joint: limit lower=-3.14159265358979 upper=1.5707963267949 effort=100.0 velocity=41.3433333333333 -> lower=-3.14159265358979 upper=1.5707963267949 effort=66.0 velocity=18.8; origin xyz=-0.003 -0.1737 0.2831 rpy=0 0 0 -> xyz=-0.003 -0.2527 0.283 rpy=0 0 0
- joint zarm_r2_joint: limit lower=-2.0943951023932 upper=0.349065850398866 effort=50.0 velocity=8.37333333333333 -> lower=-3.49065850398866 upper=0.349065850398866 effort=75.0 velocity=8.0; origin xyz=0 -0.081 0 rpy=0 0 0 -> xyz=0 0 0 rpy=0 0 0
- joint zarm_r3_joint: limit lower=-1.5707963267949 upper=1.5707963267949 effort=36.0 velocity=9.94333333333333 -> lower=-1.48352986419518 upper=1.48352986419518 effort=57.0 velocity=7.5; origin xyz=0 0 -0.104 rpy=0 0 0 -> xyz=0 0 0 rpy=0 0 0
- joint zarm_r4_joint: limit lower=-2.61799387799149 upper=0.0 effort=50.0 velocity=8.37333333333333 -> lower=-2.61799387799149 upper=0.0 effort=75.0 velocity=8.0; origin xyz=0.02 0 -0.1797 rpy=0 0 0 -> xyz=0.02 0 -0.2837 rpy=0 0 0
- joint zarm_r5_joint: limit lower=-1.5707963267949 upper=1.5707963267949 effort=12.0 velocity=7.32666666666667 -> lower=-1.5707963267949 upper=1.5707963267949 effort=14.1 velocity=17.5; origin xyz=-0.02 0 -0.1195 rpy=0 0 0 -> xyz=-0.02 0 -0.1201 rpy=0 0 0
- joint zarm_r6_joint: limit lower=-0.698131700797732 upper=1.30899693899575 effort=12.0 velocity=7.32666666666667 -> lower=-0.698131700797732 upper=1.30899693899575 effort=14.1 velocity=17.5; origin xyz=0 0 -0.114 rpy=0 0 0 -> xyz=0.0 0 -0.114 rpy=0 0 0
- joint zarm_r7_end_effector_joint: origin xyz=0 0.03 -0.17 rpy=0 0 0 -> xyz=0 0.0 -0.17 rpy=0 0 0
- joint zarm_r7_joint: limit lower=-0.698131700797732 upper=0.698131700797732 effort=12.0 velocity=7.32666666666667 -> lower=-0.698131700797732 upper=0.698131700797732 effort=14.1 velocity=17.5; origin xyz=0 0 -0.022284 rpy=0 0 0 -> xyz=0.0 0 -0.021 rpy=0 0 0

File: src/kuavo_assets/models/biped_s52/urdf/drake/biped_v3_full.urdf (robot description, URDF)
Before this commit: robot biped_s52, 32 links, 31 joints
Links:
- link waist_yaw_link: mass 18.01415568 -> 22.55935568

File: src/kuavo_assets/models/biped_s60/urdf/drake/biped_v3_arm.urdf (robot description, URDF)
Before this commit: robot biped_s45, 17 links, 16 joints
Links:
- added link knee_link, mass 5.39660196; visual mesh filename=../../meshes/knee_pitch.STL
- added link leg_link, mass 12.35650958; visual mesh filename=../../meshes/leg_pitch.STL
- added link waist_link, mass 5.4305643; visual mesh filename=../../meshes/waist_pitch.STL
- added link waist_yaw_link, mass 11.56094002; collision cylinder length=0.6 radius=0.15; visual mesh filename=../../meshes/torso.STL
- added link zarm_l7_virtual_thumb_link; collision sphere radius=0.005
- added link zarm_r7_virtual_thumb_link; collision sphere radius=0.005
- link base_link: mass 11.56094002 -> 97.77291318; geometry visual mesh filename=../../meshes/chassis.STL
- link zarm_l1_link: geometry visual mesh filename=../../meshes/l_arm_pitch.STL
- link zarm_l2_link: geometry visual mesh filename=../../meshes/l_arm_roll.STL
- link zarm_l3_link: geometry visual mesh filename=../../meshes/l_arm_yaw.STL
- link zarm_l4_link: geometry visual mesh filename=../../meshes/l_forearm.STL
- link zarm_l5_link: geometry visual mesh filename=../../meshes/l_hand_yaw.STL
- link zarm_l6_link: geometry visual mesh filename=../../meshes/l_hand_roll.STL
- link zarm_l7_link: geometry visual mesh filename=../../meshes/l_hand_pitch_noHand.STL
- link zarm_r1_link: geometry visual mesh filename=../../meshes/r_arm_pitch.STL
- link zarm_r2_link: geometry collision cylinder length=0.3 radius=0.05; visual mesh filename=../../meshes/r_arm_roll.STL
- link zarm_r3_link: geometry visual mesh filename=../../meshes/r_arm_yaw.STL
- link zarm_r4_link: geometry collision cylinder length=0.26 radius=0.05; visual mesh filename=../../meshes/r_forearm.STL
- link zarm_r5_link: geometry visual mesh filename=../../meshes/r_hand_yaw.STL
- link zarm_r6_link: geometry visual mesh filename=../../meshes/r_hand_roll.STL
- link zarm_r7_link: geometry visual mesh filename=../../meshes/r_hand_pitch_noHand.STL
Joints:
- added joint knee_joint: type revolute, parent base_link, child knee_link, origin xyz=0.2265 0.017 0.2658 rpy=0 0.0 0, axis 0 1 0, limit lower=0 upper=1.448 effort=668.53 velocity=25.33
- added joint leg_joint: type revolute, parent knee_link, child leg_link, origin xyz=-0.48618 0 0.11672 rpy=0 -0.251 0, axis 0 1 0, limit lower=-2.81 upper=0.0 effort=668.53 velocity=25.33
- added joint waist_pitch_joint: type revolute, parent leg_link, child waist_link, origin xyz=0.49384 0 0.078217 rpy=0 0.236 0, axis  0 1 0, limit lower=0.0 upper=0.9 effort=618.48 velocity=25.33
- added joint waist_yaw_joint: type revolute, parent waist_link, child waist_yaw_link, origin xyz=0.0 -0.0165 0.209 rpy=0 0 0, axis 0 0 1, limit lower=-3.238 upper=3.238 effort=618.48 velocity=25.33
- added joint zarm_l7_virtual_thumb_joint_ee: type fixed, parent zarm_l7_end_effector, child zarm_l7_virtual_thumb_link, origin xyz=0.15 0 0 rpy=0 0 0
- added joint zarm_r7_virtual_thumb_joint_ee: type fixed, parent zarm_r7_end_effector, child zarm_r7_virtual_thumb_link, origin xyz=0.15 0 0 rpy=0 0 0
- joint zarm_l1_joint: limit lower=-3.14159265358979 upper=1.5707963267949 effort=100.0 velocity=41.3433333333333 -> lower=-2.4 upper=0.6 effort=66.0 velocity=18.8; parent base_link -> waist_yaw_link
- joint zarm_l2_joint: limit lower=-0.349065850398866 upper=2.0943951023932 effort=50.0 velocity=19.154 -> lower=-0.349065850398866 upper=1.46 effort=75.0 velocity=8.0
- joint zarm_l3_joint: limit lower=-1.5707963267949 upper=1.5707963267949 effort=39.0 velocity=18.84 -> lower=-1.5707963267949 upper=0.46 effort=57.0 velocity=7.5
- joint zarm_l4_joint: limit lower=-2.61799387799149 upper=0.0 effort=50.0 velocity=18.84 -> lower=-2.61799387799149 upper=-0.2 effort=75.0 velocity=8.0
- joint zarm_l5_joint: limit lower=-1.5707963267949 upper=1.5707963267949 effort=12.0 velocity=21.666 -> lower=-1.5707963267949 upper=1.5707963267949 effort=14.1 velocity=17.5
- joint zarm_l6_joint: limit lower=-1.30899693899575 upper=0.698131700797732 effort=12.0 velocity=21.666 -> lower=-1.30899693899575 upper=0.698131700797732 effort=14.1 velocity=17.5
- joint zarm_l7_end_effector_joint: origin xyz=0 -0.03 -0.17 rpy=0 0 0 -> xyz=0 0.0 -0.17 rpy=0 0 0
- joint zarm_l7_joint: limit lower=-0.698131700797732 upper=0.698131700797732 effort=12.0 velocity=21.666 -> lower=-0.698131700797732 upper=0.698131700797732 effort=14.1 velocity=17.5
- joint zarm_r1_joint: limit lower=-3.14159265358979 upper=1.5707963267949 effort=100.0 velocity=41.3433333333333 -> lower=-2.4 upper=0.6 effort=66.0 velocity=18.8; parent base_link -> waist_yaw_link
- joint zarm_r2_joint: limit lower=-2.0943951023932 upper=0.349065850398866 effort=50.0 velocity=19.154 -> lower=-1.46 upper=0.349065850398866 effort=75.0 velocity=8.0
- joint zarm_r3_joint: limit lower=-1.5707963267949 upper=1.5707963267949 effort=39.0 velocity=18.84 -> lower=-0.46 upper=1.5707963267949 effort=57.0 velocity=7.5
- joint zarm_r4_joint: limit lower=-2.61799387799149 upper=0.0 effort=50.0 velocity=18.84 -> lower=-2.61799387799149 upper=-0.2 effort=75.0 velocity=8.0
- joint zarm_r5_joint: limit lower=-1.5707963267949 upper=1.5707963267949 effort=12.0 velocity=21.666 -> lower=-1.5707963267949 upper=1.5707963267949 effort=14.1 velocity=17.5
- joint zarm_r6_joint: limit lower=-0.698131700797732 upper=1.30899693899575 effort=12.0 velocity=21.666 -> lower=-0.698131700797732 upper=1.30899693899575 effort=14.1 velocity=17.5
- joint zarm_r7_end_effector_joint: origin xyz=0 0.03 -0.17 rpy=0 0 0 -> xyz=0 0.0 -0.17 rpy=0 0 0
- joint zarm_r7_joint: limit lower=-0.698131700797732 upper=0.698131700797732 effort=12.0 velocity=21.666 -> lower=-0.698131700797732 upper=0.698131700797732 effort=14.1 velocity=17.5
