Commit message: sync https://www.lejuhub.com/highlydynamic/kuavo-ros-control/commit/bf8cf96c4d479e46eff27ac76d565b24fe7167b3

File: src/kuavo_assets/models/biped_s52/urdf/biped_s52.urdf (robot description, URDF)
Before this commit: robot biped_s52, 48 links, 47 joints
Links:
- removed link head_rader
- added link head_camera_base, mass 0.0; visual mesh filename=package://kuavo_assets/models/biped_s52/meshes/head_camera_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
- added link head_camera_depth, mass 0.0000785398163397463; visual mesh filename=package://kuavo_assets/models/biped_s52/meshes/head_camera_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
- added link head_radar, mass 0.0; visual mesh filename=package://kuavo_assets/models/biped_s52/meshes/head_radar.S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
- added link waist_camera_base, mass 0.13300000; visual mesh filename=package://kuavo_assets/models/biped_s52/meshes/waist_camera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
- link camera_base: mass 0.00000000 -> 0.000001; geometry 
- link waist_camera: mass 0.048238 -> 0.0000785398163397463
- link waist_yaw_link: mass 19.54016 -> 19.72026
Joints:
- removed joint camera_base
- removed joint head_rader_joint
- removed joint waist_camera
- added joint camera_base_joint: type fixed, parent head_camera_depth, child camera_base, origin xyz=0 0 0 rpy=0 0 0, axis 0 0 0
- added joint head_camera_base_joint: type fixed, parent zhead_2_link, child head_camera_base, origin xyz=0.099619 0 0.032844 rpy=0 0.3406 0, axis 0 0 0
- added joint head_camera_depth_joint: type fixed, parent head_camera_base, child head_camera_depth, origin xyz=0.011715 0.0475 0.014312 rpy=0 0 0, axis 0 0 0
- added joint head_radar_joint: type fixed, parent zhead_1_link, child head_radar, origin xyz=0 0 -0.078453 rpy=0 0 0, axis 0 0 0
- added joint waist_camera_base_joint: type fixed, parent waist_yaw_link, child waist_camera_base, origin xyz=0.0787 0 -0.028149 rpy=0 0.59341 0, axis 0 0 0
- added joint waist_camera_joint: type fixed, parent waist_camera_base, child waist_camera, origin xyz=0.011715 0.0475 0.014312 rpy=0 0 0, axis 0 0 0
- joint leg_l6_joint: limit lower=-0.261799387799149 upper=0.261799387799149 effort=30.0 velocity=17.8 -> lower=-0.261799387799149 upper=0.261799387799149 effort=68.4 velocity=17.8
- joint leg_r6_joint: limit lower=-0.261799387799149 upper=0.261799387799149 effort=30.0 velocity=17.8 -> lower=-0.261799387799149 upper=0.261799387799149 effort=68.4 velocity=17.8

File: src/kuavo_assets/models/biped_s52/urdf/biped_s52_gazebo.urdf (robot description, URDF)
Before this commit: robot biped_s52, 48 links, 47 joints
Links:
- removed link head_rader
- added link head_camera_base, mass 0.0; visual mesh filename=../meshes/head_camera_base.STL
- added link head_camera_depth, mass 0.0000785398163397463; visual mesh filename=../meshes/head_camera_depth.STL
- added link head_radar, mass 0.0; visual mesh filename=../meshes/head_radar.STL
- added link waist_camera_base, mass 0.13300000; visual mesh filename=package://kuavo_assets/models/biped_s52/meshes/waist_camera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
- link camera_base: mass 0.00000000 -> 0.000001; geometry 
- link waist_camera: mass 0.048238 -> 0.0000785398163397463
- link waist_yaw_link: mass 19.54016 -> 19.72026
Joints:
- removed joint camera_base
- removed joint head_rader_joint
- removed joint waist_camera
- added joint camera_base_joint: type fixed, parent head_camera_depth, child camera_base, origin xyz=0 0 0 rpy=0 0 0, axis 0 0 0
- added joint head_camera_base_joint: type fixed, parent zhead_2_link, child head_camera_base, origin xyz=0.099619 0 0.032844 rpy=0 0.3406 0, axis 0 0 0
- added joint head_camera_depth_joint: type fixed, parent head_camera_base, child head_camera_depth, origin xyz=0.011715 0.0475 0.014312 rpy=0 0 0, axis 0 0 0
- added joint head_radar_joint: type fixed, parent zhead_1_link, child head_radar, origin xyz=0 0 -0.078453 rpy=0 0 0, axis 0 0 0
- added joint waist_camera_base_joint: type fixed, parent waist_yaw_link, child waist_camera_base, origin xyz=0.0787 0 -0.028149 rpy=0 0.59341 0, axis 0 0 0
- added joint waist_camera_joint: type fixed, parent waist_camera_base, child waist_camera, origin xyz=0.011715 0.0475 0.014312 rpy=0 0 0, axis 0 0 0
- joint leg_l6_joint: limit lower=-0.261799387799149 upper=0.261799387799149 effort=30.0 velocity=17.8 -> lower=-0.261799387799149 upper=0.261799387799149 effort=68.4 velocity=17.8
- joint leg_r6_joint: limit lower=-0.261799387799149 upper=0.261799387799149 effort=30.0 velocity=17.8 -> lower=-0.261799387799149 upper=0.261799387799149 effort=68.4 velocity=17.8

File: src/kuavo_assets/models/biped_s53/urdf/biped_s53.urdf (robot description, URDF)
Before this commit: robot biped_s53, 48 links, 47 joints
Links:
- removed link head_rader
- added link head_camera_base, mass 0.0; visual mesh filename=package://kuavo_assets/models/biped_s53/meshes/head_camera_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
- added link head_camera_depth, mass 0.0000785398163397463; visual mesh filename=package://kuavo_assets/models/biped_s53/meshes/head_camera_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
- added link head_radar, mass 0.0; visual mesh filename=package://kuavo_assets/models/biped_s53/meshes/head_radar.S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
- added link waist_camera_base, mass 0.13300000; visual mesh filename=package://kuavo_assets/models/biped_s53/meshes/waist_camera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
- link camera_base: mass 0.00000000 -> 0.000001; geometry 
- link waist_camera: mass 0.13300 -> 0.0000785398163397463
- link waist_yaw_link: mass 19.98211 -> 19.98201
Joints:
- removed joint camera_base
- removed joint head_rader_joint
- removed joint waist_camera
- added joint camera_base_joint: type fixed, parent head_camera_depth, child camera_base, origin xyz=0 0 0 rpy=0 0 0, axis 0 0 0
- added joint head_camera_base_joint: type fixed, parent zhead_2_link, child head_camera_base, origin xyz=0.099619 0 0.032844 rpy=0 0.3406 0, axis 0 0 0
- added joint head_camera_depth_joint: type fixed, parent head_camera_base, child head_camera_depth, origin xyz=0.011715 0.0475 0.014312 rpy=0 0 0, axis 0 0 0
- added joint head_radar_joint: type fixed, parent zhead_1_link, child head_radar, origin xyz=0 0 -0.078453 rpy=0 0 0, axis 0 0 0
- added joint waist_camera_base_joint: type fixed, parent waist_yaw_link, child waist_camera_base, origin xyz=0.0787 0 -0.028149 rpy=0 0.59341 0, axis 0 0 0
- added joint waist_camera_joint: type fixed, parent waist_camera_base, child waist_camera, origin xyz=0.011715 0.0475 0.014312 rpy=0 0 0, axis 0 0 0
- joint leg_l6_joint: limit lower=-0.261799387799149 upper=0.261799387799149 effort=30.0 velocity=17.8 -> lower=-0.261799387799149 upper=0.261799387799149 effort=68.4 velocity=17.8
- joint leg_r6_joint: limit lower=-0.261799387799149 upper=0.261799387799149 effort=30.0 velocity=17.8 -> lower=-0.261799387799149 upper=0.261799387799149 effort=68.4 velocity=17.8

File: src/kuavo_assets/models/biped_s53/urdf/biped_s53_gazebo.urdf (robot description, URDF)
Before this commit: robot biped_s53, 48 links, 47 joints
Links:
- removed link head_rader
- added link head_camera_base, mass 0.0; visual mesh filename=../meshes/head_camera_base.STL
- added link head_camera_depth, mass 0.0000785398163397463; visual mesh filename=../meshes/head_camera_depth.STL
- added link head_radar, mass 0.0; visual mesh filename=../meshes/head_radar.STL
- added link waist_camera_base, mass 0.13300000; visual mesh filename=../meshes/waist_camera_base.STL
- link base_link: geometry visual mesh filename=../meshes/torso.STL
- link camera_base: mass 0.00000000 -> 0.000001; geometry 
- link leg_l1_link: geometry visual mesh filename=../meshes/l_leg_roll.STL
- link leg_l2_link: geometry visual mesh filename=../meshes/l_leg_yaw.STL
- link leg_l3_link: geometry visual mesh filename=../meshes/l_leg_pitch.STL
- link leg_l4_link: geometry visual mesh filename=../meshes/l_knee.STL
- link leg_l5_link: geometry visual mesh filename=../meshes/l_foot_pitch.STL
- link leg_l6_link: geometry collision box size=0.25 0.1 0.04; visual mesh filename=../meshes/l_foot_roll.STL
- link leg_r1_link: geometry visual mesh filename=../meshes/r_leg_roll.STL
- link leg_r2_link: geometry visual mesh filename=../meshes/r_leg_yaw.STL
- link leg_r3_link: geometry visual mesh filename=../meshes/r_leg_pitch.STL
- link leg_r4_link: geometry visual mesh filename=../meshes/r_knee.STL
- link leg_r5_link: geometry visual mesh filename=../meshes/r_foot_pitch.STL
- link leg_r6_link: geometry collision box size=0.25 0.1 0.04; visual mesh filename=../meshes/r_foot_roll.STL
- link waist_camera: mass 0.048238 -> 0.0000785398163397463; geometry visual mesh filename=../meshes/waist_camera_depth.STL
- link waist_yaw_link: mass 21.63516 -> 21.90016; geometry visual mesh filename=../meshes/waist_yaw.STL
- link zarm_l1_link: geometry visual mesh filename=../meshes/l_arm_pitch.STL
- link zarm_l2_link: geometry visual mesh filename=../meshes/l_arm_roll.STL
- link zarm_l3_link: geometry visual mesh filename=../meshes/l_arm_yaw.STL
- link zarm_l4_link: geometry visual mesh filename=../meshes/l_forearm.STL
- link zarm_l5_link: geometry visual mesh filename=../meshes/l_hand_yaw.STL
- link zarm_l6_link: geometry visual mesh filename=../meshes/l_hand_roll.STL
- link zarm_l7_link: geometry visual mesh filename=../meshes/l_hand_pitch_nohand.STL
- link zarm_r1_link: geometry visual mesh filename=../meshes/r_arm_pitch.STL
- link zarm_r2_link: geometry visual mesh filename=../meshes/r_arm_roll.STL
- link zarm_r3_link: geometry visual mesh filename=../meshes/r_arm_yaw.STL
- link zarm_r4_link: geometry visual mesh filename=../meshes/r_forearm.STL
- link zarm_r5_link: geometry visual mesh filename=../meshes/r_hand_yaw.STL
- link zarm_r6_link: geometry visual mesh filename=../meshes/r_hand_roll.STL
- link zarm_r7_link: geometry collision box size=0.08 0.05 0.16; collision cylinder length=0.08 radius=0.01
- link zhead_1_link: geometry visual mesh filename=../meshes/head_yaw.STL
- link zhead_2_link: geometry visual mesh filename=../meshes/head_pitch.STL
Joints:
- removed joint camera_base
- removed joint head_rader_joint
- removed joint waist_camera
- added joint camera_base_joint: type fixed, parent head_camera_depth, child camera_base, origin xyz=0 0 0 rpy=0 0 0, axis 0 0 0
- added joint head_camera_base_joint: type fixed, parent zhead_2_link, child head_camera_base, origin xyz=0.099619 0 0.032844 rpy=0 0.3406 0, axis 0 0 0
- added joint head_camera_depth_joint: type fixed, parent head_camera_base, child head_camera_depth, origin xyz=0.011715 0.0475 0.014312 rpy=0 0 0, axis 0 0 0
- added joint head_radar_joint: type fixed, parent zhead_1_link, child head_radar, origin xyz=0 0 -0.078453 rpy=0 0 0, axis 0 0 0
- added joint waist_camera_base_joint: type fixed, parent waist_yaw_link, child waist_camera_base, origin xyz=0.0787 0 -0.028149 rpy=0 0.59341 0, axis 0 0 0
- added joint waist_camera_joint: type fixed, parent waist_camera_base, child waist_camera, origin xyz=0.011715 0.0475 0.014312 rpy=0 0 0, axis 0 0 0
- joint leg_l6_joint: limit lower=-0.261799387799149 upper=0.261799387799149 effort=30.0 velocity=17.8 -> lower=-0.261799387799149 upper=0.261799387799149 effort=68.4 velocity=17.8
- joint leg_r6_joint: limit lower=-0.261799387799149 upper=0.261799387799149 effort=30.0 velocity=17.8 -> lower=-0.261799387799149 upper=0.261799387799149 effort=68.4 velocity=17.8

File: src/kuavo_assets/models/biped_s54/urdf/biped_s54.urdf (robot description, URDF)
Before this commit: robot biped_s54, 48 links, 47 joints
Links:
- removed link head_rader
- added link head_camera_base, mass 0.0; visual mesh filename=package://kuavo_assets/models/biped_s54/meshes/head_camera_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
- added link head_camera_depth, mass 0.0000785398163397463; visual mesh filename=package://kuavo_assets/models/biped_s54/meshes/head_camera_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
- added link head_radar, mass 0.0; visual mesh filename=package://kuavo_assets/models/biped_s54/meshes/head_radar.S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
- added link waist_camera_base, mass 0.13300000; visual mesh filename=package://kuavo_assets/models/biped_s54/meshes/waist_camera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
- link camera_base: mass 0.00000000 -> 0.000001; geometry 
- link waist_camera: mass 0.13300 -> 0.0000785398163397463
- link waist_yaw_link: mass 20.23838 -> 20.50328
Joints:
- removed joint camera_base
- removed joint head_rader_joint
- removed joint waist_camera
- added joint camera_base_joint: type fixed, parent head_camera_depth, child camera_base, origin xyz=0 0 0 rpy=0 0 0, axis 0 0 0
- added joint head_camera_base_joint: type fixed, parent zhead_2_link, child head_camera_base, origin xyz=0.099619 0 0.032844 rpy=0 0.3406 0, axis 0 0 0
- added joint head_camera_depth_joint: type fixed, parent head_camera_base, child head_camera_depth, origin xyz=0.011715 0.0475 0.014312 rpy=0 0 0, axis 0 0 0
- added joint head_radar_joint: type fixed, parent zhead_1_link, child head_radar, origin xyz=0 0 -0.078453 rpy=0 0 0, axis 0 0 0
- added joint waist_camera_base_joint: type fixed, parent waist_yaw_link, child waist_camera_base, origin xyz=0.0787 0 -0.028149 rpy=0 0.59341 0, axis 0 0 0
- added joint waist_camera_joint: type fixed, parent waist_camera_base, child waist_camera, origin xyz=0.011715 0.0475 0.014312 rpy=0 0 0, axis 0 0 0
- joint leg_l6_joint: limit lower=-0.261799387799149 upper=0.261799387799149 effort=30.0 velocity=17.8 -> lower=-0.261799387799149 upper=0.261799387799149 effort=68.4 velocity=17.8
- joint leg_r6_joint: limit lower=-0.261799387799149 upper=0.261799387799149 effort=30.0 velocity=17.8 -> lower=-0.261799387799149 upper=0.261799387799149 effort=68.4 velocity=17.8

File: src/kuavo_assets/models/biped_s54/urdf/biped_s54_gazebo.urdf (robot description, URDF)
Before this commit: robot biped_s54, 48 links, 47 joints
Links:
- removed link head_rader
- added link head_camera_base, mass 0.0; visual mesh filename=../meshes/head_camera_base.STL
- added link head_camera_depth, mass 0.0000785398163397463; visual mesh filename=../meshes/head_camera_depth.STL
- added link head_radar, mass 0.0; visual mesh filename=../meshes/head_radar.STL
- added link waist_camera_base, mass 0.13300000; visual mesh filename=../meshes/waist_camera_base.STL
- link base_link: geometry visual mesh filename=../meshes/torso.STL
- link camera_base: mass 0.00000000 -> 0.000001; geometry 
- link leg_l1_link: geometry visual mesh filename=../meshes/l_leg_roll.STL
- link leg_l2_link: geometry visual mesh filename=../meshes/l_leg_yaw.STL
- link leg_l3_link: geometry visual mesh filename=../meshes/l_leg_pitch.STL
- link leg_l4_link: geometry visual mesh filename=../meshes/l_knee.STL
- link leg_l5_link: geometry visual mesh filename=../meshes/l_foot_pitch.STL
- link leg_l6_link: geometry collision box size=0.25 0.1 0.04; visual mesh filename=../meshes/l_foot_roll.STL
- link leg_r1_link: geometry visual mesh filename=../meshes/r_leg_roll.STL
- link leg_r2_link: geometry visual mesh filename=../meshes/r_leg_yaw.STL
- link leg_r3_link: geometry visual mesh filename=../meshes/r_leg_pitch.STL
- link leg_r4_link: geometry visual mesh filename=../meshes/r_knee.STL
- link leg_r5_link: geometry visual mesh filename=../meshes/r_foot_pitch.STL
- link leg_r6_link: geometry collision box size=0.25 0.1 0.04; visual mesh filename=../meshes/r_foot_roll.STL
- link waist_camera: mass 0.13300 -> 0.0000785398163397463; geometry visual mesh filename=../meshes/waist_camera_depth.STL
- link waist_yaw_link: mass 20.23838 -> 20.50328; geometry visual mesh filename=../meshes/waist_yaw.STL
- link zarm_l1_link: geometry visual mesh filename=../meshes/l_arm_pitch.STL
- link zarm_l2_link: geometry visual mesh filename=../meshes/l_arm_roll.STL
- link zarm_l3_link: geometry visual mesh filename=../meshes/l_arm_yaw.STL
- link zarm_l4_link: geometry visual mesh filename=../meshes/l_forearm.STL
- link zarm_l5_link: geometry visual mesh filename=../meshes/l_hand_yaw.STL
- link zarm_l6_link: geometry visual mesh filename=../meshes/l_hand_roll.STL
- link zarm_l7_link: geometry visual mesh filename=../meshes/l_hand_pitch_nohand.STL
- link zarm_r1_link: geometry visual mesh filename=../meshes/r_arm_pitch.STL
- link zarm_r2_link: geometry visual mesh filename=../meshes/r_arm_roll.STL
- link zarm_r3_link: geometry visual mesh filename=../meshes/r_arm_yaw.STL
- link zarm_r4_link: geometry visual mesh filename=../meshes/r_forearm.STL
- link zarm_r5_link: geometry visual mesh filename=../meshes/r_hand_yaw.STL
- link zarm_r6_link: geometry visual mesh filename=../meshes/r_hand_roll.STL
- link zarm_r7_link: geometry collision box size=0.08 0.05 0.16; collision cylinder length=0.08 radius=0.01
- link zhead_1_link: geometry visual mesh filename=../meshes/head_yaw.STL
- link zhead_2_link: geometry visual mesh filename=../meshes/head_pitch.STL
Joints:
- removed joint camera_base
- removed joint head_rader_joint
- removed joint waist_camera
- added joint camera_base_joint: type fixed, parent head_camera_depth, child camera_base, origin xyz=0 0 0 rpy=0 0 0, axis 0 0 0
- added joint head_camera_base_joint: type fixed, parent zhead_2_link, child head_camera_base, origin xyz=0.099619 0 0.032844 rpy=0 0.3406 0, axis 0 0 0
- added joint head_camera_depth_joint: type fixed, parent head_camera_base, child head_camera_depth, origin xyz=0.011715 0.0475 0.014312 rpy=0 0 0, axis 0 0 0
- added joint head_radar_joint: type fixed, parent zhead_1_link, child head_radar, origin xyz=0 0 -0.078453 rpy=0 0 0, axis 0 0 0
- added joint waist_camera_base_joint: type fixed, parent waist_yaw_link, child waist_camera_base, origin xyz=0.0787 0 -0.028149 rpy=0 0.59341 0, axis 0 0 0
- added joint waist_camera_joint: type fixed, parent waist_camera_base, child waist_camera, origin xyz=0.011715 0.0475 0.014312 rpy=0 0 0, axis 0 0 0
- joint leg_l6_joint: limit lower=-0.261799387799149 upper=0.261799387799149 effort=30.0 velocity=17.8 -> lower=-0.261799387799149 upper=0.261799387799149 effort=68.4 velocity=17.8
- joint leg_r6_joint: limit lower=-0.261799387799149 upper=0.261799387799149 effort=30.0 velocity=17.8 -> lower=-0.261799387799149 upper=0.261799387799149 effort=68.4 velocity=17.8
