Commit message: sync https://www.lejuhub.com/highlydynamic/kuavo-ros-control/commit/7ea02f6744ed785b3502846147c27472578130c5

File: src/kuavo_assets/models/biped_s52/urdf/biped_s52.urdf (robot description, URDF)
Before this commit: robot biped_s52, 48 links, 47 joints
Links:
- removed link camera_base
- removed link head_rader
- added link head_camera_base, mass 0.0; visual mesh filename=package://kuavo_assets/models/biped_s52/meshes/head_camera_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
- added link head_camera_depth, mass 0.0000785398163397463; visual mesh filename=package://kuavo_assets/models/biped_s52/meshes/head_camera_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
- added link head_radar, mass 0.0; visual mesh filename=package://kuavo_assets/models/biped_s52/meshes/head_radar.S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
- added link waist_camera_base, mass 0.13300000; visual mesh filename=package://kuavo_assets/models/biped_s52/meshes/waist_camera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
- link waist_camera: mass 0.048238 -> 0.0000785398163397463
- link waist_yaw_link: mass 19.54016 -> 19.72026
Joints:
- removed joint camera_base
- removed joint head_rader_joint
- removed joint waist_camera
- added joint head_camera_base_joint: type fixed, parent zhead_2_link, child head_camera_base, origin xyz=0.099619 0 0.032844 rpy=0 0.3406 0, axis 0 0 0
- added joint head_camera_depth_joint: type fixed, parent head_camera_base, child head_camera_depth, origin xyz=0.011715 0.0475 0.014312 rpy=0 0 0, axis 0 0 0
- added joint head_radar_joint: type fixed, parent zhead_1_link, child head_radar, origin xyz=0 0 -0.078453 rpy=0 0 0, axis 0 0 0
- added joint waist_camera_base_joint: type fixed, parent waist_yaw_link, child waist_camera_base, origin xyz=0.0787 0 -0.028149 rpy=0 0.59341 0, axis 0 0 0
- added joint waist_camera_joint: type fixed, parent waist_camera_base, child waist_camera, origin xyz=0.011715 0.0475 0.014312 rpy=0 0 0, axis 0 0 0
- joint leg_l6_joint: limit lower=-0.261799387799149 upper=0.261799387799149 effort=30.0 velocity=17.8 -> lower=-0.261799387799149 upper=0.261799387799149 effort=68.4 velocity=17.8
- joint leg_r6_joint: limit lower=-0.261799387799149 upper=0.261799387799149 effort=30.0 velocity=17.8 -> lower=-0.261799387799149 upper=0.261799387799149 effort=68.4 velocity=17.8

File: src/kuavo_assets/models/biped_s52/urdf/biped_s52_gazebo.urdf (robot description, URDF)
Before this commit: robot biped_s52, 48 links, 47 joints
Links:
- removed link camera_base
- removed link head_rader
- added link head_camera_base, mass 0.0; visual mesh filename=package://kuavo_assets/models/biped_s52/meshes/head_camera_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
- added link head_camera_depth, mass 0.0000785398163397463; visual mesh filename=package://kuavo_assets/models/biped_s52/meshes/head_camera_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
- added link head_radar, mass 0.0; visual mesh filename=package://kuavo_assets/models/biped_s52/meshes/head_radar.S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
- added link waist_camera_base, mass 0.13300000; visual mesh filename=package://kuavo_assets/models/biped_s52/meshes/waist_camera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
- link waist_camera: mass 0.048238 -> 0.0000785398163397463
- link waist_yaw_link: mass 19.54016 -> 19.72026
Joints:
- removed joint camera_base
- removed joint head_rader_joint
- removed joint waist_camera
- added joint head_camera_base_joint: type fixed, parent zhead_2_link, child head_camera_base, origin xyz=0.099619 0 0.032844 rpy=0 0.3406 0, axis 0 0 0
- added joint head_camera_depth_joint: type fixed, parent head_camera_base, child head_camera_depth, origin xyz=0.011715 0.0475 0.014312 rpy=0 0 0, axis 0 0 0
- added joint head_radar_joint: type fixed, parent zhead_1_link, child head_radar, origin xyz=0 0 -0.078453 rpy=0 0 0, axis 0 0 0
- added joint waist_camera_base_joint: type fixed, parent waist_yaw_link, child waist_camera_base, origin xyz=0.0787 0 -0.028149 rpy=0 0.59341 0, axis 0 0 0
- added joint waist_camera_joint: type fixed, parent waist_camera_base, child waist_camera, origin xyz=0.011715 0.0475 0.014312 rpy=0 0 0, axis 0 0 0
- joint leg_l6_joint: limit lower=-0.261799387799149 upper=0.261799387799149 effort=30.0 velocity=17.8 -> lower=-0.261799387799149 upper=0.261799387799149 effort=68.4 velocity=17.8
- joint leg_r6_joint: limit lower=-0.261799387799149 upper=0.261799387799149 effort=30.0 velocity=17.8 -> lower=-0.261799387799149 upper=0.261799387799149 effort=68.4 velocity=17.8

File: src/kuavo_assets/models/biped_s52/urdf/biped_s52_gazebo.xacro (robot description, xacro)
@@ -6,5 +6,5 @@
   <xacro:include filename="$(find realsense_ros_gazebo)/xacro/depthcam.xacro"/>
   <!-- d435 声明 -->
-  <xacro:realsense_d435 sensor_name="camera" parent_link="camera_base" rate="30">
+  <xacro:realsense_d435 sensor_name="camera" parent_link="head_camera_base" rate="30">
     <origin rpy="0 0 0 " xyz="0 0 0"/>
   </xacro:realsense_d435>

File: src/kuavo_assets/models/biped_s52/urdf/drake/biped_v3_arm.urdf (robot description, URDF)
Before this commit: robot biped_s52, 20 links, 19 joints
Links:
- removed link zarm_r7_virtual_thumb_link
- added link zarm_l1_ref_link; visual sphere radius=0.001
Joints:
- removed joint zarm_r7_virtual_thumb_joint_ee
- added joint zarm_l1_ref_joint: type fixed, parent waist_yaw_link, child zarm_l1_ref_link, origin xyz=-0.003 0.1737 0.2831 rpy=0 0 0

File: src/kuavo_assets/models/biped_s53/urdf/biped_s53.urdf (robot description, URDF)
Before this commit: robot biped_s53, 48 links, 47 joints
Links:
- removed link camera_base
- removed link head_rader
- added link head_camera_base, mass 0.0; visual mesh filename=package://kuavo_assets/models/biped_s53/meshes/head_camera_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
- added link head_camera_depth, mass 0.0000785398163397463; visual mesh filename=package://kuavo_assets/models/biped_s53/meshes/head_camera_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
- added link head_radar, mass 0.0; visual mesh filename=package://kuavo_assets/models/biped_s53/meshes/head_radar.S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
- added link waist_camera_base, mass 0.13300000; visual mesh filename=package://kuavo_assets/models/biped_s53/meshes/waist_camera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
- link waist_camera: mass 0.13300 -> 0.0000785398163397463
- link waist_yaw_link: mass 19.98211 -> 19.98191
Joints:
- removed joint camera_base
- removed joint head_rader_joint
- removed joint waist_camera
- added joint head_camera_base_joint: type fixed, parent zhead_2_link, child head_camera_base, origin xyz=0.099619 0 0.032844 rpy=0 0.3406 0, axis 0 0 0
- added joint head_camera_depth_joint: type fixed, parent head_camera_base, child head_camera_depth, origin xyz=0.011715 0.0475 0.014312 rpy=0 0 0, axis 0 0 0
- added joint head_radar_joint: type fixed, parent zhead_1_link, child head_radar, origin xyz=0 0 -0.078453 rpy=0 0 0, axis 0 0 0
- added joint waist_camera_base_joint: type fixed, parent waist_yaw_link, child waist_camera_base, origin xyz=0.0787 0 -0.028149 rpy=0 0.59341 0, axis 0 0 0
- added joint waist_camera_joint: type fixed, parent waist_camera_base, child waist_camera, origin xyz=0.011715 0.0475 0.014312 rpy=0 0 0, axis 0 0 0
- joint dummy_to_base_link: type floating -> fixed
- joint leg_l6_joint: limit lower=-0.261799387799149 upper=0.261799387799149 effort=30.0 velocity=17.8 -> lower=-0.261799387799149 upper=0.261799387799149 effort=68.4 velocity=17.8
- joint leg_r6_joint: limit lower=-0.261799387799149 upper=0.261799387799149 effort=30.0 velocity=17.8 -> lower=-0.261799387799149 upper=0.261799387799149 effort=68.4 velocity=17.8

File: src/kuavo_assets/models/biped_s53/urdf/biped_s53_gazebo.urdf (robot description, URDF)
Before this commit: robot biped_s53, 48 links, 47 joints
Links:
- removed link camera_base
- removed link head_rader
- added link head_camera_base, mass 0.0; visual mesh filename=package://kuavo_assets/models/biped_s53/meshes/head_camera_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
- added link head_camera_depth, mass 0.0000785398163397463; visual mesh filename=package://kuavo_assets/models/biped_s53/meshes/head_camera_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
- added link head_radar, mass 0.0; visual mesh filename=package://kuavo_assets/models/biped_s53/meshes/head_radar.S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
- added link waist_camera_base, mass 0.13300000; visual mesh filename=package://kuavo_assets/models/biped_s53/meshes/waist_camera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
- link waist_camera: mass 0.048238 -> 0.0000785398163397463
- link waist_yaw_link: mass 21.63516 -> 21.81526
Joints:
- removed joint camera_base
- removed joint head_rader_joint
- removed joint waist_camera
- added joint head_camera_base_joint: type fixed, parent zhead_2_link, child head_camera_base, origin xyz=0.099619 0 0.032844 rpy=0 0.3406 0, axis 0 0 0
- added joint head_camera_depth_joint: type fixed, parent head_camera_base, child head_camera_depth, origin xyz=0.011715 0.0475 0.014312 rpy=0 0 0, axis 0 0 0
- added joint head_radar_joint: type fixed, parent zhead_1_link, child head_radar, origin xyz=0 0 -0.078453 rpy=0 0 0, axis 0 0 0
- added joint waist_camera_base_joint: type fixed, parent waist_yaw_link, child waist_camera_base, origin xyz=0.0787 0 -0.028149 rpy=0 0.59341 0, axis 0 0 0
- added joint waist_camera_joint: type fixed, parent waist_camera_base, child waist_camera, origin xyz=0.011715 0.0475 0.014312 rpy=0 0 0, axis 0 0 0
- joint leg_l6_joint: limit lower=-0.261799387799149 upper=0.261799387799149 effort=30.0 velocity=17.8 -> lower=-0.261799387799149 upper=0.261799387799149 effort=68.4 velocity=17.8
- joint leg_r6_joint: limit lower=-0.261799387799149 upper=0.261799387799149 effort=30.0 velocity=17.8 -> lower=-0.261799387799149 upper=0.261799387799149 effort=68.4 velocity=17.8

File: src/kuavo_assets/models/biped_s53/urdf/biped_s53_gazebo.xacro (robot description, xacro)
@@ -6,5 +6,5 @@
   <xacro:include filename="$(find realsense_ros_gazebo)/xacro/depthcam.xacro"/>
   <!-- d435 声明 -->
-  <xacro:realsense_d435 sensor_name="camera" parent_link="camera_base" rate="30">
+  <xacro:realsense_d435 sensor_name="camera" parent_link="head_camera_base" rate="30">
     <origin rpy="0 0 0 " xyz="0 0 0"/>
   </xacro:realsense_d435>

File: src/kuavo_assets/models/biped_s54/urdf/biped_s54.urdf (robot description, URDF)
Before this commit: robot biped_s54, 48 links, 47 joints
Links:
- removed link camera_base
- removed link head_rader
- added link head_camera_base, mass 0.0; visual mesh filename=package://kuavo_assets/models/biped_s54/meshes/head_camera_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
- added link head_camera_depth, mass 0.0000785398163397463; visual mesh filename=package://kuavo_assets/models/biped_s54/meshes/head_camera_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
- added link head_radar, mass 0.0; visual mesh filename=package://kuavo_assets/models/biped_s54/meshes/head_radar.S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
- added link waist_camera_base, mass 0.13300000; visual mesh filename=package://kuavo_assets/models/biped_s54/meshes/waist_camera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
- link waist_camera: mass 0.13300 -> 0.0000785398163397463
- link waist_yaw_link: mass 20.23838 -> 20.50328
Joints:
- removed joint camera_base
- removed joint head_rader_joint
- removed joint waist_camera
- added joint head_camera_base_joint: type fixed, parent zhead_2_link, child head_camera_base, origin xyz=0.099619 0 0.032844 rpy=0 0.3406 0, axis 0 0 0
- added joint head_camera_depth_joint: type fixed, parent head_camera_base, child head_camera_depth, origin xyz=0.011715 0.0475 0.014312 rpy=0 0 0, axis 0 0 0
- added joint head_radar_joint: type fixed, parent zhead_1_link, child head_radar, origin xyz=0 0 -0.078453 rpy=0 0 0, axis 0 0 0
- added joint waist_camera_base_joint: type fixed, parent waist_yaw_link, child waist_camera_base, origin xyz=0.0787 0 -0.028149 rpy=0 0.59341 0, axis 0 0 0
- added joint waist_camera_joint: type fixed, parent waist_camera_base, child waist_camera, origin xyz=0.011715 0.0475 0.014312 rpy=0 0 0, axis 0 0 0
- joint leg_l6_joint: limit lower=-0.261799387799149 upper=0.261799387799149 effort=30.0 velocity=17.8 -> lower=-0.261799387799149 upper=0.261799387799149 effort=68.4 velocity=17.8
- joint leg_r6_joint: limit lower=-0.261799387799149 upper=0.261799387799149 effort=30.0 velocity=17.8 -> lower=-0.261799387799149 upper=0.261799387799149 effort=68.4 velocity=17.8

File: src/kuavo_assets/models/biped_s54/urdf/biped_s54_gazebo.urdf (robot description, URDF)
Before this commit: robot biped_s54, 48 links, 47 joints
Links:
- removed link camera_base
- removed link head_rader
- added link head_camera_base, mass 0.0; visual mesh filename=package://kuavo_assets/models/biped_s54/meshes/head_camera_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
- added link head_camera_depth, mass 0.0000785398163397463; visual mesh filename=package://kuavo_assets/models/biped_s54/meshes/head_camera_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
- added link head_radar, mass 0.0; visual mesh filename=package://kuavo_assets/models/biped_s54/meshes/head_radar.S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
- added link waist_camera_base, mass 0.13300000; visual mesh filename=package://kuavo_assets/models/biped_s54/meshes/waist_camera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
- link waist_camera: mass 0.13300 -> 0.0000785398163397463
- link waist_yaw_link: mass 20.23838 -> 20.50328
Joints:
- removed joint camera_base
- removed joint head_rader_joint
- removed joint waist_camera
- added joint head_camera_base_joint: type fixed, parent zhead_2_link, child head_camera_base, origin xyz=0.099619 0 0.032844 rpy=0 0.3406 0, axis 0 0 0
- added joint head_camera_depth_joint: type fixed, parent head_camera_base, child head_camera_depth, origin xyz=0.011715 0.0475 0.014312 rpy=0 0 0, axis 0 0 0
- added joint head_radar_joint: type fixed, parent zhead_1_link, child head_radar, origin xyz=0 0 -0.078453 rpy=0 0 0, axis 0 0 0
- added joint waist_camera_base_joint: type fixed, parent waist_yaw_link, child waist_camera_base, origin xyz=0.0787 0 -0.028149 rpy=0 0.59341 0, axis 0 0 0
- added joint waist_camera_joint: type fixed, parent waist_camera_base, child waist_camera, origin xyz=0.011715 0.0475 0.014312 rpy=0 0 0, axis 0 0 0
- joint leg_l6_joint: limit lower=-0.261799387799149 upper=0.261799387799149 effort=30.0 velocity=17.8 -> lower=-0.261799387799149 upper=0.261799387799149 effort=68.4 velocity=17.8
- joint leg_r6_joint: limit lower=-0.261799387799149 upper=0.261799387799149 effort=30.0 velocity=17.8 -> lower=-0.261799387799149 upper=0.261799387799149 effort=68.4 velocity=17.8

File: src/kuavo_assets/models/biped_s54/urdf/biped_s54_gazebo.xacro (robot description, xacro)
@@ -6,5 +6,5 @@
   <xacro:include filename="$(find realsense_ros_gazebo)/xacro/depthcam.xacro"/>
   <!-- d435 声明 -->
-  <xacro:realsense_d435 sensor_name="camera" parent_link="camera_base" rate="30">
+  <xacro:realsense_d435 sensor_name="camera" parent_link="head_camera_base" rate="30">
     <origin rpy="0 0 0 " xyz="0 0 0"/>
   </xacro:realsense_d435>
