Commit message: sync https://www.lejuhub.com/highlydynamic/kuavo-ros-control/commit/c0cc1e2dedd1ca5083617351cf8c76d075feb317

File: src/kuavo_assets/models/biped_s60/urdf/biped_s60.urdf (robot description, URDF)
Before this commit: robot biped_s60, 34 links, 33 joints
Links:
- added link camera_base, mass 0.0482361371130408; visual mesh filename=package://kuavo_assets/models/biped_s60/meshes/head_camera.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
- link camera: mass 1e-6 -> 0.0482361371130408; geometry 
- link radar: mass 1e-6 -> 0.001
- link waist_yaw_link: mass 8.79680408 -> 11.56094002
- link zarm_l1_link: mass 0.962 -> 0.91653322
- link zarm_l2_link: mass 0.57 -> 0.38767390
- link zarm_l3_link: mass 1.65 -> 1.77926875
- link zarm_l4_link: mass 0.429 -> 0.58507821; geometry collision cylinder length=0.26 radius=0.05; visual mesh filename=package://kuavo_assets/models/biped_s60/meshes/l_forearm.STL
- link zarm_l5_link: mass 0.61 -> 0.68679955
- link zarm_l6_link: mass 0.331 -> 0.39387181
- link zarm_l7_link: mass 0.64 -> 0.71537800
- link zarm_r1_link: mass 0.962 -> 0.91653322
- link zarm_r2_link: mass 0.57 -> 0.38767390
- link zarm_r3_link: mass 1.65 -> 1.77926875
- link zarm_r4_link: mass 0.429 -> 0.58507821; geometry collision cylinder length=0.26 radius=0.05; visual mesh filename=package://kuavo_assets/models/biped_s60/meshes/r_forearm.STL
- link zarm_r5_link: mass 0.61 -> 0.68679955
- link zarm_r6_link: mass 0.331 -> 0.39387181
- link zarm_r7_link: mass 0.64 -> 0.71537800
- link zhead_1_link: mass 1.06289355 -> 0.83597358; geometry collision sphere radius=0.1; visual mesh filename=package://kuavo_assets/models/biped_s60/meshes/head_yaw_new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
- link zhead_2_link: mass 0.20029579 -> 0.75473516; geometry visual mesh filename=package://kuavo_assets/models/biped_s60/meshes/head_pitch_n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
Joints:
- removed joint LB_wheel_pitch
- removed joint LB_wheel_yaw
- removed joint LF_wheel_pitch
- removed joint LF_wheel_yaw
- removed joint RB_wheel_pitch
- removed joint RB_wheel_yaw
- removed joint RF_wheel_pitch
- removed joint RF_wheel_yaw
- added joint LB_wheel_pitch_joint: type continuous, parent LB_wheel_yaw, child LB_wheel_pitch, origin xyz=0 0 -0.1103 rpy=0 0 0
- added joint LB_wheel_yaw_joint: type continuous, parent base_link, child LB_wheel_yaw, origin xyz=-0.253 0.1785 0.1853 rpy=0 0 0
- added joint LF_wheel_pitch_joint: type continuous, parent LF_wheel_yaw, child LF_wheel_pitch, origin xyz=0.0 0.0 -0.1103 rpy=0 0 0
- added joint LF_wheel_yaw_joint: type continuous, parent base_link, child LF_wheel_yaw, origin xyz=0.253 0.1785 0.1853 rpy=0 0 0
- added joint RB_wheel_pitch_joint: type continuous, parent RB_wheel_yaw, child RB_wheel_pitch, origin xyz=0 0 -0.1103 rpy=0 0 0
- added joint RB_wheel_yaw_joint: type continuous, parent base_link, child RB_wheel_yaw, origin xyz=-0.253 -0.1785 0.1853 rpy=0 0 0
- added joint RF_wheel_pitch_joint: type continuous, parent RF_wheel_yaw, child RF_wheel_pitch, origin xyz=0 0 -0.1103 rpy=0 0 0
- added joint RF_wheel_yaw_joint: type continuous, parent base_link, child RF_wheel_yaw, origin xyz=0.253 -0.1785 0.1853 rpy=0 0 0
- added joint camera_base_joint: type fixed, parent zhead_2_link, child camera_base, origin xyz=0.099478 0 0.032897 rpy=0 0.35805 0
- joint camera: origin xyz=0.094395257832706 0 0.11395418930214 rpy=0 0.310766624316135 0 -> xyz=0.011715 0.0475 0.014311 rpy=0 0 0; parent zhead_2_link -> camera_base
- joint knee_joint: origin xyz=0 0.017 0.0805 rpy=0 0.0 0 -> xyz=0.2265 0.017 0.2658 rpy=0 0.0 0
- joint leg_joint: origin xyz=-0.48618 0 0.11672 rpy=0 0.0 0 -> xyz=-0.48618 0 0.11672 rpy=0 -0.251 0
- joint radar: origin xyz=0 0 -0.0264531741828733 rpy=0 0 0 -> xyz=0 0 0.059701 rpy=0 0 0
- joint waist_pitch_joint: origin xyz=0.49384 0 0.078217 rpy=0 0 0 -> xyz=0.49384 0 0.078217 rpy=0 0.236 0
- joint waist_yaw_joint: axis  0 0 1 -> 0 0 1; limit lower=-3.14 upper=3.14 effort=267 velocity=22.5 -> lower=-3.238 upper=3.238 effort=267 velocity=22.5
- joint zarm_l1_joint: origin xyz=-0.0175 0.2917 0.20400000 rpy=0 0 0 -> xyz=0 0.1717 0.242 rpy=0 0 0
- joint zarm_l2_joint: origin xyz=0 0 0 rpy=0 0 0 -> xyz=0 0.081 0 rpy=0 0 0
- joint zarm_l4_joint: origin xyz=0.0200000000000006 0 -0.283699999999996 rpy=0 0 0 -> xyz=0.02 0 -0.2837 rpy=0 0 0
- joint zarm_l5_joint: origin xyz=-0.0200000000000025 0 -0.127037274261591 rpy=0 0 0 -> xyz=-0.02 0 -0.1195 rpy=0 0 0
- joint zarm_l6_joint: origin xyz=0.000199999999999079 0 -0.106462725738415 rpy=0 0 0 -> xyz=0.0 0 -0.114 rpy=0 0 0
- joint zarm_l7_joint: origin xyz=0 0 -0.0210004653879916 rpy=0 0 0 -> xyz=0 0 -0.021 rpy=0 0 0
- joint zarm_r1_joint: origin xyz=-0.0175 -0.2917 0.20400000 rpy=0 0 0 -> xyz=0 -0.1717 0.242 rpy=0 0 0
- joint zarm_r2_joint: origin xyz=0 0 0 rpy=0 0 0 -> xyz=0 -0.081 0 rpy=0 0 0
- joint zarm_r4_joint: origin xyz=0.0200000000000024 0 -0.2837 rpy=0 0 0 -> xyz=0.02 0 -0.2837 rpy=0 0 0
- joint zarm_r5_joint: origin xyz=-0.0200000000000001 0 -0.127037274261587 rpy=0 0 0 -> xyz=-0.02 0 -0.1195 rpy=0 0 0
- joint zarm_r6_joint: origin xyz=0 0 -0.106462725738415 rpy=0 0 0 -> xyz=0.0 0 -0.114 rpy=0 0 0
- joint zarm_r7_joint: origin xyz=0 0 -0.0209999999999999 rpy=0 0 0 -> xyz=0.0 0 -0.021 rpy=0 0 0
- joint zhead_1_joint: origin xyz=-0.01850000 0.0 0.40035 rpy=0 0 0 -> xyz=0 0 0.3164 rpy=0 0 0
- joint zhead_2_joint: origin xyz=0 0 0 rpy=0 0 0 -> xyz=0 0 0.13795 rpy=0 0 0

File: src/kuavo_assets/models/biped_s60/urdf/biped_s60_gazebo.urdf (robot description, URDF)
Before this commit: robot biped_s60, 34 links, 33 joints
Links:
- link LB_wheel_pitch: geometry collision cylinder length=0.053 radius=0.075; visual mesh filename=package://kuavo_assets/models/biped_s60/meshes/LB_wheel_pit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
- link LF_wheel_pitch: geometry collision cylinder length=0.053 radius=0.075; visual mesh filename=package://kuavo_assets/models/biped_s60/meshes/LF_wheel_pit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
- link RB_wheel_pitch: geometry collision cylinder length=0.053 radius=0.075; visual mesh filename=package://kuavo_assets/models/biped_s60/meshes/RB_wheel_pit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
- link RF_wheel_pitch: geometry collision cylinder length=0.053 radius=0.075; visual mesh filename=package://kuavo_assets/models/biped_s60/meshes/RF_wheel_pit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
- link camera: mass 1e-6 -> 0.001
- link radar: mass 1e-6 -> 0.001
- link waist_yaw_link: mass 8.79680408 -> 11.56094002
- link zarm_l1_link: mass 0.962 -> 0.91653322
- link zarm_l2_link: mass 0.57 -> 0.38767390
- link zarm_l3_link: mass 1.65 -> 1.77926875
- link zarm_l4_link: mass 0.429 -> 0.58507821; geometry visual mesh filename=package://kuavo_assets/models/biped_s60/meshes/l_forearm.STL
- link zarm_l5_link: mass 0.61 -> 0.68679955
- link zarm_l6_link: mass 0.331 -> 0.39387181
- link zarm_l7_link: mass 0.64 -> 0.71537800
- link zarm_r1_link: mass 0.962 -> 0.91653322
- link zarm_r2_link: mass 0.57 -> 0.38767390
- link zarm_r3_link: mass 1.65 -> 1.77926875
- link zarm_r4_link: mass 0.429 -> 0.58507821; geometry visual mesh filename=package://kuavo_assets/models/biped_s60/meshes/r_forearm.STL
- link zarm_r5_link: mass 0.61 -> 0.68679955
- link zarm_r6_link: mass 0.331 -> 0.39387181
- link zarm_r7_link: mass 0.64 -> 0.71537800
- link zhead_1_link: mass 1.06289355 -> 0.83597358; geometry collision sphere radius=0.1; visual mesh filename=package://kuavo_assets/models/biped_s60/meshes/head_yaw_new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
- link zhead_2_link: mass 0.20029579 -> 0.75473516; geometry visual mesh filename=package://kuavo_assets/models/biped_s60/meshes/head_pitch_n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
Joints:
- joint LB_wheel_pitch_joint: origin xyz=-2.0599051378023E-05 -0.0359499999999999 -0.110254588925895 rpy=0 0 0 -> xyz=0 0 -0.1103 rpy=0 0 0
- joint LB_wheel_yaw_joint: origin xyz=-0.479499999999996 0.178499999999997 -0.000500000000000111 rpy=0 0 0 -> xyz=-0.253 0.1785 0.1853 rpy=0 0 0
- joint LF_wheel_pitch_joint: origin xyz=-2.0599051378134E-05 -0.03595 -0.110254588925895 rpy=0 0 0 -> xyz=0.0 0.0 -0.1103 rpy=0 0 0
- joint LF_wheel_yaw_joint: origin xyz=0.0265000000000065 0.1785 -0.000500000000000105 rpy=0 0 0 -> xyz=0.253 0.1785 0.1853 rpy=0 0 0
- joint RB_wheel_pitch_joint: origin xyz=0 0.0359499999999987 -0.110055652556463 rpy=0 0 0 -> xyz=0 0 -0.1103 rpy=0 0 0
- joint RB_wheel_yaw_joint: origin xyz=-0.479499999999985 -0.178500000000001 -0.000500000000000111 rpy=0 0 0 -> xyz=-0.253 -0.1785 0.1853 rpy=0 0 0
- joint RF_wheel_pitch_joint: origin xyz=0 0.03595 -0.110056 rpy=0 0 0 -> xyz=0 0 -0.1103 rpy=0 0 0
- joint RF_wheel_yaw_joint: origin xyz=0.0265000000000133 -0.178499999999998 -0.000500000000000111 rpy=0 0 0 -> xyz=0.253 -0.1785 0.1853 rpy=0 0 0
- joint camera: origin xyz=0.094395257832706 0 0.11395418930214 rpy=0 0.310766624316135 0 -> xyz=0.099478 0 0.032897 rpy=0 0.35805 0
- joint knee_joint: origin xyz=0 0.017 0.0805 rpy=0 0.0 0 -> xyz=0.2265 0.017 0.2658 rpy=0 0.0 0
- joint leg_joint: origin xyz=-0.48618 0 0.11672 rpy=0 0 0 -> xyz=-0.48618 0 0.11672 rpy=0 -0.251 0
- joint radar: origin xyz=0 0 -0.0264531741828733 rpy=0 0 0 -> xyz=0 0 0.059701 rpy=0 0 0
- joint waist_pitch_joint: origin xyz=0.49384 0 0.078217 rpy=0 0 0 -> xyz=0.49384 0 0.078217 rpy=0 0.236 0
- joint waist_yaw_joint: axis  0 0 1 -> 0 0 1; limit lower=-3.14 upper=3.14 effort=267 velocity=22.5 -> lower=-3.238 upper=3.238 effort=267 velocity=22.5
- joint zarm_l1_joint: origin xyz=-0.0175 0.2917 0.20400000 rpy=0 0 0 -> xyz=0 0.1717 0.242 rpy=0 0 0
- joint zarm_l2_joint: origin xyz=0 0 0 rpy=0 0 0 -> xyz=0 0.081 0 rpy=0 0 0
- joint zarm_l4_joint: origin xyz=0.0200000000000006 0 -0.283699999999996 rpy=0 0 0 -> xyz=0.02 0 -0.2837 rpy=0 0 0
- joint zarm_l5_joint: origin xyz=-0.0200000000000025 0 -0.127037274261591 rpy=0 0 0 -> xyz=-0.02 0 -0.1195 rpy=0 0 0
- joint zarm_l6_joint: origin xyz=0.000199999999999079 0 -0.106462725738415 rpy=0 0 0 -> xyz=0.0 0 -0.114 rpy=0 0 0
- joint zarm_l7_joint: origin xyz=0 0 -0.0210004653879916 rpy=0 0 0 -> xyz=0 0 -0.021 rpy=0 0 0
- joint zarm_r1_joint: origin xyz=-0.0175 -0.2917 0.20400000 rpy=0 0 0 -> xyz=0 -0.1717 0.242 rpy=0 0 0
- joint zarm_r2_joint: origin xyz=0 0 0 rpy=0 0 0 -> xyz=0 -0.081 0 rpy=0 0 0
- joint zarm_r4_joint: origin xyz=0.0200000000000024 0 -0.2837 rpy=0 0 0 -> xyz=0.02 0 -0.2837 rpy=0 0 0
- joint zarm_r5_joint: origin xyz=-0.0200000000000001 0 -0.127037274261587 rpy=0 0 0 -> xyz=-0.02 0 -0.1195 rpy=0 0 0
- joint zarm_r6_joint: origin xyz=0 0 -0.106462725738415 rpy=0 0 0 -> xyz=0.0 0 -0.114 rpy=0 0 0
- joint zarm_r7_joint: origin xyz=0 0 -0.0209999999999999 rpy=0 0 0 -> xyz=0.0 0 -0.021 rpy=0 0 0
- joint zhead_1_joint: origin xyz=-0.01850000 0.0 0.40035 rpy=0 0 0 -> xyz=0 0 0.3164 rpy=0 0 0
- joint zhead_2_joint: origin xyz=0 0 0 rpy=0 0 0 -> xyz=0 0 0.13795 rpy=0 0 0

Commit message: sync https://www.lejuhub.com/highlydynamic/kuavo-ros-control/commit/99f23d40a562a2b71cd419a3c1ae3bd883a9d948

File: src/kuavo_assets/models/biped_s60/urdf/biped_s60.urdf (robot description, URDF)
Before this commit: robot biped_s60, 39 links, 38 joints
Joints:
- joint floating_base: child base_link -> dummy_link; parent dummy_link -> base_link

File: src/kuavo_assets/models/biped_s60/urdf/biped_s60_gazebo.urdf (robot description, URDF)
Before this commit: robot biped_s60, 34 links, 33 joints
Joints:
- joint floating_base: child base_link -> dummy_link; parent dummy_link -> base_link

File: src/kuavo_assets/models/biped_s60/urdf/drake/biped_v3_arm.urdf (robot description, URDF)
Before this commit: robot biped_s45, 17 links, 16 joints
Links:
- added link knee_link, mass 5.39660196; visual mesh filename=../../meshes/knee_pitch.STL
- added link leg_link, mass 12.35650958; visual mesh filename=../../meshes/leg_pitch.STL
- added link waist_link, mass 5.4305643; visual mesh filename=../../meshes/waist_pitch.STL
- added link waist_yaw_link, mass 11.56094002; collision cylinder length=0.6 radius=0.15; visual mesh filename=../../meshes/torso.STL
- added link zarm_l7_virtual_thumb_link; collision sphere radius=0.005
- added link zarm_r7_virtual_thumb_link; collision sphere radius=0.005
- link base_link: mass 11.56094002 -> 97.77291318; geometry visual mesh filename=../../meshes/chassis.STL
- link zarm_r2_link: geometry collision cylinder length=0.3 radius=0.05; visual mesh filename=../../meshes/r_arm_roll.STL
- link zarm_r4_link: geometry collision cylinder length=0.26 radius=0.05; visual mesh filename=../../meshes/r_forearm.STL
Joints:
- added joint knee_joint: type revolute, parent base_link, child knee_link, origin xyz=0.2265 0.017 0.2658 rpy=0 0.0 0, axis 0 1 0, limit lower=0 upper=1.448 effort=668.53 velocity=25.33
- added joint leg_joint: type revolute, parent knee_link, child leg_link, origin xyz=-0.48618 0 0.11672 rpy=0 -0.251 0, axis 0 1 0, limit lower=-2.81 upper=0.0 effort=668.53 velocity=25.33
- added joint waist_pitch_joint: type revolute, parent leg_link, child waist_link, origin xyz=0.49384 0 0.078217 rpy=0 0.236 0, axis  0 1 0, limit lower=0.0 upper=0.9 effort=618.48 velocity=25.33
- added joint waist_yaw_joint: type revolute, parent waist_link, child waist_yaw_link, origin xyz=0.0 -0.0165 0.209 rpy=0 0 0, axis 0 0 1, limit lower=-3.238 upper=3.238 effort=618.48 velocity=25.33
- added joint zarm_l7_virtual_thumb_joint_ee: type fixed, parent zarm_l7_end_effector, child zarm_l7_virtual_thumb_link, origin xyz=0.15 0 0 rpy=0 0 0
- added joint zarm_r7_virtual_thumb_joint_ee: type fixed, parent zarm_r7_end_effector, child zarm_r7_virtual_thumb_link, origin xyz=0.15 0 0 rpy=0 0 0
- joint zarm_l1_joint: limit lower=-3.14159265358979 upper=1.5707963267949 effort=66.0 velocity=18.8 -> lower=-2.4 upper=0.6 effort=66.0 velocity=18.8; origin xyz=0 0.2527 0.242 rpy=0 0 0 -> xyz=0 0.1717 0.242 rpy=0 0 0; parent base_link -> waist_yaw_link
- joint zarm_l2_joint: limit lower=-0.349065850398866 upper=3.49065850398866 effort=75.0 velocity=8.0 -> lower=-0.349065850398866 upper=1.46 effort=75.0 velocity=8.0; origin xyz=0 0 0 rpy=0 0 0 -> xyz=0 0.081 0 rpy=0 0 0
- joint zarm_l3_joint: limit lower=-1.48352986419518 upper=1.48352986419518 effort=57.0 velocity=7.5 -> lower=-1.5707963267949 upper=0.46 effort=57.0 velocity=7.5
- joint zarm_r1_joint: limit lower=-3.14159265358979 upper=1.5707963267949 effort=66.0 velocity=18.8 -> lower=-2.4 upper=0.6 effort=66.0 velocity=18.8; origin xyz=0 -0.2527 0.242 rpy=0 0 0 -> xyz=0 -0.1717 0.242 rpy=0 0 0; parent base_link -> waist_yaw_link
- joint zarm_r2_joint: limit lower=-3.49065850398866 upper=0.349065850398866 effort=75.0 velocity=8.0 -> lower=-1.46 upper=0.349065850398866 effort=75.0 velocity=8.0; origin xyz=0 0 0 rpy=0 0 0 -> xyz=0 -0.081 0 rpy=0 0 0
- joint zarm_r3_joint: limit lower=-1.48352986419518 upper=1.48352986419518 effort=57.0 velocity=7.5 -> lower=-0.46 upper=1.5707963267949 effort=57.0 velocity=7.5

File: src/kuavo_assets/models/biped_s61/urdf/biped_s61.urdf (robot description, URDF)
Before this commit: robot biped_s61, 36 links, 35 joints
Links:
- removed link camera
- removed link camera_base
- added link head_camera_base, mass 0.0482361371130408; visual mesh filename=package://kuavo_assets/models/biped_s61/meshes/head_camera.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
- added link head_camera_depth, mass 0.0482361371130408
Joints:
- removed joint camera
- removed joint camera_base_joint
- added joint head_camera_base_joint: type fixed, parent zhead_2_link, child head_camera_base, origin xyz=0.099619 0 0.032844 rpy=0 0.3406 0
- added joint head_camera_depth_joint: type fixed, parent head_camera_base, child head_camera_depth, origin xyz=0.011715 0.0475 0.014311 rpy=0 0 0
- joint floating_base: child base_link -> dummy_link; parent dummy_link -> base_link

File: src/kuavo_assets/models/biped_s61/urdf/biped_s61_gazebo.urdf (robot description, URDF)
Before this commit: robot biped_s61, 39 links, 38 joints
Links:
- removed link camera
- added link head_camera_base, mass 0.001; visual mesh filename=package://kuavo_assets/models/biped_s61/meshes/head_camera.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
- added link head_camera_depth, mass 0.001
Joints:
- removed joint camera
- added joint head_camera_base_joint: type fixed, parent zhead_2_link, child head_camera_base, origin xyz=0.099619 0 0.032844 rpy=0 0.3406 0
- added joint head_camera_depth_joint: type fixed, parent head_camera_base, child head_camera_depth, origin xyz=0.011715 0.0475 0.014311 rpy=0 0 0
- joint floating_base: child base_link -> dummy_link; parent dummy_link -> base_link

File: src/kuavo_assets/models/biped_s61/urdf/biped_s61_gazebo.xacro (robot description, xacro)
@@ -5,5 +5,5 @@
   <!-- 可选：深度相机（如不需要可移除本段） -->
   <xacro:include filename="$(find realsense_ros_gazebo)/xacro/depthcam.xacro"/>
-  <xacro:realsense_d435 sensor_name="camera" parent_link="camera" rate="30">
+  <xacro:realsense_d435 sensor_name="camera" parent_link="head_camera_base" rate="30">
     <origin rpy="0 0 0" xyz="0 0 0"/>
   </xacro:realsense_d435>

File: src/kuavo_assets/models/biped_s61/urdf/drake/biped_v3_arm.urdf (robot description, URDF)
Before this commit: robot biped_s45, 17 links, 16 joints
Links:
- added link base_to_joint, mass 7.27493629; visual mesh filename=../../meshes/knee_link.STL
- added link knee_link, mass 13.41361777; visual mesh filename=../../meshes/leg_Link.STL
- added link leg_link, mass 9.78118294; visual mesh filename=../../meshes/waist_pitch_Link.STL
- added link waist_link, mass 4.65997944; visual mesh filename=../../meshes/waist_yaw_Link.STL
- added link waist_yaw_link, mass 11.56094002; collision cylinder length=0.6 radius=0.15; visual mesh filename=../../meshes/torso.STL
- added link zarm_l7_end_effector_1
- added link zarm_l7_end_effector_2
- added link zarm_l7_virtual_thumb_link; collision sphere radius=0.005
- added link zarm_r7_end_effector_1
- added link zarm_r7_end_effector_2
- added link zarm_r7_virtual_thumb_link; collision sphere radius=0.005
- link base_link: mass 11.56094002 -> 121.0; geometry collision cylinder length=0.32 radius=0.37; visual mesh filename=../../meshes/base_link.STL
Joints:
- added joint base_to_joint: type fixed, parent base_link, child base_to_joint, origin xyz=0.098 0 0.27064321 rpy=0 0 0
- added joint knee_joint: type revolute, parent base_to_joint, child knee_link, origin xyz=0 0 0.1055 rpy=0 0 0, axis 0 1 0, limit lower=0 upper=1.448 effort=668.53 velocity=25.33
- added joint leg_joint: type revolute, parent knee_link, child leg_link, origin xyz=-0.46521 0 0.18325 rpy=0 0 0, axis 0 1 0, limit lower=-2.81 upper=0.0 effort=668.53 velocity=25.33
- added joint waist_pitch_joint: type revolute, parent leg_link, child waist_link, origin xyz=0.48296 0 0.12941 rpy=0 0 0, axis 0 1 0, limit lower=0.0 upper=0.9 effort=618.48 velocity=25.33
- added joint waist_yaw_joint: type revolute, parent waist_link, child waist_yaw_link, origin xyz=0 0 0.235 rpy=0 0 0, axis 0 0 1, limit lower=-3.14159265358979 upper=3.14159265358979 effort=618.48 velocity=25.33
- added joint zarm_l7_end_effector_1_joint: type fixed, parent zarm_l7_link, child zarm_l7_end_effector_1, origin xyz=0 0.0 -0.08 rpy=0 0 0
- added joint zarm_l7_end_effector_2_joint: type fixed, parent zarm_l7_link, child zarm_l7_end_effector_2, origin xyz=0.03 0.0 -0.17 rpy=0 0 0
- added joint zarm_l7_virtual_thumb_joint_ee: type fixed, parent zarm_l7_end_effector, child zarm_l7_virtual_thumb_link, origin xyz=0.15 0 0 rpy=0 0 0
- added joint zarm_r7_end_effector_1_joint: type fixed, parent zarm_r7_link, child zarm_r7_end_effector_1, origin xyz=0 0.0 -0.08 rpy=0 0 0
- added joint zarm_r7_end_effector_2_joint: type fixed, parent zarm_r7_link, child zarm_r7_end_effector_2, origin xyz=0.03 0.0 -0.17 rpy=0 0 0
- added joint zarm_r7_virtual_thumb_joint_ee: type fixed, parent zarm_r7_end_effector, child zarm_r7_virtual_thumb_link, origin xyz=0.15 0 0 rpy=0 0 0
- joint zarm_l1_joint: parent base_link -> waist_yaw_link
- joint zarm_r1_joint: parent base_link -> waist_yaw_link
