Commit message: sync https://www.lejuhub.com/highlydynamic/kuavo-ros-control/commit/135829a997544480aedf0944ccf04a55ce892c69

File: src/kuavo_assets/models/biped_s40/urdf/biped_s40.urdf (robot description, URDF)
Before this commit: robot biped_s40, 46 links, 45 joints
Links:
- link base_link: mass 22.6719 -> 22.6889

File: src/kuavo_assets/models/biped_s40/urdf/biped_s40_gazebo.urdf (robot description, URDF)
Before this commit: robot biped_s40, 46 links, 45 joints
Links:
- link base_link: mass 22.6719 -> 22.6889

File: src/kuavo_assets/models/biped_s40/urdf/drake/biped_v3.urdf (robot description, URDF)
Before this commit: robot biped_v3, 13 links, 12 joints
Links:
- link torso: mass 33.6709 -> 33.6879

File: src/kuavo_assets/models/biped_s40/urdf/drake/biped_v3_all_joint.urdf (robot description, URDF)
Before this commit: robot biped_v3_all_joint, 35 links, 30 joints
Links:
- link torso: mass 23.55403 -> 23.57103

File: src/kuavo_assets/models/biped_s40/urdf/drake/biped_v3_full.urdf (robot description, URDF)
Before this commit: robot biped_v3_full, 27 links, 26 joints
Links:
- link torso: mass 24.1969 -> 24.2139

Commit message: sync https://www.lejuhub.com/highlydynamic/kuavo-ros-control/commit/b549b1ee37a11da2d6e52858abc5b742d4198347

File: src/kuavo_assets/models/biped_s40/urdf/biped_s40.urdf (robot description, URDF)
Before this commit: robot biped_s40, 46 links, 45 joints
Links:
- link base_link: mass 22.6889 -> 22.6719

File: src/kuavo_assets/models/biped_s40/urdf/biped_s40_gazebo.urdf (robot description, URDF)
Before this commit: robot biped_s40, 46 links, 45 joints
Links:
- link base_link: mass 22.6889 -> 22.6719

File: src/kuavo_assets/models/biped_s40/urdf/drake/biped_v3.urdf (robot description, URDF)
Before this commit: robot biped_v3, 13 links, 12 joints
Links:
- link torso: mass 33.6879 -> 33.6709

File: src/kuavo_assets/models/biped_s40/urdf/drake/biped_v3_all_joint.urdf (robot description, URDF)
Before this commit: robot biped_v3_all_joint, 35 links, 30 joints
Links:
- link torso: mass 23.57103 -> 23.55403

File: src/kuavo_assets/models/biped_s40/urdf/drake/biped_v3_full.urdf (robot description, URDF)
Before this commit: robot biped_v3_full, 27 links, 26 joints
Links:
- link torso: mass 24.2139 -> 24.1969
