Commit message: sync https://www.lejuhub.com/highlydynamic/kuavo-ros-control/commit/d5bc0442038a6c377a3c34de2c88710d314d8f19

File: src/kuavo_assets/models/biped_s40/urdf/biped_s40_gazebo.urdf (robot description, URDF)
Before this commit: robot biped_s40, 46 links, 45 joints
Joints:
- removed joint dummy_to_base_link
- added joint base_link_to_dummy_link: type fixed, parent base_link, child dummy_link, origin xyz=0 0 0 rpy=0 0 0

Commit message: sync https://www.lejuhub.com/highlydynamic/kuavo-ros-control/commit/9948e96a872cd6f952b6d0768c2b8046fb59aabf

File: src/kuavo_assets/models/biped_s40/urdf/biped_s40_gazebo.urdf (robot description, URDF)
Before this commit: robot biped_s40, 46 links, 45 joints
Links:
- link base_link: mass 22.6889 -> 22.6719
