Commit message: sync https://www.lejuhub.com/highlydynamic/kuavo-ros-control/commit/fbe93f17eb09bb747a1d693ce282cbf61c6bff55

File: src/kuavo_assets/models/biped_s40/urdf/biped_s40_gazebo.urdf (robot description, URDF)
Before this commit: robot biped_s40, 46 links, 45 joints
Links:
- link base_link: mass 22.6719 -> 22.6889
