Commit message: sync https://www.lejuhub.com/highlydynamic/kuavo-ros-control/commit/4e98c7d9f2dfef5c7dade2df07f620a283888d85

File: src/kuavo_assets/models/biped_s300049/urdf/biped_s300049.urdf (robot description, URDF)
Before this commit: robot biped_s300049, 73 links, 72 joints
Links:
- removed link l_Index_prox
- removed link l_index_dist
- removed link l_little_dist
- removed link l_little_prox
- removed link l_middle_dist
- removed link l_middle_prox
- removed link l_palm
- removed link l_ring_dist
- removed link l_ring_prox
- removed link l_thumb_dist
- removed link l_thumb_prox
- removed link r_index_dist
- removed link r_index_prox
- removed link r_little_dist
- removed link r_little_prox
- removed link r_middle_dist
- removed link r_middle_prox
- removed link r_palm
- removed link r_ring_dist
- removed link r_ring_prox
- removed link r_thumb_dist
- removed link r_thumb_prox
- added link l_hand_base_link, mass 0.4185; collision mesh filename=package://kuavo_assets/models/biped_s300049/L6V3.1_leju/L6V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; visual mesh filename=package://kuavo_assets/models/biped_s300049/L6V3.1_leju/L6V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
- added link l_index_distal, mass 0.018408; collision mesh filename=package://kuavo_assets/models/biped_s300049/L6V3.1_leju/L6V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; visual mesh filename=package://kuavo_assets/models/biped_s300049/L6V3.1_leju/L6V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
- added link l_index_proximal, mass 0.008553; collision mesh filename=package://kuavo_assets/models/biped_s300049/L6V3.1_leju/L6V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; visual mesh filename=package://kuavo_assets/models/biped_s300049/L6V3.1_leju/L6V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
- added link l_middle_distal, mass 0.018408; collision mesh filename=package://kuavo_assets/models/biped_s300049/L6V3.1_leju/L6V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; visual mesh filename=package://kuavo_assets/models/biped_s300049/L6V3.1_leju/L6V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
- added link l_middle_proximal, mass 0.008553; collision mesh filename=package://kuavo_assets/models/biped_s300049/L6V3.1_leju/L6V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; visual mesh filename=package://kuavo_assets/models/biped_s300049/L6V3.1_leju/L6V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
- added link l_pinky_distal, mass 0.018408; collision mesh filename=package://kuavo_assets/models/biped_s300049/L6V3.1_leju/L6V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; visual mesh filename=package://kuavo_assets/models/biped_s300049/L6V3.1_leju/L6V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
- added link l_pinky_proximal, mass 0.008553; collision mesh filename=package://kuavo_assets/models/biped_s300049/L6V3.1_leju/L6V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; visual mesh filename=package://kuavo_assets/models/biped_s300049/L6V3.1_leju/L6V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
- added link l_ring_distal, mass 0.018408; collision mesh filename=package://kuavo_assets/models/biped_s300049/L6V3.1_leju/L6V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; visual mesh filename=package://kuavo_assets/models/biped_s300049/L6V3.1_leju/L6V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
- added link l_ring_proximal, mass 0.008553; collision mesh filename=package://kuavo_assets/models/biped_s300049/L6V3.1_leju/L6V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; visual mesh filename=package://kuavo_assets/models/biped_s300049/L6V3.1_leju/L6V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
- added link l_thumb_distal, mass 0.018; collision mesh filename=package://kuavo_assets/models/biped_s300049/L6V3.1_leju/L6V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; visual mesh filename=package://kuavo_assets/models/biped_s300049/L6V3.1_leju/L6V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
- added link l_thumb_metacarpals, mass 0.065; collision mesh filename=package://kuavo_assets/models/biped_s300049/L6V3.1_leju/L6V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; visual mesh filename=package://kuavo_assets/models/biped_s300049/L6V3.1_leju/L6V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
- added link l_thumb_metacarpals_base1, mass 0.01; collision mesh filename=package://kuavo_assets/models/biped_s300049/L6V3.1_leju/L6V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; visual mesh filename=package://kuavo_assets/models/biped_s300049/L6V3.1_leju/L6V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
- added link l_wrist_ft_link, mass 0.161981; collision mesh filename=package://kuavo_assets/models/biped_s300049/L6V3.1_leju/L6V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 scale=0.001 0.001 0.001; visual mesh filename=package://kuavo_assets/models/biped_s300049/L6V3.1_leju/L6V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 scale=0.001 0.001 0.001
- added link r_hand_base_link, mass 0.4185; collision mesh filename=package://kuavo_assets/models/biped_s300049/L6V3.1_leju/L6V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; visual mesh filename=package://kuavo_assets/models/biped_s300049/L6V3.1_leju/L6V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
- added link r_index_distal, mass 0.018408; collision mesh filename=package://kuavo_assets/models/biped_s300049/L6V3.1_leju/L6V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; visual mesh filename=package://kuavo_assets/models/biped_s300049/L6V3.1_leju/L6V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
- added link r_index_proximal, mass 0.008553; collision mesh filename=package://kuavo_assets/models/biped_s300049/L6V3.1_leju/L6V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; visual mesh filename=package://kuavo_assets/models/biped_s300049/L6V3.1_leju/L6V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
- added link r_middle_distal, mass 0.018408; collision mesh filename=package://kuavo_assets/models/biped_s300049/L6V3.1_leju/L6V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; visual mesh filename=package://kuavo_assets/models/biped_s300049/L6V3.1_leju/L6V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
- added link r_middle_proximal, mass 0.008553; collision mesh filename=package://kuavo_assets/models/biped_s300049/L6V3.1_leju/L6V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; visual mesh filename=package://kuavo_assets/models/biped_s300049/L6V3.1_leju/L6V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
- added link r_pinky_distal, mass 0.018408; collision mesh filename=package://kuavo_assets/models/biped_s300049/L6V3.1_leju/L6V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; visual mesh filename=package://kuavo_assets/models/biped_s300049/L6V3.1_leju/L6V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
- added link r_pinky_proximal, mass 0.008553; collision mesh filename=package://kuavo_assets/models/biped_s300049/L6V3.1_leju/L6V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; visual mesh filename=package://kuavo_assets/models/biped_s300049/L6V3.1_leju/L6V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
- added link r_ring_distal, mass 0.018408; collision mesh filename=package://kuavo_assets/models/biped_s300049/L6V3.1_leju/L6V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; visual mesh filename=package://kuavo_assets/models/biped_s300049/L6V3.1_leju/L6V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
- added link r_ring_proximal, mass 0.008553; collision mesh filename=package://kuavo_assets/models/biped_s300049/L6V3.1_leju/L6V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; visual mesh filename=package://kuavo_assets/models/biped_s300049/L6V3.1_leju/L6V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
- added link r_thumb_distal, mass 0.018; collision mesh filename=package://kuavo_assets/models/biped_s300049/L6V3.1_leju/L6V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; visual mesh filename=package://kuavo_assets/models/biped_s300049/L6V3.1_leju/L6V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
- added link r_thumb_metacarpals, mass 0.065; collision mesh filename=package://kuavo_assets/models/biped_s300049/L6V3.1_leju/L6V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; visual mesh filename=package://kuavo_assets/models/biped_s300049/L6V3.1_leju/L6V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
- added link r_thumb_metacarpals_base1, mass 0.01; collision mesh filename=package://kuavo_assets/models/biped_s300049/L6V3.1_leju/L6V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; visual mesh filename=package://kuavo_assets/models/biped_s300049/L6V3.1_leju/L6V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
- added link r_wrist_ft_link, mass 0.161981; collision mesh filename=package://kuavo_assets/models/biped_s300049/L6V3.1_leju/L6V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 scale=0.001 0.001 0.001; visual mesh filename=package://kuavo_assets/models/biped_s300049/L6V3.1_leju/L6V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 scale=0.001 0.001 0.001
Joints:
- removed joint l_indexMCP
- removed joint l_indexPIP
- removed joint l_littleMCP
- removed joint l_littlePIP
- removed joint l_middleMCP
- removed joint l_middlePIP
- removed joint l_palm_fixed_joint
- removed joint l_ringMCP
- removed joint l_ringPIP
- removed joint l_thumbCMC
- removed joint l_thumbMCP
- removed joint r_indexMCP
- removed joint r_indexPIP
- removed joint r_littleMCP
- removed joint r_littlePIP
- removed joint r_middleMCP
- removed joint r_middlePIP
- removed joint r_palm_fixed_joint
- removed joint r_ringMCP
- removed joint r_ringPIP
- removed joint r_thumbCMC
- removed joint r_thumbMCP
- added joint l_index_dip: type revolute, parent l_index_proximal, child l_index_distal, origin xyz=0.001001 -0.000537 0.028003 rpy=0 0 0, axis 0 1 0, limit lower=0 upper=1.277039 effort=0 velocity=3.1, mimic joint=l_index_mcp_pitch multiplier=1.125676 offset=0
- added joint l_index_mcp_pitch: type revolute, parent l_hand_base_link, child l_index_proximal, origin xyz=-0.00066821 -0.028967 0.11722 rpy=0 0 0, axis 0 1 0, limit lower=0 upper=1.134464 effort=0.574 velocity=6.10
- added joint l_middle_dip: type revolute, parent l_middle_proximal, child l_middle_distal, origin xyz=0.000994 0.000058 0.028008 rpy=0 0 0, axis 0 1 0, limit lower=0 upper=1.277039 effort=0 velocity=3.1, mimic joint=l_middle_mcp_pitch multiplier=1.125676 offset=0
- added joint l_middle_mcp_pitch: type revolute, parent l_hand_base_link, child l_middle_proximal, origin xyz=-0.00066821 -0.0089013 0.12322 rpy=0 0 0, axis 0 1 0, limit lower=0 upper=1.134464 effort=0.574 velocity=6.10
- added joint l_pinky_dip: type revolute, parent l_pinky_proximal, child l_pinky_distal, origin xyz=0.000979 0.001534 0.027967 rpy=0 0 0, axis 0 1 0, limit lower=0 upper=1.277039 effort=0 velocity=3.1, mimic joint=l_pinky_mcp_pitch multiplier=1.125676 offset=0
- added joint l_pinky_mcp_pitch: type revolute, parent l_hand_base_link, child l_pinky_proximal, origin xyz=-0.00067852 0.029814 0.11424 rpy=0 0 0, axis 0 1 0, limit lower=0 upper=1.134464 effort=0.574 velocity=6.10
- added joint l_ring_dip: type revolute, parent l_ring_proximal, child l_ring_distal, origin xyz=0.000979 0.001534 0.027967 rpy=0 0 0, axis 0 1 0, limit lower=0 upper=1.277039 effort=0 velocity=3.1, mimic joint=l_ring_mcp_pitch multiplier=1.125676 offset=0
- added joint l_ring_mcp_pitch: type revolute, parent l_hand_base_link, child l_ring_proximal, origin xyz=-0.00067368 0.010717 0.11822 rpy=0 0 0, axis 0 1 0, limit lower=0 upper=1.134464 effort=0.574 velocity=6.10
- added joint l_thumb_cmc_pitch: type revolute, parent l_thumb_metacarpals_base1, child l_thumb_metacarpals, origin xyz=0.0057298 -0.01332 0.0027456 rpy=1.1083 0 0.40143, axis -1 0 0, limit lower=0 upper=0.837758 effort=1.008 velocity=3.47
- added joint l_thumb_cmc_roll: type revolute, parent l_hand_base_link, child l_thumb_metacarpals_base1, origin xyz=0.0078133 -0.029898 0.026692 rpy=-0.034907 0 0, axis 0 0 1, limit lower=-0.087266 upper=1.256637 effort=0.588 velocity=5.95
- added joint l_thumb_dip: type revolute, parent l_thumb_metacarpals, child l_thumb_distal, origin xyz=0 0.0061 0.0827 rpy=0 0 0, axis -1 0 0, limit lower=0 upper=0.963287 effort=0 velocity=1.7, mimic joint=l_thumb_cmc_pitch multiplier=1.226495 offset=0
- added joint l_wrist_ft_to_hand: type fixed, parent l_wrist_ft_link, child l_hand_base_link, origin xyz=0 0 -0.065 rpy=0 3.1415926 1.5707963
- added joint r_index_dip: type revolute, parent r_index_proximal, child r_index_distal, origin xyz=0.0009359 0 0.028002 rpy=0 0 0, axis 0 1 0, limit lower=0 upper=1.277039 effort=0 velocity=3.1, mimic joint=r_index_mcp_pitch multiplier=1.125676 offset=0
- added joint r_index_mcp_pitch: type revolute, parent r_hand_base_link, child r_index_proximal, origin xyz=-0.00066821 0.033467 0.11622 rpy=-0.087266 0 0, axis 0 1 0, limit lower=0 upper=1.134464 effort=0.574 velocity=6.10
- added joint r_middle_dip: type revolute, parent r_middle_proximal, child r_middle_distal, origin xyz=0.0009359 0 0.028002 rpy=0 0 0, axis 0 1 0, limit lower=0 upper=1.277039 effort=0 velocity=3.1, mimic joint=r_middle_mcp_pitch multiplier=1.125676 offset=0
- added joint r_middle_mcp_pitch: type revolute, parent r_hand_base_link, child r_middle_proximal, origin xyz=-0.00066821 0.0134013 0.12272 rpy=-0.034907 0 0, axis 0 1 0, limit lower=0 upper=1.134464 effort=0.574 velocity=6.10
- added joint r_pinky_dip: type revolute, parent r_pinky_proximal, child r_pinky_distal, origin xyz=0.0009359 0 0.028002 rpy=0 0 0, axis 0 1 0, limit lower=0 upper=1.277039 effort=0 velocity=3.1, mimic joint=r_pinky_mcp_pitch multiplier=1.125676 offset=0
- added joint r_pinky_mcp_pitch: type revolute, parent r_hand_base_link, child r_pinky_proximal, origin xyz=-0.00067852 -0.025314 0.11474 rpy=0.05236 0 0, axis 0 1 0, limit lower=0 upper=1.134464 effort=0.574 velocity=6.10
- added joint r_ring_dip: type revolute, parent r_ring_proximal, child r_ring_distal, origin xyz=0.0009359 0 0.028002 rpy=0 0 0, axis 0 1 0, limit lower=0 upper=1.277039 effort=0 velocity=3.1, mimic joint=r_ring_mcp_pitch multiplier=1.125676 offset=0
- added joint r_ring_mcp_pitch: type revolute, parent r_hand_base_link, child r_ring_proximal, origin xyz=-0.00067368 -0.006217 0.11872 rpy=0.017453 0 0, axis 0 1 0, limit lower=0 upper=1.134464 effort=0.574 velocity=6.10
- added joint r_thumb_cmc_pitch: type revolute, parent r_thumb_metacarpals_base1, child r_thumb_metacarpals, origin xyz=0.0054997 0.013314 0.0032166 rpy=-1.0762 0.013637 -0.40121, axis 1 0 0, limit lower=0 upper=0.837758 effort=1.008 velocity=3.47
- added joint r_thumb_cmc_roll: type revolute, parent r_hand_base_link, child r_thumb_metacarpals_base1, origin xyz=0.0078133 0.030812 0.025678 rpy=-0.034907 0 0, axis 0 0.034899 -0.99939, limit lower=-0.087266 upper=1.256637 effort=0.588 velocity=5.95
- added joint r_thumb_dip: type revolute, parent r_thumb_metacarpals, child r_thumb_distal, origin xyz=0 -0.0061 0.0827 rpy=0 0 0, axis 1 0 0, limit lower=0 upper=0.963287 effort=0 velocity=1.7, mimic joint=r_thumb_cmc_pitch multiplier=1.226495 offset=0
- added joint r_wrist_ft_to_hand: type fixed, parent r_wrist_ft_link, child r_hand_base_link, origin xyz=0 0 -0.065 rpy=-3.1415926 0 1.5707963
- added joint zarm_l7_to_l_wrist_ft: type fixed, parent zarm_l7_link, child l_wrist_ft_link, origin xyz=0 0 0 rpy=0 0 0
- added joint zarm_r7_to_r_wrist_ft: type fixed, parent zarm_r7_link, child r_wrist_ft_link, origin xyz=0 0 0 rpy=0 0 0

File: src/kuavo_assets/models/biped_s400049/urdf/biped_s400049.urdf (robot description, URDF)
Before this commit: robot biped_s400049, 73 links, 72 joints
Links:
- removed link l_Index_prox
- removed link l_index_dist
- removed link l_little_dist
- removed link l_little_prox
- removed link l_middle_dist
- removed link l_middle_prox
- removed link l_palm
- removed link l_ring_dist
- removed link l_ring_prox
- removed link l_thumb_dist
- removed link l_thumb_prox
- removed link r_index_dist
- removed link r_index_prox
- removed link r_little_dist
- removed link r_little_prox
- removed link r_middle_dist
- removed link r_middle_prox
- removed link r_palm
- removed link r_ring_dist
- removed link r_ring_prox
- removed link r_thumb_dist
- removed link r_thumb_prox
Joints:
- removed joint l_indexMCP
- removed joint l_indexPIP
- removed joint l_littleMCP
- removed joint l_littlePIP
- removed joint l_middleMCP
- removed joint l_middlePIP
- removed joint l_palm_fixed_joint
- removed joint l_ringMCP
- removed joint l_ringPIP
- removed joint l_thumbCMC
- removed joint l_thumbMCP
- removed joint r_indexMCP
- removed joint r_indexPIP
- removed joint r_littleMCP
- removed joint r_littlePIP
- removed joint r_middleMCP
- removed joint r_middlePIP
- removed joint r_palm_fixed_joint
- removed joint r_ringMCP
- removed joint r_ringPIP
- removed joint r_thumbCMC
- removed joint r_thumbMCP

Commit message: sync https://www.lejuhub.com/highlydynamic/kuavo-ros-control/commit/6dfd12cd8d5d5c397fdeee8815ce3b05d4bc44b4

File: src/kuavo_assets/models/biped_s300049/urdf/biped_s300049.urdf (robot description, URDF)
Before this commit: robot biped_s300049, 77 links, 76 joints
Links:
- link base_link: mass 28.27893803 -> 26.71633803

Commit message: sync https://www.lejuhub.com/highlydynamic/kuavo-ros-control/commit/b8743ae4542980fc851291d8921b9457faea872f

File: src/kuavo_assets/models/biped_s300049/urdf/biped_s300049.urdf (robot description, URDF)
Before this commit: robot biped_s300049, 77 links, 76 joints
Joints:
- removed joint l_thumb_cmc_roll
- removed joint l_thumb_dip
- removed joint r_thumb_cmc_roll
- removed joint r_thumb_dip
- added joint l_thumb_cmc_yaw: type revolute, parent l_hand_base_link, child l_thumb_metacarpals_base1, origin xyz=0.0078133 -0.029898 0.026692 rpy=-0.034907 0 0, axis 0 0 1, limit lower=-0.087266 upper=1.256637 effort=0.588 velocity=5.95
- added joint l_thumb_ip: type revolute, parent l_thumb_metacarpals, child l_thumb_distal, origin xyz=0 0.0061 0.0827 rpy=0 0 0, axis -1 0 0, limit lower=0 upper=0.963287 effort=0 velocity=1.7, mimic joint=l_thumb_cmc_pitch multiplier=1.226495 offset=0
- added joint r_thumb_cmc_yaw: type revolute, parent r_hand_base_link, child r_thumb_metacarpals_base1, origin xyz=0.0078133 0.030812 0.025678 rpy=-0.034907 0 0, axis 0 0.034899 -0.99939, limit lower=-0.087266 upper=1.256637 effort=0.588 velocity=5.95
- added joint r_thumb_ip: type revolute, parent r_thumb_metacarpals, child r_thumb_distal, origin xyz=0 -0.0061 0.0827 rpy=0 0 0, axis 1 0 0, limit lower=0 upper=0.963287 effort=0 velocity=1.7, mimic joint=r_thumb_cmc_pitch multiplier=1.226495 offset=0
- joint r_wrist_ft_to_hand: origin xyz=0 0 -0.065 rpy=-3.1415926 0 1.5707963 -> xyz=0 0 -0.065 rpy=0 3.1415926 -1.5707963
- joint zarm_r3_joint: axis 0 0 1 -> 0 1 0
- joint zarm_r5_joint: axis 0 0 1 -> 0 1 0

Commit message: sync https://www.lejuhub.com/highlydynamic/kuavo-ros-control/commit/d21d2f5e9787aa5481a95aa8af40b91a9464af37

File: src/kuavo_assets/models/biped_s300049/urdf/biped_s300049.urdf (robot description, URDF)
Before this commit: robot biped_s300049, 77 links, 76 joints
Links:
- link base_link: mass 26.71633803 -> 27.81233803
