Commit message: sync https://www.lejuhub.com/highlydynamic/kuavo-ros-control/commit/8b94b4ea445857a93a295e0332eb3a14b357265b

File: src/kuavo_assets/models/biped_s56/urdf/biped_s56.urdf (robot description, URDF)
Before this commit: robot biped_s56, 50 links, 49 joints
Links:
- link leg_l5_link: mass 0.07554 -> 0.33065201
- link leg_l6_link: mass 0.60538 -> 0.85589925
- link leg_r5_link: mass 0.07554 -> 0.33065201
- link leg_r6_link: mass 0.60538 -> 0.85589925
- link waist_camera: mass 0.001 -> 0.0000785398163397463
- link waist_camera_base: mass 0.13300 -> 0.13300000
- link waist_yaw_link: mass 19.98099 -> 19.98211
Joints:
- joint l_foot_heel_joint: origin xyz=-0.073164 0.0 -0.0595 rpy=0 0 0 -> xyz=-0.07316377 0.0 -0.0365 rpy=0 0 0
- joint l_foot_toe_joint: origin xyz=0.17084 0.0 -0.0595 rpy=0 0 0 -> xyz=0.17083623 0.0 -0.0365 rpy=0 0 0
- joint leg_l5_joint: origin xyz=0.002 0 -0.416 rpy=0 0 0 -> xyz=0 0 -0.416 rpy=0 0 0
- joint leg_l6_joint: origin xyz=0 0 0 rpy=0 0 0 -> xyz=0 0 -0.023 rpy=0 0 0
- joint leg_r5_joint: origin xyz=0.002 0 -0.416 rpy=0 0 0 -> xyz=0 0 -0.416 rpy=0 0 0
- joint leg_r6_joint: origin xyz=0 0 0 rpy=0 0 0 -> xyz=0 0 -0.023 rpy=0 0 0
- joint ll_foot_heel_joint: origin xyz=-0.073164 0.05 -0.0595 rpy=0 0 0 -> xyz=-0.07316377 0.05 -0.0365 rpy=0 0 0
- joint ll_foot_toe_joint: origin xyz=0.17084 0.05 -0.0595 rpy=0 0 0 -> xyz=0.17083623 0.05 -0.0365 rpy=0 0 0
- joint lr_foot_heel_joint: origin xyz=-0.073164 -0.05 -0.0595 rpy=0 0 0 -> xyz=-0.07316377 -0.05 -0.0365 rpy=0 0 0
- joint lr_foot_toe_joint: origin xyz=0.17084 -0.05 -0.0595 rpy=0 0 0 -> xyz=0.17083623 -0.05 -0.0365 rpy=0 0 0
- joint r_foot_heel_joint: origin xyz=-0.073164 0.0 -0.0595 rpy=0 0 0 -> xyz=-0.07316377 0.0 -0.0365 rpy=0 0 0
- joint r_foot_toe_joint: origin xyz=0.17084 0.0 -0.0595 rpy=0 0 0 -> xyz=0.17083623 0.0 -0.0365 rpy=0 0 0
- joint rl_foot_heel_joint: origin xyz=-0.073164 0.05 -0.0595 rpy=0 0 0 -> xyz=-0.07316377 0.05 -0.0365 rpy=0 0 0
- joint rl_foot_toe_joint: origin xyz=0.17084 0.05 -0.0595 rpy=0 0 0 -> xyz=0.17083623 0.05 -0.0365 rpy=0 0 0
- joint rr_foot_heel_joint: origin xyz=-0.073164 -0.05 -0.0595 rpy=0 0 0 -> xyz=-0.07316377 -0.05 -0.0365 rpy=0 0 0
- joint rr_foot_toe_joint: origin xyz=0.17084 -0.05 -0.0595 rpy=0 0 0 -> xyz=0.17083623 -0.05 -0.0365 rpy=0 0 0
- joint waist_camera_base_joint: origin xyz=0.09462 0 -0.010454 rpy=0 1.0472 0 -> xyz=0.0787 0 -0.028149 rpy=0 0.59341 0
- joint waist_yaw_joint: origin xyz=0 0 0.111 rpy=0 0 0 -> xyz=0 0 0.1114 rpy=0 0 0
- joint zarm_l1_joint: origin xyz=-0.003 0.253 0.2834 rpy=0 0 0 -> xyz=-0.003 0.2527 0.283 rpy=0 0 0
- joint zarm_r1_joint: origin xyz=-0.003 -0.253 0.2834 rpy=0 0 0 -> xyz=-0.003 -0.2527 0.283 rpy=0 0 0
- joint zhead_1_joint: origin xyz=-0.003 0.0 0.49125 rpy=0 0 0 -> xyz=-0.003 0.0 0.49535 rpy=0 0 0

File: src/kuavo_assets/models/biped_s56/urdf/biped_s56_gazebo.urdf (robot description, URDF)
Before this commit: robot biped_s56, 48 links, 47 joints
Links:
- removed link camera_base
- removed link head_rader
- added link head_camera_base, mass 0.0; visual mesh filename=package://kuavo_assets/models/biped_s56/meshes/head_camera_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
- added link head_camera_depth, mass 0.0000785398163397463; visual mesh filename=package://kuavo_assets/models/biped_s56/meshes/head_camera_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
- added link head_radar, mass 0.0; visual mesh filename=package://kuavo_assets/models/biped_s56/meshes/head_radar.S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
- added link waist_camera_base, mass 0.13300000; visual mesh filename=package://kuavo_assets/models/biped_s56/meshes/waist_camera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
- link waist_camera: mass 0.048238 -> 0.0000785398163397463
Joints:
- removed joint camera_base
- removed joint head_rader_joint
- removed joint waist_camera
- added joint head_camera_base_joint: type fixed, parent zhead_2_link, child head_camera_base, origin xyz=0.099619 0 0.032844 rpy=0 0.3406 0, axis 0 0 0
- added joint head_camera_depth_joint: type fixed, parent head_camera_base, child head_camera_depth, origin xyz=0.011715 0.0475 0.014312 rpy=0 0 0, axis 0 0 0
- added joint head_radar_joint: type fixed, parent zhead_1_link, child head_radar, origin xyz=0 0 -0.078453 rpy=0 0 0, axis 0 0 0
- added joint waist_camera_base_joint: type fixed, parent waist_yaw_link, child waist_camera_base, origin xyz=0.0787 0 -0.028149 rpy=0 0.59341 0, axis 0 0 0
- added joint waist_camera_joint: type fixed, parent waist_camera_base, child waist_camera, origin xyz=0.011715 0.0475 0.014312 rpy=0 0 0, axis 0 0 0
- joint leg_r6_joint: origin xyz=0 0 0 rpy=0 0 0 -> xyz=0 0 -0.023 rpy=0 0 0

File: src/kuavo_assets/models/biped_s56/urdf/drake/biped_v3_all_joint.urdf (robot description, URDF)
Before this commit: robot biped_v3_all_joint, 35 links, 30 joints
Joints:
- joint leg_r6_joint: origin xyz=0 0 0 rpy=0 0 0 -> xyz=0 0 -0.023 rpy=0 0 0

Commit message: sync https://www.lejuhub.com/highlydynamic/kuavo-ros-control/commit/93bef0cadb2f78a5cd4b7dc085bcdfcc0f178344

File: src/kuavo_assets/models/biped_s56/urdf/biped_s56.urdf (robot description, URDF)
Before this commit: robot biped_s56, 50 links, 49 joints
Links:
- link waist_camera: mass 0.0000785398163397463 -> 7.8539816339743E-05; geometry visual mesh filename=../meshes/waist_camera_depth.STL
- link waist_camera_base: geometry visual mesh filename=../meshes/waist_camera_base.STL
Joints:
- joint waist_camera_base_joint: origin xyz=0.0787 0 -0.028149 rpy=0 0.59341 0 -> xyz=0.09462 0 -0.010454 rpy=0 1.0472 0
