Commit message: sync https://www.lejuhub.com/highlydynamic/kuavo-ros-control/commit/9327920ea3320a1ac3ee11cab436bd2be7f1b6b9

File: src/kuavo_assets/models/biped_s100045/urdf/biped_s100045.urdf (robot description, URDF)
Before this commit: robot biped_s100045, 47 links, 46 joints
Links:
- link zarm_l1_link: mass 0.962 -> 0.95200000
- link zarm_l2_link: mass 0.57 -> 0.38500000
- link zarm_l3_link: mass 1.65 -> 1.75450000
- link zarm_l4_link: mass 0.429 -> 0.60780000
- link zarm_l5_link: mass 0.203 -> 0.63690000
- link zarm_l6_link: mass 0.111 -> 0.47390000
- link zarm_r1_link: mass 0.962 -> 0.95200000
- link zarm_r2_link: mass 0.57 -> 0.38500000
- link zarm_r3_link: mass 1.65 -> 1.75450000
- link zarm_r4_link: mass 0.429 -> 0.60780000
- link zarm_r5_link: mass 0.203 -> 0.63690000
- link zarm_r6_link: mass 0.111 -> 0.47390000

File: src/kuavo_assets/models/biped_s100045/urdf/biped_s100045_gazebo.urdf (robot description, URDF)
Before this commit: robot biped_s100045, 47 links, 46 joints
Links:
- link zarm_l1_link: mass 0.962 -> 0.95200000
- link zarm_l2_link: mass 0.57 -> 0.38500000
- link zarm_l3_link: mass 1.65 -> 1.75450000
- link zarm_l4_link: mass 0.429 -> 0.60780000
- link zarm_l5_link: mass 0.61 -> 0.63690000
- link zarm_l6_link: mass 0.331 -> 0.47390000
- link zarm_r1_link: mass 0.962 -> 0.95200000
- link zarm_r2_link: mass 0.57 -> 0.38500000
- link zarm_r3_link: mass 1.65 -> 1.75450000
- link zarm_r4_link: mass 0.429 -> 0.60780000
- link zarm_r5_link: mass 0.61 -> 0.63690000
- link zarm_r6_link: mass 0.331 -> 0.47390000

File: src/kuavo_assets/models/biped_s100045/urdf/drake/biped_v3_arm.urdf (robot description, URDF)
Before this commit: robot biped_s100045, 19 links, 18 joints
Links:
- link zarm_l1_link: mass 0.962 -> 0.95200000
- link zarm_l2_link: mass 0.57 -> 0.38500000
- link zarm_l3_link: mass 1.65 -> 1.75450000
- link zarm_l4_link: mass 0.429 -> 0.60780000
- link zarm_l5_link: mass 0.61 -> 0.63690000
- link zarm_l6_link: mass 0.331 -> 0.47390000
- link zarm_r1_link: mass 0.962 -> 0.95200000
- link zarm_r2_link: mass 0.57 -> 0.38500000
- link zarm_r3_link: mass 1.65 -> 1.75450000
- link zarm_r4_link: mass 0.429 -> 0.60780000
- link zarm_r5_link: mass 0.61 -> 0.63690000
- link zarm_r6_link: mass 0.331 -> 0.47390000

File: src/kuavo_assets/models/biped_s100049/urdf/biped_s100049.urdf (robot description, URDF)
Before this commit: robot biped_s100049, 47 links, 46 joints
Links:
- link zarm_l1_link: mass 0.962 -> 0.95200000
- link zarm_l2_link: mass 0.57 -> 0.38500000
- link zarm_l3_link: mass 1.65 -> 1.75450000
- link zarm_l4_link: mass 0.429 -> 0.60780000
- link zarm_l5_link: mass 0.61 -> 0.63690000
- link zarm_l6_link: mass 0.331 -> 0.47390000
- link zarm_r1_link: mass 0.962 -> 0.95200000
- link zarm_r2_link: mass 0.57 -> 0.38500000
- link zarm_r3_link: mass 1.65 -> 1.75450000
- link zarm_r4_link: mass 0.429 -> 0.60780000
- link zarm_r5_link: mass 0.61 -> 0.63690000
- link zarm_r6_link: mass 0.331 -> 0.47390000

File: src/kuavo_assets/models/biped_s100049/urdf/biped_s100049_gazebo.urdf (robot description, URDF)
Before this commit: robot biped_s100049, 47 links, 46 joints
Links:
- link zarm_l1_link: mass 0.962 -> 0.95200000
- link zarm_l2_link: mass 0.57 -> 0.38500000
- link zarm_l3_link: mass 1.65 -> 1.75450000
- link zarm_l4_link: mass 0.429 -> 0.60780000
- link zarm_l5_link: mass 0.61 -> 0.63690000
- link zarm_l6_link: mass 0.331 -> 0.47390000
- link zarm_r1_link: mass 0.962 -> 0.95200000
- link zarm_r2_link: mass 0.57 -> 0.38500000
- link zarm_r3_link: mass 1.65 -> 1.75450000
- link zarm_r4_link: mass 0.429 -> 0.60780000
- link zarm_r5_link: mass 0.61 -> 0.63690000
- link zarm_r6_link: mass 0.331 -> 0.47390000

File: src/kuavo_assets/models/biped_s100049/urdf/drake/biped_v3_arm.urdf (robot description, URDF)
Before this commit: robot biped_s100049, 19 links, 18 joints
Links:
- link zarm_l1_link: mass 0.962 -> 0.95200000
- link zarm_l2_link: mass 0.57 -> 0.38500000
- link zarm_l3_link: mass 1.65 -> 1.75450000
- link zarm_l4_link: mass 0.429 -> 0.60780000
- link zarm_l5_link: mass 0.61 -> 0.63690000
- link zarm_l6_link: mass 0.331 -> 0.47390000
- link zarm_r1_link: mass 0.962 -> 0.95200000
- link zarm_r2_link: mass 0.57 -> 0.38500000
- link zarm_r3_link: mass 1.65 -> 1.75450000
- link zarm_r4_link: mass 0.429 -> 0.60780000
- link zarm_r5_link: mass 0.61 -> 0.63690000
- link zarm_r6_link: mass 0.331 -> 0.47390000

File: src/kuavo_assets/models/biped_s200049/urdf/biped_s200049.urdf (robot description, URDF)
Before this commit: robot biped_s200049, 65 links, 64 joints
Links:
- link zarm_l1_link: mass 0.962 -> 0.95200000
- link zarm_l2_link: mass 0.57 -> 0.38500000
- link zarm_l3_link: mass 1.65 -> 1.75450000
- link zarm_l4_link: mass 0.429 -> 0.60780000
- link zarm_l5_link: mass 0.61 -> 0.63690000
- link zarm_l6_link: mass 0.331 -> 0.47390000
- link zarm_r1_link: mass 0.962 -> 0.95200000
- link zarm_r2_link: mass 0.57 -> 0.38500000
- link zarm_r3_link: mass 1.65 -> 1.75450000
- link zarm_r4_link: mass 0.429 -> 0.60780000
- link zarm_r5_link: mass 0.61 -> 0.63690000
- link zarm_r6_link: mass 0.331 -> 0.47390000

File: src/kuavo_assets/models/biped_s200049/urdf/biped_s200049_gazebo.urdf (robot description, URDF)
Before this commit: robot biped_s200049, 63 links, 62 joints
Links:
- link zarm_l1_link: mass 0.962 -> 0.95200000
- link zarm_l2_link: mass 0.57 -> 0.38500000
- link zarm_l3_link: mass 1.65 -> 1.75450000
- link zarm_l4_link: mass 0.429 -> 0.60780000
- link zarm_l5_link: mass 0.61 -> 0.63690000
- link zarm_l6_link: mass 0.331 -> 0.47390000
- link zarm_r1_link: mass 0.962 -> 0.95200000
- link zarm_r2_link: mass 0.57 -> 0.38500000
- link zarm_r3_link: mass 1.65 -> 1.75450000
- link zarm_r4_link: mass 0.429 -> 0.60780000
- link zarm_r5_link: mass 0.61 -> 0.63690000
- link zarm_r6_link: mass 0.331 -> 0.47390000

File: src/kuavo_assets/models/biped_s200049/urdf/drake/biped_v3_arm.urdf (robot description, URDF)
Before this commit: robot biped_s200049, 19 links, 18 joints
Links:
- link zarm_l1_link: mass 0.962 -> 0.95200000
- link zarm_l2_link: mass 0.57 -> 0.38500000
- link zarm_l3_link: mass 1.65 -> 1.75450000
- link zarm_l4_link: mass 0.429 -> 0.60780000
- link zarm_l5_link: mass 0.61 -> 0.63690000
- link zarm_l6_link: mass 0.331 -> 0.47390000
- link zarm_r1_link: mass 0.962 -> 0.95200000
- link zarm_r2_link: mass 0.57 -> 0.38500000
- link zarm_r3_link: mass 1.65 -> 1.75450000
- link zarm_r4_link: mass 0.429 -> 0.60780000
- link zarm_r5_link: mass 0.61 -> 0.63690000
- link zarm_r6_link: mass 0.331 -> 0.47390000

File: src/kuavo_assets/models/biped_s60/urdf/drake/biped_v3_arm.urdf (robot description, URDF)
Before this commit: robot biped_s45, 17 links, 16 joints
Links:
- added link knee_link, mass 5.39660196; visual mesh filename=../../meshes/knee_pitch.STL
- added link leg_link, mass 12.35650958; visual mesh filename=../../meshes/leg_pitch.STL
- added link waist_link, mass 5.4305643; visual mesh filename=../../meshes/waist_pitch.STL
- added link waist_yaw_link, mass 11.56094002; collision cylinder length=0.6 radius=0.15; visual mesh filename=../../meshes/torso.STL
- added link zarm_l7_virtual_thumb_link; collision sphere radius=0.005
- added link zarm_r7_virtual_thumb_link; collision sphere radius=0.005
- link base_link: mass 11.56094002 -> 97.77291318; geometry visual mesh filename=../../meshes/chassis.STL
- link zarm_r2_link: geometry collision cylinder length=0.3 radius=0.05; visual mesh filename=../../meshes/r_arm_roll.STL
- link zarm_r4_link: geometry collision cylinder length=0.26 radius=0.05; visual mesh filename=../../meshes/r_forearm.STL
Joints:
- added joint knee_joint: type revolute, parent base_link, child knee_link, origin xyz=0.2265 0.017 0.2658 rpy=0 0.0 0, axis 0 1 0, limit lower=0 upper=1.448 effort=668.53 velocity=25.33
- added joint leg_joint: type revolute, parent knee_link, child leg_link, origin xyz=-0.48618 0 0.11672 rpy=0 -0.251 0, axis 0 1 0, limit lower=-2.81 upper=0.0 effort=668.53 velocity=25.33
- added joint waist_pitch_joint: type revolute, parent leg_link, child waist_link, origin xyz=0.49384 0 0.078217 rpy=0 0.236 0, axis  0 1 0, limit lower=0.0 upper=0.9 effort=618.48 velocity=25.33
- added joint waist_yaw_joint: type revolute, parent waist_link, child waist_yaw_link, origin xyz=0.0 -0.0165 0.209 rpy=0 0 0, axis 0 0 1, limit lower=-3.238 upper=3.238 effort=618.48 velocity=25.33
- added joint zarm_l7_virtual_thumb_joint_ee: type fixed, parent zarm_l7_end_effector, child zarm_l7_virtual_thumb_link, origin xyz=0.15 0 0 rpy=0 0 0
- added joint zarm_r7_virtual_thumb_joint_ee: type fixed, parent zarm_r7_end_effector, child zarm_r7_virtual_thumb_link, origin xyz=0.15 0 0 rpy=0 0 0
- joint zarm_l1_joint: limit lower=-3.14159265358979 upper=1.5707963267949 effort=66.0 velocity=18.8 -> lower=-2.4 upper=0.6 effort=66.0 velocity=18.8; origin xyz=0 0.2527 0.242 rpy=0 0 0 -> xyz=0 0.1717 0.242 rpy=0 0 0; parent base_link -> waist_yaw_link
- joint zarm_l2_joint: limit lower=-0.349065850398866 upper=3.49065850398866 effort=75.0 velocity=8.0 -> lower=-0.349065850398866 upper=1.46 effort=75.0 velocity=8.0; origin xyz=0 0 0 rpy=0 0 0 -> xyz=0 0.081 0 rpy=0 0 0
- joint zarm_l3_joint: limit lower=-1.48352986419518 upper=1.48352986419518 effort=57.0 velocity=7.5 -> lower=-1.5707963267949 upper=0.46 effort=57.0 velocity=7.5
- joint zarm_l4_joint: limit lower=-2.61799387799149 upper=0.0 effort=75.0 velocity=8.0 -> lower=-2.61799387799149 upper=-0.2 effort=75.0 velocity=8.0
- joint zarm_r1_joint: limit lower=-3.14159265358979 upper=1.5707963267949 effort=66.0 velocity=18.8 -> lower=-2.4 upper=0.6 effort=66.0 velocity=18.8; origin xyz=0 -0.2527 0.242 rpy=0 0 0 -> xyz=0 -0.1717 0.242 rpy=0 0 0; parent base_link -> waist_yaw_link
- joint zarm_r2_joint: limit lower=-3.49065850398866 upper=0.349065850398866 effort=75.0 velocity=8.0 -> lower=-1.46 upper=0.349065850398866 effort=75.0 velocity=8.0; origin xyz=0 0 0 rpy=0 0 0 -> xyz=0 -0.081 0 rpy=0 0 0
- joint zarm_r3_joint: limit lower=-1.48352986419518 upper=1.48352986419518 effort=57.0 velocity=7.5 -> lower=-0.46 upper=1.5707963267949 effort=57.0 velocity=7.5
- joint zarm_r4_joint: limit lower=-2.61799387799149 upper=0.0 effort=75.0 velocity=8.0 -> lower=-2.61799387799149 upper=-0.2 effort=75.0 velocity=8.0

Commit message: sync https://www.lejuhub.com/highlydynamic/kuavo-ros-control/commit/06073a50df5a2f3439762ce50e6622434b5db753

File: src/kuavo_assets/models/biped_s100045/urdf/biped_s100045.urdf (robot description, URDF)
Before this commit: robot biped_s100045, 47 links, 46 joints
Joints:
- removed joint dummy_to_base_link
- added joint base_link_to_dummy_link: type fixed, parent base_link, child dummy_link, origin xyz=0 0 0 rpy=0 0 0

File: src/kuavo_assets/models/biped_s100045/urdf/biped_s100045_gazebo.urdf (robot description, URDF)
Before this commit: robot biped_s100045, 47 links, 46 joints
Joints:
- removed joint dummy_to_base_link
- added joint base_link_to_dummy_link: type fixed, parent base_link, child dummy_link, origin xyz=0 0 0 rpy=0 0 0

File: src/kuavo_assets/models/biped_s100049/urdf/biped_s100049.urdf (robot description, URDF)
Before this commit: robot biped_s100049, 47 links, 46 joints
Joints:
- removed joint dummy_to_base_link
- added joint base_link_to_dummy_link: type fixed, parent base_link, child dummy_link, origin xyz=0 0 0 rpy=0 0 0

File: src/kuavo_assets/models/biped_s100049/urdf/biped_s100049_gazebo.urdf (robot description, URDF)
Before this commit: robot biped_s100049, 47 links, 46 joints
Joints:
- removed joint dummy_to_base_link
- added joint base_link_to_dummy_link: type fixed, parent base_link, child dummy_link, origin xyz=0 0 0 rpy=0 0 0

File: src/kuavo_assets/models/biped_s11/urdf/biped_s11.urdf (robot description, URDF)
Before this commit: robot biped_s11, 37 links, 36 joints
Joints:
- removed joint dummy_to_base_link
- added joint base_link_to_dummy_link: type fixed, parent base_link, child dummy_link, origin xyz=0 0 0 rpy=0 0 0

File: src/kuavo_assets/models/biped_s13/urdf/biped_s13_gazebo.urdf (robot description, URDF)
Before this commit: robot biped_s13, 39 links, 38 joints
Joints:
- removed joint dummy_to_base_link
- added joint base_link_to_dummy_link: type fixed, parent base_link, child dummy_link, origin xyz=0 0 0 rpy=0 0 0

File: src/kuavo_assets/models/biped_s14/urdf/biped_s14.urdf (robot description, URDF)
Before this commit: robot biped_s14, 41 links, 40 joints
Joints:
- removed joint dummy_to_base_link
- added joint base_link_to_dummy_link: type fixed, parent base_link, child dummy_link, origin xyz=0 0 0 rpy=0 0 0

File: src/kuavo_assets/models/biped_s14/urdf/biped_s14_gazebo.urdf (robot description, URDF)
Before this commit: robot biped_s14, 41 links, 40 joints
Joints:
- removed joint dummy_to_base_link
- added joint base_link_to_dummy_link: type fixed, parent base_link, child dummy_link, origin xyz=0 0 0 rpy=0 0 0

File: src/kuavo_assets/models/biped_s16/urdf/biped_s16.urdf (robot description, URDF)
Before this commit: robot biped_s16, 41 links, 40 joints
Joints:
- removed joint dummy_to_base_link
- added joint base_link_to_dummy_link: type fixed, parent base_link, child dummy_link, origin xyz=0 0 0 rpy=0 0 0

File: src/kuavo_assets/models/biped_s16/urdf/biped_s16_gazebo.urdf (robot description, URDF)
Before this commit: robot biped_s16, 41 links, 40 joints
Joints:
- removed joint dummy_to_base_link
- added joint base_link_to_dummy_link: type fixed, parent base_link, child dummy_link, origin xyz=0 0 0 rpy=0 0 0

File: src/kuavo_assets/models/biped_s17/urdf/biped_s17.urdf (robot description, URDF)
Before this commit: robot biped_s17, 43 links, 42 joints
Joints:
- removed joint dummy_to_base_link
- added joint base_link_to_dummy_link: type fixed, parent base_link, child dummy_link, origin xyz=0 0 0 rpy=0 0 0

File: src/kuavo_assets/models/biped_s17/urdf/biped_s17_gazebo.urdf (robot description, URDF)
Before this commit: robot biped_s17, 43 links, 42 joints
Joints:
- removed joint dummy_to_base_link
- added joint base_link_to_dummy_link: type fixed, parent base_link, child dummy_link, origin xyz=0 0 0 rpy=0 0 0

File: src/kuavo_assets/models/biped_s200049/urdf/biped_s200049.urdf (robot description, URDF)
Before this commit: robot biped_s200049, 65 links, 64 joints
Joints:
- removed joint dummy_to_base_link
- added joint base_link_to_dummy_link: type fixed, parent base_link, child dummy_link, origin xyz=0 0 0 rpy=0 0 0

File: src/kuavo_assets/models/biped_s200049/urdf/biped_s200049_gazebo.urdf (robot description, URDF)
Before this commit: robot biped_s200049, 63 links, 62 joints
Joints:
- removed joint dummy_to_base_link
- added joint base_link_to_dummy_link: type fixed, parent base_link, child dummy_link, origin xyz=0 0 0 rpy=0 0 0

File: src/kuavo_assets/models/biped_s200053/urdf/biped_s200053.urdf (robot description, URDF)
Before this commit: robot biped_s200053, 76 links, 75 joints
Joints:
- removed joint dummy_to_base_link
- added joint base_link_to_dummy_link: type fixed, parent base_link, child dummy_link, origin xyz=0 0 0 rpy=0 0 0

File: src/kuavo_assets/models/biped_s200053/urdf/biped_s200053_gazebo.urdf (robot description, URDF)
Before this commit: robot biped_s53, 48 links, 47 joints
Joints:
- removed joint dummy_to_base_link
- added joint base_link_to_dummy_link: type fixed, parent base_link, child dummy_link, origin xyz=0 0 0 rpy=0 0 0

File: src/kuavo_assets/models/biped_s200053/urdf/drake/biped_v3_full.urdf (robot description, URDF)
Before this commit: robot biped_s53, 32 links, 31 joints
Joints:
- removed joint dummy_to_base_link
- added joint base_link_to_dummy_link: type fixed, parent base_link, child dummy_link, origin xyz=0 0 0 rpy=0 0 0

File: src/kuavo_assets/models/biped_s200062/urdf/biped_s200062.urdf (robot description, URDF)
Before this commit: robot biped_s200062, 64 links, 63 joints
Joints:
- removed joint floating_base
- added joint base_link_to_dummy_link: type fixed, parent base_link, child dummy_link, origin xyz=0 0 0 rpy=0 0 0

File: src/kuavo_assets/models/biped_s200062/urdf/biped_s200062_gazebo.urdf (robot description, URDF)
Before this commit: robot biped_s200062, 39 links, 38 joints
Joints:
- removed joint floating_base
- added joint base_link_to_dummy_link: type fixed, parent base_link, child dummy_link, origin xyz=0 0 0 rpy=0 0 0

File: src/kuavo_assets/models/biped_s300049/urdf/biped_s300049_gazebo.urdf (robot description, URDF)
Before this commit: robot biped_s300049, 69 links, 68 joints
Joints:
- removed joint dummy_to_base_link
- added joint base_link_to_dummy_link: type fixed, parent base_link, child dummy_link, origin xyz=0 0 0 rpy=0 0 0
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