Commit message: sync https://www.lejuhub.com/highlydynamic/kuavo-ros-control/commit/a6bd805759b0f84dd1a9451440552aabac36ab47

File: src/kuavo_assets/models/biped_s56/urdf/drake/Lleg.urdf (robot description, URDF)
Before this commit: robot Lleg, 7 links, 4 joints
Joints:
- joint l_foot_pitch_joint: origin xyz=0 0.0 -0.346 rpy=0 0 0 -> xyz=0 0 -0.416 rpy=0 0 0
- joint l_foot_roll_joint: origin xyz=0 0 0 rpy=0 0 0 -> xyz=0 0 -0.023 rpy=0 0 0
- joint l_l_bar_y: origin xyz=0 0.0318 -0.09 rpy=0 0 0 -> xyz=0.0535 0 -0.1883 rpy=0 0 0
- joint l_r_bar_y: origin xyz=0 -0.0362 -0.153 rpy=0 0 0 -> xyz=0.0535 0 -0.0983 rpy=0 0 0

File: src/kuavo_assets/models/biped_s56/urdf/drake/Rleg.urdf (robot description, URDF)
Before this commit: robot Rleg, 7 links, 4 joints
Joints:
- joint r_foot_pitch_joint: origin xyz=0 0 -0.346 rpy=0 0 0 -> xyz=0 0 -0.416 rpy=0 0 0
- joint r_foot_roll_joint: origin xyz=0 0 0 rpy=0 0 0 -> xyz=0 0 -0.023 rpy=0 0 0
- joint r_l_bar_y: origin xyz=0 0.0362 -0.153 rpy=0 0 0 -> xyz=0.0535 0 -0.0983 rpy=0 0 0
- joint r_r_bar_y: origin xyz=0 -0.0318 -0.09 rpy=0 0 0 -> xyz=0.0535 0 -0.1883 rpy=0 0 0

File: src/kuavo_assets/models/biped_s56/urdf/drake/biped_v3_all_joint.urdf (robot description, URDF)
Before this commit: robot biped_v3_all_joint, 35 links, 30 joints
Links:
- link leg_l1_link: mass 1.71093115 -> 1.55641
- link leg_l2_link: mass 0.58029165 -> 0.75873
- link leg_l3_link: mass 4.50393141 -> 6.68074
- link leg_l4_link: mass 1.62776815 -> 3.64666
- link leg_r1_link: mass 1.71093008 -> 1.55641
- link leg_r2_link: mass 0.58029165 -> 0.75873
- link leg_r3_link: mass 4.50385993 -> 6.68074
- link leg_r4_link: mass 1.62655699 -> 3.64666
Joints:
- joint l_l_bar_y: origin xyz=0 0.0318 -0.09 rpy=0 0 0 -> xyz=0.0535 0 -0.1883 rpy=0 0 0
- joint l_r_bar_y: origin xyz=0 -0.0362 -0.153 rpy=0 0 0 -> xyz=0.0535 0 -0.0983 rpy=0 0 0
- joint leg_l1_joint: limit lower=-0.314159265358979 upper=0.663225115757845 effort=180.0 velocity=23.55 -> lower=-0.314159265358979 upper=0.663225115757845 effort=127.0 velocity=10.4; origin xyz=-0.0024999 0.087 -0.066 rpy=0 0 0 -> xyz=0.0 0.095075 -0.066 rpy=0 0 0
- joint leg_l2_joint: limit lower=-0.872664625997165 upper=0.785398163397448 effort=100.0 velocity=41.3433333333333 -> lower=-0.785398163397448 upper=1.91986217719376 effort=71.0 velocity=8.7
- joint leg_l3_joint: limit lower=-2.00712863979348 upper=1.5707963267949 effort=100.0 velocity=41.3433333333333 -> lower=-1.91986217719376 upper=1.5707963267949 effort=132 velocity=12.7; origin xyz=0.000500354536093913 -0.00100000000000011 -0.1287 rpy=0 0 0 -> xyz=0 0 -0.1437 rpy=0 0 0
- joint leg_l4_joint: limit lower=0.0 upper=2.53072741539178 effort=180.0 velocity=23.55 -> lower=0.0 upper=2.53072741539178 effort=280.0 velocity=10.4; origin xyz=-6.87185435835039E-05 0 -0.284 rpy=0 0 0 -> xyz=-0.0011639 0 -0.284 rpy=0 0 0
- joint leg_l5_joint: limit lower=-0.872664625997165 upper=0.349065850398866 effort=36.0 velocity=23.0266666666667 -> lower=-0.872664625997165 upper=0.349065850398866 effort=91.6 velocity=17.8; origin xyz=-0.000431635992531742 0 -0.346000000000001 rpy=0 0 0 -> xyz=0.00 0 -0.416 rpy=0 0 0
- joint leg_l6_joint: limit lower=-0.261799387799149 upper=0.261799387799149 effort=36.0 velocity=23.0266666666667 -> lower=-0.261799387799149 upper=0.261799387799149 effort=30.0 velocity=17.8
- joint leg_r1_joint: limit lower=-0.663225115757845 upper=0.314159265358979 effort=180.0 velocity=23.55 -> lower=-0.663225115757845 upper=0.314159265358979 effort=127.0 velocity=10.4; origin xyz=-0.0024999 -0.087 -0.066 rpy=0 0 0 -> xyz=0.0 -0.095075 -0.066 rpy=0 0 0
- joint leg_r2_joint: limit lower=-0.785398163397448 upper=0.872664625997165 effort=100.0 velocity=41.3433333333333 -> lower=-1.91986217719376 upper=0.785398163397448 effort=71.0 velocity=8.7
- joint leg_r3_joint: limit lower=-2.00712863979348 upper=1.5707963267949 effort=100.0 velocity=41.3433333333333 -> lower=-1.91986217719376 upper=1.5707963267949 effort=132.0 velocity=12.7; origin xyz=-4.88006581312577E-05 0 -0.1287 rpy=0 0 0 -> xyz=0 0 -0.1437 rpy=0 0 0
- joint leg_r4_joint: limit lower=0.0 upper=2.53072741539178 effort=180.0 velocity=23.55 -> lower=0.0 upper=2.53072741539178 effort=280.0 velocity=10.4; origin xyz=0.000147138572785148 0 -0.283999982974744 rpy=0 0 0 -> xyz=-0.0011639 0 -0.284 rpy=0 0 0
- joint leg_r5_joint: limit lower=-0.872664625997165 upper=0.349065850398866 effort=36.0 velocity=23.0266666666667 -> lower=-0.872664625997165 upper=0.349065850398866 effort=91.6 velocity=17.8; origin xyz=0.000119806050928577 0 -0.345999979257963 rpy=0 0 0 -> xyz=0.000 0 -0.416 rpy=0 0 0
- joint leg_r6_joint: limit lower=-0.261799387799149 upper=0.261799387799149 effort=36.0 velocity=23.0266666666667 -> lower=-0.261799387799149 upper=0.261799387799149 effort=30.0 velocity=17.8
- joint r_l_bar_y: origin xyz=0 0.0362 -0.153 rpy=0 0 0 -> xyz=0.0535 0 -0.0983 rpy=0 0 0
- joint r_r_bar_y: origin xyz=0 -0.0318 -0.09 rpy=0 0 0 -> xyz=0.0535 0 -0.1883 rpy=0 0 0
