Commit message: sync https://www.lejuhub.com/highlydynamic/kuavo-ros-control/commit/cc872949deee084a7cd1fb99050b49299960824b

File: src/kuavo_assets/models/biped_s17/urdf/biped_s17_gazebo.urdf (robot description, URDF)
Before this commit: robot biped_s17, 43 links, 42 joints
Links:
- link base_link: mass 6.61137344 -> 5.27737344

File: src/kuavo_assets/models/biped_s17/urdf/drake/biped_v3.urdf (robot description, URDF)
Before this commit: robot biped_v3, 14 links, 13 joints
Links:
- link torso: mass 17.90214703 -> 16.56814703
