Commit message: sync https://www.lejuhub.com/highlydynamic/kuavo-ros-control/commit/daa191fa1378f8b8a23eb8931ed4a79e2c19454a

File: src/kuavo_assets/models/biped_s17/urdf/biped_s17.urdf (robot description, URDF)
Before this commit: robot biped_s17, 39 links, 38 joints
Links:
- link waist_yaw_link: mass 4.8567 -> 6.9767

File: src/kuavo_assets/models/biped_s17/urdf/biped_s17_gazebo.urdf (robot description, URDF)
Before this commit: robot biped_s17, 39 links, 38 joints
Links:
- link waist_yaw_link: mass 4.8567 -> 6.9767

File: src/kuavo_assets/models/biped_s17/urdf/drake/biped_v3.urdf (robot description, URDF)
Before this commit: robot biped_v3, 14 links, 13 joints
Links:
- link torso: mass 16.1291 -> 18.2491

File: src/kuavo_assets/models/biped_s17/urdf/drake/biped_v3_all_joint.urdf (robot description, URDF)
Before this commit: robot biped_v3_all_joint, 30 links, 25 joints
Links:
- link torso: mass 9.4582 -> 11.5782

File: src/kuavo_assets/models/biped_s17/urdf/drake/biped_v3_full.urdf (robot description, URDF)
Before this commit: robot biped_v3_full, 22 links, 21 joints
Links:
- link torso: mass 9.8296 -> 11.9496

File: src/kuavo_assets/models/biped_s60/urdf/biped_s60.urdf (robot description, URDF)
Before this commit: robot biped_s60, 35 links, 34 joints
Links:
- added link zarm_l7_end_effector_1
- added link zarm_l7_end_effector_2
- added link zarm_r7_end_effector_1
- added link zarm_r7_end_effector_2
Joints:
- added joint zarm_l7_end_effector_1_joint: type fixed, parent zarm_l7_link, child zarm_l7_end_effector_1, origin xyz=0 0.0 -0.08 rpy=0 0 0
- added joint zarm_l7_end_effector_2_joint: type fixed, parent zarm_l7_link, child zarm_l7_end_effector_2, origin xyz=0.03 0.0 -0.17 rpy=0 0 0
- added joint zarm_r7_end_effector_1_joint: type fixed, parent zarm_r7_link, child zarm_r7_end_effector_1, origin xyz=0 0.0 -0.08 rpy=0 0 0
- added joint zarm_r7_end_effector_2_joint: type fixed, parent zarm_r7_link, child zarm_r7_end_effector_2, origin xyz=0.03 0.0 -0.17 rpy=0 0 0
- joint zarm_l7_end_effector_joint: origin xyz=0 -0.03 -0.17 rpy=0 0 0 -> xyz=0 0.0 -0.17 rpy=0 0 0
- joint zarm_r7_end_effector_joint: origin xyz=0 0.03 -0.17 rpy=0 0 0 -> xyz=0 0.0 -0.17 rpy=0 0 0

File: src/kuavo_assets/models/biped_s61/urdf/biped_s61.urdf (robot description, URDF)
Before this commit: robot biped_s61, 32 links, 31 joints
Links:
- added link zarm_l7_end_effector_1
- added link zarm_l7_end_effector_2
- added link zarm_r7_end_effector_1
- added link zarm_r7_end_effector_2
Joints:
- added joint zarm_l7_end_effector_1_joint: type fixed, parent zarm_l7_link, child zarm_l7_end_effector_1, origin xyz=0 0.0 -0.08 rpy=0 0 0
- added joint zarm_l7_end_effector_2_joint: type fixed, parent zarm_l7_link, child zarm_l7_end_effector_2, origin xyz=0.03 0.0 -0.17 rpy=0 0 0
- added joint zarm_r7_end_effector_1_joint: type fixed, parent zarm_r7_link, child zarm_r7_end_effector_1, origin xyz=0 0.0 -0.08 rpy=0 0 0
- added joint zarm_r7_end_effector_2_joint: type fixed, parent zarm_r7_link, child zarm_r7_end_effector_2, origin xyz=0.03 0.0 -0.17 rpy=0 0 0

Commit message: sync https://www.lejuhub.com/highlydynamic/kuavo-ros-control/commit/4df36fa943c669aeb679d515c1c2554fd36a097e

File: src/kuavo_assets/models/biped_s17/urdf/biped_s17.urdf (robot description, URDF)
Before this commit: robot biped_s17, 39 links, 38 joints
Links:
- removed link waist_yaw_link
- added link camera_base, mass 0.00001000; visual mesh filename=package://kuavo_assets/models/biped_s17/meshes/head_camera_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
- added link head_radar, mass 0.00000100; visual mesh filename=package://kuavo_assets/models/biped_s17/meshes/head_radar.S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
- added link l_handball, mass 0.17660000; visual mesh filename=package://kuavo_assets/models/biped_s17/meshes/l_handball.S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
- added link r_handball, mass 0.17660000; visual mesh filename=package://kuavo_assets/models/biped_s17/meshes/r_handball.S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
- added link torso, mass 8.37744703; collision box size=0.14 0.2 0.26; collision cylinder length=0.125 radius=0.008
- link base_link: mass 4.8567 -> 5.27737344
- link leg_l1_link: mass 0.62568928 -> 0.6865
- link leg_l2_link: mass 2.03159924 -> 2.054
- link leg_l3_link: mass 3.38846623 -> 3.2746
- link leg_l4_link: mass 2.61852 -> 2.4454
- link leg_l5_link: mass 0.10854305 -> 0.1314
- link leg_l6_link: mass 0.43610846 -> 0.5783271
- link leg_r1_link: mass 0.62568928 -> 0.6865
- link leg_r2_link: mass 2.03159924 -> 2.054
- link leg_r3_link: mass 3.38846623 -> 3.2746
- link leg_r4_link: mass 2.61852 -> 2.4454
- link leg_r5_link: mass 0.10854305 -> 0.1314
- link leg_r6_link: mass 0.43610846 -> 0.5783271
- link zarm_l1_link: mass 0.80328906 -> 0.84760000
- link zarm_l2_link: mass 0.32360735 -> 0.36680000
- link zarm_l3_link: mass 1.46578996 -> 1.51660000
- link zarm_l4_link: mass 0.42136972 -> 0.34500000
- link zarm_r1_link: mass 0.80328906 -> 0.84760000
- link zarm_r2_link: mass 0.32360735 -> 0.36680000
- link zarm_r3_link: mass 1.46578996 -> 1.51660000
- link zarm_r4_link: mass 0.42136972 -> 0.34500000
- link zhead_1_link: mass 1.03077542 -> 1.07555742
- link zhead_2_link: mass 0.33654975 -> 0.61000000
Joints:
- added joint camera_base_joint: type fixed, parent zhead_2_link, child camera_base, origin xyz=0.047118 0 0.051192 rpy=0 0.27152 0
- added joint head_radar_joint: type fixed, parent zhead_1_link, child head_radar, origin xyz=0 0 -0.026453 rpy=0 0 0
- added joint l_handball_joint: type fixed, parent zarm_l4_link, child l_handball, origin xyz=0 0 -0.085236 rpy=0 0 0
- added joint r_handball_joint: type fixed, parent zarm_r4_link, child r_handball, origin xyz=0 0 -0.085236 rpy=0 0 0
- joint leg_l1_joint: origin xyz=0.0 0.12441237 -0.22115341 rpy=0 0 0 -> xyz=0 0.12441 -0.22265 rpy=0 0 0
- joint leg_r1_joint: origin xyz=0.0 -0.12441237 -0.22115341 rpy=0 0 0 -> xyz=0.0 -0.12441 -0.22265 rpy=0 0 0
- joint waist_yaw_joint: child waist_yaw_link -> torso
- joint zarm_l1_joint: origin xyz=0.0 0.18100293 0.23992606 rpy=0 0 0 -> xyz=0 0.181 0.23843 rpy=0 0 0; parent waist_yaw_link -> torso
- joint zarm_l4_joint: origin xyz=0 0.0 -0.20533 rpy=0 0 0 -> xyz=0 0 -0.2085 rpy=0 0 0
- joint zarm_r1_joint: origin xyz=0.0 -0.18100293 0.23992606 rpy=0 0 0 -> xyz=0 -0.181 0.23843 rpy=0 0 0; parent waist_yaw_link -> torso
- joint zarm_r4_joint: origin xyz=0 -0.0 -0.20533 rpy=0 0 0 -> xyz=0 0 -0.2085 rpy=0 0 0
- joint zhead_1_joint: origin xyz=0.004 0 0.35618 rpy=0 0 0 -> xyz=0.0042 0 0.35369 rpy=0 0 0; parent waist_yaw_link -> torso

File: src/kuavo_assets/models/biped_s17/urdf/biped_s17_gazebo.urdf (robot description, URDF)
Before this commit: robot biped_s17, 39 links, 38 joints
Links:
- removed link waist_yaw_link
- added link camera_base, mass 0.00001000; visual mesh filename=package://kuavo_assets/models/biped_s17/meshes/head_camera_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
- added link head_radar, mass 0.00000100; visual mesh filename=package://kuavo_assets/models/biped_s17/meshes/head_radar.S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
- added link l_handball, mass 0.17660000; visual mesh filename=package://kuavo_assets/models/biped_s17/meshes/l_handball.S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
- added link r_handball, mass 0.17660000; visual mesh filename=package://kuavo_assets/models/biped_s17/meshes/r_handball.S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
- added link torso, mass 8.37744703; collision box size=0.14 0.2 0.26; collision cylinder length=0.013 radius=0.005
- link base_link: mass 4.8567 -> 5.27737344
- link leg_l1_link: mass 0.62568928 -> 0.6865
- link leg_l2_link: mass 2.03159924 -> 2.054
- link leg_l3_link: mass 3.38846623 -> 3.2746
- link leg_l4_link: mass 2.61852 -> 2.4454
- link leg_l5_link: mass 0.10854305 -> 0.1314
- link leg_l6_link: mass 0.43610846 -> 0.5783271
- link leg_r1_link: mass 0.62568928 -> 0.6865
- link leg_r2_link: mass 2.03159924 -> 2.054
- link leg_r3_link: mass 3.38846623 -> 3.2746
- link leg_r4_link: mass 2.61852 -> 2.4454
- link leg_r5_link: mass 0.10854305 -> 0.1314
- link leg_r6_link: mass 0.43610846 -> 0.5783271
- link zarm_l1_link: mass 0.80328906 -> 0.84760000
- link zarm_l2_link: mass 0.32360735 -> 0.36680000
- link zarm_l3_link: mass 1.46578996 -> 1.51660000
- link zarm_l4_link: mass 0.42136972 -> 0.34500000
- link zarm_r1_link: mass 0.80328906 -> 0.84760000
- link zarm_r2_link: mass 0.32360735 -> 0.36680000
- link zarm_r3_link: mass 1.46578996 -> 1.51660000
- link zarm_r4_link: mass 0.42136972 -> 0.34500000
- link zhead_1_link: mass 1.03077542 -> 1.07555742
- link zhead_2_link: mass 0.33654975 -> 0.61000000
Joints:
- added joint camera_base_joint: type fixed, parent zhead_2_link, child camera_base, origin xyz=0.047118 0 0.051192 rpy=0 0.27152 0
- added joint head_radar_joint: type fixed, parent zhead_1_link, child head_radar, origin xyz=0 0 -0.026453 rpy=0 0 0
- added joint l_handball_joint: type fixed, parent zarm_l4_link, child l_handball, origin xyz=0 0 -0.085236 rpy=0 0 0
- added joint r_handball_joint: type fixed, parent zarm_r4_link, child r_handball, origin xyz=0 0 -0.085236 rpy=0 0 0
- joint leg_l1_joint: origin xyz=0.0 0.12441237 -0.22115341 rpy=0 0 0 -> xyz=0 0.12441 -0.22265 rpy=0 0 0
- joint leg_l5_joint: limit lower=-0.872664625997165 upper=0.523598775598299 effort=37 velocity=17.0 -> lower=-0.872664625997165 upper=0.523598775598299 effort=74 velocity=17.0
- joint leg_l6_joint: limit lower=-0.261799387799149 upper=0.261799387799149 effort=37 velocity=17.0 -> lower=-0.261799387799149 upper=0.261799387799149 effort=74 velocity=17.0
- joint leg_r1_joint: origin xyz=0.0 -0.12441237 -0.22115341 rpy=0 0 0 -> xyz=0.0 -0.12441 -0.22265 rpy=0 0 0
- joint leg_r5_joint: limit lower=-0.872664625997165 upper=0.523598775598299 effort=37 velocity=17.0 -> lower=-0.872664625997165 upper=0.523598775598299 effort=74 velocity=17.0
- joint leg_r6_joint: limit lower=-0.261799387799149 upper=0.261799387799149 effort=37 velocity=17.0 -> lower=-0.261799387799149 upper=0.261799387799149 effort=74 velocity=17.0
- joint waist_yaw_joint: child waist_yaw_link -> torso
- joint zarm_l1_joint: origin xyz=0.0 0.18100293 0.23992606 rpy=0 0 0 -> xyz=0 0.181 0.23843 rpy=0 0 0; parent waist_yaw_link -> torso
- joint zarm_l4_joint: origin xyz=0 0.0 -0.20533 rpy=0 0 0 -> xyz=0 0 -0.2085 rpy=0 0 0
- joint zarm_r1_joint: origin xyz=0.0 -0.18100293 0.23992606 rpy=0 0 0 -> xyz=0 -0.181 0.23843 rpy=0 0 0; parent waist_yaw_link -> torso
- joint zarm_r4_joint: origin xyz=0 -0.0 -0.20533 rpy=0 0 0 -> xyz=0 0 -0.2085 rpy=0 0 0
- joint zhead_1_joint: origin xyz=0.004 0 0.35618 rpy=0 0 0 -> xyz=0.0042 0 0.35369 rpy=0 0 0; parent waist_yaw_link -> torso

File: src/kuavo_assets/models/biped_s17/urdf/drake/biped_v3_full.urdf (robot description, URDF)
Before this commit: robot biped_v3_full, 22 links, 21 joints
Links:
- link leg_l1_link: mass 0.62568928 -> 0.6865
- link leg_l2_link: mass 2.03159924 -> 2.054
- link leg_l3_link: mass 3.38846623 -> 3.2746
- link leg_l4_link: mass 2.61852 -> 2.4454
- link leg_l5_link: mass 0.10854305 -> 0.1314
- link leg_l6_link: mass 0.43610846 -> 0.5783271
- link leg_r1_link: mass 0.62568928 -> 0.6865
- link leg_r2_link: mass 2.03159924 -> 2.054
- link leg_r3_link: mass 3.38846623 -> 3.2746
- link leg_r4_link: mass 2.61852 -> 2.4454
- link leg_r5_link: mass 0.10854305 -> 0.1314
- link leg_r6_link: mass 0.43610846 -> 0.5783271
- link torso: mass 11.9496 -> 9.63014703
- link waist: mass 4.853 -> 5.27737344
- link zarm_l1_link: mass 0.80328906 -> 0.84760000
- link zarm_l2_link: mass 0.32360735 -> 0.36680000
- link zarm_l3_link: mass 1.46578996 -> 1.51660000
- link zarm_l4_link: mass 0.42136972 -> 0.34500000
- link zarm_r1_link: mass 0.80328906 -> 0.84760000
- link zarm_r2_link: mass 0.32360735 -> 0.36680000
- link zarm_r3_link: mass 1.46578996 -> 1.51660000
- link zarm_r4_link: mass 0.42136972 -> 0.34500000
Joints:
- joint leg_l1_joint: limit lower=-3.228 upper=2.44346 effort=180 velocity=23.55 -> lower=-3.228 upper=2.44346 effort=150 velocity=14.6; origin xyz=0.0 0.12441237 -0.22115341 rpy=0 0 0 -> xyz=0 0.12441 -0.22265 rpy=0 0 0
- joint leg_l2_joint: limit lower=-0.837758 upper=2.40855 effort=100 velocity=41.3433333333333 -> lower=-0.837758 upper=2.40855 effort=150 velocity=14.6
- joint leg_l3_joint: limit lower=-1.7453 upper=1.7453 effort=100 velocity=41.3433333333333 -> lower=-1.7453 upper=1.7453 effort=70 velocity=12.0
- joint leg_l4_joint: limit lower=-0.08726646 upper=2.530727 effort=180 velocity=23.55 -> lower=-0.08726646 upper=2.530727 effort=150 velocity=14.6
- joint leg_l5_joint: limit lower=-0.872664625997165 upper=0.523598775598299 effort=36.0 velocity=23.0266666666667 -> lower=-0.872664625997165 upper=0.523598775598299 effort=74 velocity=17.0
- joint leg_l6_joint: limit lower=-0.261799387799149 upper=0.261799387799149 effort=36 velocity=23.0266666666667 -> lower=-0.261799387799149 upper=0.261799387799149 effort=74 velocity=17.0
- joint leg_r1_joint: limit lower=-3.228 upper=2.44346 effort=180 velocity=23.55 -> lower=-2.44346 upper=3.228 effort=150 velocity=14.6; origin xyz=0.0 -0.12441237 -0.22115341 rpy=0 0 0 -> xyz=0.0 -0.12441 -0.22265 rpy=0 0 0
- joint leg_r2_joint: limit lower=-2.40855 upper=0.837758 effort=100 velocity=41.3433333333333 -> lower=-2.40855 upper=0.837758 effort=150 velocity=14.6
- joint leg_r3_joint: limit lower=-1.7453 upper=1.7453 effort=100 velocity=41.3433333333333 -> lower=-1.7453 upper=1.7453 effort=70 velocity=12.0
- joint leg_r4_joint: limit lower=-0.08726646 upper=2.530727 effort=180 velocity=23.55 -> lower=-0.08726646 upper=2.530727 effort=150 velocity=14.6
- joint leg_r5_joint: limit lower=-0.872664625997165 upper=0.523598775598299 effort=36.0 velocity=23.0266666666667 -> lower=-0.872664625997165 upper=0.523598775598299 effort=74 velocity=17.0
- joint leg_r6_joint: limit lower=-0.261799387799149 upper=0.261799387799149 effort=36 velocity=23.0266666666667 -> lower=-0.261799387799149 upper=0.261799387799149 effort=74 velocity=17.0
- joint zarm_l1_joint: limit lower=-3.14159265358979 upper=2.0943951023932 effort=12 velocity=7.32666666666667 -> lower=-3.14159265358979 upper=2.0943951023932 effort=14.1 velocity=10.5; origin xyz=0.0 0.18100293 0.23992606 rpy=0 0 0 -> xyz=0 0.181 0.23843 rpy=0 0 0
- joint zarm_l2_joint: limit lower=-0.52 upper=3.316 effort=12 velocity=7.32666666666667 -> lower=-0.52 upper=3.316 effort=37 velocity=15.0
- joint zarm_l3_joint: limit lower=-1.5707963267949 upper=1.5707963267949 effort=12 velocity=7.32666666666667 -> lower=-1.5707963267949 upper=1.5707963267949 effort=37 velocity=15.0
- joint zarm_l4_joint: limit lower=-2.26892802759263 upper=0.08726 effort=12 velocity=7.32666666666667 -> lower=-2.26892802759263 upper=0.08726 effort=37 velocity=15.0; origin xyz=0 0.0 -0.20533 rpy=0 0 0 -> xyz=0 0 -0.2085 rpy=0 0 0
- joint zarm_r1_joint: limit lower=-3.14159265358979 upper=2.0943951023932 effort=12 velocity=7.32666666666667 -> lower=-3.14159265358979 upper=2.0943951023932 effort=14.1 velocity=10.5; origin xyz=0.0 -0.18100293 0.23992606 rpy=0 0 0 -> xyz=0 -0.181 0.23843 rpy=0 0 0
- joint zarm_r2_joint: limit lower=-3.3161 upper=0.52 effort=12 velocity=7.32666666666667 -> lower=-3.3161 upper=0.52 effort=37.0 velocity=15.0
- joint zarm_r3_joint: limit lower=-1.5707963267949 upper=1.5707963267949 effort=12 velocity=7.32666666666667 -> lower=-1.5707963267949 upper=1.5707963267949 effort=37.0 velocity=15.0
- joint zarm_r4_joint: limit lower=-2.26892802759263 upper=0.08726 effort=12 velocity=7.32666666666667 -> lower=-2.26892802759263 upper=0.08726 effort=37.0 velocity=15.0; origin xyz=0 -0.0 -0.20533 rpy=0 0 0 -> xyz=0 0 -0.2085 rpy=0 0 0

Commit message: sync https://www.lejuhub.com/highlydynamic/kuavo-ros-control/commit/8ed1b83bd492ce0cdf2bffa03f0b52e8d59f0902

File: src/kuavo_assets/models/biped_s17/urdf/biped_s17.urdf (robot description, URDF)
Before this commit: robot biped_s17, 43 links, 42 joints
Links:
- link base_link: mass 5.27737344 -> 6.61137344

File: src/kuavo_assets/models/biped_s17/urdf/biped_s17_gazebo.urdf (robot description, URDF)
Before this commit: robot biped_s17, 43 links, 42 joints
Links:
- link base_link: mass 5.27737344 -> 6.61137344
