Commit message: sync https://www.lejuhub.com/highlydynamic/kuavo-ros-control/commit/c665c08de2c124bf54b19fd394808ea2caee9fea

File: src/kuavo_assets/models/biped_s17/urdf/biped_s17.urdf (robot description, URDF)
Before this commit: robot biped_s17, 43 links, 42 joints
Links:
- link base_link: mass 5.27737344 -> 6.61137344
Joints:
- removed joint dummy_to_base_link
- added joint base_link_to_dummy_link: type fixed, parent base_link, child dummy_link, origin xyz=0 0 0 rpy=0 0 0

File: src/kuavo_assets/models/biped_s17/urdf/biped_s17_gazebo.urdf (robot description, URDF)
Before this commit: robot biped_s17, 43 links, 42 joints
Links:
- link base_link: mass 5.27737344 -> 6.61137344
Joints:
- removed joint dummy_to_base_link
- added joint base_link_to_dummy_link: type fixed, parent base_link, child dummy_link, origin xyz=0 0 0 rpy=0 0 0

File: src/kuavo_assets/models/biped_s40/urdf/biped_s40_gazebo.urdf (robot description, URDF)
Before this commit: robot biped_s40, 46 links, 45 joints
Joints:
- removed joint dummy_to_base_link
- added joint base_link_to_dummy_link: type fixed, parent base_link, child dummy_link, origin xyz=0 0 0 rpy=0 0 0

File: src/kuavo_assets/models/biped_s56/urdf/biped_s56.urdf (robot description, URDF)
Before this commit: robot biped_s56, 50 links, 49 joints
Links:
- link leg_l5_link: mass 0.07554 -> 0.33065201
- link leg_l6_link: mass 0.60538 -> 0.85589925
- link leg_r5_link: mass 0.07554 -> 0.33065201
- link leg_r6_link: mass 0.60538 -> 0.85589925
- link waist_camera: mass 0.001 -> 7.8539816339743E-05; geometry visual mesh filename=../meshes/waist_camera_depth.STL
- link waist_camera_base: mass 0.13300 -> 0.13300000; geometry visual mesh filename=../meshes/waist_camera_base.STL
- link waist_yaw_link: mass 19.98099 -> 19.98211
Joints:
- removed joint dummy_to_base_link
- added joint base_link_to_dummy_link: type fixed, parent base_link, child dummy_link, origin xyz=0 0 0 rpy=0 0 0
- joint l_foot_heel_joint: origin xyz=-0.073164 0.0 -0.0595 rpy=0 0 0 -> xyz=-0.07316377 0.0 -0.0365 rpy=0 0 0
- joint l_foot_toe_joint: origin xyz=0.17084 0.0 -0.0595 rpy=0 0 0 -> xyz=0.17083623 0.0 -0.0365 rpy=0 0 0
- joint leg_l5_joint: origin xyz=0.002 0 -0.416 rpy=0 0 0 -> xyz=0 0 -0.416 rpy=0 0 0
- joint leg_l6_joint: origin xyz=0 0 0 rpy=0 0 0 -> xyz=0 0 -0.023 rpy=0 0 0
- joint leg_r5_joint: origin xyz=0.002 0 -0.416 rpy=0 0 0 -> xyz=0 0 -0.416 rpy=0 0 0
- joint leg_r6_joint: origin xyz=0 0 0 rpy=0 0 0 -> xyz=0 0 -0.023 rpy=0 0 0
- joint ll_foot_heel_joint: origin xyz=-0.073164 0.05 -0.0595 rpy=0 0 0 -> xyz=-0.07316377 0.05 -0.0365 rpy=0 0 0
- joint ll_foot_toe_joint: origin xyz=0.17084 0.05 -0.0595 rpy=0 0 0 -> xyz=0.17083623 0.05 -0.0365 rpy=0 0 0
- joint lr_foot_heel_joint: origin xyz=-0.073164 -0.05 -0.0595 rpy=0 0 0 -> xyz=-0.07316377 -0.05 -0.0365 rpy=0 0 0
- joint lr_foot_toe_joint: origin xyz=0.17084 -0.05 -0.0595 rpy=0 0 0 -> xyz=0.17083623 -0.05 -0.0365 rpy=0 0 0
- joint r_foot_heel_joint: origin xyz=-0.073164 0.0 -0.0595 rpy=0 0 0 -> xyz=-0.07316377 0.0 -0.0365 rpy=0 0 0
- joint r_foot_toe_joint: origin xyz=0.17084 0.0 -0.0595 rpy=0 0 0 -> xyz=0.17083623 0.0 -0.0365 rpy=0 0 0
- joint rl_foot_heel_joint: origin xyz=-0.073164 0.05 -0.0595 rpy=0 0 0 -> xyz=-0.07316377 0.05 -0.0365 rpy=0 0 0
- joint rl_foot_toe_joint: origin xyz=0.17084 0.05 -0.0595 rpy=0 0 0 -> xyz=0.17083623 0.05 -0.0365 rpy=0 0 0
- joint rr_foot_heel_joint: origin xyz=-0.073164 -0.05 -0.0595 rpy=0 0 0 -> xyz=-0.07316377 -0.05 -0.0365 rpy=0 0 0
- joint rr_foot_toe_joint: origin xyz=0.17084 -0.05 -0.0595 rpy=0 0 0 -> xyz=0.17083623 -0.05 -0.0365 rpy=0 0 0
- joint waist_yaw_joint: origin xyz=0 0 0.111 rpy=0 0 0 -> xyz=0 0 0.1114 rpy=0 0 0
- joint zarm_l1_joint: origin xyz=-0.003 0.253 0.2834 rpy=0 0 0 -> xyz=-0.003 0.2527 0.283 rpy=0 0 0
- joint zarm_r1_joint: origin xyz=-0.003 -0.253 0.2834 rpy=0 0 0 -> xyz=-0.003 -0.2527 0.283 rpy=0 0 0
- joint zhead_1_joint: origin xyz=-0.003 0.0 0.49125 rpy=0 0 0 -> xyz=-0.003 0.0 0.49535 rpy=0 0 0

File: src/kuavo_assets/models/biped_s56/urdf/biped_s56_gazebo.urdf (robot description, URDF)
Before this commit: robot biped_s56, 48 links, 47 joints
Links:
- removed link camera_base
- removed link head_rader
- added link head_camera_base, mass 0.0; visual mesh filename=package://kuavo_assets/models/biped_s56/meshes/head_camera_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
- added link head_camera_depth, mass 0.0000785398163397463; visual mesh filename=package://kuavo_assets/models/biped_s56/meshes/head_camera_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
- added link head_radar, mass 0.0; visual mesh filename=package://kuavo_assets/models/biped_s56/meshes/head_radar.S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
- added link waist_camera_base, mass 0.13300000; visual mesh filename=package://kuavo_assets/models/biped_s56/meshes/waist_camera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
- link waist_camera: mass 0.048238 -> 0.0000785398163397463
Joints:
- removed joint camera_base
- removed joint dummy_to_base_link
- removed joint head_rader_joint
- removed joint waist_camera
- added joint base_link_to_dummy_link: type fixed, parent base_link, child dummy_link, origin xyz=0 0 0 rpy=0 0 0
- added joint head_camera_base_joint: type fixed, parent zhead_2_link, child head_camera_base, origin xyz=0.099619 0 0.032844 rpy=0 0.3406 0, axis 0 0 0
- added joint head_camera_depth_joint: type fixed, parent head_camera_base, child head_camera_depth, origin xyz=0.011715 0.0475 0.014312 rpy=0 0 0, axis 0 0 0
- added joint head_radar_joint: type fixed, parent zhead_1_link, child head_radar, origin xyz=0 0 -0.078453 rpy=0 0 0, axis 0 0 0
- added joint waist_camera_base_joint: type fixed, parent waist_yaw_link, child waist_camera_base, origin xyz=0.0787 0 -0.028149 rpy=0 0.59341 0, axis 0 0 0
- added joint waist_camera_joint: type fixed, parent waist_camera_base, child waist_camera, origin xyz=0.011715 0.0475 0.014312 rpy=0 0 0, axis 0 0 0
- joint leg_r6_joint: origin xyz=0 0 0 rpy=0 0 0 -> xyz=0 0 -0.023 rpy=0 0 0

File: src/kuavo_assets/models/biped_s56/urdf/biped_s56_gazebo.xacro (robot description, xacro)
@@ -6,5 +6,5 @@
   <xacro:include filename="$(find realsense_ros_gazebo)/xacro/depthcam.xacro"/>
   <!-- d435 声明 -->
-  <xacro:realsense_d435 sensor_name="camera" parent_link="camera_base" rate="30">
+  <xacro:realsense_d435 sensor_name="camera" parent_link="head_camera_base" rate="30">
     <origin rpy="0 0 0 " xyz="0 0 0"/>
   </xacro:realsense_d435>

File: src/kuavo_assets/models/biped_s56/urdf/drake/biped_v3_all_joint.urdf (robot description, URDF)
Before this commit: robot biped_v3_all_joint, 35 links, 30 joints
Links:
- link leg_l1_link: mass 1.71093115 -> 1.55641
- link leg_l2_link: mass 0.58029165 -> 0.75873
- link leg_l3_link: mass 4.50393141 -> 6.68074
- link leg_l4_link: mass 1.62776815 -> 3.64666
- link leg_r1_link: mass 1.71093008 -> 1.55641
- link leg_r2_link: mass 0.58029165 -> 0.75873
- link leg_r3_link: mass 4.50385993 -> 6.68074
- link leg_r4_link: mass 1.62655699 -> 3.64666
Joints:
- joint l_l_bar_y: origin xyz=0 0.0318 -0.09 rpy=0 0 0 -> xyz=0.0535 0 -0.1883 rpy=0 0 0
- joint l_r_bar_y: origin xyz=0 -0.0362 -0.153 rpy=0 0 0 -> xyz=0.0535 0 -0.0983 rpy=0 0 0
- joint leg_l1_joint: limit lower=-0.314159265358979 upper=0.663225115757845 effort=180.0 velocity=23.55 -> lower=-0.314159265358979 upper=0.663225115757845 effort=127.0 velocity=10.4; origin xyz=-0.0024999 0.087 -0.066 rpy=0 0 0 -> xyz=0.0 0.095075 -0.066 rpy=0 0 0
- joint leg_l2_joint: limit lower=-0.872664625997165 upper=0.785398163397448 effort=100.0 velocity=41.3433333333333 -> lower=-0.785398163397448 upper=1.91986217719376 effort=71.0 velocity=8.7
- joint leg_l3_joint: limit lower=-2.00712863979348 upper=1.5707963267949 effort=100.0 velocity=41.3433333333333 -> lower=-1.91986217719376 upper=1.5707963267949 effort=132 velocity=12.7; origin xyz=0.000500354536093913 -0.00100000000000011 -0.1287 rpy=0 0 0 -> xyz=0 0 -0.1437 rpy=0 0 0
- joint leg_l4_joint: limit lower=0.0 upper=2.53072741539178 effort=180.0 velocity=23.55 -> lower=0.0 upper=2.53072741539178 effort=280.0 velocity=10.4; origin xyz=-6.87185435835039E-05 0 -0.284 rpy=0 0 0 -> xyz=-0.0011639 0 -0.284 rpy=0 0 0
- joint leg_l5_joint: limit lower=-0.872664625997165 upper=0.349065850398866 effort=36.0 velocity=23.0266666666667 -> lower=-0.872664625997165 upper=0.349065850398866 effort=91.6 velocity=17.8; origin xyz=-0.000431635992531742 0 -0.346000000000001 rpy=0 0 0 -> xyz=0.00 0 -0.416 rpy=0 0 0
- joint leg_l6_joint: limit lower=-0.261799387799149 upper=0.261799387799149 effort=36.0 velocity=23.0266666666667 -> lower=-0.261799387799149 upper=0.261799387799149 effort=30.0 velocity=17.8
- joint leg_r1_joint: limit lower=-0.663225115757845 upper=0.314159265358979 effort=180.0 velocity=23.55 -> lower=-0.663225115757845 upper=0.314159265358979 effort=127.0 velocity=10.4; origin xyz=-0.0024999 -0.087 -0.066 rpy=0 0 0 -> xyz=0.0 -0.095075 -0.066 rpy=0 0 0
- joint leg_r2_joint: limit lower=-0.785398163397448 upper=0.872664625997165 effort=100.0 velocity=41.3433333333333 -> lower=-1.91986217719376 upper=0.785398163397448 effort=71.0 velocity=8.7
- joint leg_r3_joint: limit lower=-2.00712863979348 upper=1.5707963267949 effort=100.0 velocity=41.3433333333333 -> lower=-1.91986217719376 upper=1.5707963267949 effort=132.0 velocity=12.7; origin xyz=-4.88006581312577E-05 0 -0.1287 rpy=0 0 0 -> xyz=0 0 -0.1437 rpy=0 0 0
- joint leg_r4_joint: limit lower=0.0 upper=2.53072741539178 effort=180.0 velocity=23.55 -> lower=0.0 upper=2.53072741539178 effort=280.0 velocity=10.4; origin xyz=0.000147138572785148 0 -0.283999982974744 rpy=0 0 0 -> xyz=-0.0011639 0 -0.284 rpy=0 0 0
- joint leg_r5_joint: limit lower=-0.872664625997165 upper=0.349065850398866 effort=36.0 velocity=23.0266666666667 -> lower=-0.872664625997165 upper=0.349065850398866 effort=91.6 velocity=17.8; origin xyz=0.000119806050928577 0 -0.345999979257963 rpy=0 0 0 -> xyz=0.000 0 -0.416 rpy=0 0 0
- joint leg_r6_joint: limit lower=-0.261799387799149 upper=0.261799387799149 effort=36.0 velocity=23.0266666666667 -> lower=-0.261799387799149 upper=0.261799387799149 effort=30.0 velocity=17.8; origin xyz=0 0 0 rpy=0 0 0 -> xyz=0 0 -0.023 rpy=0 0 0
- joint r_l_bar_y: origin xyz=0 0.0362 -0.153 rpy=0 0 0 -> xyz=0.0535 0 -0.0983 rpy=0 0 0
- joint r_r_bar_y: origin xyz=0 -0.0318 -0.09 rpy=0 0 0 -> xyz=0.0535 0 -0.1883 rpy=0 0 0

Commit message: sync https://www.lejuhub.com/highlydynamic/kuavo-ros-control/commit/128f196dbc67aeea536e4db051b68e9662559a15

File: src/kuavo_assets/models/biped_s17/urdf/biped_s17.urdf (robot description, URDF)
Before this commit: robot biped_s17, 43 links, 42 joints
Joints:
- joint zhead_1_joint: origin xyz=0.0042 0 0.35369 rpy=0 0 0 -> xyz=0.0042 0 0.35469 rpy=0 0 0

File: src/kuavo_assets/models/biped_s17/urdf/biped_s17_gazebo.urdf (robot description, URDF)
Before this commit: robot biped_s17, 43 links, 42 joints
Joints:
- joint zhead_1_joint: origin xyz=0.0042 0 0.35369 rpy=0 0 0 -> xyz=0.0042 0 0.35469 rpy=0 0 0

Commit message: sync https://www.lejuhub.com/highlydynamic/kuavo-ros-control/commit/1c853b776b54ccb01a0f7a9fbe29a4151ab340fa

File: src/kuavo_assets/models/biped_s17/urdf/biped_s17.urdf (robot description, URDF)
Before this commit: robot biped_s17, 43 links, 42 joints
Links:
- link base_link: mass 6.61137344 -> 5.27737344

Commit message: sync https://www.lejuhub.com/highlydynamic/kuavo-ros-control/commit/6f0789ee5a527ef737ce02917e4f21db8a91f054

File: src/kuavo_assets/models/biped_s17/urdf/biped_s17.urdf (robot description, URDF)
Before this commit: robot biped_s17, 43 links, 42 joints
Links:
- link base_link: mass 6.61137344 -> 5.27737344
Joints:
- joint zhead_1_joint: origin xyz=0.0042 0 0.35369 rpy=0 0 0 -> xyz=0.0042 0 0.35469 rpy=0 0 0

File: src/kuavo_assets/models/biped_s17/urdf/biped_s17_gazebo.urdf (robot description, URDF)
Before this commit: robot biped_s17, 43 links, 42 joints
Links:
- link base_link: mass 6.61137344 -> 5.27737344
Joints:
- joint zhead_1_joint: origin xyz=0.0042 0 0.35369 rpy=0 0 0 -> xyz=0.0042 0 0.35469 rpy=0 0 0

File: src/kuavo_assets/models/biped_s17/urdf/drake/biped_v3_all_joint.urdf (robot description, URDF)
Before this commit: robot biped_v3_all_joint, 30 links, 25 joints
Links:
- link torso: mass 11.10734703 -> 9.77334703

File: src/kuavo_assets/models/biped_s17/urdf/drake/biped_v3_full.urdf (robot description, URDF)
Before this commit: robot biped_v3_full, 22 links, 21 joints
Links:
- link torso: mass 11.75014703 -> 10.41614703

File: src/kuavo_assets/models/biped_s40/urdf/biped_s40_gazebo.urdf (robot description, URDF)
Before this commit: robot biped_s40, 46 links, 45 joints
Links:
- link base_link: mass 22.6719 -> 22.6889

File: src/kuavo_assets/models/biped_s63/urdf/biped_s63.urdf (robot description, URDF)
Before this commit: robot biped_s63, 36 links, 35 joints
Joints:
- joint zhead_1_joint: origin xyz=0 0 0.43485 rpy=0 0 0 -> xyz=0 0 0.43935 rpy=0 0 0

File: src/kuavo_assets/models/biped_s63/urdf/biped_s63_gazebo.urdf (robot description, URDF)
Before this commit: robot biped_s63, 40 links, 39 joints
Joints:
- joint zhead_1_joint: origin xyz=0 0 0.43485 rpy=0 0 0 -> xyz=0 0 0.43935 rpy=0 0 0
