Commit message: sync https://www.lejuhub.com/highlydynamic/kuavo-ros-control/commit/3eb57342ffdf3ab20d45d793be22c771440a4ed1

File: src/kuavo_assets/models/biped_s63/urdf/drake/biped_v3_arm.urdf (robot description, URDF)
Before this commit: robot biped_s45, 17 links, 16 joints
Links:
- added link base_to_joint, mass 7.34488200; visual mesh filename=../../meshes/knee_link.STL
- added link knee_link, mass 13.60706531; visual mesh filename=../../meshes/knee_pitch.STL
- added link leg_link, mass 9.43091394; visual mesh filename=../../meshes/leg_pitch.STL
- added link waist_link, mass 8.15311772; visual mesh filename=../../meshes/waist_pitch.STL
- added link waist_yaw_link, mass 12.64200813; collision cylinder length=0.6 radius=0.15; visual mesh filename=../../meshes/torso.STL
- added link zarm_l7_end_effector_1
- added link zarm_l7_end_effector_2
- added link zarm_l7_virtual_thumb_link; collision sphere radius=0.005
- added link zarm_r7_end_effector_1
- added link zarm_r7_end_effector_2
- added link zarm_r7_virtual_thumb_link; collision sphere radius=0.005
- link base_link: mass 11.56094002 -> 129.40001; geometry collision cylinder length=0.32 radius=0.37; visual mesh filename=../../meshes/chassis.STL
- link zarm_l1_link: mass 0.91653322 -> 1.01295970
- link zarm_l2_link: mass 0.38767390 -> 0.43788857; geometry collision cylinder length=0.3 radius=0.05; visual mesh filename=../../meshes/l_arm_roll.STL
- link zarm_l3_link: mass 1.77926875 -> 1.83544700
- link zarm_l4_link: mass 0.58507821 -> 0.65770374; geometry collision cylinder length=0.26 radius=0.05; visual mesh filename=../../meshes/l_forearm.STL
- link zarm_l5_link: mass 0.68679955 -> 0.67878399
- link zarm_l6_link: mass 0.39387181 -> 0.51230538
- link zarm_l7_link: mass 0.71537800 -> 0.7374; geometry collision cylinder length=0.14 radius=0.04; visual mesh filename=../../meshes/l_hand_pitch_noHand.STL
- link zarm_r1_link: mass 0.91653322 -> 1.01295970
- link zarm_r2_link: mass 0.38767390 -> 0.43788857; geometry collision cylinder length=0.3 radius=0.05; visual mesh filename=../../meshes/r_arm_roll.STL
- link zarm_r3_link: mass 1.77926875 -> 1.83544700
- link zarm_r4_link: mass 0.58507821 -> 0.65770374; geometry collision cylinder length=0.26 radius=0.05; visual mesh filename=../../meshes/r_forearm.STL
- link zarm_r5_link: mass 0.68679955 -> 0.67878399
- link zarm_r6_link: mass 0.39387181 -> 0.51230538
- link zarm_r7_link: mass 0.71537800 -> 0.7374; geometry collision cylinder length=0.14 radius=0.04; visual mesh filename=../../meshes/r_hand_pitch_noHand.STL
Joints:
- added joint base_to_joint: type fixed, parent base_link, child base_to_joint, origin xyz=0.093 0 0.30085 rpy=0 0 0, axis 0 1 0
- added joint knee_joint: type revolute, parent base_to_joint, child knee_link, origin xyz=0 0 0.1055 rpy=0 0 0, axis 0 1 0, limit lower=0 upper=1.44862327915529 effort=668.53 velocity=25.33
- added joint leg_joint: type revolute, parent knee_link, child leg_link, origin xyz=-0.46521 0 0.18325 rpy=0 0 0, axis 0 1 0, limit lower=-2.80998009571087 upper=0.0 effort=668.53 velocity=25.33
- added joint waist_pitch_joint: type revolute, parent leg_link, child waist_link, origin xyz=0.48296 0 0.12941 rpy=0 0 0, axis 0 1 0, limit lower=-0.15707963267949 upper=2.9845130209103 effort=618.48 velocity=25.33
- added joint waist_yaw_joint: type revolute, parent waist_link, child waist_yaw_link, origin xyz=0 0 0.25 rpy=0 0 0, axis 0 0 1, limit lower=-3.14159265358979 upper=3.14159265358979 effort=618.48 velocity=25.33
- added joint zarm_l7_end_effector_1_joint: type fixed, parent zarm_l7_link, child zarm_l7_end_effector_1, origin xyz=0 0.0 -0.08 rpy=0 0 0
- added joint zarm_l7_end_effector_2_joint: type fixed, parent zarm_l7_link, child zarm_l7_end_effector_2, origin xyz=0.03 0.0 -0.17 rpy=0 0 0
- added joint zarm_l7_virtual_thumb_joint_ee: type fixed, parent zarm_l7_end_effector, child zarm_l7_virtual_thumb_link, origin xyz=0.15 0 0 rpy=0 0 0
- added joint zarm_r7_end_effector_1_joint: type fixed, parent zarm_r7_link, child zarm_r7_end_effector_1, origin xyz=0 0.0 -0.08 rpy=0 0 0
- added joint zarm_r7_end_effector_2_joint: type fixed, parent zarm_r7_link, child zarm_r7_end_effector_2, origin xyz=0.03 0.0 -0.17 rpy=0 0 0
- added joint zarm_r7_virtual_thumb_joint_ee: type fixed, parent zarm_r7_end_effector, child zarm_r7_virtual_thumb_link, origin xyz=0.15 0 0 rpy=0 0 0
- joint zarm_l1_joint: limit lower=-3.14159265358979 upper=1.5707963267949 effort=66.0 velocity=18.8 -> lower=-2.4 upper=0.6 effort=85.0 velocity=13.0; origin xyz=0 0.2527 0.242 rpy=0 0 0 -> xyz=0 0.253 0.227 rpy=0 0 0; parent base_link -> waist_yaw_link
- joint zarm_l2_joint: limit lower=-0.349065850398866 upper=3.49065850398866 effort=75.0 velocity=8.0 -> lower=-0.349065850398866 upper=1.46 effort=75.0 velocity=8.0
- joint zarm_l3_joint: limit lower=-1.48352986419518 upper=1.48352986419518 effort=57.0 velocity=7.5 -> lower=-1.5707963267949 upper=0.46 effort=57.0 velocity=7.5
- joint zarm_r1_joint: limit lower=-3.14159265358979 upper=1.5707963267949 effort=66.0 velocity=18.8 -> lower=-2.4 upper=0.6 effort=85.0 velocity=13.0; origin xyz=0 -0.2527 0.242 rpy=0 0 0 -> xyz=0 -0.253 0.227 rpy=0 0 0; parent base_link -> waist_yaw_link
- joint zarm_r2_joint: limit lower=-3.49065850398866 upper=0.349065850398866 effort=75.0 velocity=8.0 -> lower=-1.46 upper=0.349065850398866 effort=75.0 velocity=8.0
- joint zarm_r3_joint: limit lower=-1.48352986419518 upper=1.48352986419518 effort=57.0 velocity=7.5 -> lower=-0.46 upper=1.5707963267949 effort=57.0 velocity=7.5
