Commit message: sync https://www.lejuhub.com/highlydynamic/kuavo-ros-control/commit/a59e92419f5618b8882bc23496d0ef9aaff863cd

File: src/kuavo_assets/models/wheel_arm_upper_body/urdf/drake/wheel_v3_arm_only.urdf (robot description, URDF)
Before this commit: robot biped_s62, 28 links, 27 joints
Links:
- link zarm_l7_link: mass 0.71537800 -> 0.0542110173081966
- link zarm_r7_link: mass 0.71537800 -> 0.11660000
