Commit message: sync https://www.lejuhub.com/highlydynamic/kuavo-ros-control/commit/5cdd6f9cda3e8e25afe0f3a7a7531ae1a563b242

File: src/kuavo_assets/models/biped_s200049/urdf/drake/biped_v3_arm.urdf (robot description, URDF)
Before this commit: robot biped_s200049, 19 links, 18 joints
Joints:
- joint zarm_l7_end_effector_joint: origin xyz=0 0 -0.17 rpy=0 0 0 -> xyz=0 -0.03 -0.17 rpy=0 0 0
- joint zarm_r7_end_effector_joint: origin xyz=0 0 -0.17 rpy=0 0 0 -> xyz=0 0.03 -0.17 rpy=0 0 0
