Commit message: sync https://www.lejuhub.com/highlydynamic/kuavo-ros-control/commit/bb977f7ff3954b61b401493bb51530a5b534942b

File: src/kuavo_assets/models/biped_s400055/urdf/biped_s400055.urdf (robot description, URDF)
Before this commit: robot biped_s400055, 74 links, 73 joints
Links:
- link leg_l3_link: geometry collision cylinder length=0.04 radius=0.06; collision cylinder length=0.25 radius=0.065
- link leg_l4_link: geometry collision cylinder length=0.3 radius=0.05; visual mesh filename=package://kuavo_assets/models/biped_s400055/meshes/l_knee.S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
- link leg_l6_link: geometry collision box size=0.042 0.096 0.0108; collision box size=0.09 0.1 0.0108
- link leg_r3_link: geometry collision cylinder length=0.04 radius=0.06; collision cylinder length=0.25 radius=0.065
- link leg_r4_link: geometry collision cylinder length=0.3 radius=0.05; visual mesh filename=package://kuavo_assets/models/biped_s400055/meshes/r_knee.S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
- link leg_r6_link: geometry collision box size=0.042 0.096 0.0108; collision box size=0.09 0.1 0.0108
- link waist_yaw_link: geometry collision cylinder length=0.06 radius=0.13; collision cylinder length=0.12 radius=0.13
- link zarm_l1_link: geometry collision cylinder length=0.04 radius=0.05; visual mesh filename=package://kuavo_assets/models/biped_s400055/meshes/l_arm_pi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
- link zarm_l3_link: geometry collision cylinder length=0.14 radius=0.045; visual mesh filename=package://kuavo_assets/models/biped_s400055/meshes/l_arm_ya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
- link zarm_l4_link: geometry collision cylinder length=0.18 radius=0.045; visual mesh filename=package://kuavo_assets/models/biped_s400055/meshes/l_forear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
- link zarm_l7_link: geometry collision box size=0.08 0.05 0.16; collision cylinder length=0.08 radius=0.01
- link zarm_r1_link: geometry collision cylinder length=0.04 radius=0.05; visual mesh filename=package://kuavo_assets/models/biped_s400055/meshes/r_arm_pi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
- link zarm_r3_link: geometry collision cylinder length=0.14 radius=0.045; visual mesh filename=package://kuavo_assets/models/biped_s400055/meshes/r_arm_ya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
- link zarm_r4_link: geometry collision cylinder length=0.18 radius=0.045; visual mesh filename=package://kuavo_assets/models/biped_s400055/meshes/r_forear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
- link zarm_r7_link: geometry collision box size=0.08 0.05 0.16; collision cylinder length=0.08 radius=0.01
Joints:
- joint l_hand_base_joint: origin xyz=0 0 -0.07 rpy=0 3.14159265358979 0 -> xyz=0 0 -0.053 rpy=0 3.14159265358979 0
- joint l_index_j1: type fixed -> revolute
- joint l_index_j2: type fixed -> revolute
- joint l_index_j3: type fixed -> revolute
- joint l_little_j1: type fixed -> revolute
- joint l_little_j2: type fixed -> revolute
- joint l_little_j3: type fixed -> revolute
- joint l_middle_j1: type fixed -> revolute
- joint l_middle_j2: type fixed -> revolute
- joint l_thumb_j1: type fixed -> revolute
- joint l_thumb_j2: type fixed -> revolute
- joint l_thumb_j3: type fixed -> revolute
- joint r_hand_base_joint: origin xyz=0 0 -0.07 rpy=3.14159265358979 0 0 -> xyz=0 0 -0.053 rpy=3.14159265358979 0 0
- joint r_index_j1: type fixed -> revolute
- joint r_index_j2: type fixed -> revolute
- joint r_index_j3: type fixed -> revolute
- joint r_little_j1: type fixed -> revolute
- joint r_little_j2: type fixed -> revolute
- joint r_little_j3: type fixed -> revolute
- joint r_middle_j1: type fixed -> revolute
- joint r_middle_j2: type fixed -> revolute
- joint r_thumb_j1: type fixed -> revolute
- joint r_thumb_j2: type fixed -> revolute
- joint r_thumb_j3: type fixed -> revolute

File: src/kuavo_assets/models/biped_s400055/urdf/biped_s400055_gazebo.urdf (robot description, URDF)
Before this commit: robot biped_s55, 74 links, 73 joints
Links:
- link base_link: geometry visual mesh filename=package://kuavo_assets/models/biped_s400055/meshes/torso.STL
- link head_camera_base: geometry visual mesh filename=package://kuavo_assets/models/biped_s400055/meshes/head_cam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
- link head_camera_depth: geometry visual mesh filename=package://kuavo_assets/models/biped_s400055/meshes/head_cam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
- link head_radar: geometry visual mesh filename=package://kuavo_assets/models/biped_s400055/meshes/head_rad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
- link leg_l1_link: geometry visual mesh filename=package://kuavo_assets/models/biped_s400055/meshes/l_leg_ro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
- link leg_l2_link: geometry visual mesh filename=package://kuavo_assets/models/biped_s400055/meshes/l_leg_ya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
- link leg_l3_link: geometry visual mesh filename=package://kuavo_assets/models/biped_s400055/meshes/l_leg_pi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
- link leg_l4_link: geometry visual mesh filename=package://kuavo_assets/models/biped_s400055/meshes/l_knee.S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
- link leg_l5_link: geometry visual mesh filename=package://kuavo_assets/models/biped_s400055/meshes/l_foot_p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
- link leg_l6_link: geometry collision box size=0.25 0.1 0.04; visual mesh filename=package://kuavo_assets/models/biped_s400055/meshes/l_foot_r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
- link leg_r1_link: geometry visual mesh filename=package://kuavo_assets/models/biped_s400055/meshes/r_leg_ro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
- link leg_r2_link: geometry visual mesh filename=package://kuavo_assets/models/biped_s400055/meshes/r_leg_ya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
- link leg_r3_link: geometry visual mesh filename=package://kuavo_assets/models/biped_s400055/meshes/r_leg_pi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
- link leg_r4_link: geometry visual mesh filename=package://kuavo_assets/models/biped_s400055/meshes/r_knee.S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
- link leg_r5_link: geometry visual mesh filename=package://kuavo_assets/models/biped_s400055/meshes/r_foot_p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
- link leg_r6_link: geometry collision box size=0.25 0.1 0.04; visual mesh filename=package://kuavo_assets/models/biped_s400055/meshes/r_foot_r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
- link waist_camera: geometry visual mesh filename=package://kuavo_assets/models/biped_s400055/meshes/waist_ca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
- link waist_camera_base: geometry visual mesh filename=package://kuavo_assets/models/biped_s400055/meshes/waist_ca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
- link waist_yaw_link: geometry visual mesh filename=package://kuavo_assets/models/biped_s400055/meshes/waist_ya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
- link zarm_l1_link: geometry visual mesh filename=package://kuavo_assets/models/biped_s400055/meshes/l_arm_pi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
- link zarm_l2_link: geometry visual mesh filename=package://kuavo_assets/models/biped_s400055/meshes/l_arm_ro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
- link zarm_l3_link: geometry visual mesh filename=package://kuavo_assets/models/biped_s400055/meshes/l_arm_ya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
- link zarm_l4_link: geometry visual mesh filename=package://kuavo_assets/models/biped_s400055/meshes/l_forear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
- link zarm_l5_link: geometry visual mesh filename=package://kuavo_assets/models/biped_s400055/meshes/l_hand_y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
- link zarm_l6_link: geometry visual mesh filename=package://kuavo_assets/models/biped_s400055/meshes/l_hand_r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
- link zarm_l7_link: geometry collision box size=0.08 0.05 0.16; collision cylinder length=0.08 radius=0.01
- link zarm_r1_link: geometry visual mesh filename=package://kuavo_assets/models/biped_s400055/meshes/r_arm_pi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
- link zarm_r2_link: geometry visual mesh filename=package://kuavo_assets/models/biped_s400055/meshes/r_arm_ro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
- link zarm_r3_link: geometry visual mesh filename=package://kuavo_assets/models/biped_s400055/meshes/r_arm_ya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
- link zarm_r4_link: geometry visual mesh filename=package://kuavo_assets/models/biped_s400055/meshes/r_forear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
- link zarm_r5_link: geometry visual mesh filename=package://kuavo_assets/models/biped_s400055/meshes/r_hand_y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
- link zarm_r6_link: geometry visual mesh filename=package://kuavo_assets/models/biped_s400055/meshes/r_hand_r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
- link zarm_r7_link: geometry collision box size=0.08 0.05 0.16; collision cylinder length=0.08 radius=0.01
- link zhead_1_link: geometry visual mesh filename=package://kuavo_assets/models/biped_s400055/meshes/head_yaw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
- link zhead_2_link: geometry visual mesh filename=package://kuavo_assets/models/biped_s400055/meshes/head_pit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
Joints:
- joint l_hand_base_joint: origin xyz=0 0 -0.07 rpy=0 3.14159265358979 0 -> xyz=0 0 -0.053 rpy=0 3.14159265358979 0
- joint r_hand_base_joint: origin xyz=0 0 -0.07 rpy=3.14159265358979 0 0 -> xyz=0 0 -0.053 rpy=3.14159265358979 0 0

File: src/kuavo_assets/models/biped_s400055/urdf/drake/biped_v3_all_joint.urdf (robot description, URDF)
Before this commit: robot biped_v3_all_joint, 59 links, 54 joints
Links:
- link zarm_l7_link: geometry visual mesh filename=../../meshes/l_hand_pitch.STL
- link zarm_r7_link: geometry visual mesh filename=../../meshes/r_hand_pitch.STL
Joints:
- joint l_hand_base_joint: origin xyz=0 0 -0.07 rpy=0 3.14159265358979 0 -> xyz=0 0 -0.053 rpy=0 3.14159265358979 0
- joint r_hand_base_joint: origin xyz=0 0 -0.07 rpy=3.14159265358979 0 0 -> xyz=0 0 -0.053 rpy=3.14159265358979 0 0

File: src/kuavo_assets/models/biped_s400055/urdf/drake/biped_v3_arm.urdf (robot description, URDF)
Before this commit: robot biped_s55, 44 links, 43 joints
Joints:
- joint l_hand_base_joint: origin xyz=0 0 -0.07 rpy=0 3.14159265358979 0 -> xyz=0 0 -0.053 rpy=0 3.14159265358979 0
- joint r_hand_base_joint: origin xyz=0 0 -0.07 rpy=3.14159265358979 0 0 -> xyz=0 0 -0.053 rpy=3.14159265358979 0 0

File: src/kuavo_assets/models/biped_s400055/urdf/drake/biped_v3_full.urdf (robot description, URDF)
Before this commit: robot biped_s55, 56 links, 55 joints
Links:
- link zarm_l7_link: geometry visual mesh filename=../../meshes/l_hand_pitch.STL
- link zarm_r7_link: geometry visual mesh filename=../../meshes/r_hand_pitch.STL
Joints:
- joint l_hand_base_joint: origin xyz=0 0 -0.07 rpy=0 3.14159265358979 0 -> xyz=0 0 -0.053 rpy=0 3.14159265358979 0
- joint r_hand_base_joint: origin xyz=0 0 -0.07 rpy=3.14159265358979 0 0 -> xyz=0 0 -0.053 rpy=3.14159265358979 0 0

File: src/kuavo_assets/models/biped_s400062/urdf/biped_s400062.urdf (robot description, URDF)
Before this commit: robot biped_s62, 56 links, 55 joints
Links:
- added link zarm_l7_end_effector_1
- added link zarm_l7_end_effector_2
- added link zarm_r7_end_effector_1
- added link zarm_r7_end_effector_2
- link base_link: geometry collision cylinder length=0.32 radius=0.37; visual mesh filename=package://kuavo_assets/models/biped_s400062/meshes/base_lin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
- link base_to_joint: geometry visual mesh filename=package://kuavo_assets/models/biped_s400062/meshes/knee_lin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
- link head_camera_base: geometry visual mesh filename=package://kuavo_assets/models/biped_s400062/meshes/head_cam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
- link knee_link: geometry visual mesh filename=package://kuavo_assets/models/biped_s400062/meshes/leg_Link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
- link leg_link: geometry visual mesh filename=package://kuavo_assets/models/biped_s400062/meshes/waist_pi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
- link radar: geometry visual mesh filename=package://kuavo_assets/models/biped_s400062/meshes/head_rad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
- link waist_link: geometry visual mesh filename=package://kuavo_assets/models/biped_s400062/meshes/waist_ya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
- link waist_yaw_link: geometry collision cylinder length=0.6 radius=0.15; visual mesh filename=package://kuavo_assets/models/biped_s400062/meshes/torso.STL
- link wheel_left_behind: geometry collision cylinder length=0.03 radius=0.13035; visual mesh filename=package://kuavo_assets/models/biped_s400062/meshes/wheel_le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
- link wheel_left_front: geometry collision cylinder length=0.03 radius=0.13035; visual mesh filename=package://kuavo_assets/models/biped_s400062/meshes/wheel_le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
- link wheel_right_behind: geometry collision cylinder length=0.03 radius=0.13035; visual mesh filename=package://kuavo_assets/models/biped_s400062/meshes/wheel_ri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
- link wheel_right_front: geometry collision cylinder length=0.03 radius=0.13035; visual mesh filename=package://kuavo_assets/models/biped_s400062/meshes/wheel_ri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
- link zarm_l1_link: geometry visual mesh filename=package://kuavo_assets/models/biped_s400062/meshes/l_arm_pi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
- link zarm_l2_link: geometry collision cylinder length=0.3 radius=0.05; visual mesh filename=package://kuavo_assets/models/biped_s400062/meshes/l_arm_ro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
- link zarm_l3_link: geometry visual mesh filename=package://kuavo_assets/models/biped_s400062/meshes/l_arm_ya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
- link zarm_l4_link: geometry collision cylinder length=0.26 radius=0.05; visual mesh filename=package://kuavo_assets/models/biped_s400062/meshes/l_forear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
- link zarm_l5_link: geometry visual mesh filename=package://kuavo_assets/models/biped_s400062/meshes/l_hand_y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
- link zarm_l6_link: geometry visual mesh filename=package://kuavo_assets/models/biped_s400062/meshes/l_hand_r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
- link zarm_l7_end_effector: geometry collision sphere radius=0.005
- link zarm_l7_link: geometry collision cylinder length=0.14 radius=0.04; visual mesh filename=package://kuavo_assets/models/biped_s400062/meshes/l_hand_p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
- link zarm_r1_link: geometry visual mesh filename=package://kuavo_assets/models/biped_s400062/meshes/r_arm_pi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
- link zarm_r2_link: geometry collision cylinder length=0.3 radius=0.05; visual mesh filename=package://kuavo_assets/models/biped_s400062/meshes/r_arm_ro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
- link zarm_r3_link: geometry visual mesh filename=package://kuavo_assets/models/biped_s400062/meshes/r_arm_ya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
- link zarm_r4_link: geometry collision cylinder length=0.26 radius=0.05; visual mesh filename=package://kuavo_assets/models/biped_s400062/meshes/r_forear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
- link zarm_r5_link: geometry visual mesh filename=package://kuavo_assets/models/biped_s400062/meshes/r_hand_y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
- link zarm_r6_link: geometry visual mesh filename=package://kuavo_assets/models/biped_s400062/meshes/r_hand_r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
- link zarm_r7_end_effector: geometry collision sphere radius=0.005
- link zarm_r7_link: geometry collision cylinder length=0.14 radius=0.04; visual mesh filename=package://kuavo_assets/models/biped_s400062/meshes/r_hand_p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
- link zhead_1_link: geometry collision sphere radius=0.1; visual mesh filename=package://kuavo_assets/models/biped_s400062/meshes/head_yaw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
- link zhead_2_link: geometry visual mesh filename=package://kuavo_assets/models/biped_s400062/meshes/head_pit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
Joints:
- added joint zarm_l7_end_effector_1_joint: type fixed, parent zarm_l7_link, child zarm_l7_end_effector_1, origin xyz=0 0.0 -0.08 rpy=0 0 0
- added joint zarm_l7_end_effector_2_joint: type fixed, parent zarm_l7_link, child zarm_l7_end_effector_2, origin xyz=0.03 0.0 -0.17 rpy=0 0 0
- added joint zarm_r7_end_effector_1_joint: type fixed, parent zarm_r7_link, child zarm_r7_end_effector_1, origin xyz=0 0.0 -0.08 rpy=0 0 0
- added joint zarm_r7_end_effector_2_joint: type fixed, parent zarm_r7_link, child zarm_r7_end_effector_2, origin xyz=0.03 0.0 -0.17 rpy=0 0 0
- joint l_hand_base_joint: origin xyz=0 0 -0.07 rpy=0 3.14159265358979 0 -> xyz=0 0 -0.053 rpy=0 3.14159265358979 0
- joint l_index_j1: type fixed -> revolute
- joint l_index_j2: type fixed -> revolute
- joint l_index_j3: type fixed -> revolute
- joint l_little_j1: type fixed -> revolute
- joint l_little_j2: type fixed -> revolute
- joint l_little_j3: type fixed -> revolute
- joint l_middle_j1: type fixed -> revolute
- joint l_middle_j2: type fixed -> revolute
- joint l_thumb_j1: type fixed -> revolute
- joint l_thumb_j2: type fixed -> revolute
- joint l_thumb_j3: type fixed -> revolute
- joint r_hand_base_joint: origin xyz=0 0 -0.07 rpy=3.14159265358979 0 0 -> xyz=0 0 -0.053 rpy=3.14159265358979 0 0
- joint r_index_j1: type fixed -> revolute
- joint r_index_j2: type fixed -> revolute
- joint r_index_j3: type fixed -> revolute
- joint r_little_j1: type fixed -> revolute
- joint r_little_j2: type fixed -> revolute
- joint r_little_j3: type fixed -> revolute
- joint r_middle_j1: type fixed -> revolute
- joint r_middle_j2: type fixed -> revolute
- joint r_thumb_j1: type fixed -> revolute
- joint r_thumb_j2: type fixed -> revolute
- joint r_thumb_j3: type fixed -> revolute
- joint zarm_l7_end_effector_joint: origin xyz=0 -0.03 -0.17 rpy=0 0 0 -> xyz=0 0.0 -0.17 rpy=0 0 0
- joint zarm_l7_joint: origin xyz=0 0 -0.0210004653879916 rpy=0 0 0 -> xyz=0 0 -0.021 rpy=0 0 0
- joint zarm_r7_end_effector_joint: origin xyz=0 0.03 -0.17 rpy=0 0 0 -> xyz=0 0.0 -0.17 rpy=0 0 0
- joint zarm_r7_joint: origin xyz=0 0 -0.0209999999999999 rpy=0 0 0 -> xyz=0.0 0 -0.021 rpy=0 0 0

File: src/kuavo_assets/models/biped_s400062/urdf/biped_s400062_gazebo.urdf (robot description, URDF)
Before this commit: robot biped_s62, 64 links, 63 joints
Links:
- link base_link: geometry visual mesh filename=package://kuavo_assets/models/biped_s400062/meshes/base_lin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
- link base_to_joint: geometry visual mesh filename=package://kuavo_assets/models/biped_s400062/meshes/knee_lin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
- link head_camera_base: geometry visual mesh filename=package://kuavo_assets/models/biped_s400062/meshes/head_cam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
- link knee_link: geometry visual mesh filename=package://kuavo_assets/models/biped_s400062/meshes/leg_Link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
- link leg_link: geometry visual mesh filename=package://kuavo_assets/models/biped_s400062/meshes/waist_pi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
- link radar: geometry visual mesh filename=package://kuavo_assets/models/biped_s400062/meshes/head_rad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
- link waist_pitch_link: geometry visual mesh filename=package://kuavo_assets/models/biped_s400062/meshes/waist_ya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
- link waist_yaw_link: geometry visual mesh filename=package://kuavo_assets/models/biped_s400062/meshes/torso.STL
- link wheel_left_behind: geometry visual mesh filename=package://kuavo_assets/models/biped_s400062/meshes/wheel_le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
- link wheel_left_front: geometry visual mesh filename=package://kuavo_assets/models/biped_s400062/meshes/wheel_le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
- link wheel_right_behind: geometry visual mesh filename=package://kuavo_assets/models/biped_s400062/meshes/wheel_ri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
- link wheel_right_front: geometry visual mesh filename=package://kuavo_assets/models/biped_s400062/meshes/wheel_ri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
- link zarm_l1_link: geometry visual mesh filename=package://kuavo_assets/models/biped_s400062/meshes/l_arm_pi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
- link zarm_l2_link: geometry visual mesh filename=package://kuavo_assets/models/biped_s400062/meshes/l_arm_ro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
- link zarm_l3_link: geometry visual mesh filename=package://kuavo_assets/models/biped_s400062/meshes/l_arm_ya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
- link zarm_l4_link: geometry visual mesh filename=package://kuavo_assets/models/biped_s400062/meshes/l_forear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
- link zarm_l5_link: geometry visual mesh filename=package://kuavo_assets/models/biped_s400062/meshes/l_hand_y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
- link zarm_l6_link: geometry visual mesh filename=package://kuavo_assets/models/biped_s400062/meshes/l_hand_r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
- link zarm_l7_end_effector: geometry collision sphere radius=0.005
- link zarm_l7_link: geometry visual mesh filename=package://kuavo_assets/models/biped_s400062/meshes/l_hand_p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
- link zarm_r1_link: geometry visual mesh filename=package://kuavo_assets/models/biped_s400062/meshes/r_arm_pi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
- link zarm_r2_link: geometry visual mesh filename=package://kuavo_assets/models/biped_s400062/meshes/r_arm_ro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
- link zarm_r3_link: geometry visual mesh filename=package://kuavo_assets/models/biped_s400062/meshes/r_arm_ya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
- link zarm_r4_link: geometry visual mesh filename=package://kuavo_assets/models/biped_s400062/meshes/r_forear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
- link zarm_r5_link: geometry visual mesh filename=package://kuavo_assets/models/biped_s400062/meshes/r_hand_y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
- link zarm_r6_link: geometry visual mesh filename=package://kuavo_assets/models/biped_s400062/meshes/r_hand_r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
- link zarm_r7_end_effector: geometry collision sphere radius=0.005
- link zarm_r7_link: geometry visual mesh filename=package://kuavo_assets/models/biped_s400062/meshes/r_hand_p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
- link zhead_1_link: geometry visual mesh filename=package://kuavo_assets/models/biped_s400062/meshes/head_yaw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
- link zhead_2_link: geometry visual mesh filename=package://kuavo_assets/models/biped_s400062/meshes/head_pit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
Joints:
- joint l_hand_base_joint: origin xyz=0 0 -0.07 rpy=0 3.14159265358979 0 -> xyz=0 0 -0.053 rpy=0 3.14159265358979 0
- joint r_hand_base_joint: origin xyz=0 0 -0.07 rpy=3.14159265358979 0 0 -> xyz=0 0 -0.053 rpy=3.14159265358979 0 0
- joint zarm_l7_end_effector_joint: origin xyz=0 -0.03 -0.17 rpy=0 0 0 -> xyz=0 0.0 -0.17 rpy=0 0 0
- joint zarm_l7_joint: origin xyz=0 0 -0.0210004653879916 rpy=0 0 0 -> xyz=0 0 -0.021 rpy=0 0 0
- joint zarm_r7_end_effector_joint: origin xyz=0 0.03 -0.17 rpy=0 0 0 -> xyz=0 0.0 -0.17 rpy=0 0 0
- joint zarm_r7_joint: origin xyz=0 0 -0.0209999999999999 rpy=0 0 0 -> xyz=0.0 0 -0.021 rpy=0 0 0

File: src/kuavo_assets/models/biped_s400062/urdf/drake/Larm.urdf (robot description, URDF)
Before this commit: robot Larm, 7 links, 7 joints
Links:
- link l_forearm_pitch: geometry visual mesh filename=../../meshes/l_forearm.STL

File: src/kuavo_assets/models/biped_s400062/urdf/drake/Rarm.urdf (robot description, URDF)
Before this commit: robot Rarm, 7 links, 7 joints
Links:
- link r_forearm_pitch: geometry visual mesh filename=../../meshes/r_forearm.STL

File: src/kuavo_assets/models/biped_s400062/urdf/drake/biped_v3_arm.urdf (robot description, URDF)
Before this commit: robot biped_s62, 48 links, 47 joints
Links:
- added link zarm_l7_end_effector_1
- added link zarm_l7_end_effector_2
- added link zarm_r7_end_effector_1
- added link zarm_r7_end_effector_2
- link zarm_l7_end_effector: geometry collision sphere radius=0.005
- link zarm_l7_link: geometry visual mesh filename=../../meshes/l_hand_pitch.STL
- link zarm_r7_end_effector: geometry collision sphere radius=0.005
- link zarm_r7_link: geometry visual mesh filename=../../meshes/r_hand_pitch.STL
Joints:
- added joint zarm_l7_end_effector_1_joint: type fixed, parent zarm_l7_link, child zarm_l7_end_effector_1, origin xyz=0 0.0 -0.08 rpy=0 0 0
- added joint zarm_l7_end_effector_2_joint: type fixed, parent zarm_l7_link, child zarm_l7_end_effector_2, origin xyz=0.03 0.0 -0.17 rpy=0 0 0
- added joint zarm_r7_end_effector_1_joint: type fixed, parent zarm_r7_link, child zarm_r7_end_effector_1, origin xyz=0 0.0 -0.08 rpy=0 0 0
- added joint zarm_r7_end_effector_2_joint: type fixed, parent zarm_r7_link, child zarm_r7_end_effector_2, origin xyz=0.03 0.0 -0.17 rpy=0 0 0
- joint l_hand_base_joint: origin xyz=0 0 -0.07 rpy=0 3.14159265358979 0 -> xyz=0 0 -0.053 rpy=0 3.14159265358979 0
- joint r_hand_base_joint: origin xyz=0 0 -0.07 rpy=3.14159265358979 0 0 -> xyz=0 0 -0.053 rpy=3.14159265358979 0 0
- joint zarm_l7_end_effector_joint: origin xyz=0 0 -0.17 rpy=0 0 0 -> xyz=0 0.0 -0.17 rpy=0 0 0
- joint zarm_r7_end_effector_joint: origin xyz=0 0 -0.17 rpy=0 0 0 -> xyz=0 0.0 -0.17 rpy=0 0 0
