Commit message: sync https://www.lejuhub.com/highlydynamic/kuavo-ros-control/commit/bb977f7ff3954b61b401493bb51530a5b534942b

File: src/kuavo_assets/models/biped_s400062/urdf/drake/biped_v3_arm_only.urdf (robot description, URDF)
Before this commit: robot biped_s62, 48 links, 47 joints
Links:
- added link zarm_l7_end_effector_1
- added link zarm_l7_end_effector_2
- added link zarm_r7_end_effector_1
- added link zarm_r7_end_effector_2
- link zarm_l7_end_effector: geometry collision sphere radius=0.005
- link zarm_l7_link: geometry visual mesh filename=../../meshes/l_hand_pitch.STL
- link zarm_r7_end_effector: geometry collision sphere radius=0.005
- link zarm_r7_link: geometry visual mesh filename=../../meshes/r_hand_pitch.STL
Joints:
- added joint zarm_l7_end_effector_1_joint: type fixed, parent zarm_l7_link, child zarm_l7_end_effector_1, origin xyz=0 0.0 -0.08 rpy=0 0 0
- added joint zarm_l7_end_effector_2_joint: type fixed, parent zarm_l7_link, child zarm_l7_end_effector_2, origin xyz=0.03 0.0 -0.17 rpy=0 0 0
- added joint zarm_r7_end_effector_1_joint: type fixed, parent zarm_r7_link, child zarm_r7_end_effector_1, origin xyz=0 0.0 -0.08 rpy=0 0 0
- added joint zarm_r7_end_effector_2_joint: type fixed, parent zarm_r7_link, child zarm_r7_end_effector_2, origin xyz=0.03 0.0 -0.17 rpy=0 0 0
- joint l_hand_base_joint: origin xyz=0 0 -0.07 rpy=0 3.14159265358979 0 -> xyz=0 0 -0.053 rpy=0 3.14159265358979 0
- joint r_hand_base_joint: origin xyz=0 0 -0.07 rpy=3.14159265358979 0 0 -> xyz=0 0 -0.053 rpy=3.14159265358979 0 0
- joint zarm_l7_end_effector_joint: origin xyz=0 0 -0.17 rpy=0 0 0 -> xyz=0 0.0 -0.17 rpy=0 0 0
- joint zarm_r7_end_effector_joint: origin xyz=0 0 -0.17 rpy=0 0 0 -> xyz=0 0.0 -0.17 rpy=0 0 0

File: src/kuavo_assets/models/biped_s400062/urdf/drake/biped_v3_full.urdf (robot description, URDF)
Before this commit: robot biped_v3_full, 47 links, 46 joints
Links:
- link zarm_l7_link: geometry visual mesh filename=../../meshes/l_hand_pitch.STL
- link zarm_r7_link: geometry visual mesh filename=../../meshes/r_hand_pitch.STL
Joints:
- joint l_hand_base_joint: origin xyz=0 0 -0.07 rpy=0 3.14159265358979 0 -> xyz=0 0 -0.053 rpy=0 3.14159265358979 0
- joint r_hand_base_joint: origin xyz=0 0 -0.07 rpy=3.14159265358979 0 0 -> xyz=0 0 -0.053 rpy=3.14159265358979 0 0

File: src/kuavo_assets/models/biped_s400062/urdf/drake/biped_v3_upper_body.urdf (robot description, URDF)
Before this commit: robot biped_s62, 43 links, 42 joints
Links:
- added link zarm_l7_end_effector_1
- added link zarm_l7_end_effector_2
- added link zarm_r7_end_effector_1
- added link zarm_r7_end_effector_2
- link zarm_l7_end_effector: geometry collision sphere radius=0.005
- link zarm_l7_link: geometry visual mesh filename=../../meshes/l_hand_pitch.STL
- link zarm_r7_end_effector: geometry collision sphere radius=0.005
- link zarm_r7_link: geometry visual mesh filename=../../meshes/r_hand_pitch.STL
Joints:
- added joint zarm_l7_end_effector_1_joint: type fixed, parent zarm_l7_link, child zarm_l7_end_effector_1, origin xyz=0 0.0 -0.08 rpy=0 0 0
- added joint zarm_l7_end_effector_2_joint: type fixed, parent zarm_l7_link, child zarm_l7_end_effector_2, origin xyz=0.03 0.0 -0.17 rpy=0 0 0
- added joint zarm_r7_end_effector_1_joint: type fixed, parent zarm_r7_link, child zarm_r7_end_effector_1, origin xyz=0 0.0 -0.08 rpy=0 0 0
- added joint zarm_r7_end_effector_2_joint: type fixed, parent zarm_r7_link, child zarm_r7_end_effector_2, origin xyz=0.03 0.0 -0.17 rpy=0 0 0
- joint l_hand_base_joint: origin xyz=0 0 -0.07 rpy=0 3.14159265358979 0 -> xyz=0 0 -0.053 rpy=0 3.14159265358979 0
- joint r_hand_base_joint: origin xyz=0 0 -0.07 rpy=3.14159265358979 0 0 -> xyz=0 0 -0.053 rpy=3.14159265358979 0 0
- joint zarm_l7_end_effector_joint: origin xyz=0 0 -0.17 rpy=0 0 0 -> xyz=0 0.0 -0.17 rpy=0 0 0
- joint zarm_r7_end_effector_joint: origin xyz=0 0 -0.17 rpy=0 0 0 -> xyz=0 0.0 -0.17 rpy=0 0 0
