Commit message: sync https://www.lejuhub.com/highlydynamic/kuavo-ros-control/commit/6cea279df3d42f9fbfcd0bb26aa241da5ad7aecd

File: src/kuavo_assets/models/biped_s400062/urdf/biped_s400062.urdf (robot description, URDF)
Before this commit: robot biped_s400062, 60 links, 59 joints
Links:
- removed link head_camera_depth
- added link cam_h_link, mass 0.0482361371130408
- added link cam_l_link
- added link cam_r_link
- added link camera_l_base, mass 1.07678764383011; collision mesh filename=package://kuavo_assets/models/biped_s400062/meshes/camera_l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; visual mesh filename=package://kuavo_assets/models/biped_s400062/meshes/camera_l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
- added link camera_l_color_link
- added link camera_l_depth_link
- added link camera_r_base, mass 1.07678764383011; collision mesh filename=package://kuavo_assets/models/biped_s400062/meshes/camera_r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; visual mesh filename=package://kuavo_assets/models/biped_s400062/meshes/camera_r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
- added link camera_r_color_link
- added link camera_r_depth_link
Joints:
- removed joint head_camera_depth_joint
- added joint cam_h_link_joint: type fixed, parent head_camera_base, child cam_h_link, origin xyz=0.011715 0.0475 0.014311 rpy=0 0 0
- added joint camera_l_base_joint: type fixed, parent zarm_l7_link, child camera_l_base, origin xyz=0.093563 -0.015735 0.021967 rpy=-2.2353 1.1377 -2.1889, axis 0 0 0
- added joint camera_l_color_frame: type fixed, parent camera_l_base, child camera_l_color_link, origin xyz=0.0109 0.009 0.021 rpy=0 0 0
- added joint camera_l_depth_frame: type fixed, parent camera_l_base, child camera_l_depth_link, origin xyz=0.0109 -0.009 0.021 rpy=0 0 0
- added joint camera_r_base_joint: type fixed, parent zarm_r7_link, child camera_r_base, origin xyz=0.134 0.015735 0.0111 rpy=2.2353 1.1377 2.1889, axis 0 0 0
- added joint camera_r_color_frame: type fixed, parent camera_r_base, child camera_r_color_link, origin xyz=0.0109 0.009 -0.021 rpy=3.14159265358979 0 0
- added joint camera_r_depth_frame: type fixed, parent camera_r_base, child camera_r_depth_link, origin xyz=0.0109 -0.009 -0.021 rpy=3.14159265358979 0 0
- added joint camera_to_realcam_l_frame: type fixed, parent camera_l_base, child cam_l_link, origin xyz=0.0146 0.00 0.021 rpy=0 0 0
- added joint camera_to_realcam_r_frame: type fixed, parent camera_r_base, child cam_r_link, origin xyz=0.0146 0.00 -0.021 rpy=3.14159265358979 0 0

File: src/kuavo_assets/models/biped_s400062/urdf/biped_s400062_gazebo.urdf (robot description, URDF)
Before this commit: robot biped_s400062, 64 links, 63 joints
Links:
- removed link head_camera_depth
- added link cam_h_link, mass 0.001
Joints:
- removed joint head_camera_depth_joint
- added joint cam_h_link_joint: type fixed, parent head_camera_base, child cam_h_link, origin xyz=0.011715 0.0475 0.014311 rpy=0 0 0

File: src/kuavo_assets/models/biped_s400063/urdf/biped_s400063.urdf (robot description, URDF)
Before this commit: robot biped_s400063, 60 links, 59 joints
Links:
- removed link head_camera_depth
- added link cam_h_link, mass 0.0; visual mesh filename=package://kuavo_assets/models/biped_s400063/meshes/head_cam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
- added link cam_l_link
- added link cam_r_link
- added link camera_l_base, mass 1.07678764383011; collision mesh filename=package://kuavo_assets/models/biped_s400063/meshes/camera_l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; visual mesh filename=package://kuavo_assets/models/biped_s400063/meshes/camera_l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
- added link camera_l_color_link
- added link camera_l_depth_link
- added link camera_r_base, mass 1.07678764383011; collision mesh filename=package://kuavo_assets/models/biped_s400063/meshes/camera_r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; visual mesh filename=package://kuavo_assets/models/biped_s400063/meshes/camera_r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
- added link camera_r_color_link
- added link camera_r_depth_link
Joints:
- removed joint head_camera_depth_joint
- added joint cam_h_link_joint: type fixed, parent head_camera_base, child cam_h_link, origin xyz=0.011715 0.0475 0.014311 rpy=0 0 0
- added joint camera_l_base_joint: type fixed, parent zarm_l7_link, child camera_l_base, origin xyz=0.093563 -0.015735 0.021967 rpy=-2.2353 1.1377 -2.1889, axis 0 0 0
- added joint camera_l_color_frame: type fixed, parent camera_l_base, child camera_l_color_link, origin xyz=0.0109 0.009 0.021 rpy=0 0 0
- added joint camera_l_depth_frame: type fixed, parent camera_l_base, child camera_l_depth_link, origin xyz=0.0109 -0.009 0.021 rpy=0 0 0
- added joint camera_r_base_joint: type fixed, parent zarm_r7_link, child camera_r_base, origin xyz=0.134 0.015735 0.0111 rpy=2.2353 1.1377 2.1889, axis 0 0 0
- added joint camera_r_color_frame: type fixed, parent camera_r_base, child camera_r_color_link, origin xyz=0.0109 0.009 -0.021 rpy=3.14159265358979 0 0
- added joint camera_r_depth_frame: type fixed, parent camera_r_base, child camera_r_depth_link, origin xyz=0.0109 -0.009 -0.021 rpy=3.14159265358979 0 0
- added joint camera_to_realcam_l_frame: type fixed, parent camera_l_base, child cam_l_link, origin xyz=0.0146 0.00 0.021 rpy=0 0 0
- added joint camera_to_realcam_r_frame: type fixed, parent camera_r_base, child cam_r_link, origin xyz=0.0146 0.00 -0.021 rpy=3.14159265358979 0 0

File: src/kuavo_assets/models/biped_s400063/urdf/biped_s400063_gazebo.urdf (robot description, URDF)
Before this commit: robot biped_s400063, 64 links, 63 joints
Links:
- removed link head_camera_depth
- added link cam_h_link, mass 0.0; visual mesh filename=package://kuavo_assets/models/biped_s400063/meshes/head_cam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
Joints:
- removed joint head_camera_depth_joint
- added joint cam_h_link_joint: type fixed, parent head_camera_base, child cam_h_link, origin xyz=0.011715 0.0475 0.014311 rpy=0 0 0
