Commit message: sync https://www.lejuhub.com/highlydynamic/kuavo-ros-control/commit/7de5e3056d13f589807967907f1e57179189f905

File: src/kuavo_assets/models/biped_s500053/urdf/drake/biped_v3_arm.urdf (robot description, URDF)
Before this commit: robot biped_s500053, 62 links, 61 joints
Joints:
- joint l_index_dip: axis 0 1 0 -> (none); limit lower=0 upper=1.43 effort=100 velocity=1 -> (none); mimic joint=l_index_mcp_pitch multiplier=0.89 offset=0 -> (none); type revolute -> fixed
- joint l_index_mcp_pitch: axis 0 1 0 -> (none); limit lower=0 upper=1.60 effort=100 velocity=1 -> (none); type revolute -> fixed
- joint l_middle_dip: axis 0 1 0 -> (none); limit lower=0 upper=1.43 effort=100 velocity=1 -> (none); mimic joint=l_middle_mcp_pitch multiplier=0.89 offset=0 -> (none); type revolute -> fixed
- joint l_middle_mcp_pitch: axis 0 1 0 -> (none); limit lower=0 upper=1.60 effort=100 velocity=1 -> (none); type revolute -> fixed
- joint l_pinky_dip: axis 0 1 0 -> (none); limit lower=0 upper=1.43 effort=100 velocity=1 -> (none); mimic joint=l_pinky_mcp_pitch multiplier=0.89 offset=0 -> (none); type revolute -> fixed
- joint l_pinky_mcp_pitch: axis 0 1 0 -> (none); limit lower=0 upper=1.60 effort=100 velocity=1 -> (none); type revolute -> fixed
- joint l_ring_dip: axis 0 1 0 -> (none); limit lower=0 upper=1.43 effort=100 velocity=1 -> (none); mimic joint=l_ring_mcp_pitch multiplier=0.89 offset=0 -> (none); type revolute -> fixed
- joint l_ring_mcp_pitch: axis 0 1 0 -> (none); limit lower=0 upper=1.60 effort=100 velocity=1 -> (none); type revolute -> fixed
- joint l_thumb_cmc_pitch: axis 0 1 0 -> (none); limit lower=0 upper=0.58 effort=100 velocity=1 -> (none); type revolute -> fixed
- joint l_thumb_cmc_yaw: axis 0 0 1 -> (none); limit lower=0 upper=1.3 effort=100 velocity=1 -> (none); type revolute -> fixed
- joint l_thumb_ip: axis 0 1 0 -> (none); limit lower=0 upper=1.08 effort=100 velocity=1 -> (none); mimic joint=l_thumb_cmc_pitch multiplier=2.29 offset=0 -> (none); type revolute -> fixed
- joint r_index_dip: axis 0 1 0 -> (none); limit lower=0 upper=1.43 effort=100 velocity=1 -> (none); mimic joint=r_index_mcp_pitch multiplier=0.89 offset=0 -> (none); type revolute -> fixed
- joint r_index_mcp_pitch: axis 0 1 0 -> (none); limit lower=0 upper=1.60 effort=100 velocity=1 -> (none); type revolute -> fixed
- joint r_middle_dip: axis 0 1 0 -> (none); limit lower=0 upper=1.43 effort=100 velocity=1 -> (none); mimic joint=r_middle_mcp_pitch multiplier=0.89 offset=0 -> (none); type revolute -> fixed
- joint r_middle_mcp_pitch: axis 0 1 0 -> (none); limit lower=0 upper=1.60 effort=100 velocity=1 -> (none); type revolute -> fixed
- joint r_pinky_dip: axis 0 1 0 -> (none); limit lower=0 upper=1.43 effort=100 velocity=1 -> (none); mimic joint=r_pinky_mcp_pitch multiplier=0.89 offset=0 -> (none); type revolute -> fixed
- joint r_pinky_mcp_pitch: axis 0 1 0 -> (none); limit lower=0 upper=1.60 effort=100 velocity=1 -> (none); type revolute -> fixed
- joint r_ring_dip: axis 0 1 0 -> (none); limit lower=0 upper=1.43 effort=100 velocity=1 -> (none); mimic joint=r_ring_mcp_pitch multiplier=0.89 offset=0 -> (none); type revolute -> fixed
- joint r_ring_mcp_pitch: axis 0 1 0 -> (none); limit lower=0 upper=1.60 effort=100 velocity=1 -> (none); type revolute -> fixed
- joint r_thumb_cmc_pitch: axis 0 1 0 -> (none); limit lower=0 upper=0.58 effort=100 velocity=1 -> (none); type revolute -> fixed
- joint r_thumb_cmc_yaw: axis 0 0 -1 -> (none); limit lower=0 upper=1.36 effort=100 velocity=1 -> (none); type revolute -> fixed
- joint r_thumb_ip: axis 0 1 0 -> (none); limit lower=0 upper=1.08 effort=100 velocity=1 -> (none); mimic joint=r_thumb_cmc_pitch multiplier=1.86 offset=0 -> (none); type revolute -> fixed

File: src/kuavo_assets/models/biped_s500055/urdf/drake/biped_v3_arm.urdf (robot description, URDF)
Before this commit: robot biped_s500055, 60 links, 59 joints
Joints:
- joint l_index_dip: axis 0 1 0 -> (none); limit lower=0 upper=1.43 effort=100 velocity=1 -> (none); mimic joint=l_index_mcp_pitch multiplier=0.89 offset=0 -> (none); type revolute -> fixed
- joint l_index_mcp_pitch: axis 0 1 0 -> (none); limit lower=0 upper=1.60 effort=100 velocity=1 -> (none); type revolute -> fixed
- joint l_middle_dip: axis 0 1 0 -> (none); limit lower=0 upper=1.43 effort=100 velocity=1 -> (none); mimic joint=l_middle_mcp_pitch multiplier=0.89 offset=0 -> (none); type revolute -> fixed
- joint l_middle_mcp_pitch: axis 0 1 0 -> (none); limit lower=0 upper=1.60 effort=100 velocity=1 -> (none); type revolute -> fixed
- joint l_pinky_dip: axis 0 1 0 -> (none); limit lower=0 upper=1.43 effort=100 velocity=1 -> (none); mimic joint=l_pinky_mcp_pitch multiplier=0.89 offset=0 -> (none); type revolute -> fixed
- joint l_pinky_mcp_pitch: axis 0 1 0 -> (none); limit lower=0 upper=1.60 effort=100 velocity=1 -> (none); type revolute -> fixed
- joint l_ring_dip: axis 0 1 0 -> (none); limit lower=0 upper=1.43 effort=100 velocity=1 -> (none); mimic joint=l_ring_mcp_pitch multiplier=0.89 offset=0 -> (none); type revolute -> fixed
- joint l_ring_mcp_pitch: axis 0 1 0 -> (none); limit lower=0 upper=1.60 effort=100 velocity=1 -> (none); type revolute -> fixed
- joint l_thumb_cmc_pitch: axis 0 1 0 -> (none); limit lower=0 upper=0.58 effort=100 velocity=1 -> (none); type revolute -> fixed
- joint l_thumb_cmc_yaw: axis 0 0 1 -> (none); limit lower=0 upper=1.3 effort=100 velocity=1 -> (none); type revolute -> fixed
- joint l_thumb_ip: axis 0 1 0 -> (none); limit lower=0 upper=1.08 effort=100 velocity=1 -> (none); mimic joint=l_thumb_cmc_pitch multiplier=2.29 offset=0 -> (none); type revolute -> fixed
- joint r_index_dip: axis 0 1 0 -> (none); limit lower=0 upper=1.43 effort=100 velocity=1 -> (none); mimic joint=r_index_mcp_pitch multiplier=0.89 offset=0 -> (none); type revolute -> fixed
- joint r_index_mcp_pitch: axis 0 1 0 -> (none); limit lower=0 upper=1.60 effort=100 velocity=1 -> (none); type revolute -> fixed
- joint r_middle_dip: axis 0 1 0 -> (none); limit lower=0 upper=1.43 effort=100 velocity=1 -> (none); mimic joint=r_middle_mcp_pitch multiplier=0.89 offset=0 -> (none); type revolute -> fixed
- joint r_middle_mcp_pitch: axis 0 1 0 -> (none); limit lower=0 upper=1.60 effort=100 velocity=1 -> (none); type revolute -> fixed
- joint r_pinky_dip: axis 0 1 0 -> (none); limit lower=0 upper=1.43 effort=100 velocity=1 -> (none); mimic joint=r_pinky_mcp_pitch multiplier=0.89 offset=0 -> (none); type revolute -> fixed
- joint r_pinky_mcp_pitch: axis 0 1 0 -> (none); limit lower=0 upper=1.60 effort=100 velocity=1 -> (none); type revolute -> fixed
- joint r_ring_dip: axis 0 1 0 -> (none); limit lower=0 upper=1.43 effort=100 velocity=1 -> (none); mimic joint=r_ring_mcp_pitch multiplier=0.89 offset=0 -> (none); type revolute -> fixed
- joint r_ring_mcp_pitch: axis 0 1 0 -> (none); limit lower=0 upper=1.60 effort=100 velocity=1 -> (none); type revolute -> fixed
- joint r_thumb_cmc_pitch: axis 0 1 0 -> (none); limit lower=0 upper=0.58 effort=100 velocity=1 -> (none); type revolute -> fixed
- joint r_thumb_cmc_yaw: axis 0 0 -1 -> (none); limit lower=0 upper=1.36 effort=100 velocity=1 -> (none); type revolute -> fixed
- joint r_thumb_ip: axis 0 1 0 -> (none); limit lower=0 upper=1.08 effort=100 velocity=1 -> (none); mimic joint=r_thumb_cmc_pitch multiplier=1.86 offset=0 -> (none); type revolute -> fixed

File: src/kuavo_assets/models/biped_s500062/urdf/drake/biped_v3_arm.urdf (robot description, URDF)
Before this commit: robot biped_s500062, 52 links, 51 joints
Joints:
- joint l_index_dip: axis 0 1 0 -> (none); limit lower=0 upper=1.43 effort=100 velocity=1 -> (none); mimic joint=l_index_mcp_pitch multiplier=0.89 offset=0 -> (none); type revolute -> fixed
- joint l_index_mcp_pitch: axis 0 1 0 -> (none); limit lower=0 upper=1.60 effort=100 velocity=1 -> (none); type revolute -> fixed
- joint l_middle_dip: axis 0 1 0 -> (none); limit lower=0 upper=1.43 effort=100 velocity=1 -> (none); mimic joint=l_middle_mcp_pitch multiplier=0.89 offset=0 -> (none); type revolute -> fixed
- joint l_middle_mcp_pitch: axis 0 1 0 -> (none); limit lower=0 upper=1.60 effort=100 velocity=1 -> (none); type revolute -> fixed
- joint l_pinky_dip: axis 0 1 0 -> (none); limit lower=0 upper=1.43 effort=100 velocity=1 -> (none); mimic joint=l_pinky_mcp_pitch multiplier=0.89 offset=0 -> (none); type revolute -> fixed
- joint l_pinky_mcp_pitch: axis 0 1 0 -> (none); limit lower=0 upper=1.60 effort=100 velocity=1 -> (none); type revolute -> fixed
- joint l_ring_dip: axis 0 1 0 -> (none); limit lower=0 upper=1.43 effort=100 velocity=1 -> (none); mimic joint=l_ring_mcp_pitch multiplier=0.89 offset=0 -> (none); type revolute -> fixed
- joint l_ring_mcp_pitch: axis 0 1 0 -> (none); limit lower=0 upper=1.60 effort=100 velocity=1 -> (none); type revolute -> fixed
- joint l_thumb_cmc_pitch: axis 0 1 0 -> (none); limit lower=0 upper=0.58 effort=100 velocity=1 -> (none); type revolute -> fixed
- joint l_thumb_cmc_yaw: axis 0 0 1 -> (none); limit lower=0 upper=1.3 effort=100 velocity=1 -> (none); type revolute -> fixed
- joint l_thumb_ip: axis 0 1 0 -> (none); limit lower=0 upper=1.08 effort=100 velocity=1 -> (none); mimic joint=l_thumb_cmc_pitch multiplier=2.29 offset=0 -> (none); type revolute -> fixed
- joint r_index_dip: axis 0 1 0 -> (none); limit lower=0 upper=1.43 effort=100 velocity=1 -> (none); mimic joint=r_index_mcp_pitch multiplier=0.89 offset=0 -> (none); type revolute -> fixed
- joint r_index_mcp_pitch: axis 0 1 0 -> (none); limit lower=0 upper=1.60 effort=100 velocity=1 -> (none); type revolute -> fixed
- joint r_middle_dip: axis 0 1 0 -> (none); limit lower=0 upper=1.43 effort=100 velocity=1 -> (none); mimic joint=r_middle_mcp_pitch multiplier=0.89 offset=0 -> (none); type revolute -> fixed
- joint r_middle_mcp_pitch: axis 0 1 0 -> (none); limit lower=0 upper=1.60 effort=100 velocity=1 -> (none); type revolute -> fixed
- joint r_pinky_dip: axis 0 1 0 -> (none); limit lower=0 upper=1.43 effort=100 velocity=1 -> (none); mimic joint=r_pinky_mcp_pitch multiplier=0.89 offset=0 -> (none); type revolute -> fixed
- joint r_pinky_mcp_pitch: axis 0 1 0 -> (none); limit lower=0 upper=1.60 effort=100 velocity=1 -> (none); type revolute -> fixed
- joint r_ring_dip: axis 0 1 0 -> (none); limit lower=0 upper=1.43 effort=100 velocity=1 -> (none); mimic joint=r_ring_mcp_pitch multiplier=0.89 offset=0 -> (none); type revolute -> fixed
- joint r_ring_mcp_pitch: axis 0 1 0 -> (none); limit lower=0 upper=1.60 effort=100 velocity=1 -> (none); type revolute -> fixed
- joint r_thumb_cmc_pitch: axis 0 1 0 -> (none); limit lower=0 upper=0.58 effort=100 velocity=1 -> (none); type revolute -> fixed
- joint r_thumb_cmc_yaw: axis 0 0 -1 -> (none); limit lower=0 upper=1.36 effort=100 velocity=1 -> (none); type revolute -> fixed
- joint r_thumb_ip: axis 0 1 0 -> (none); limit lower=0 upper=1.08 effort=100 velocity=1 -> (none); mimic joint=r_thumb_cmc_pitch multiplier=1.86 offset=0 -> (none); type revolute -> fixed

File: src/kuavo_assets/models/biped_s500063/urdf/drake/biped_v3_arm.urdf (robot description, URDF)
Before this commit: robot biped_s500063, 52 links, 51 joints
Joints:
- joint l_index_dip: axis 0 1 0 -> (none); limit lower=0 upper=1.43 effort=100 velocity=1 -> (none); mimic joint=l_index_mcp_pitch multiplier=0.89 offset=0 -> (none); type revolute -> fixed
- joint l_index_mcp_pitch: axis 0 1 0 -> (none); limit lower=0 upper=1.60 effort=100 velocity=1 -> (none); type revolute -> fixed
- joint l_middle_dip: axis 0 1 0 -> (none); limit lower=0 upper=1.43 effort=100 velocity=1 -> (none); mimic joint=l_middle_mcp_pitch multiplier=0.89 offset=0 -> (none); type revolute -> fixed
- joint l_middle_mcp_pitch: axis 0 1 0 -> (none); limit lower=0 upper=1.60 effort=100 velocity=1 -> (none); type revolute -> fixed
- joint l_pinky_dip: axis 0 1 0 -> (none); limit lower=0 upper=1.43 effort=100 velocity=1 -> (none); mimic joint=l_pinky_mcp_pitch multiplier=0.89 offset=0 -> (none); type revolute -> fixed
- joint l_pinky_mcp_pitch: axis 0 1 0 -> (none); limit lower=0 upper=1.60 effort=100 velocity=1 -> (none); type revolute -> fixed
- joint l_ring_dip: axis 0 1 0 -> (none); limit lower=0 upper=1.43 effort=100 velocity=1 -> (none); mimic joint=l_ring_mcp_pitch multiplier=0.89 offset=0 -> (none); type revolute -> fixed
- joint l_ring_mcp_pitch: axis 0 1 0 -> (none); limit lower=0 upper=1.60 effort=100 velocity=1 -> (none); type revolute -> fixed
- joint l_thumb_cmc_pitch: axis 0 1 0 -> (none); limit lower=0 upper=0.58 effort=100 velocity=1 -> (none); type revolute -> fixed
- joint l_thumb_cmc_yaw: axis 0 0 1 -> (none); limit lower=0 upper=1.3 effort=100 velocity=1 -> (none); type revolute -> fixed
- joint l_thumb_ip: axis 0 1 0 -> (none); limit lower=0 upper=1.08 effort=100 velocity=1 -> (none); mimic joint=l_thumb_cmc_pitch multiplier=2.29 offset=0 -> (none); type revolute -> fixed
- joint r_index_dip: axis 0 1 0 -> (none); limit lower=0 upper=1.43 effort=100 velocity=1 -> (none); mimic joint=r_index_mcp_pitch multiplier=0.89 offset=0 -> (none); type revolute -> fixed
- joint r_index_mcp_pitch: axis 0 1 0 -> (none); limit lower=0 upper=1.60 effort=100 velocity=1 -> (none); type revolute -> fixed
- joint r_middle_dip: axis 0 1 0 -> (none); limit lower=0 upper=1.43 effort=100 velocity=1 -> (none); mimic joint=r_middle_mcp_pitch multiplier=0.89 offset=0 -> (none); type revolute -> fixed
- joint r_middle_mcp_pitch: axis 0 1 0 -> (none); limit lower=0 upper=1.60 effort=100 velocity=1 -> (none); type revolute -> fixed
- joint r_pinky_dip: axis 0 1 0 -> (none); limit lower=0 upper=1.43 effort=100 velocity=1 -> (none); mimic joint=r_pinky_mcp_pitch multiplier=0.89 offset=0 -> (none); type revolute -> fixed
- joint r_pinky_mcp_pitch: axis 0 1 0 -> (none); limit lower=0 upper=1.60 effort=100 velocity=1 -> (none); type revolute -> fixed
- joint r_ring_dip: axis 0 1 0 -> (none); limit lower=0 upper=1.43 effort=100 velocity=1 -> (none); mimic joint=r_ring_mcp_pitch multiplier=0.89 offset=0 -> (none); type revolute -> fixed
- joint r_ring_mcp_pitch: axis 0 1 0 -> (none); limit lower=0 upper=1.60 effort=100 velocity=1 -> (none); type revolute -> fixed
- joint r_thumb_cmc_pitch: axis 0 1 0 -> (none); limit lower=0 upper=0.58 effort=100 velocity=1 -> (none); type revolute -> fixed
- joint r_thumb_cmc_yaw: axis 0 0 -1 -> (none); limit lower=0 upper=1.36 effort=100 velocity=1 -> (none); type revolute -> fixed
- joint r_thumb_ip: axis 0 1 0 -> (none); limit lower=0 upper=1.08 effort=100 velocity=1 -> (none); mimic joint=r_thumb_cmc_pitch multiplier=1.86 offset=0 -> (none); type revolute -> fixed
