Commit message: sync https://www.lejuhub.com/highlydynamic/kuavo-ros-control/commit/f9b8ead0d27ffc0c4a0e63c22ac095d3adbc1677

File: src/kuavo_assets/models/biped_s200062/urdf/drake/biped_v3_upper_body.urdf (robot description, URDF)
Before this commit: robot biped_s200062, 28 links, 27 joints
Joints:
- joint waist_yaw_joint: origin xyz=0 0 0.235 rpy=0 0 0 -> xyz=0 0 0.250 rpy=0 0 0
- joint zarm_l1_joint: origin xyz=0 0.2527 0.242 rpy=0 0 0 -> xyz=0 0.2527 0.227 rpy=0 0 0
- joint zarm_r1_joint: origin xyz=0 -0.2527 0.242 rpy=0 0 0 -> xyz=0 -0.2527 0.227 rpy=0 0 0

Commit message: sync https://www.lejuhub.com/highlydynamic/kuavo-ros-control/commit/db0aae75cbfd7470dbf84435384325b5ce8cf835

File: src/kuavo_assets/models/biped_s200062/urdf/drake/biped_v3_upper_body.urdf (robot description, URDF)
Before this commit: robot biped_s200062, 28 links, 27 joints
Links:
- removed link base_to_joint
- removed link knee_link
- removed link leg_link
- removed link waist_link
- removed link waist_yaw_link
Joints:
- removed joint base_to_joint
- removed joint knee_joint
- removed joint leg_joint
- removed joint waist_pitch_joint
- removed joint waist_yaw_joint
- joint zarm_l1_joint: parent waist_yaw_link -> base_link
- joint zarm_r1_joint: parent waist_yaw_link -> base_link

File: src/kuavo_assets/models/biped_s200063/urdf/drake/biped_v3_upper_body.urdf (robot description, URDF)
Before this commit: robot biped_s200063, 40 links, 39 joints
Links:
- removed link base_to_joint
- removed link knee_link
- removed link leg_link
- removed link waist_link
- removed link waist_yaw_link
Joints:
- removed joint base_to_joint
- removed joint knee_joint
- removed joint leg_joint
- removed joint waist_pitch_joint
- removed joint waist_yaw_joint
- joint zarm_l1_joint: origin xyz=0 0.2527 0.227 rpy=0 0 0 -> xyz=0 0.253 0.227 rpy=0 0 0; parent waist_yaw_link -> base_link
- joint zarm_r1_joint: origin xyz=0 -0.2527 0.227 rpy=0 0 0 -> xyz=0 -0.253 0.227 rpy=0 0 0; parent waist_yaw_link -> base_link
