Commit message: sync https://www.lejuhub.com/highlydynamic/kuavo-ros-control/commit/b890a834b7fa9562f89b7f2cc50ea32cb26ddd92

File: src/kuavo_assets/models/biped_s100049/urdf/biped_s100049.urdf (robot description, URDF)
Before this commit: robot biped_s100049, 81 links, 80 joints
Links:
- removed link camera
- removed link camera_l_color_link
- removed link camera_l_depth_link
- removed link camera_r_color_link
- removed link camera_r_depth_link
- removed link l_camera_link
- removed link l_d405_camera
- removed link r_d405_camera
- added link cam_h_link
- added link l_camera_link_connect, mass 0.09000000; collision mesh filename=package://kuavo_assets/models/biped_s100049/meshes/l_camera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; visual mesh filename=package://kuavo_assets/models/biped_s100049/meshes/l_camera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
- link camera_base: geometry visual mesh filename=package://kuavo_assets/models/biped_s100049/meshes/camera.S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
Joints:
- removed joint camera
- removed joint camera_l_color_frame
- removed joint camera_l_depth_frame
- removed joint camera_r_color_frame
- removed joint camera_r_depth_frame
- removed joint l_d405_camera_joint
- removed joint r_d405_camera_joint
- added joint camera_to_realcam_h_frame: type fixed, parent camera_base, child cam_h_link, origin xyz=0.015645 0.0475 0.01431109357346 rpy=0 0 0
- joint camera_l_base_joint: parent l_camera_link -> l_camera_link_connect
- joint l_camera_link_joint: child l_camera_link -> l_camera_link_connect

File: src/kuavo_assets/models/biped_s100049/urdf/biped_s100049_gazebo.urdf (robot description, URDF)
Before this commit: robot biped_s100049, 47 links, 46 joints
Links:
- removed link camera
- added link cam_h_link
- link camera_base: geometry visual mesh filename=package://kuavo_assets/models/biped_s100049/meshes/camera.S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
Joints:
- removed joint camera
- added joint camera_to_realcam_h_frame: type fixed, parent camera_base, child cam_h_link, origin xyz=0.015645 0.0475 0.01431109357346 rpy=0 0 0
- joint camera_base: origin xyz=0.0828919080642966 0 0.119165137551254 rpy=0 0.488692190558416 0 -> xyz=0.0932759773834307 0 0.145322661773667 rpy=3.14159265358979 0.383972435438723 0

File: src/kuavo_assets/models/biped_s200049/urdf/biped_s200049.urdf (robot description, URDF)
Before this commit: robot biped_s200049, 76 links, 75 joints
Links:
- removed link camera
- removed link camera_l_color_link
- removed link camera_l_depth_link
- removed link camera_r_color_link
- removed link camera_r_depth_link
- link camera_base: geometry visual mesh filename=package://kuavo_assets/models/biped_s200049/meshes/camera.S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
Joints:
- removed joint camera
- removed joint camera_l_color_frame
- removed joint camera_l_depth_frame
- removed joint camera_r_color_frame
- removed joint camera_r_depth_frame
- joint camera_to_realcam_h_frame: origin xyz=0.00 0.00 0.0 rpy=0 0 0 -> xyz=0.015645 0.0475 0.01431109357346 rpy=0 0 0; parent camera -> camera_base

File: src/kuavo_assets/models/biped_s200049/urdf/biped_s200049_gazebo.urdf (robot description, URDF)
Before this commit: robot biped_s200049, 76 links, 75 joints
Links:
- removed link camera
- removed link camera_l_color_link
- removed link camera_l_depth_link
- removed link camera_r_color_link
- removed link camera_r_depth_link
- link camera_base: geometry visual mesh filename=package://kuavo_assets/models/biped_s200049/meshes/camera.S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
Joints:
- removed joint camera
- removed joint camera_l_color_frame
- removed joint camera_l_depth_frame
- removed joint camera_r_color_frame
- removed joint camera_r_depth_frame
- joint camera_to_realcam_h_frame: origin xyz=0.00 0.00 0.0 rpy=0 0 0 -> xyz=0.015645 0.0475 0.01431109357346 rpy=0 0 0; parent camera -> camera_base
